Commit message: 一応全体ができた

File: ginko_description/models/ginko_auto/urdf/modules/leg_r.urdf.xacro (robot description, xacro)
@@ -125,5 +125,5 @@
 	    	<mimic joint="${name}_joint1" multiplier="-1" offset="0"/>
 	  	</joint>
-		<!-- lower link (upper-1st) -->
+		<!-- parallel link (lower-1st) -->
 		<link name="${name}_link4">
 			<!-- Collision created from STL mesh without color -->
@@ -155,5 +155,5 @@
 			<limit effort="1000.0" lower="-1.3" upper="0.7854" velocity="0.5"/>
 		</joint>
-		<!-- lower link (upper-2nd) -->
+		<!-- parallel link (lower-2nd) -->
 		<link name="${name}_link5">
 			<!-- Collision created from STL mesh without color -->

File: ginko_description/models/ginko_auto/urdf/robot.urdf.xacro (robot description, xacro)
@@ -1,5 +1,9 @@
 <?xml version="1.0"?>
 <robot name="ginko" xmlns:xacro="http://www.ros.org/wiki/xacro">
+	<xacro:include filename="$(find ginko_description)/models/ginko_auto/urdf/modules/body.urdf.xacro"/>
 	<xacro:include filename="$(find ginko_description)/models/ginko_auto/urdf/modules/leg_r.urdf.xacro"/>
+	<xacro:include filename="$(find ginko_description)/models/ginko_auto/urdf/modules/leg_l.urdf.xacro"/>
+	<xacro:include filename="$(find ginko_description)/models/ginko_auto/urdf/modules/arm_r.urdf.xacro"/>
+	<xacro:include filename="$(find ginko_description)/models/ginko_auto/urdf/modules/arm_l.urdf.xacro"/>
 	<link name="world"/>
 	<link name="base"/>
@@ -8,30 +12,9 @@
 		<child link="base"/>
 	</joint>
-<!-- 	<link name="leg_r_link0">
-		<collision>
-			<origin xyz="0 0 0" rpy="0 0 0"/>
-			<geometry>
-				<mesh filename="package://ginko_description/models/ginko_auto/meshes/stl/link02_r_femoral.stl"/>
-			</geometry>
-		</collision>
-		<visual>
-			<origin xyz="0 0 0" rpy="0 0 0"/>
-			<geometry>
-				<mesh filename="package://ginko_description/models/ginko_auto/meshes/dae/link02_r_femoral.dae"/>
-			</geometry>
-		</visual>
-		<inertial>
-			<origin xyz="0 0 0" rpy="0 0 0"/>
-			<mass value="6.1"/>
-			<inertia ixx="0.0001" ixy="0.0" ixz="0.0" iyy="0.0001" iyz="0.0" izz="0.0001"/>
-		</inertial>
-	</link>
-	<joint name="fixed_on_base" type="fixed">
-	    <parent link="base"/>
-		<child link="leg_r_link0"/>
-	    <origin xyz="0 0 0" rpy="0 0 0"/>
-	    <axis xyz="0 0 0"/>
-	</joint> -->
-	<xacro:leg_r name="leg_r" parent="base"/>
+	<xacro:body name="body" parent="base"/>
+	<xacro:leg_r name="leg_r" parent="body_leg_r_link"/>
+	<xacro:leg_l name="leg_l" parent="body_leg_l_link"/>
+	<xacro:arm_r name="arm_r" parent="body_arm_r_link"/>
+	<xacro:arm_l name="arm_l" parent="body_arm_l_link"/>
 <!-- 	<xacro:include filename="$(find ginko_description)/models/ginko_auto/urdf/modules/leg_r.urdf.xacro">
 		<param name="name" value="leg_r"/>
