Commit message: open manipulatorの書き方に寄せた

File: ginko_description/models/ginko_auto/urdf/modules/arm_l.urdf.xacro (robot description, xacro)
@@ -62,4 +62,13 @@
 			<axis xyz="1 0 0"/>
 			<limit effort="1000.0" lower="-0.85" upper="1.18" velocity="0.5"/>
+		</joint>
+		<link name="${name}_link1_rev"/>
+		<joint name="${name}_joint1_rev" type="revolute">
+			<parent link="${name}_link0"/>
+			<child  link="${name}_link1_rev"/>
+			<origin xyz="-0.0562 0.0246 0" rpy="-0.3927 3.1416 0"/>
+			<axis xyz="1 0 0"/>
+	    	<limit effort="1000.0" lower="-3.141593" upper="3.141593" velocity="0.5"/>
+	    	<mimic joint="${name}_joint1" multiplier="-1" offset="0"/>
 		</joint>
 		<!-- scissors -->

File: ginko_description/models/ginko_auto/urdf/modules/arm_r.urdf.xacro (robot description, xacro)
@@ -62,4 +62,13 @@
 			<axis xyz="-1 0 0"/>
 			<limit effort="1000.0" lower="-0.85" upper="1.18" velocity="0.5"/>
+		</joint>
+		<link name="${name}_link1_rev"/>
+		<joint name="${name}_joint1_rev" type="revolute">
+			<parent link="${name}_link0"/>
+			<child  link="${name}_link1_rev"/>
+			<origin xyz="-0.0562 -0.0246 0" rpy="0.3927 3.1416 0"/>
+			<axis xyz="-1 0 0"/>
+	    	<limit effort="1000.0" lower="-3.141593" upper="3.141593" velocity="0.5"/>
+	    	<mimic joint="${name}_joint1" multiplier="-1" offset="0"/>
 		</joint>
 		<!-- scissors -->

Commit message: ゴールポジション表示用のlaunchファイルを作った

File: ginko_description/models/ginko_auto/urdf/modules/arm_l.urdf.xacro (robot description, xacro)
@@ -70,5 +70,5 @@
 			<axis xyz="1 0 0"/>
 	    	<limit effort="1000.0" lower="-3.141593" upper="3.141593" velocity="0.5"/>
-	    	<mimic joint="${name}_joint1" multiplier="-1" offset="0"/>
+	    	<!-- <mimic joint="${name}_joint1" multiplier="-1" offset="0"/>  -->
 		</joint>
 		<!-- scissors -->

File: ginko_description/models/ginko_auto/urdf/modules/arm_l_mimic.urdf.xacro (robot description, xacro)
@@ -1,5 +1,5 @@
 <?xml version="1.0"?>
-<robot name="arm_r" xmlns:xacro="http://www.ros.org/wiki/xacro">
-	<xacro:macro name="arm_r" params="name parent">
+<robot name="arm_l" xmlns:xacro="http://www.ros.org/wiki/xacro">
+	<xacro:macro name="arm_l" params="name parent">
 	<!-- <xacro:property name="name" value="leg"/> -->
 		<!-- shoulder pitch. -->
@@ -9,5 +9,5 @@
 				<origin xyz="0 0 0" rpy="0 0 0"/>
 				<geometry>
-					<mesh filename="package://ginko_description/models/ginko_auto/meshes/stl/link09_r_arm01.stl"/>
+					<mesh filename="package://ginko_description/models/ginko_auto/meshes/stl/link09_l_arm01.stl"/>
 				</geometry>
 			</collision>
@@ -16,5 +16,5 @@
 				<origin xyz="0 0 0" rpy="0 0 0"/>
 				<geometry>
-					<mesh filename="package://ginko_description/models/ginko_auto/meshes/dae/link09_r_arm01.dae"/>
+					<mesh filename="package://ginko_description/models/ginko_auto/meshes/dae/link09_l_arm01.dae"/>
 				</geometry>
 			</visual>
@@ -30,5 +30,5 @@
 			<child link="${name}_link0"/>
 		    <origin xyz="0 0 0" rpy="0 0 0"/>
-		    <axis xyz="0 1 0"/>
+		    <axis xyz="0 -1 0"/>
 			<limit effort="1000.0" lower="-2.6" upper="2.6" velocity="0.5"/>
 		</joint>
@@ -39,5 +39,5 @@
 				<origin xyz="0 0 0" rpy="0 0 0"/>
 	    		<geometry>
-					<mesh filename="package://ginko_description/models/ginko_auto/meshes/stl/link10_r_arm02.stl"/>
+					<mesh filename="package://ginko_description/models/ginko_auto/meshes/stl/link10_l_arm02.stl"/>
 	    		</geometry>
 			</collision>
@@ -46,5 +46,5 @@
 				<origin xyz="0 0 0" rpy="0 0 0"/>
 	    		<geometry>
-					<mesh filename="package://ginko_description/models/ginko_auto/meshes/dae/link10_r_arm02.dae"/>
+					<mesh filename="package://ginko_description/models/ginko_auto/meshes/dae/link10_l_arm02.dae"/>
 	    		</geometry>
 			</visual>
@@ -59,5 +59,5 @@
 			<parent link="${name}_link0"/>
 			<child  link="${name}_link1"/>
-			<origin xyz="0.035 -0.0246 0" rpy="-0.3927 0 0"/>
+			<origin xyz="0.035 0.0246 0" rpy="0.3927 0 0"/>
 			<axis xyz="1 0 0"/>
 			<limit effort="1000.0" lower="-0.85" upper="1.18" velocity="0.5"/>
@@ -67,8 +67,8 @@
 			<parent link="${name}_link0"/>
 			<child  link="${name}_link1_rev"/>
-			<origin xyz="-0.0562 -0.0246 0" rpy="0.3927 3.1416 0"/>
+			<origin xyz="-0.0562 0.0246 0" rpy="-0.3927 3.1416 0"/>
 			<axis xyz="1 0 0"/>
 	    	<limit effort="1000.0" lower="-3.141593" upper="3.141593" velocity="0.5"/>
-	    	<!-- <mimic joint="${name}_joint1" multiplier="-1" offset="0"/>  -->
+	    	<mimic joint="${name}_joint1" multiplier="-1" offset="0"/>
 		</joint>
 		<!-- scissors -->
@@ -78,5 +78,5 @@
 				<origin xyz="0 0 0" rpy="0 0 0"/>
 	    		<geometry>
-					<mesh filename="package://ginko_description/models/ginko_auto/meshes/stl/link11_r_scissor01.stl"/>
+					<mesh filename="package://ginko_description/models/ginko_auto/meshes/stl/link11_l_scissor01.stl"/>
 	    		</geometry>
 			</collision>
@@ -85,5 +85,5 @@
 				<origin xyz="0 0 0" rpy="0 0 0"/>
 	    		<geometry>
-					<mesh filename="package://ginko_description/models/ginko_auto/meshes/dae/link11_r_scissor01.dae"/>
+					<mesh filename="package://ginko_description/models/ginko_auto/meshes/dae/link11_l_scissor01.dae"/>
 	    		</geometry>
 			</visual>
@@ -98,6 +98,6 @@
 	    	<parent link="${name}_link1"/>
 	    	<child  link="${name}_link2"/>
-	    	<origin xyz="0.0092 -0.0784 -0.0933" rpy="0 0.7854 0"/>
-	    	<axis xyz="0 -1 0"/>
+	    	<origin xyz="0.0092 0.0784 -0.0933" rpy="0 0.7854 0"/>
+	    	<axis xyz="0 1 0"/>
 	    	<limit effort="1000.0" lower="-2.36" upper="2.36" velocity="0.5"/>
 	  	</joint>
@@ -107,5 +107,5 @@
 				<origin xyz="0 0 0" rpy="0 0 0"/>
 	    		<geometry>
-					<mesh filename="package://ginko_description/models/ginko_auto/meshes/stl/link12_r_scissor02.stl"/>
+					<mesh filename="package://ginko_description/models/ginko_auto/meshes/stl/link12_l_scissor02.stl"/>
 	    		</geometry>
 			</collision>
@@ -114,5 +114,5 @@
 				<origin xyz="0 0 0" rpy="0 0 0"/>
 	    		<geometry>
-					<mesh filename="package://ginko_description/models/ginko_auto/meshes/dae/link12_r_scissor02.dae"/>
+					<mesh filename="package://ginko_description/models/ginko_auto/meshes/dae/link12_l_scissor02.dae"/>
 	    		</geometry>
 			</visual>
@@ -127,6 +127,6 @@
 	    	<parent link="${name}_link1"/>
 	    	<child  link="${name}_link3"/>
-	    	<origin xyz="0.0092 -0.0219 -0.0933" rpy="0 0.7854 0"/>
-	    	<axis xyz="0 -1 0"/>
+	    	<origin xyz="0.0092 0.0219 -0.0933" rpy="0 0.7854 0"/>
+	    	<axis xyz="0 1 0"/>
 	    	<limit effort="1000.0" lower="-2.36" upper="2.36" velocity="0.5"/>
 	  	</joint>
@@ -150,5 +150,5 @@
 	    	<parent link="${name}_link1"/>
 	    	<child  link="${name}_urg_link"/>
-	    	<origin xyz="-0.04675 -0.00655 -0.0483" rpy="0 1.57 1.57"/>
+	    	<origin xyz="-0.04675 0.00655 -0.0483" rpy="0 1.57 -1.57"/>
 	  	</joint>
 	</xacro:macro>

File: ginko_description/models/ginko_auto/urdf/modules/arm_r_mimic.urdf.xacro (robot description, xacro)
@@ -70,5 +70,5 @@
 			<axis xyz="1 0 0"/>
 	    	<limit effort="1000.0" lower="-3.141593" upper="3.141593" velocity="0.5"/>
-	    	<!-- <mimic joint="${name}_joint1" multiplier="-1" offset="0"/>  -->
+	    	<mimic joint="${name}_joint1" multiplier="-1" offset="0"/>
 		</joint>
 		<!-- scissors -->

Commit message: URDFを更新

File: ginko_description/models/ginko_auto/urdf/modules/arm_l.urdf.xacro (robot description, xacro)
@@ -98,5 +98,5 @@
 	    	<parent link="${name}_link1"/>
 	    	<child  link="${name}_link2"/>
-	    	<origin xyz="0.0092 0.0784 -0.0933" rpy="0 0.7854 0"/>
+	    	<origin xyz="0.0092 0.0547 -0.11295" rpy="0 0.7854 0"/>
 	    	<axis xyz="0 1 0"/>
 	    	<limit effort="1000.0" lower="-2.36" upper="2.36" velocity="0.5"/>
@@ -127,5 +127,5 @@
 	    	<parent link="${name}_link1"/>
 	    	<child  link="${name}_link3"/>
-	    	<origin xyz="0.0092 0.0219 -0.0933" rpy="0 0.7854 0"/>
+	    	<origin xyz="0.0092 -0.0018 -0.11295" rpy="0 0.7854 0"/>
 	    	<axis xyz="0 1 0"/>
 	    	<limit effort="1000.0" lower="-2.36" upper="2.36" velocity="0.5"/>
@@ -150,5 +150,5 @@
 	    	<parent link="${name}_link1"/>
 	    	<child  link="${name}_urg_link"/>
-	    	<origin xyz="-0.04675 0.00655 -0.0483" rpy="0 1.57 -1.57"/>
+	    	<origin xyz="-0.0456 -0.01715 -0.06795" rpy="0 1.57 -1.57"/>
 	  	</joint>
 	</xacro:macro>

File: ginko_description/models/ginko_auto/urdf/modules/arm_r.urdf.xacro (robot description, xacro)
@@ -98,5 +98,5 @@
 	    	<parent link="${name}_link1"/>
 	    	<child  link="${name}_link2"/>
-	    	<origin xyz="0.0092 -0.0784 -0.0933" rpy="0 0.7854 0"/>
+	    	<origin xyz="0.0092 -0.0547 -0.11295" rpy="0 0.7854 0"/>
 	    	<axis xyz="0 -1 0"/>
 	    	<limit effort="1000.0" lower="-2.36" upper="2.36" velocity="0.5"/>
@@ -127,5 +127,5 @@
 	    	<parent link="${name}_link1"/>
 	    	<child  link="${name}_link3"/>
-	    	<origin xyz="0.0092 -0.0219 -0.0933" rpy="0 0.7854 0"/>
+	    	<origin xyz="0.0092 0.0018 -0.11295" rpy="0 0.7854 0"/>
 	    	<axis xyz="0 -1 0"/>
 	    	<limit effort="1000.0" lower="-2.36" upper="2.36" velocity="0.5"/>
@@ -150,5 +150,5 @@
 	    	<parent link="${name}_link1"/>
 	    	<child  link="${name}_urg_link"/>
-	    	<origin xyz="-0.04675 -0.00655 -0.0483" rpy="0 1.57 1.57"/>
+	    	<origin xyz="-0.0456 0.01715 -0.06795" rpy="0 1.57 1.57"/>
 	  	</joint>
 	</xacro:macro>

File: ginko_description/models/ginko_auto/urdf/modules/body.urdf.xacro (robot description, xacro)
@@ -66,5 +66,5 @@
 		    <parent link="${name}_link0"/>
 			<child link="${name}_arm_r_link"/>
-		    <origin xyz="0 -0.0903 0.04865" rpy="0 0 0"/>
+		    <origin xyz="0 -0.10683 0.05115" rpy="0 0 0"/>
 		    <axis xyz="0 -1 0"/>
 		</joint>
@@ -73,5 +73,5 @@
 		    <parent link="${name}_link0"/>
 			<child link="${name}_arm_l_link"/>
-		    <origin xyz="0 0.0903 0.04865" rpy="0 0 0"/>
+		    <origin xyz="0 0.10683 0.05115" rpy="0 0 0"/>
 		    <axis xyz="0 1 0"/>
 		</joint>
@@ -80,5 +80,5 @@
 		    <parent link="${name}_link1"/>
 			<child link="${name}_leg_r_link"/>
-		    <origin xyz="0.0263 -0.0411 -0.0434" rpy="0 0 0"/>
+		    <origin xyz="0.0205 0.0 -0.0409" rpy="0 0 0"/>
 		    <axis xyz="0 1 0"/>
 		</joint>
@@ -87,5 +87,5 @@
 		    <parent link="${name}_link1"/>
 			<child link="${name}_leg_l_link"/>
-		    <origin xyz="0.0263 0.0411 -0.0434" rpy="0 0 0"/>
+		    <origin xyz="-0.0404 0.0 -0.0409" rpy="0 0 0"/>
 		    <axis xyz="0 1 0"/>
 		</joint>

File: ginko_description/models/ginko_auto/urdf/modules/leg_l.urdf.xacro (robot description, xacro)
@@ -29,5 +29,5 @@
 		    <parent link="${parent}"/>
 			<child link="${name}_link0"/>
-		    <origin xyz="0 0 0" rpy="0.39217 0 0"/>
+		    <origin xyz="0 0 0" rpy="0 0 0"/>
 		    <axis xyz="1 0 0"/>
 			<limit effort="1000.0" lower="-0.8" upper="1.1781" velocity="0.5"/>
@@ -59,5 +59,5 @@
 			<parent link="${name}_link0"/>
 			<child  link="${name}_link1"/>
-			<origin xyz="-0.0163 -0.0148 -0.0364" rpy="0 0.7854 0"/>
+			<origin xyz="0.0433 0.0175 -0.0481" rpy="0 0.7854 0"/>
 			<axis xyz="0 -1 0"/>
 			<limit effort="1000.0" lower="-1.3" upper="0.7854" velocity="0.5"/>
@@ -89,5 +89,5 @@
 	    	<parent link="${name}_link0"/>
 	    	<child  link="${name}_link2"/>
-	    	<origin xyz="-0.0376 -0.0148 -0.04845" rpy="0 0.7854 0"/>
+	    	<origin xyz="0.022 0.0175 -0.06015" rpy="0 0.7854 0"/>
 	    	<axis xyz="0 -1 0"/>
 	    	<limit effort="1000.0" lower="-3.141593" upper="3.141593" velocity="0.5"/>

File: ginko_description/models/ginko_auto/urdf/modules/leg_l_mimic.urdf.xacro (robot description, xacro)
@@ -29,5 +29,5 @@
 		    <parent link="${parent}"/>
 			<child link="${name}_link0"/>
-		    <origin xyz="0 0 0" rpy="0.39217 0 0"/>
+		    <origin xyz="0 0 0" rpy="0 0 0"/>
 		    <axis xyz="1 0 0"/>
 			<limit effort="1000.0" lower="-0.8" upper="1.1781" velocity="0.5"/>
@@ -59,5 +59,5 @@
 			<parent link="${name}_link0"/>
 			<child  link="${name}_link1"/>
-			<origin xyz="-0.0163 -0.0148 -0.0364" rpy="0 0.7854 0"/>
+			<origin xyz="0.0433 0.0175 -0.0481" rpy="0 0.7854 0"/>
 			<axis xyz="0 -1 0"/>
 			<limit effort="1000.0" lower="-1.3" upper="0.7854" velocity="0.5"/>
@@ -89,5 +89,5 @@
 	    	<parent link="${name}_link0"/>
 	    	<child  link="${name}_link2"/>
-	    	<origin xyz="-0.0376 -0.0148 -0.04845" rpy="0 0.7854 0"/>
+	    	<origin xyz="0.022 0.0175 -0.06015" rpy="0 0.7854 0"/>
 	    	<axis xyz="0 -1 0"/>
 	    	<limit effort="1000.0" lower="-3.141593" upper="3.141593" velocity="0.5"/>

File: ginko_description/models/ginko_auto/urdf/modules/leg_r.urdf.xacro (robot description, xacro)
@@ -29,5 +29,5 @@
 		    <parent link="${parent}"/>
 			<child link="${name}_link0"/>
-		    <origin xyz="0 0 0" rpy="-0.39217 0 0"/>
+		    <origin xyz="0 0 0" rpy="0 0 0"/>
 		    <axis xyz="1 0 0"/>
 			<limit effort="1000.0" lower="-1.1781" upper="0.8" velocity="0.5"/>
@@ -59,5 +59,5 @@
 			<parent link="${name}_link0"/>
 			<child  link="${name}_link1"/>
-			<origin xyz="-0.0163 0.0148 -0.0364" rpy="0 0.7854 0"/>
+			<origin xyz="-0.0176 -0.0175 -0.0481" rpy="0 0.7854 0"/>
 			<axis xyz="0 1 0"/>
 			<limit effort="1000.0" lower="-0.7854" upper="1.3" velocity="0.5"/>
@@ -89,5 +89,5 @@
 	    	<parent link="${name}_link0"/>
 	    	<child  link="${name}_link2"/>
-	    	<origin xyz="-0.0376 0.0148 -0.04845" rpy="0 0.7854 0"/>
+	    	<origin xyz="-0.0389 -0.0175 -0.06015" rpy="0 0.7854 0"/>
 	    	<axis xyz="0 1 0"/>
 	    	<limit effort="1000.0" lower="-3.141593" upper="3.141593" velocity="0.5"/>

File: ginko_description/models/ginko_auto/urdf/modules/leg_r_mimic.urdf.xacro (robot description, xacro)
@@ -29,5 +29,5 @@
 		    <parent link="${parent}"/>
 			<child link="${name}_link0"/>
-		    <origin xyz="0 0 0" rpy="-0.39217 0 0"/>
+		    <origin xyz="0 0 0" rpy="0 0 0"/>
 		    <axis xyz="1 0 0"/>
 			<limit effort="1000.0" lower="-1.1781" upper="0.8" velocity="0.5"/>
@@ -59,5 +59,5 @@
 			<parent link="${name}_link0"/>
 			<child  link="${name}_link1"/>
-			<origin xyz="-0.0163 0.0148 -0.0364" rpy="0 0.7854 0"/>
+			<origin xyz="-0.0176 -0.0175 -0.0481" rpy="0 0.7854 0"/>
 			<axis xyz="0 1 0"/>
 			<limit effort="1000.0" lower="-0.7854" upper="1.3" velocity="0.5"/>
@@ -89,5 +89,5 @@
 	    	<parent link="${name}_link0"/>
 	    	<child  link="${name}_link2"/>
-	    	<origin xyz="-0.0376 0.0148 -0.04845" rpy="0 0.7854 0"/>
+	    	<origin xyz="-0.0389 -0.0175 -0.06015" rpy="0 0.7854 0"/>
 	    	<axis xyz="0 1 0"/>
 	    	<limit effort="1000.0" lower="-3.141593" upper="3.141593" velocity="0.5"/>

Commit message: URDF修正、サーボのオフセットを補正

File: ginko_description/models/ginko_auto/urdf/modules/arm_l.urdf.xacro (robot description, xacro)
@@ -29,5 +29,5 @@
 		    <parent link="${parent}"/>
 			<child link="${name}_link0"/>
-		    <origin xyz="0 0 0" rpy="0 0 0"/>
+		    <origin xyz="0 0 0" rpy="0 0.3927 0"/>
 		    <axis xyz="0 -1 0"/>
 			<limit effort="1000.0" lower="-2.6" upper="2.6" velocity="0.5"/>
@@ -59,5 +59,5 @@
 			<parent link="${name}_link0"/>
 			<child  link="${name}_link1"/>
-			<origin xyz="0.035 0.0246 0" rpy="0.3927 0 0"/>
+			<origin xyz="0.035 0.0246 0" rpy="1.1781 0 0"/>
 			<axis xyz="1 0 0"/>
 			<limit effort="1000.0" lower="-0.85" upper="1.18" velocity="0.5"/>
@@ -67,5 +67,5 @@
 			<parent link="${name}_link0"/>
 			<child  link="${name}_link1_rev"/>
-			<origin xyz="-0.0562 0.0246 0" rpy="-0.3927 3.1416 0"/>
+			<origin xyz="-0.0562 0.0246 0" rpy="-1.1781 0 3.1416"/>
 			<axis xyz="1 0 0"/>
 	    	<limit effort="1000.0" lower="-3.141593" upper="3.141593" velocity="0.5"/>

File: ginko_description/models/ginko_auto/urdf/modules/arm_r.urdf.xacro (robot description, xacro)
@@ -29,5 +29,5 @@
 		    <parent link="${parent}"/>
 			<child link="${name}_link0"/>
-		    <origin xyz="0 0 0" rpy="0 0 0"/>
+		    <origin xyz="0 0 0" rpy="0 0.3927 0"/>
 		    <axis xyz="0 1 0"/>
 			<limit effort="1000.0" lower="-2.6" upper="2.6" velocity="0.5"/>
@@ -59,5 +59,5 @@
 			<parent link="${name}_link0"/>
 			<child  link="${name}_link1"/>
-			<origin xyz="0.035 -0.0246 0" rpy="-0.3927 0 0"/>
+			<origin xyz="0.035 -0.0246 0" rpy="-1.1781 0 0"/>
 			<axis xyz="1 0 0"/>
 			<limit effort="1000.0" lower="-0.85" upper="1.18" velocity="0.5"/>
@@ -67,5 +67,5 @@
 			<parent link="${name}_link0"/>
 			<child  link="${name}_link1_rev"/>
-			<origin xyz="-0.0562 -0.0246 0" rpy="0.3927 3.1416 0"/>
+			<origin xyz="-0.0562 -0.0246 0" rpy="1.1781 0 3.1416"/>
 			<axis xyz="1 0 0"/>
 	    	<limit effort="1000.0" lower="-3.141593" upper="3.141593" velocity="0.5"/>

File: ginko_description/models/ginko_auto/urdf/modules/leg_l.urdf.xacro (robot description, xacro)
@@ -30,5 +30,5 @@
 			<child link="${name}_link0"/>
 		    <origin xyz="0 0 0" rpy="0 0 0"/>
-		    <axis xyz="1 0 0"/>
+		    <axis xyz="-1 0 0"/>
 			<limit effort="1000.0" lower="-0.8" upper="1.1781" velocity="0.5"/>
 		</joint>

Commit message: 胴体のみで動作確認中

File: ginko_description/models/ginko_auto/urdf/modules/arm_l.urdf.xacro (robot description, xacro)
@@ -20,9 +20,9 @@
 			</visual>
 			<!-- nothing worth -->
-			<inertial>
+<!-- 			<inertial>
 				<origin xyz="0 0 0" rpy="0 0 0"/>
 				<mass value="6.1"/>
 				<inertia ixx="0.0001" ixy="0.0" ixz="0.0" iyy="0.0001" iyz="0.0" izz="0.0001"/>
-			</inertial>
+			</inertial> -->
 		</link>
 		<joint name="${name}_joint0" type="revolute">

File: ginko_description/models/ginko_auto/urdf/modules/body.urdf.xacro (robot description, xacro)
@@ -16,12 +16,15 @@
 				<origin xyz="0 0 0" rpy="0 0 0"/>
 				<geometry>
-					<mesh filename="package://ginko_description/models/ginko_auto/meshes/dae/link00_chest.dae"/>
+					<mesh filename="package://ginko_description/models/ginko_auto/meshes/stl/link00_chest.stl"/>
+					<!-- <mesh filename="package://ginko_description/models/ginko_auto/meshes/dae/link00_chest.dae"/> -->
 				</geometry>
 			</visual>
-			<!-- nothing worth -->
 			<inertial>
-				<origin xyz="0 0 0" rpy="0 0 0"/>
-				<mass value="6.1"/>
-				<inertia ixx="0.0001" ixy="0.0" ixz="0.0" iyy="0.0001" iyz="0.0" izz="0.0001"/>
+				<mass value="0.45002697"/>
+				<origin xyz="0.00026100 0.00002855 0.04624115" rpy="0 0 0"/>
+				<inertia
+					ixx="0.00220956"
+					ixy="-0.00000074" iyy="0.00093793"
+					ixz="0.00003667" iyz="-0.00000052" izz="0.00247546"/>
 			</inertial>
 		</link>
@@ -48,9 +51,11 @@
 	    		</geometry>
 			</visual>
-			<!-- nothing worth -->
 			<inertial>
-				<origin xyz="0 0 0" rpy="0 0 0"/>
-				<mass value="6.1"/>
-				<inertia ixx="0.0001" ixy="0.0" ixz="0.0" iyy="0.0001" iyz="0.0" izz="0.0001"/>
+				<mass value="0.33312665"/>
+				<origin xyz="-0.01135452 -0.00000134 -0.02720222" rpy="0 0 0"/>
+				<inertia
+					ixx="0.00015328"
+					ixy="0.00000003" iyy="0.00073745"
+					ixz="0.00001078" iyz="0.00000000" izz="0.00073107"/>
 			</inertial>
 		</link>

File: ginko_description/models/ginko_auto/urdf/robot_gazebo.urdf.xacro (robot description, xacro)
@@ -4,7 +4,7 @@
   <xacro:include filename="$(find ginko_description)/models/ginko_auto/urdf/gazebo_modules/body.gazebo"/>
   <!-- Import all Gazebo-customization elements, including Gazebo colors -->
-  <xacro:include filename="$(find rrbot_description)/urdf/rrbot.gazebo" />
+  <!-- <xacro:include filename="$(find rrbot_description)/urdf/rrbot.gazebo" /> -->
   <!-- Import Rviz colors -->
-  <xacro:include filename="$(find rrbot_description)/urdf/materials.xacro" />
+  <!-- <xacro:include filename="$(find rrbot_description)/urdf/materials.xacro" /> -->
   <!-- Used for fixing robot to Gazebo 'base_link' -->
   <link name="base"/>
