Commit message: 腕が反映できない

File: ginko_description/models/ginko_auto/urdf/modules/arm_l.urdf.xacro (robot description, xacro)
@@ -9,5 +9,6 @@
 				<origin xyz="0 0 0" rpy="0 0 0"/>
 				<geometry>
-					<mesh filename="package://ginko_description/models/ginko_auto/meshes/stl/link09_l_arm01.stl"/>
+					<mesh filename="package://ginko_description/models/ginko_auto/meshes/stl/link01_waist.stl"/>
+					<!-- <mesh filename="package://ginko_description/models/ginko_auto/meshes/stl/link09_l_arm01.stl"/> -->
 				</geometry>
 			</collision>
@@ -16,13 +17,18 @@
 				<origin xyz="0 0 0" rpy="0 0 0"/>
 				<geometry>
-					<mesh filename="package://ginko_description/models/ginko_auto/meshes/dae/link09_l_arm01.dae"/>
+					<mesh filename="package://ginko_description/models/ginko_auto/meshes/stl/link01_waist.stl"/>
+					<!-- <mesh filename="package://ginko_description/models/ginko_auto/meshes/stl/link09_l_arm01.stl"/> -->
+					<!-- <mesh filename="package://ginko_description/models/ginko_auto/meshes/dae/link09_l_arm01.dae"/> -->
 				</geometry>
 			</visual>
 			<!-- nothing worth -->
-<!-- 			<inertial>
-				<origin xyz="0 0 0" rpy="0 0 0"/>
-				<mass value="6.1"/>
-				<inertia ixx="0.0001" ixy="0.0" ixz="0.0" iyy="0.0001" iyz="0.0" izz="0.0001"/>
-			</inertial> -->
+			<inertial>
+				<mass value="0.01356014"/>
+				<origin xyz="-0.01125790 0.00529265 0.00000000" rpy="0 0 0"/>
+				<inertia
+					ixx="0.00000235"
+					ixy="0.00000004" iyy="0.00001670"
+					ixz="0.00000000" iyz="0.00000000" izz="0.00001606"/>
+			</inertial>
 		</link>
 		<joint name="${name}_joint0" type="revolute">
@@ -46,12 +52,16 @@
 				<origin xyz="0 0 0" rpy="0 0 0"/>
 	    		<geometry>
-					<mesh filename="package://ginko_description/models/ginko_auto/meshes/dae/link10_l_arm02.dae"/>
+					<mesh filename="package://ginko_description/models/ginko_auto/meshes/stl/link10_l_arm02.stl"/>
+					<!-- <mesh filename="package://ginko_description/models/ginko_auto/meshes/dae/link10_l_arm02.dae"/> -->
 	    		</geometry>
 			</visual>
 			<!-- nothing worth -->
 			<inertial>
-				<origin xyz="0 0 0" rpy="0 0 0"/>
-				<mass value="6.1"/>
-				<inertia ixx="0.0001" ixy="0.0" ixz="0.0" iyy="0.0001" iyz="0.0" izz="0.0001"/>
+				<mass value="0.33139947"/>
+				<origin xyz="-0.02612786 0.02650564 -0.06333369" rpy="0 0 0"/>
+				<inertia
+					ixx="0.00115128"
+					ixy="0.00015366" iyy="0.00113572"
+					ixz="-0.00031848" iyz="-0.00037104" izz="0.00064743"/>
 			</inertial>
 		</link>
@@ -85,12 +95,16 @@
 				<origin xyz="0 0 0" rpy="0 0 0"/>
 	    		<geometry>
-					<mesh filename="package://ginko_description/models/ginko_auto/meshes/dae/link11_l_scissor01.dae"/>
+					<mesh filename="package://ginko_description/models/ginko_auto/meshes/stl/link11_l_scissor01.stl"/>
+					<!-- <mesh filename="package://ginko_description/models/ginko_auto/meshes/dae/link11_l_scissor01.dae"/> -->
 	    		</geometry>
 			</visual>
 			<!-- nothing worth -->
 			<inertial>
-				<origin xyz="0 0 0" rpy="0 0 0"/>
-				<mass value="6.1"/>
-				<inertia ixx="0.0001" ixy="0.0" ixz="0.0" iyy="0.0001" iyz="0.0" izz="0.0001"/>
+				<mass value="0.03287850"/>
+				<origin xyz="0.08234859 -0.030246866 0.00514112" rpy="0 0 0"/>
+				<inertia
+					ixx="0.00002277"
+					ixy="-0.00000014" iyy="0.00008197"
+					ixz="-0.00000058" iyz="-0.00000001" izz="0.00010105"/>
 			</inertial>
 		</link>
@@ -114,12 +128,16 @@
 				<origin xyz="0 0 0" rpy="0 0 0"/>
 	    		<geometry>
-					<mesh filename="package://ginko_description/models/ginko_auto/meshes/dae/link12_l_scissor02.dae"/>
+					<mesh filename="package://ginko_description/models/ginko_auto/meshes/stl/link12_l_scissor02.stl"/>
+					<!-- <mesh filename="package://ginko_description/models/ginko_auto/meshes/dae/link12_l_scissor02.dae"/> -->
 	    		</geometry>
 			</visual>
 			<!-- nothing worth -->
 			<inertial>
-				<origin xyz="0 0 0" rpy="0 0 0"/>
-				<mass value="6.1"/>
-				<inertia ixx="0.0001" ixy="0.0" ixz="0.0" iyy="0.0001" iyz="0.0" izz="0.0001"/>
+				<mass value="0.02936110"/>
+				<origin xyz="0.07807033 0.02515230 -0.00665437" rpy="0 0 0"/>
+				<inertia
+					ixx="0.00001452"
+					ixy="0.00000023" iyy="0.00006407"
+					ixz="-0.00000245" iyz="-0.00000002" izz="0.00008024"/>
 			</inertial>
 		</link>
@@ -133,16 +151,26 @@
 	  	<!-- LiDAR -->
 		<link name="${name}_urg_link">
+	    	<collision>
+				<origin xyz="0 0 0" rpy="0 0 0"/>
+	    		<geometry>
+					<mesh filename="package://ginko_description/models/ginko_auto/meshes/stl/urg.stl"/>
+	    		</geometry>
+			</collision>
 			<!-- Visualisation created from Color dae -->
 	    	<visual>
 				<origin xyz="0 0 0" rpy="0 0 0"/>
 	    		<geometry>
-					<mesh filename="package://ginko_description/models/ginko_auto/meshes/dae/urg.dae"/>
+	    			<mesh filename="package://ginko_description/models/ginko_auto/meshes/stl/urg.stl"/>
+					<!-- <mesh filename="package://ginko_description/models/ginko_auto/meshes/dae/urg.dae"/> -->
 	    		</geometry>
 			</visual>
 			<!-- nothing worth -->
 			<inertial>
-				<origin xyz="0 0 0" rpy="0 0 0"/>
-				<mass value="6.1"/>
-				<inertia ixx="0.0001" ixy="0.0" ixz="0.0" iyy="0.0001" iyz="0.0" izz="0.0001"/>
+				<mass value="0.16705492"/>
+				<origin xyz="-0.00014579 0.00000831 -0.02360505" rpy="0 0 0"/>
+				<inertia
+					ixx="0.00008801"
+					ixy="0.00000000" iyy="0.00008854"
+					ixz="-0.00000049" iyz="-0.00000004" izz="0.00006019"/>
 			</inertial>
 		</link>

File: ginko_description/models/ginko_auto/urdf/robot_gazebo.urdf.xacro (robot description, xacro)
@@ -3,4 +3,6 @@
   <xacro:include filename="$(find ginko_description)/models/ginko_auto/urdf/modules/body.urdf.xacro"/>
   <xacro:include filename="$(find ginko_description)/models/ginko_auto/urdf/gazebo_modules/body.gazebo"/>
+  <xacro:include filename="$(find ginko_description)/models/ginko_auto/urdf/modules/arm_l.urdf.xacro"/>
+  <xacro:include filename="$(find ginko_description)/models/ginko_auto/urdf/gazebo_modules/arm_l.gazebo"/>
   <!-- Import all Gazebo-customization elements, including Gazebo colors -->
   <!-- <xacro:include filename="$(find rrbot_description)/urdf/rrbot.gazebo" /> -->
@@ -9,5 +11,8 @@
   <!-- Used for fixing robot to Gazebo 'base_link' -->
   <link name="base"/>
-  <xacro:body name="body" parent="base"/>
-  <xacro:body_gazebo name="body" parent="base"/>
+  <!-- <xacro:body name="body" parent="base"/> -->
+  <!-- <xacro:body_gazebo name="body"/> -->
+<!--   <xacro:arm_l name="arm_l" parent="body_arm_l_link"/> -->
+  <xacro:arm_l name="arm_l" parent="base"/>
+  <!-- <xacro:arm_l_gazebo name="arm_l"/> -->
 </robot>

Commit message: gazeboは実体のないfix linkを挟むとダメらしい

File: ginko_description/models/ginko_auto/urdf/modules/arm_l.urdf.xacro (robot description, xacro)
@@ -9,6 +9,6 @@
 				<origin xyz="0 0 0" rpy="0 0 0"/>
 				<geometry>
-					<mesh filename="package://ginko_description/models/ginko_auto/meshes/stl/link01_waist.stl"/>
-					<!-- <mesh filename="package://ginko_description/models/ginko_auto/meshes/stl/link09_l_arm01.stl"/> -->
+					<!-- <mesh filename="package://ginko_description/models/ginko_auto/meshes/stl/link01_waist.stl"/> -->
+					<mesh filename="package://ginko_description/models/ginko_auto/meshes/stl/link09_l_arm01.stl"/>
 				</geometry>
 			</collision>
@@ -17,6 +17,6 @@
 				<origin xyz="0 0 0" rpy="0 0 0"/>
 				<geometry>
-					<mesh filename="package://ginko_description/models/ginko_auto/meshes/stl/link01_waist.stl"/>
-					<!-- <mesh filename="package://ginko_description/models/ginko_auto/meshes/stl/link09_l_arm01.stl"/> -->
+					<!-- <mesh filename="package://ginko_description/models/ginko_auto/meshes/stl/link01_waist.stl"/> -->
+					<mesh filename="package://ginko_description/models/ginko_auto/meshes/stl/link09_l_arm01.stl"/>
 					<!-- <mesh filename="package://ginko_description/models/ginko_auto/meshes/dae/link09_l_arm01.dae"/> -->
 				</geometry>
@@ -35,5 +35,5 @@
 		    <parent link="${parent}"/>
 			<child link="${name}_link0"/>
-		    <origin xyz="0 0 0" rpy="0 0.3927 0"/>
+		    <origin xyz="0 0.10683 0.05115" rpy="0 0.3927 0"/>
 		    <axis xyz="0 -1 0"/>
 			<limit effort="1000.0" lower="-2.6" upper="2.6" velocity="0.5"/>

File: ginko_description/models/ginko_auto/urdf/modules/body.urdf.xacro (robot description, xacro)
@@ -77,5 +77,5 @@
 		    <axis xyz="0 -1 0"/>
 		</joint>
-		<link name="${name}_arm_l_link"/>
+<!-- 		<link name="${name}_arm_l_link"/>
 		<joint name="${name}_joint3" type="fixed">
 		    <parent link="${name}_link0"/>
@@ -83,5 +83,5 @@
 		    <origin xyz="0 0.10683 0.05115" rpy="0 0 0"/>
 		    <axis xyz="0 1 0"/>
-		</joint>
+		</joint> -->
 		<link name="${name}_leg_r_link"/>
 		<joint name="${name}_joint4" type="fixed">

File: ginko_description/models/ginko_auto/urdf/robot_gazebo.urdf.xacro (robot description, xacro)
@@ -11,8 +11,8 @@
   <!-- Used for fixing robot to Gazebo 'base_link' -->
   <link name="base"/>
-  <!-- <xacro:body name="body" parent="base"/> -->
+  <xacro:body name="body" parent="base"/>
   <!-- <xacro:body_gazebo name="body"/> -->
-<!--   <xacro:arm_l name="arm_l" parent="body_arm_l_link"/> -->
-  <xacro:arm_l name="arm_l" parent="base"/>
-  <!-- <xacro:arm_l_gazebo name="arm_l"/> -->
+  <!-- <xacro:arm_l name="arm_l" parent="body_arm_l_link"/> -->
+  <xacro:arm_l name="arm_l" parent="body_link0"/>
+  <xacro:arm_l_gazebo name="arm_l"/>
 </robot>
