Commit message: 回転方向を合わせた

File: ginko_description/models/ginko_auto/urdf/modules/arm_r.urdf.xacro (robot description, xacro)
@@ -60,5 +60,5 @@
 			<child  link="${name}_link1"/>
 			<origin xyz="0.035 -0.0246 0" rpy="-0.3927 0 0"/>
-			<axis xyz="-1 0 0"/>
+			<axis xyz="1 0 0"/>
 			<limit effort="1000.0" lower="-0.85" upper="1.18" velocity="0.5"/>
 		</joint>
@@ -68,5 +68,5 @@
 			<child  link="${name}_link1_rev"/>
 			<origin xyz="-0.0562 -0.0246 0" rpy="0.3927 3.1416 0"/>
-			<axis xyz="-1 0 0"/>
+			<axis xyz="1 0 0"/>
 	    	<limit effort="1000.0" lower="-3.141593" upper="3.141593" velocity="0.5"/>
 	    	<mimic joint="${name}_joint1" multiplier="-1" offset="0"/>

File: ginko_description/models/ginko_auto/urdf/modules/leg_l.urdf.xacro (robot description, xacro)
@@ -121,7 +121,7 @@
 	    	<child  link="${name}_link3"/>
 	    	<origin xyz="0.1 0.0 0.0" rpy="0 -0.7854 0"/>
-	    	<axis xyz="0 -1 0"/>
+	    	<axis xyz="0 1 0"/>
 	    	<limit effort="1000.0" lower="-3.141593" upper="3.141593" velocity="0.5"/>
-	    	<!-- <mimic joint="${name}_joint1" multiplier="-1" offset="0"/>  -->
+	    	<!-- <mimic joint="${name}_joint1" multiplier="1" offset="0"/>  -->
 	  	</joint>
 		<!-- parallel link (lower-1st) -->
@@ -213,7 +213,7 @@
 	    	<child  link="${name}_link6"/>
 	    	<origin xyz="0.1 0.0 0.0" rpy="0 -2.3562 0"/>
-	    	<axis xyz="0 -1 0"/>
+	    	<axis xyz="0 1 0"/>
 	    	<limit effort="1000.0" lower="-3.141593" upper="3.141593" velocity="0.5"/>
-	    	<!-- <mimic joint="${name}_joint4" multiplier="-1" offset="0"/>  -->
+	    	<!-- <mimic joint="${name}_joint4" multiplier="1" offset="0"/>  -->
 	  	</joint>
 		<link name="${name}_link7">
@@ -275,4 +275,29 @@
 	    	<limit effort="1000.0" lower="-2.6" upper="2.6" velocity="0.5"/>
 	  	</joint>
+ <!-- toe edges -->
+		<link name="${name}_toe_link0"/>
+		<joint name="${name}_toe_joint0" type="fixed">
+	    	<parent link="${name}_link8"/>
+	    	<child  link="${name}_toe_link0"/>
+	    	<origin xyz="0.064 0.040 -0.005" rpy="0 0 0"/>
+	  	</joint>
+		<link name="${name}_toe_link1"/>
+		<joint name="${name}_toe_joint1" type="fixed">
+	    	<parent link="${name}_link8"/>
+	    	<child  link="${name}_toe_link1"/>
+	    	<origin xyz="-0.064 0.040 -0.005" rpy="0 0 0"/>
+	  	</joint>
+		<link name="${name}_toe_link2"/>
+		<joint name="${name}_toe_joint2" type="fixed">
+	    	<parent link="${name}_link8"/>
+	    	<child  link="${name}_toe_link2"/>
+	    	<origin xyz="-0.064 -0.040 -0.005" rpy="0 0 0"/>
+	  	</joint>
+		<link name="${name}_toe_link3"/>
+		<joint name="${name}_toe_joint3" type="fixed">
+	    	<parent link="${name}_link8"/>
+	    	<child  link="${name}_toe_link3"/>
+	    	<origin xyz="0.064 -0.040 -0.005" rpy="0 0 0"/>
+	  	</joint>
 	</xacro:macro>
 </robot>

File: ginko_description/models/ginko_auto/urdf/modules/leg_r.urdf.xacro (robot description, xacro)
@@ -121,7 +121,7 @@
 	    	<child  link="${name}_link3"/>
 	    	<origin xyz="0.1 0.0 0.0" rpy="0 -0.7854 0"/>
-	    	<axis xyz="0 1 0"/>
+	    	<axis xyz="0 -1 0"/>
 	    	<limit effort="1000.0" lower="-3.141593" upper="3.141593" velocity="0.5"/>
-	    	<!-- <mimic joint="${name}_joint1" multiplier="-1" offset="0"/>  -->
+	    	<!-- <mimic joint="${name}_joint1" multiplier="1" offset="0"/>  -->
 	  	</joint>
 		<!-- parallel link (lower-1st) -->
@@ -213,7 +213,7 @@
 	    	<child  link="${name}_link6"/>
 	    	<origin xyz="0.1 0.0 0.0" rpy="0 -2.3562 0"/>
-	    	<axis xyz="0 1 0"/>
+	    	<axis xyz="0 -1 0"/>
 	    	<limit effort="1000.0" lower="-3.141593" upper="3.141593" velocity="0.5"/>
-	    	<!-- <mimic joint="${name}_joint4" multiplier="-1" offset="0"/>  -->
+	    	<!-- <mimic joint="${name}_joint4" multiplier="1" offset="0"/>  -->
 	  	</joint>
 		<link name="${name}_link7">
@@ -275,4 +275,29 @@
 	    	<limit effort="1000.0" lower="-2.6" upper="2.6" velocity="0.5"/>
 	  	</joint>
+ <!-- toe edges -->
+		<link name="${name}_toe_link0"/>
+		<joint name="${name}_toe_joint0" type="fixed">
+	    	<parent link="${name}_link8"/>
+	    	<child  link="${name}_toe_link0"/>
+	    	<origin xyz="0.064 0.040 -0.005" rpy="0 0 0"/>
+	  	</joint>
+		<link name="${name}_toe_link1"/>
+		<joint name="${name}_toe_joint1" type="fixed">
+	    	<parent link="${name}_link8"/>
+	    	<child  link="${name}_toe_link1"/>
+	    	<origin xyz="-0.064 0.040 -0.005" rpy="0 0 0"/>
+	  	</joint>
+		<link name="${name}_toe_link2"/>
+		<joint name="${name}_toe_joint2" type="fixed">
+	    	<parent link="${name}_link8"/>
+	    	<child  link="${name}_toe_link2"/>
+	    	<origin xyz="-0.064 -0.040 -0.005" rpy="0 0 0"/>
+	  	</joint>
+		<link name="${name}_toe_link3"/>
+		<joint name="${name}_toe_joint3" type="fixed">
+	    	<parent link="${name}_link8"/>
+	    	<child  link="${name}_toe_link3"/>
+	    	<origin xyz="0.064 -0.040 -0.005" rpy="0 0 0"/>
+	  	</joint>
 	</xacro:macro>
 </robot>

Commit message: 右腕を取り付け

File: ginko_description/models/ginko_auto/urdf/modules/arm_r.urdf.xacro (robot description, xacro)
@@ -16,5 +16,6 @@
 				<origin xyz="0 0 0" rpy="0 0 0"/>
 				<geometry>
-					<mesh filename="package://ginko_description/models/ginko_auto/meshes/dae/link09_r_arm01.dae"/>
+					<mesh filename="package://ginko_description/models/ginko_auto/meshes/stl/link09_r_arm01.stl"/>
+					<!-- <mesh filename="package://ginko_description/models/ginko_auto/meshes/dae/link09_r_arm01.dae"/> -->
 				</geometry>
 			</visual>
@@ -29,5 +30,5 @@
 		    <parent link="${parent}"/>
 			<child link="${name}_link0"/>
-		    <origin xyz="0 0 0" rpy="0 0.3927 0"/>
+		    <origin xyz="0 -0.10683 0.05115" rpy="0 0.3927 0"/>
 		    <axis xyz="0 1 0"/>
 			<limit effort="1000.0" lower="-2.6" upper="2.6" velocity="0.5"/>
@@ -46,5 +47,6 @@
 				<origin xyz="0 0 0" rpy="0 0 0"/>
 	    		<geometry>
-					<mesh filename="package://ginko_description/models/ginko_auto/meshes/dae/link10_r_arm02.dae"/>
+					<mesh filename="package://ginko_description/models/ginko_auto/meshes/stl/link10_r_arm02.stl"/>
+					<!-- <mesh filename="package://ginko_description/models/ginko_auto/meshes/dae/link10_r_arm02.dae"/> -->
 	    		</geometry>
 			</visual>
@@ -85,5 +87,6 @@
 				<origin xyz="0 0 0" rpy="0 0 0"/>
 	    		<geometry>
-					<mesh filename="package://ginko_description/models/ginko_auto/meshes/dae/link11_r_scissor01.dae"/>
+					<mesh filename="package://ginko_description/models/ginko_auto/meshes/stl/link11_r_scissor01.stl"/>
+					<!-- <mesh filename="package://ginko_description/models/ginko_auto/meshes/dae/link11_r_scissor01.dae"/> -->
 	    		</geometry>
 			</visual>
@@ -114,5 +117,6 @@
 				<origin xyz="0 0 0" rpy="0 0 0"/>
 	    		<geometry>
-					<mesh filename="package://ginko_description/models/ginko_auto/meshes/dae/link12_r_scissor02.dae"/>
+					<mesh filename="package://ginko_description/models/ginko_auto/meshes/stl/link12_r_scissor02.stl"/>
+					<!-- <mesh filename="package://ginko_description/models/ginko_auto/meshes/dae/link12_r_scissor02.dae"/> -->
 	    		</geometry>
 			</visual>
@@ -133,16 +137,26 @@
 	  	<!-- LiDAR -->
 		<link name="${name}_urg_link">
+	    	<collision>
+				<origin xyz="0 0 0" rpy="0 0 0"/>
+	    		<geometry>
+					<mesh filename="package://ginko_description/models/ginko_auto/meshes/stl/urg.stl"/>
+	    		</geometry>
+			</collision>
 			<!-- Visualisation created from Color dae -->
 	    	<visual>
 				<origin xyz="0 0 0" rpy="0 0 0"/>
 	    		<geometry>
-					<mesh filename="package://ginko_description/models/ginko_auto/meshes/dae/urg.dae"/>
+	    			<mesh filename="package://ginko_description/models/ginko_auto/meshes/stl/urg.stl"/>
+					<!-- <mesh filename="package://ginko_description/models/ginko_auto/meshes/dae/urg.dae"/> -->
 	    		</geometry>
 			</visual>
 			<!-- nothing worth -->
 			<inertial>
-				<origin xyz="0 0 0" rpy="0 0 0"/>
-				<mass value="6.1"/>
-				<inertia ixx="0.0001" ixy="0.0" ixz="0.0" iyy="0.0001" iyz="0.0" izz="0.0001"/>
+				<mass value="0.16705492"/>
+				<origin xyz="-0.00014579 0.00000831 -0.02360505" rpy="0 0 0"/>
+				<inertia
+					ixx="0.00008801"
+					ixy="0.00000000" iyy="0.00008854"
+					ixz="-0.00000049" iyz="-0.00000004" izz="0.00006019"/>
 			</inertial>
 		</link>

File: ginko_description/models/ginko_auto/urdf/modules/body.urdf.xacro (robot description, xacro)
@@ -70,5 +70,5 @@
 			<limit effort="1000.0" lower="-2.6" upper="2.6" velocity="0.5"/>
 		</joint>
-		<link name="${name}_arm_r_link"/>
+<!-- 		<link name="${name}_arm_r_link"/>
 		<joint name="${name}_joint2" type="fixed">
 		    <parent link="${name}_link0"/>
@@ -76,5 +76,5 @@
 		    <origin xyz="0 -0.10683 0.05115" rpy="0 0 0"/>
 		    <axis xyz="0 -1 0"/>
-		</joint>
+		</joint> -->
 <!-- 		<link name="${name}_arm_l_link"/>
 		<joint name="${name}_joint3" type="fixed">

File: ginko_description/models/ginko_auto/urdf/robot_gazebo.urdf.xacro (robot description, xacro)
@@ -5,4 +5,6 @@
   <xacro:include filename="$(find ginko_description)/models/ginko_auto/urdf/modules/arm_l.urdf.xacro"/>
   <xacro:include filename="$(find ginko_description)/models/ginko_auto/urdf/gazebo_modules/arm_l.gazebo"/>
+  <xacro:include filename="$(find ginko_description)/models/ginko_auto/urdf/modules/arm_r.urdf.xacro"/>
+  <xacro:include filename="$(find ginko_description)/models/ginko_auto/urdf/gazebo_modules/arm_r.gazebo"/>
   <!-- Import all Gazebo-customization elements, including Gazebo colors -->
   <!-- <xacro:include filename="$(find rrbot_description)/urdf/rrbot.gazebo" /> -->
@@ -16,3 +18,5 @@
   <xacro:arm_l name="arm_l" parent="body_link0"/>
   <xacro:arm_l_gazebo name="arm_l"/>
+  <xacro:arm_r name="arm_r" parent="body_link0"/>
+  <xacro:arm_r_gazebo name="arm_r"/>
 </robot>
