Commit message: URDFにジャイロの位置を追加

File: ginko_description/models/ginko_auto/urdf/modules/body.urdf.xacro (robot description, xacro)
@@ -32,5 +32,5 @@
 		    <axis xyz="0 0 1"/>
 		</joint>
-		<!-- parallel link (upper-1st) -->
+		<!-- waist -->
 		<link name="${name}_link1">
 			<!-- Collision created from STL mesh without color -->
@@ -90,4 +90,10 @@
 		    <axis xyz="0 1 0"/>
 		</joint>
+		<link name="${name}_imu_link"/>
+		<joint name="${name}_imu_joint" type="fixed">
+	    	<parent link="${name}_link1"/>
+	    	<child  link="${name}_imu_link"/>
+	    	<origin xyz="-0.09 0 -0.0379" rpy="0 1.5708 0"/>
+	  	</joint>
 	</xacro:macro>
 </robot>

Commit message: デモに向けてパラメータ調整

File: ginko_description/models/ginko_auto/urdf/modules/body.urdf.xacro (robot description, xacro)
@@ -94,5 +94,6 @@
 	    	<parent link="${name}_link1"/>
 	    	<child  link="${name}_imu_link"/>
-	    	<origin xyz="-0.09 0 -0.0379" rpy="0 1.5708 0"/>
+	    	<origin xyz="-0.09 0 -0.0379" rpy="0 1.51 0"/>
+<!-- 	    	<origin xyz="-0.09 0 -0.0379" rpy="0 1.5708 0"/> -->
 	  	</joint>
 	</xacro:macro>

Commit message: トピック名を整理、rqt_graphを見やすくした

File: ginko_description/models/ginko_auto/urdf/modules/body.urdf.xacro (robot description, xacro)
@@ -94,7 +94,18 @@
 	    	<parent link="${name}_link1"/>
 	    	<child  link="${name}_imu_link"/>
-	    	<origin xyz="-0.09 0 -0.0379" rpy="0 1.51 0"/>
-<!-- 	    	<origin xyz="-0.09 0 -0.0379" rpy="0 1.5708 0"/> -->
+	    	<origin xyz="-0.09 0 -0.0379" rpy="0 1.5708 0"/>
 	  	</joint>
+<!-- 		<link name="${name}_imu_link_dummy"/>
+		<joint name="${name}_imu_joint_dummy" type="fixed">
+	    	<parent link="${name}_link1"/>
+	    	<child  link="${name}_imu_link_dummy"/>
+	    	<origin xyz="-0.09 0 -0.0379" rpy="0 1.48 0"/>
+	  	</joint>
+		<link name="${name}_imu_link"/>
+		<joint name="${name}_imu_joint" type="fixed">
+	    	<parent link="${name}_imu_link_dummy"/>
+	    	<child  link="${name}_imu_link"/>
+	    	<origin xyz="0 0 0" rpy="0 0 -0.025"/>
+	  	</joint> -->
 	</xacro:macro>
 </robot>

Commit message: 大枠ができてきた

File: ginko_description/models/ginko_auto/urdf/modules/body.urdf.xacro (robot description, xacro)
@@ -90,22 +90,16 @@
 		    <axis xyz="0 1 0"/>
 		</joint>
-		<link name="${name}_imu_link"/>
-		<joint name="${name}_imu_joint" type="fixed">
+		<link name="${name}_imu_attached_link"/>
+		<joint name="${name}_imu_attached_joint" type="fixed">
 	    	<parent link="${name}_link1"/>
-	    	<child  link="${name}_imu_link"/>
+	    	<child  link="${name}_imu_attached_link"/>
 	    	<origin xyz="-0.09 0 -0.0379" rpy="0 1.5708 0"/>
 	  	</joint>
-<!-- 		<link name="${name}_imu_link_dummy"/>
-		<joint name="${name}_imu_joint_dummy" type="fixed">
+		<link name="${name}_imu_base_link"/>
+		<joint name="${name}_imu_base_joint" type="fixed">
 	    	<parent link="${name}_link1"/>
-	    	<child  link="${name}_imu_link_dummy"/>
-	    	<origin xyz="-0.09 0 -0.0379" rpy="0 1.48 0"/>
+	    	<child  link="${name}_imu_base_link"/>
+	    	<origin xyz="-0.09 0 -0.0379" rpy="0 0 0"/>
 	  	</joint>
-		<link name="${name}_imu_link"/>
-		<joint name="${name}_imu_joint" type="fixed">
-	    	<parent link="${name}_imu_link_dummy"/>
-	    	<child  link="${name}_imu_link"/>
-	    	<origin xyz="0 0 0" rpy="0 0 -0.025"/>
-	  	</joint> -->
 	</xacro:macro>
 </robot>

Commit message: gazeboでうまく色がつかないので読み込むモデルをstlに変更

File: ginko_description/models/ginko_auto/urdf/modules/body.urdf.xacro (robot description, xacro)
@@ -16,4 +16,5 @@
 				<origin xyz="0 0 0" rpy="0 0 0"/>
 				<geometry>
+					<!-- <mesh filename="package://ginko_description/models/ginko_auto/meshes/obj/link00_chest.obj"/> -->
 					<mesh filename="package://ginko_description/models/ginko_auto/meshes/stl/link00_chest.stl"/>
 					<!-- <mesh filename="package://ginko_description/models/ginko_auto/meshes/dae/link00_chest.dae"/> -->
@@ -48,5 +49,7 @@
 				<origin xyz="0 0 0" rpy="0 0 0"/>
 	    		<geometry>
-					<mesh filename="package://ginko_description/models/ginko_auto/meshes/dae/link01_waist.dae"/>
+	    			<!-- <mesh filename="package://ginko_description/models/ginko_auto/meshes/obj/link01_waist.obj"/> -->
+					<mesh filename="package://ginko_description/models/ginko_auto/meshes/stl/link01_waist.stl"/>
+					<!-- <mesh filename="package://ginko_description/models/ginko_auto/meshes/dae/link01_waist.dae"/> -->
 	    		</geometry>
 			</visual>

Commit message: 胴体に1kg程度の錘を追加

File: ginko_description/models/ginko_auto/urdf/modules/body.urdf.xacro (robot description, xacro)
@@ -22,10 +22,10 @@
 			</visual>
 			<inertial>
-				<mass value="0.45002697"/>
-				<origin xyz="0.00026100 0.00002855 0.04624115" rpy="0 0 0"/>
+				<mass value="1.41502697"/>
+				<origin xyz="0.00008301 0.00000908 0.03819562" rpy="0 0 0"/>
 				<inertia
-					ixx="0.00220956"
-					ixy="-0.00000074" iyy="0.00093793"
-					ixz="0.00003667" iyz="-0.00000052" izz="0.00247546"/>
+					ixx="0.00454987"
+					ixy="-0.00000074" iyy="0.00327828"
+					ixz="0.00004210" iyz="-0.00000007" izz="0.00287757"/>
 			</inertial>
 		</link>

Commit message: 左足検証中

File: ginko_description/models/ginko_auto/urdf/modules/body.urdf.xacro (robot description, xacro)
@@ -91,5 +91,5 @@
 		    <axis xyz="0 1 0"/>
 		</joint>
-		<link name="${name}_leg_l_link"/>
+<!-- 		<link name="${name}_leg_l_link"/>
 		<joint name="${name}_joint5" type="fixed">
 		    <parent link="${name}_link1"/>
@@ -97,5 +97,5 @@
 		    <origin xyz="-0.0404 0.0 -0.0409" rpy="0 0 0"/>
 		    <axis xyz="0 1 0"/>
-		</joint>
+		</joint> -->
 		<link name="${name}_imu_attached_link"/>
 		<joint name="${name}_imu_attached_joint" type="fixed">

File: ginko_description/models/ginko_auto/urdf/modules/leg_l.urdf.xacro (robot description, xacro)
@@ -16,12 +16,15 @@
 				<origin xyz="0 0 0" rpy="0 0 0"/>
 				<geometry>
-					<mesh filename="package://ginko_description/models/ginko_auto/meshes/dae/link02_l_femoral.dae"/>
+					<mesh filename="package://ginko_description/models/ginko_auto/meshes/stl/link02_l_femoral.stl"/>
+					<!-- <mesh filename="package://ginko_description/models/ginko_auto/meshes/dae/link02_l_femoral.dae"/> -->
 				</geometry>
 			</visual>
-			<!-- nothing worth -->
-			<inertial>
-				<origin xyz="0 0 0" rpy="0 0 0"/>
-				<mass value="6.1"/>
-				<inertia ixx="0.0001" ixy="0.0" ixz="0.0" iyy="0.0001" iyz="0.0" izz="0.0001"/>
+			<inertial>
+				<mass value="0.03433352"/>
+				<origin xyz="0.02930795 0.03723759 -0.02605386" rpy="0 0 0"/>
+				<inertia
+					ixx="0.00002443"
+					ixy="-0.00000021" iyy="0.00002287"
+					ixz="-0.00000021" iyz="-0.00000391" izz="0.00002983"/>
 			</inertial>
 		</link>
@@ -29,5 +32,5 @@
 		    <parent link="${parent}"/>
 			<child link="${name}_link0"/>
-		    <origin xyz="0 0 0" rpy="0 0 0"/>
+			<origin xyz="-0.0404 0.0 -0.0409" rpy="0 0 0"/>
 		    <axis xyz="-1 0 0"/>
 			<limit effort="1000.0" lower="-0.8" upper="1.1781" velocity="0.5"/>
@@ -46,12 +49,15 @@
 				<origin xyz="0 0 0" rpy="0 0 0"/>
 	    		<geometry>
-					<mesh filename="package://ginko_description/models/ginko_auto/meshes/dae/link03_l_leg01.dae"/>
-	    		</geometry>
-			</visual>
-			<!-- nothing worth -->
-			<inertial>
-				<origin xyz="0 0 0" rpy="0 0 0"/>
-				<mass value="6.1"/>
-				<inertia ixx="0.0001" ixy="0.0" ixz="0.0" iyy="0.0001" iyz="0.0" izz="0.0001"/>
+					<mesh filename="package://ginko_description/models/ginko_auto/meshes/stl/link03_l_leg01.stl"/>
+					<!-- <mesh filename="package://ginko_description/models/ginko_auto/meshes/dae/link03_l_leg01.dae"/> -->
+	    		</geometry>
+			</visual>
+			<inertial>
+				<mass value="0.18525692"/>
+				<origin xyz="0.05000000 0.03285059 0.00068146" rpy="0 0 0"/>
+				<inertia
+					ixx="0.00041331"
+					ixy="-0.00003605" iyy="0.00027917"
+					ixz="-0.00000000" iyz="-0.00000184" izz="0.00066510"/>
 			</inertial>
 		</link>
@@ -76,12 +82,15 @@
 				<origin xyz="0 0 0" rpy="0 0 0"/>
 	    		<geometry>
-					<mesh filename="package://ginko_description/models/ginko_auto/meshes/dae/link04_l_leg02.dae"/>
-	    		</geometry>
-			</visual>
-			<!-- nothing worth -->
-			<inertial>
-				<origin xyz="0 0 0" rpy="0 0 0"/>
-				<mass value="6.1"/>
-				<inertia ixx="0.0001" ixy="0.0" ixz="0.0" iyy="0.0001" iyz="0.0" izz="0.0001"/>
+					<mesh filename="package://ginko_description/models/ginko_auto/meshes/stl/link04_l_leg02.stl"/>
+					<!-- <mesh filename="package://ginko_description/models/ginko_auto/meshes/dae/link04_l_leg02.dae"/> -->
+	    		</geometry>
+			</visual>
+			<inertial>
+				<mass value="0.01646643"/>
+				<origin xyz="0.05000000 0.02495100 -0.00491150" rpy="0 0 0"/>
+				<inertia
+					ixx="0.00000640"
+					ixy="0.00000000" iyy="0.00001642"
+					ixz="0.00000000" iyz="0.00000000" izz="0.00002264"/>
 			</inertial>
 		</link>
@@ -92,9 +101,8 @@
 	    	<axis xyz="0 -1 0"/>
 	    	<limit effort="1000.0" lower="-3.141593" upper="3.141593" velocity="0.5"/>
-	    	<mimic joint="${name}_joint1" multiplier="1" offset="0"/>
+	    	<!-- <mimic joint="${name}_joint1" multiplier="1" offset="0"/>  -->
 	  	</joint>
 		<!-- knee -->
-		<link name="${name}_link3">
-			<!-- Collision created from STL mesh without color -->
+<!-- 		<link name="${name}_link3">
 	    	<collision>
 				<origin xyz="0 0 0" rpy="0 0 0"/>
@@ -103,5 +111,4 @@
 	    		</geometry>
 			</collision>
-			<!-- Visualisation created from Color dae -->
 	    	<visual>
 				<origin xyz="0 0 0" rpy="0 0 0"/>
@@ -110,5 +117,4 @@
 	    		</geometry>
 			</visual>
-			<!-- nothing worth -->
 			<inertial>
 				<origin xyz="0 0 0" rpy="0 0 0"/>
@@ -123,9 +129,7 @@
 	    	<axis xyz="0 1 0"/>
 	    	<limit effort="1000.0" lower="-3.141593" upper="3.141593" velocity="0.5"/>
-	    	<!-- <mimic joint="${name}_joint1" multiplier="1" offset="0"/>  -->
-	  	</joint>
+	  	</joint> -->
 		<!-- parallel link (lower-1st) -->
-		<link name="${name}_link4">
-			<!-- Collision created from STL mesh without color -->
+<!-- 		<link name="${name}_link4">
 			<collision>
 				<origin xyz="0 0 0" rpy="0 0 0"/>
@@ -134,5 +138,4 @@
 	    		</geometry>
 			</collision>
-			<!-- Visualisation created from Color dae -->
 	    	<visual>
 				<origin xyz="0 0 0" rpy="0 0 0"/>
@@ -141,5 +144,4 @@
 	    		</geometry>
 			</visual>
-			<!-- nothing worth -->
 			<inertial>
 				<origin xyz="0 0 0" rpy="0 0 0"/>
@@ -154,8 +156,7 @@
 			<axis xyz="0 -1 0"/>
 			<limit effort="1000.0" lower="-0.7854" upper="1.3" velocity="0.5"/>
-		</joint>
+		</joint> -->
 		<!-- parallel link (lower-2nd) -->
-		<link name="${name}_link5">
-			<!-- Collision created from STL mesh without color -->
+<!-- 		<link name="${name}_link5">
 	    	<collision>
 				<origin xyz="0 0 0" rpy="0 0 0"/>
@@ -164,5 +165,4 @@
 	    		</geometry>
 			</collision>
-			<!-- Visualisation created from Color dae -->
 	    	<visual>
 				<origin xyz="0 0 0" rpy="0 0 0"/>
@@ -171,5 +171,4 @@
 	    		</geometry>
 			</visual>
-			<!-- nothing worth -->
 			<inertial>
 				<origin xyz="0 0 0" rpy="0 0 0"/>
@@ -185,8 +184,7 @@
 	    	<limit effort="1000.0" lower="-3.141593" upper="3.141593" velocity="0.5"/>
 	    	<mimic joint="${name}_joint4" multiplier="1" offset="0"/>
-	  	</joint>
+	  	</joint> -->
 		<!-- toe -->
-		<link name="${name}_link6">
-			<!-- Collision created from STL mesh without color -->
+<!-- 		<link name="${name}_link6">
 	    	<collision>
 				<origin xyz="0 0 0" rpy="0 0 0"/>
@@ -195,5 +193,4 @@
 	    		</geometry>
 			</collision>
-			<!-- Visualisation created from Color dae -->
 	    	<visual>
 				<origin xyz="0 0 0" rpy="0 0 0"/>
@@ -202,5 +199,4 @@
 	    		</geometry>
 			</visual>
-			<!-- nothing worth -->
 			<inertial>
 				<origin xyz="0 0 0" rpy="0 0 0"/>
@@ -215,8 +211,6 @@
 	    	<axis xyz="0 1 0"/>
 	    	<limit effort="1000.0" lower="-3.141593" upper="3.141593" velocity="0.5"/>
-	    	<!-- <mimic joint="${name}_joint4" multiplier="1" offset="0"/>  -->
 	  	</joint>
 		<link name="${name}_link7">
-			<!-- Collision created from STL mesh without color -->
 	    	<collision>
 				<origin xyz="0 0 0" rpy="0 0 0"/>
@@ -225,5 +219,4 @@
 	    		</geometry>
 			</collision>
-			<!-- Visualisation created from Color dae -->
 	    	<visual>
 				<origin xyz="0 0 0" rpy="0 0 0"/>
@@ -232,5 +225,4 @@
 	    		</geometry>
 			</visual>
-			<!-- nothing worth -->
 			<inertial>
 				<origin xyz="0 0 0" rpy="0 0 0"/>
@@ -247,5 +239,4 @@
 	  	</joint>
 		<link name="${name}_link8">
-			<!-- Collision created from STL mesh without color -->
 	    	<collision>
 				<origin xyz="0 0 0" rpy="0 0 0"/>
@@ -254,5 +245,4 @@
 	    		</geometry>
 			</collision>
-			<!-- Visualisation created from Color dae -->
 	    	<visual>
 				<origin xyz="0 0 0" rpy="0 0 0"/>
@@ -261,5 +251,4 @@
 	    		</geometry>
 			</visual>
-			<!-- nothing worth -->
 			<inertial>
 				<origin xyz="0 0 0" rpy="0 0 0"/>
@@ -274,7 +263,7 @@
 	    	<axis xyz="0 0 1"/>
 	    	<limit effort="1000.0" lower="-2.6" upper="2.6" velocity="0.5"/>
-	  	</joint>
+	  	</joint> -->
  <!-- toe edges -->
-		<link name="${name}_toe_link0"/>
+<!-- 		<link name="${name}_toe_link0"/>
 		<joint name="${name}_toe_joint0" type="fixed">
 	    	<parent link="${name}_link8"/>
@@ -305,5 +294,5 @@
 	    	<child  link="${name}_toe_center"/>
 	    	<origin xyz="0.0 0.0 -0.005" rpy="0 0 0"/>
-	  	</joint>
+	  	</joint> -->
 	</xacro:macro>
 </robot>

File: ginko_description/models/ginko_auto/urdf/robot_gazebo.urdf.xacro (robot description, xacro)
@@ -7,4 +7,6 @@
   <xacro:include filename="$(find ginko_description)/models/ginko_auto/urdf/modules/arm_r.urdf.xacro"/>
   <xacro:include filename="$(find ginko_description)/models/ginko_auto/urdf/gazebo_modules/arm_r.gazebo"/>
+  <xacro:include filename="$(find ginko_description)/models/ginko_auto/urdf/modules/leg_l.urdf.xacro"/>
+  <xacro:include filename="$(find ginko_description)/models/ginko_auto/urdf/gazebo_modules/leg_l.gazebo"/>
   <!-- Import all Gazebo-customization elements, including Gazebo colors -->
   <!-- <xacro:include filename="$(find rrbot_description)/urdf/rrbot.gazebo" /> -->
@@ -20,3 +22,5 @@
   <xacro:arm_r name="arm_r" parent="body_link0"/>
   <xacro:arm_r_gazebo name="arm_r"/>
+  <xacro:leg_l name="leg_l" parent="body_link1"/>
+  <xacro:leg_l_gazebo name="leg_l"/>
 </robot>
