Commit message: サーボの動きに対応してrvizで動きが見えるようにした

File: ginko_description/models/ginko_auto/urdf/modules/leg_l.urdf.xacro (robot description, xacro)
@@ -123,5 +123,5 @@
 	    	<axis xyz="0 -1 0"/>
 	    	<limit effort="1000.0" lower="-3.141593" upper="3.141593" velocity="0.5"/>
-	    	<mimic joint="${name}_joint1" multiplier="-1" offset="0"/>
+	    	<!-- <mimic joint="${name}_joint1" multiplier="-1" offset="0"/>  -->
 	  	</joint>
 		<!-- parallel link (lower-1st) -->
@@ -215,5 +215,5 @@
 	    	<axis xyz="0 -1 0"/>
 	    	<limit effort="1000.0" lower="-3.141593" upper="3.141593" velocity="0.5"/>
-	    	<mimic joint="${name}_joint4" multiplier="-1" offset="0"/>
+	    	<!-- <mimic joint="${name}_joint4" multiplier="-1" offset="0"/>  -->
 	  	</joint>
 		<link name="${name}_link7">

File: ginko_description/models/ginko_auto/urdf/modules/leg_l_mimic.urdf.xacro (robot description, xacro)
@@ -1,5 +1,5 @@
 <?xml version="1.0"?>
-<robot name="leg_r" xmlns:xacro="http://www.ros.org/wiki/xacro">
-	<xacro:macro name="leg_r" params="name parent">
+<robot name="leg_l" xmlns:xacro="http://www.ros.org/wiki/xacro">
+	<xacro:macro name="leg_l" params="name parent">
 	<!-- <xacro:property name="name" value="leg"/> -->
 		<!-- Link conencts from body. Femoral first. -->
@@ -9,5 +9,5 @@
 				<origin xyz="0 0 0" rpy="0 0 0"/>
 				<geometry>
-					<mesh filename="package://ginko_description/models/ginko_auto/meshes/stl/link02_r_femoral.stl"/>
+					<mesh filename="package://ginko_description/models/ginko_auto/meshes/stl/link02_l_femoral.stl"/>
 				</geometry>
 			</collision>
@@ -16,5 +16,5 @@
 				<origin xyz="0 0 0" rpy="0 0 0"/>
 				<geometry>
-					<mesh filename="package://ginko_description/models/ginko_auto/meshes/dae/link02_r_femoral.dae"/>
+					<mesh filename="package://ginko_description/models/ginko_auto/meshes/dae/link02_l_femoral.dae"/>
 				</geometry>
 			</visual>
@@ -29,7 +29,7 @@
 		    <parent link="${parent}"/>
 			<child link="${name}_link0"/>
-		    <origin xyz="0 0 0" rpy="-0.39217 0 0"/>
+		    <origin xyz="0 0 0" rpy="0.39217 0 0"/>
 		    <axis xyz="1 0 0"/>
-			<limit effort="1000.0" lower="-1.1781" upper="0.8" velocity="0.5"/>
+			<limit effort="1000.0" lower="-0.8" upper="1.1781" velocity="0.5"/>
 		</joint>
 		<!-- parallel link (upper-1st) -->
@@ -39,12 +39,12 @@
 				<origin xyz="0 0 0" rpy="0 0 0"/>
 	    		<geometry>
-					<mesh filename="package://ginko_description/models/ginko_auto/meshes/stl/link03_r_leg01.stl"/>
-	    		</geometry>
-			</collision>
-			<!-- Visualisation created from Color dae -->
-	    	<visual>
-				<origin xyz="0 0 0" rpy="0 0 0"/>
-	    		<geometry>
-					<mesh filename="package://ginko_description/models/ginko_auto/meshes/dae/link03_r_leg01.dae"/>
+					<mesh filename="package://ginko_description/models/ginko_auto/meshes/stl/link03_l_leg01.stl"/>
+	    		</geometry>
+			</collision>
+			<!-- Visualisation created from Color dae -->
+	    	<visual>
+				<origin xyz="0 0 0" rpy="0 0 0"/>
+	    		<geometry>
+					<mesh filename="package://ginko_description/models/ginko_auto/meshes/dae/link03_l_leg01.dae"/>
 	    		</geometry>
 			</visual>
@@ -59,7 +59,7 @@
 			<parent link="${name}_link0"/>
 			<child  link="${name}_link1"/>
-			<origin xyz="-0.0163 0.0148 -0.0364" rpy="0 0.7854 0"/>
-			<axis xyz="0 1 0"/>
-			<limit effort="1000.0" lower="-0.7854" upper="1.3" velocity="0.5"/>
+			<origin xyz="-0.0163 -0.0148 -0.0364" rpy="0 0.7854 0"/>
+			<axis xyz="0 -1 0"/>
+			<limit effort="1000.0" lower="-1.3" upper="0.7854" velocity="0.5"/>
 		</joint>
 		<!-- parallel link (upper-2nd) -->
@@ -69,12 +69,12 @@
 				<origin xyz="0 0 0" rpy="0 0 0"/>
 	    		<geometry>
-					<mesh filename="package://ginko_description/models/ginko_auto/meshes/stl/link04_r_leg02.stl"/>
-	    		</geometry>
-			</collision>
-			<!-- Visualisation created from Color dae -->
-	    	<visual>
-				<origin xyz="0 0 0" rpy="0 0 0"/>
-	    		<geometry>
-					<mesh filename="package://ginko_description/models/ginko_auto/meshes/dae/link04_r_leg02.dae"/>
+					<mesh filename="package://ginko_description/models/ginko_auto/meshes/stl/link04_l_leg02.stl"/>
+	    		</geometry>
+			</collision>
+			<!-- Visualisation created from Color dae -->
+	    	<visual>
+				<origin xyz="0 0 0" rpy="0 0 0"/>
+	    		<geometry>
+					<mesh filename="package://ginko_description/models/ginko_auto/meshes/dae/link04_l_leg02.dae"/>
 	    		</geometry>
 			</visual>
@@ -89,6 +89,6 @@
 	    	<parent link="${name}_link0"/>
 	    	<child  link="${name}_link2"/>
-	    	<origin xyz="-0.0376 0.0148 -0.04845" rpy="0 0.7854 0"/>
-	    	<axis xyz="0 1 0"/>
+	    	<origin xyz="-0.0376 -0.0148 -0.04845" rpy="0 0.7854 0"/>
+	    	<axis xyz="0 -1 0"/>
 	    	<limit effort="1000.0" lower="-3.141593" upper="3.141593" velocity="0.5"/>
 	    	<mimic joint="${name}_joint1" multiplier="1" offset="0"/>
@@ -100,12 +100,12 @@
 				<origin xyz="0 0 0" rpy="0 0 0"/>
 	    		<geometry>
-					<mesh filename="package://ginko_description/models/ginko_auto/meshes/stl/link05_r_knee.stl"/>
-	    		</geometry>
-			</collision>
-			<!-- Visualisation created from Color dae -->
-	    	<visual>
-				<origin xyz="0 0 0" rpy="0 0 0"/>
-	    		<geometry>
-					<mesh filename="package://ginko_description/models/ginko_auto/meshes/dae/link05_r_knee.dae"/>
+					<mesh filename="package://ginko_description/models/ginko_auto/meshes/stl/link05_l_knee.stl"/>
+	    		</geometry>
+			</collision>
+			<!-- Visualisation created from Color dae -->
+	    	<visual>
+				<origin xyz="0 0 0" rpy="0 0 0"/>
+	    		<geometry>
+					<mesh filename="package://ginko_description/models/ginko_auto/meshes/dae/link05_l_knee.dae"/>
 	    		</geometry>
 			</visual>
@@ -121,7 +121,7 @@
 	    	<child  link="${name}_link3"/>
 	    	<origin xyz="0.1 0.0 0.0" rpy="0 -0.7854 0"/>
-	    	<axis xyz="0 1 0"/>
-	    	<limit effort="1000.0" lower="-3.141593" upper="3.141593" velocity="0.5"/>
-	    	<!-- <mimic joint="${name}_joint1" multiplier="-1" offset="0"/>  -->
+	    	<axis xyz="0 -1 0"/>
+	    	<limit effort="1000.0" lower="-3.141593" upper="3.141593" velocity="0.5"/>
+	    	<mimic joint="${name}_joint1" multiplier="-1" offset="0"/>
 	  	</joint>
 		<!-- parallel link (lower-1st) -->
@@ -131,12 +131,12 @@
 				<origin xyz="0 0 0" rpy="0 0 0"/>
 	    		<geometry>
-					<mesh filename="package://ginko_description/models/ginko_auto/meshes/stl/link03_r_leg01.stl"/>
-	    		</geometry>
-			</collision>
-			<!-- Visualisation created from Color dae -->
-	    	<visual>
-				<origin xyz="0 0 0" rpy="0 0 0"/>
-	    		<geometry>
-					<mesh filename="package://ginko_description/models/ginko_auto/meshes/dae/link03_r_leg01.dae"/>
+					<mesh filename="package://ginko_description/models/ginko_auto/meshes/stl/link03_l_leg01.stl"/>
+	    		</geometry>
+			</collision>
+			<!-- Visualisation created from Color dae -->
+	    	<visual>
+				<origin xyz="0 0 0" rpy="0 0 0"/>
+	    		<geometry>
+					<mesh filename="package://ginko_description/models/ginko_auto/meshes/dae/link03_l_leg01.dae"/>
 	    		</geometry>
 			</visual>
@@ -152,6 +152,6 @@
 			<child  link="${name}_link4"/>
 			<origin xyz="0 0 -0.0386" rpy="0 2.3562 0"/>
-			<axis xyz="0 1 0"/>
-			<limit effort="1000.0" lower="-1.3" upper="0.7854" velocity="0.5"/>
+			<axis xyz="0 -1 0"/>
+			<limit effort="1000.0" lower="-0.7854" upper="1.3" velocity="0.5"/>
 		</joint>
 		<!-- parallel link (lower-2nd) -->
@@ -161,12 +161,12 @@
 				<origin xyz="0 0 0" rpy="0 0 0"/>
 	    		<geometry>
-					<mesh filename="package://ginko_description/models/ginko_auto/meshes/stl/link04_r_leg02.stl"/>
-	    		</geometry>
-			</collision>
-			<!-- Visualisation created from Color dae -->
-	    	<visual>
-				<origin xyz="0 0 0" rpy="0 0 0"/>
-	    		<geometry>
-					<mesh filename="package://ginko_description/models/ginko_auto/meshes/dae/link04_r_leg02.dae"/>
+					<mesh filename="package://ginko_description/models/ginko_auto/meshes/stl/link04_l_leg02.stl"/>
+	    		</geometry>
+			</collision>
+			<!-- Visualisation created from Color dae -->
+	    	<visual>
+				<origin xyz="0 0 0" rpy="0 0 0"/>
+	    		<geometry>
+					<mesh filename="package://ginko_description/models/ginko_auto/meshes/dae/link04_l_leg02.dae"/>
 	    		</geometry>
 			</visual>
@@ -182,5 +182,5 @@
 	    	<child  link="${name}_link5"/>
 	    	<origin xyz="-0.0213 0 -0.02655" rpy="0 2.3562 0"/>
-	    	<axis xyz="0 1 0"/>
+	    	<axis xyz="0 -1 0"/>
 	    	<limit effort="1000.0" lower="-3.141593" upper="3.141593" velocity="0.5"/>
 	    	<mimic joint="${name}_joint4" multiplier="1" offset="0"/>
@@ -192,12 +192,12 @@
 				<origin xyz="0 0 0" rpy="0 0 0"/>
 	    		<geometry>
-					<mesh filename="package://ginko_description/models/ginko_auto/meshes/stl/link06_r_toe01.stl"/>
-	    		</geometry>
-			</collision>
-			<!-- Visualisation created from Color dae -->
-	    	<visual>
-				<origin xyz="0 0 0" rpy="0 0 0"/>
-	    		<geometry>
-					<mesh filename="package://ginko_description/models/ginko_auto/meshes/dae/link06_r_toe01.dae"/>
+					<mesh filename="package://ginko_description/models/ginko_auto/meshes/stl/link06_l_toe01.stl"/>
+	    		</geometry>
+			</collision>
+			<!-- Visualisation created from Color dae -->
+	    	<visual>
+				<origin xyz="0 0 0" rpy="0 0 0"/>
+	    		<geometry>
+					<mesh filename="package://ginko_description/models/ginko_auto/meshes/dae/link06_l_toe01.dae"/>
 	    		</geometry>
 			</visual>
@@ -213,7 +213,7 @@
 	    	<child  link="${name}_link6"/>
 	    	<origin xyz="0.1 0.0 0.0" rpy="0 -2.3562 0"/>
-	    	<axis xyz="0 1 0"/>
-	    	<limit effort="1000.0" lower="-3.141593" upper="3.141593" velocity="0.5"/>
-	    	<!-- <mimic joint="${name}_joint4" multiplier="-1" offset="0"/>  -->
+	    	<axis xyz="0 -1 0"/>
+	    	<limit effort="1000.0" lower="-3.141593" upper="3.141593" velocity="0.5"/>
+	    	<mimic joint="${name}_joint4" multiplier="-1" offset="0"/>
 	  	</joint>
 		<link name="${name}_link7">
@@ -222,12 +222,12 @@
 				<origin xyz="0 0 0" rpy="0 0 0"/>
 	    		<geometry>
-					<mesh filename="package://ginko_description/models/ginko_auto/meshes/stl/link07_r_toe02.stl"/>
-	    		</geometry>
-			</collision>
-			<!-- Visualisation created from Color dae -->
-	    	<visual>
-				<origin xyz="0 0 0" rpy="0 0 0"/>
-	    		<geometry>
-					<mesh filename="package://ginko_description/models/ginko_auto/meshes/dae/link07_r_toe02.dae"/>
+					<mesh filename="package://ginko_description/models/ginko_auto/meshes/stl/link07_l_toe02.stl"/>
+	    		</geometry>
+			</collision>
+			<!-- Visualisation created from Color dae -->
+	    	<visual>
+				<origin xyz="0 0 0" rpy="0 0 0"/>
+	    		<geometry>
+					<mesh filename="package://ginko_description/models/ginko_auto/meshes/dae/link07_l_toe02.dae"/>
 	    		</geometry>
 			</visual>
@@ -242,5 +242,5 @@
 	    	<parent link="${name}_link6"/>
 	    	<child  link="${name}_link7"/>
-	    	<origin xyz="-0.028 -0.02475 -0.0391" rpy="0 0 0"/>
+	    	<origin xyz="-0.028 0.02475 -0.0391" rpy="0 0 0"/>
 	    	<axis xyz="-1 0 0"/>
 	    	<limit effort="1000.0" lower="-1.6" upper="1.6" velocity="0.5"/>
@@ -251,12 +251,12 @@
 				<origin xyz="0 0 0" rpy="0 0 0"/>
 	    		<geometry>
-					<mesh filename="package://ginko_description/models/ginko_auto/meshes/stl/link08_r_toe03.stl"/>
-	    		</geometry>
-			</collision>
-			<!-- Visualisation created from Color dae -->
-	    	<visual>
-				<origin xyz="0 0 0" rpy="0 0 0"/>
-	    		<geometry>
-					<mesh filename="package://ginko_description/models/ginko_auto/meshes/dae/link08_r_toe03.dae"/>
+					<mesh filename="package://ginko_description/models/ginko_auto/meshes/stl/link08_l_toe03.stl"/>
+	    		</geometry>
+			</collision>
+			<!-- Visualisation created from Color dae -->
+	    	<visual>
+				<origin xyz="0 0 0" rpy="0 0 0"/>
+	    		<geometry>
+					<mesh filename="package://ginko_description/models/ginko_auto/meshes/dae/link08_l_toe03.dae"/>
 	    		</geometry>
 			</visual>

File: ginko_description/models/ginko_auto/urdf/modules/leg_r.urdf_mimic.xacro (robot description, xacro)
@@ -123,5 +123,5 @@
 	    	<axis xyz="0 1 0"/>
 	    	<limit effort="1000.0" lower="-3.141593" upper="3.141593" velocity="0.5"/>
-	    	<!-- <mimic joint="${name}_joint1" multiplier="-1" offset="0"/>  -->
+	    	<mimic joint="${name}_joint1" multiplier="-1" offset="0"/>
 	  	</joint>
 		<!-- parallel link (lower-1st) -->
@@ -215,5 +215,5 @@
 	    	<axis xyz="0 1 0"/>
 	    	<limit effort="1000.0" lower="-3.141593" upper="3.141593" velocity="0.5"/>
-	    	<!-- <mimic joint="${name}_joint4" multiplier="-1" offset="0"/>  -->
+	    	<mimic joint="${name}_joint4" multiplier="-1" offset="0"/>
 	  	</joint>
 		<link name="${name}_link7">

Commit message: 足裏中心をurdfに追加

File: ginko_description/models/ginko_auto/urdf/modules/leg_l.urdf.xacro (robot description, xacro)
@@ -300,4 +300,10 @@
 	    	<origin xyz="0.064 -0.040 -0.005" rpy="0 0 0"/>
 	  	</joint>
+		<link name="${name}_toe_link0"/>
+		<joint name="${name}_toe_center" type="fixed">
+	    	<parent link="${name}_link8"/>
+	    	<child  link="${name}_toe_link0"/>
+	    	<origin xyz="0.0 0.0 -0.005" rpy="0 0 0"/>
+	  	</joint>
 	</xacro:macro>
 </robot>

File: ginko_description/models/ginko_auto/urdf/modules/leg_r.urdf.xacro (robot description, xacro)
@@ -300,4 +300,10 @@
 	    	<origin xyz="0.064 -0.040 -0.005" rpy="0 0 0"/>
 	  	</joint>
+		<link name="${name}_toe_link0"/>
+		<joint name="${name}_toe_center" type="fixed">
+	    	<parent link="${name}_link8"/>
+	    	<child  link="${name}_toe_link0"/>
+	    	<origin xyz="0.0 0.0 -0.005" rpy="0 0 0"/>
+	  	</joint>
 	</xacro:macro>
 </robot>

Commit message: 両足裏の接地点を求めた

File: ginko_description/models/ginko_auto/urdf/modules/leg_l.urdf.xacro (robot description, xacro)
@@ -300,8 +300,8 @@
 	    	<origin xyz="0.064 -0.040 -0.005" rpy="0 0 0"/>
 	  	</joint>
-		<link name="${name}_toe_link0"/>
-		<joint name="${name}_toe_center" type="fixed">
-	    	<parent link="${name}_link8"/>
-	    	<child  link="${name}_toe_link0"/>
+		<link name="${name}_toe_center"/>
+		<joint name="${name}_toe_center_joint" type="fixed">
+	    	<parent link="${name}_link8"/>
+	    	<child  link="${name}_toe_center"/>
 	    	<origin xyz="0.0 0.0 -0.005" rpy="0 0 0"/>
 	  	</joint>

File: ginko_description/models/ginko_auto/urdf/modules/leg_r.urdf.xacro (robot description, xacro)
@@ -300,8 +300,8 @@
 	    	<origin xyz="0.064 -0.040 -0.005" rpy="0 0 0"/>
 	  	</joint>
-		<link name="${name}_toe_link0"/>
-		<joint name="${name}_toe_center" type="fixed">
-	    	<parent link="${name}_link8"/>
-	    	<child  link="${name}_toe_link0"/>
+		<link name="${name}_toe_center"/>
+		<joint name="${name}_toe_center_joint" type="fixed">
+	    	<parent link="${name}_link8"/>
+	    	<child  link="${name}_toe_center"/>
 	    	<origin xyz="0.0 0.0 -0.005" rpy="0 0 0"/>
 	  	</joint>

Commit message: 左足の途中

File: ginko_description/models/ginko_auto/urdf/modules/leg_l.urdf.xacro (robot description, xacro)
@@ -104,5 +104,5 @@
 	  	</joint>
 		<!-- knee -->
-<!-- 		<link name="${name}_link3">
+		<link name="${name}_link3">
 	    	<collision>
 				<origin xyz="0 0 0" rpy="0 0 0"/>
@@ -114,5 +114,6 @@
 				<origin xyz="0 0 0" rpy="0 0 0"/>
 	    		<geometry>
-					<mesh filename="package://ginko_description/models/ginko_auto/meshes/dae/link05_l_knee.dae"/>
+					<mesh filename="package://ginko_description/models/ginko_auto/meshes/stl/link05_l_knee.stl"/>
+					<!-- <mesh filename="package://ginko_description/models/ginko_auto/meshes/dae/link05_l_knee.dae"/> -->
 	    		</geometry>
 			</visual>
@@ -129,5 +130,5 @@
 	    	<axis xyz="0 1 0"/>
 	    	<limit effort="1000.0" lower="-3.141593" upper="3.141593" velocity="0.5"/>
-	  	</joint> -->
+	  	</joint>
 		<!-- parallel link (lower-1st) -->
 <!-- 		<link name="${name}_link4">

File: ginko_description/models/ginko_auto/urdf/robot_gazebo.urdf.xacro (robot description, xacro)
@@ -16,10 +16,9 @@
   <link name="base"/>
   <xacro:body name="body" parent="base"/>
-  <!-- <xacro:body_gazebo name="body"/> -->
-  <!-- <xacro:arm_l name="arm_l" parent="body_arm_l_link"/> -->
-  <xacro:arm_l name="arm_l" parent="body_link0"/>
+  <xacro:body_gazebo name="body"/>
+<!--   <xacro:arm_l name="arm_l" parent="body_link0"/>
   <xacro:arm_l_gazebo name="arm_l"/>
   <xacro:arm_r name="arm_r" parent="body_link0"/>
-  <xacro:arm_r_gazebo name="arm_r"/>
+  <xacro:arm_r_gazebo name="arm_r"/> -->
   <xacro:leg_l name="leg_l" parent="body_link1"/>
   <xacro:leg_l_gazebo name="leg_l"/>

Commit message: 左足動作確認完了

File: ginko_description/models/ginko_auto/urdf/modules/leg_l.urdf.xacro (robot description, xacro)
@@ -132,5 +132,5 @@
 	  	</joint>
 		<!-- parallel link (lower-1st) -->
-<!-- 		<link name="${name}_link4">
+		<link name="${name}_link4">
 			<collision>
 				<origin xyz="0 0 0" rpy="0 0 0"/>
@@ -142,11 +142,14 @@
 				<origin xyz="0 0 0" rpy="0 0 0"/>
 	    		<geometry>
-					<mesh filename="package://ginko_description/models/ginko_auto/meshes/dae/link03_l_leg01.dae"/>
-	    		</geometry>
-			</visual>
-			<inertial>
-				<origin xyz="0 0 0" rpy="0 0 0"/>
-				<mass value="6.1"/>
-				<inertia ixx="0.0001" ixy="0.0" ixz="0.0" iyy="0.0001" iyz="0.0" izz="0.0001"/>
+					<mesh filename="package://ginko_description/models/ginko_auto/meshes/stl/link03_l_leg01.stl"/>
+	    		</geometry>
+			</visual>
+			<inertial>
+				<mass value="0.18525692"/>
+				<origin xyz="0.05000000 0.03285059 0.00068146" rpy="0 0 0"/>
+				<inertia
+					ixx="0.00041331"
+					ixy="-0.00003605" iyy="0.00027917"
+					ixz="-0.00000000" iyz="-0.00000184" izz="0.00066510"/>
 			</inertial>
 		</link>
@@ -157,7 +160,7 @@
 			<axis xyz="0 -1 0"/>
 			<limit effort="1000.0" lower="-0.7854" upper="1.3" velocity="0.5"/>
-		</joint> -->
+		</joint>
 		<!-- parallel link (lower-2nd) -->
-<!-- 		<link name="${name}_link5">
+		<link name="${name}_link5">
 	    	<collision>
 				<origin xyz="0 0 0" rpy="0 0 0"/>
@@ -169,11 +172,14 @@
 				<origin xyz="0 0 0" rpy="0 0 0"/>
 	    		<geometry>
-					<mesh filename="package://ginko_description/models/ginko_auto/meshes/dae/link04_l_leg02.dae"/>
-	    		</geometry>
-			</visual>
-			<inertial>
-				<origin xyz="0 0 0" rpy="0 0 0"/>
-				<mass value="6.1"/>
-				<inertia ixx="0.0001" ixy="0.0" ixz="0.0" iyy="0.0001" iyz="0.0" izz="0.0001"/>
+					<mesh filename="package://ginko_description/models/ginko_auto/meshes/stl/link04_l_leg02.stl"/>
+	    		</geometry>
+			</visual>
+			<inertial>
+				<mass value="0.01646643"/>
+				<origin xyz="0.05000000 0.02495100 -0.00491150" rpy="0 0 0"/>
+				<inertia
+					ixx="0.00000640"
+					ixy="0.00000000" iyy="0.00001642"
+					ixz="0.00000000" iyz="0.00000000" izz="0.00002264"/>
 			</inertial>
 		</link>
@@ -185,7 +191,7 @@
 	    	<limit effort="1000.0" lower="-3.141593" upper="3.141593" velocity="0.5"/>
 	    	<mimic joint="${name}_joint4" multiplier="1" offset="0"/>
-	  	</joint> -->
+	  	</joint>
 		<!-- toe -->
-<!-- 		<link name="${name}_link6">
+		<link name="${name}_link6">
 	    	<collision>
 				<origin xyz="0 0 0" rpy="0 0 0"/>
@@ -197,11 +203,14 @@
 				<origin xyz="0 0 0" rpy="0 0 0"/>
 	    		<geometry>
-					<mesh filename="package://ginko_description/models/ginko_auto/meshes/dae/link06_l_toe01.dae"/>
-	    		</geometry>
-			</visual>
-			<inertial>
-				<origin xyz="0 0 0" rpy="0 0 0"/>
-				<mass value="6.1"/>
-				<inertia ixx="0.0001" ixy="0.0" ixz="0.0" iyy="0.0001" iyz="0.0" izz="0.0001"/>
+					<mesh filename="package://ginko_description/models/ginko_auto/meshes/stl/link06_l_toe01.stl"/>
+	    		</geometry>
+			</visual>
+			<inertial>
+				<mass value="0.08799204"/>
+				<origin xyz="-0.04166125 0.02463880 -0.02586249" rpy="0 0 0"/>
+				<inertia
+					ixx="0.00002815"
+					ixy="-0.00000041" iyy="0.00006846"
+					ixz="0.00000980" iyz="-0.00000026" izz="0.00006529"/>
 			</inertial>
 		</link>
@@ -223,11 +232,14 @@
 				<origin xyz="0 0 0" rpy="0 0 0"/>
 	    		<geometry>
-					<mesh filename="package://ginko_description/models/ginko_auto/meshes/dae/link07_l_toe02.dae"/>
-	    		</geometry>
-			</visual>
-			<inertial>
-				<origin xyz="0 0 0" rpy="0 0 0"/>
-				<mass value="6.1"/>
-				<inertia ixx="0.0001" ixy="0.0" ixz="0.0" iyy="0.0001" iyz="0.0" izz="0.0001"/>
+					<mesh filename="package://ginko_description/models/ginko_auto/meshes/stl/link07_l_toe02.stl"/>
+	    		</geometry>
+			</visual>
+			<inertial>
+				<mass value="0.10920041"/>
+				<origin xyz="0.02658756 0.00000053 -0.01782468" rpy="0 0 0"/>
+				<inertia
+					ixx="0.00003853"
+					ixy="0.00000000" iyy="0.00005192"
+					ixz="-0.00000479" iyz="0.00000000" izz="0.00003521"/>
 			</inertial>
 		</link>
@@ -249,11 +261,14 @@
 				<origin xyz="0 0 0" rpy="0 0 0"/>
 	    		<geometry>
-					<mesh filename="package://ginko_description/models/ginko_auto/meshes/dae/link08_l_toe03.dae"/>
-	    		</geometry>
-			</visual>
-			<inertial>
-				<origin xyz="0 0 0" rpy="0 0 0"/>
-				<mass value="6.1"/>
-				<inertia ixx="0.0001" ixy="0.0" ixz="0.0" iyy="0.0001" iyz="0.0" izz="0.0001"/>
+					<mesh filename="package://ginko_description/models/ginko_auto/meshes/stl/link08_l_toe03.stl"/>
+	    		</geometry>
+			</visual>
+			<inertial>
+				<mass value="0.05363111"/>
+				<origin xyz="0.00000000 0.00000000 -0.00269342" rpy="0 0 0"/>
+				<inertia
+					ixx="0.00002877"
+					ixy="0.00000000" iyy="0.00007083"
+					ixz="0.00000000" iyz="-0.00000000" izz="0.00009934"/>
 			</inertial>
 		</link>
@@ -264,5 +279,5 @@
 	    	<axis xyz="0 0 1"/>
 	    	<limit effort="1000.0" lower="-2.6" upper="2.6" velocity="0.5"/>
-	  	</joint> -->
+	  	</joint>
  <!-- toe edges -->
 <!-- 		<link name="${name}_toe_link0"/>
