Commit message: 体全体をgazeboで再現

File: ginko_description/models/ginko_auto/urdf/goal.urdf.xacro (robot description, xacro)
@@ -18,8 +18,8 @@
 	<xacro:arm_l name="arm_l" parent="body_arm_l_link"/> -->
 	<xacro:body name="goal_body" parent="base"/>
-	<xacro:leg_r name="goal_leg_r" parent="goal_body_leg_r_link"/>
-	<xacro:leg_l name="goal_leg_l" parent="goal_body_leg_l_link"/>
-	<xacro:arm_r name="goal_arm_r" parent="goal_body_arm_r_link"/>
-	<xacro:arm_l name="goal_arm_l" parent="goal_body_arm_l_link"/>
+	<xacro:leg_r name="goal_leg_r" parent="goal_body_link1"/>
+	<xacro:leg_l name="goal_leg_l" parent="goal_body_link1"/>
+	<xacro:arm_r name="goal_arm_r" parent="goal_body_link0"/>
+	<xacro:arm_l name="goal_arm_l" parent="goal_body_link0"/>
 	<!-- <xacro:include filename="robot.transmission.xacro" /> -->
 	<!-- <xacro:include filename="robot.gazebo.xacro" /> -->

File: ginko_description/models/ginko_auto/urdf/modules/body.urdf.xacro (robot description, xacro)
@@ -84,5 +84,5 @@
 		    <axis xyz="0 1 0"/>
 		</joint> -->
-		<link name="${name}_leg_r_link"/>
+<!-- 		<link name="${name}_leg_r_link"/>
 		<joint name="${name}_joint4" type="fixed">
 		    <parent link="${name}_link1"/>
@@ -90,5 +90,5 @@
 		    <origin xyz="0.0205 0.0 -0.0409" rpy="0 0 0"/>
 		    <axis xyz="0 1 0"/>
-		</joint>
+		</joint> -->
 <!-- 		<link name="${name}_leg_l_link"/>
 		<joint name="${name}_joint5" type="fixed">

File: ginko_description/models/ginko_auto/urdf/modules/leg_l.urdf.xacro (robot description, xacro)
@@ -119,7 +119,10 @@
 			</visual>
 			<inertial>
-				<origin xyz="0 0 0" rpy="0 0 0"/>
-				<mass value="6.1"/>
-				<inertia ixx="0.0001" ixy="0.0" ixz="0.0" iyy="0.0001" iyz="0.0" izz="0.0001"/>
+				<mass value="0.01781176"/>
+				<origin xyz="0.00393357 0.02364163 -0.01930000" rpy="0 0 0"/>
+				<inertia
+					ixx="0.00001301"
+					ixy="0.00000008" iyy="0.00000700"
+					ixz="0.00000000" iyz="0.00000000" izz="0.00001388"/>
 			</inertial>
 		</link>
@@ -281,5 +284,5 @@
 	  	</joint>
  <!-- toe edges -->
-<!-- 		<link name="${name}_toe_link0"/>
+		<link name="${name}_toe_link0"/>
 		<joint name="${name}_toe_joint0" type="fixed">
 	    	<parent link="${name}_link8"/>
@@ -310,5 +313,5 @@
 	    	<child  link="${name}_toe_center"/>
 	    	<origin xyz="0.0 0.0 -0.005" rpy="0 0 0"/>
-	  	</joint> -->
+	  	</joint>
 	</xacro:macro>
 </robot>

File: ginko_description/models/ginko_auto/urdf/modules/leg_r.urdf.xacro (robot description, xacro)
@@ -5,5 +5,4 @@
 		<!-- Link conencts from body. Femoral first. -->
 		<link name="${name}_link0">
-			<!-- Collision created from STL mesh without color -->
 			<collision>
 				<origin xyz="0 0 0" rpy="0 0 0"/>
@@ -12,16 +11,17 @@
 				</geometry>
 			</collision>
-			<!-- Visualisation created from Color dae -->
 			<visual>
 				<origin xyz="0 0 0" rpy="0 0 0"/>
 				<geometry>
-					<mesh filename="package://ginko_description/models/ginko_auto/meshes/dae/link02_r_femoral.dae"/>
+					<mesh filename="package://ginko_description/models/ginko_auto/meshes/stl/link02_r_femoral.stl"/>
 				</geometry>
 			</visual>
-			<!-- nothing worth -->
-			<inertial>
-				<origin xyz="0 0 0" rpy="0 0 0"/>
-				<mass value="6.1"/>
-				<inertia ixx="0.0001" ixy="0.0" ixz="0.0" iyy="0.0001" iyz="0.0" izz="0.0001"/>
+			<inertial>
+				<mass value="0.03431457"/>
+				<origin xyz="-0.02905818 -0.03723481 -0.02604954" rpy="0 0 0"/>
+				<inertia
+					ixx="0.00002441"
+					ixy="0.00000001" iyy="0.00002285"
+					ixz="0.00000021" iyz="0.00000391" izz="0.00002980"/>
 			</inertial>
 		</link>
@@ -29,5 +29,5 @@
 		    <parent link="${parent}"/>
 			<child link="${name}_link0"/>
-		    <origin xyz="0 0 0" rpy="0 0 0"/>
+		    <origin xyz="0.0205 0.0 -0.0409" rpy="0 0 0"/>
 		    <axis xyz="1 0 0"/>
 			<limit effort="1000.0" lower="-1.1781" upper="0.8" velocity="0.5"/>
@@ -35,5 +35,4 @@
 		<!-- parallel link (upper-1st) -->
 		<link name="${name}_link1">
-			<!-- Collision created from STL mesh without color -->
 			<collision>
 				<origin xyz="0 0 0" rpy="0 0 0"/>
@@ -42,16 +41,17 @@
 	    		</geometry>
 			</collision>
-			<!-- Visualisation created from Color dae -->
-	    	<visual>
-				<origin xyz="0 0 0" rpy="0 0 0"/>
-	    		<geometry>
-					<mesh filename="package://ginko_description/models/ginko_auto/meshes/dae/link03_r_leg01.dae"/>
-	    		</geometry>
-			</visual>
-			<!-- nothing worth -->
-			<inertial>
-				<origin xyz="0 0 0" rpy="0 0 0"/>
-				<mass value="6.1"/>
-				<inertia ixx="0.0001" ixy="0.0" ixz="0.0" iyy="0.0001" iyz="0.0" izz="0.0001"/>
+	    	<visual>
+				<origin xyz="0 0 0" rpy="0 0 0"/>
+	    		<geometry>
+					<mesh filename="package://ginko_description/models/ginko_auto/meshes/stl/link03_r_leg01.stl"/>
+	    		</geometry>
+			</visual>
+			<inertial>
+				<mass value="0.18525690"/>
+				<origin xyz="0.05000000 -0.01719078 0.00068146" rpy="0 0 0"/>
+				<inertia
+					ixx="0.00055489"
+					ixy="-0.00004242" iyy="0.00027917"
+					ixz="0.00000000" iyz="-0.00000175" izz="0.00081028"/>
 			</inertial>
 		</link>
@@ -65,5 +65,4 @@
 		<!-- parallel link (upper-2nd) -->
 		<link name="${name}_link2">
-			<!-- Collision created from STL mesh without color -->
 	    	<collision>
 				<origin xyz="0 0 0" rpy="0 0 0"/>
@@ -72,16 +71,17 @@
 	    		</geometry>
 			</collision>
-			<!-- Visualisation created from Color dae -->
-	    	<visual>
-				<origin xyz="0 0 0" rpy="0 0 0"/>
-	    		<geometry>
-					<mesh filename="package://ginko_description/models/ginko_auto/meshes/dae/link04_r_leg02.dae"/>
-	    		</geometry>
-			</visual>
-			<!-- nothing worth -->
-			<inertial>
-				<origin xyz="0 0 0" rpy="0 0 0"/>
-				<mass value="6.1"/>
-				<inertia ixx="0.0001" ixy="0.0" ixz="0.0" iyy="0.0001" iyz="0.0" izz="0.0001"/>
+	    	<visual>
+				<origin xyz="0 0 0" rpy="0 0 0"/>
+	    		<geometry>
+					<mesh filename="package://ginko_description/models/ginko_auto/meshes/stl/link04_r_leg02.stl"/>
+	    		</geometry>
+			</visual>
+			<inertial>
+				<mass value="0.01646643"/>
+				<origin xyz="0.05000000 -0.02495100 -0.00491150" rpy="0 0 0"/>
+				<inertia
+					ixx="0.00000640"
+					ixy="0.00000000" iyy="0.00001642"
+					ixz="0.00000000" iyz="0.00000000" izz="0.00002264"/>
 			</inertial>
 		</link>
@@ -96,5 +96,4 @@
 		<!-- knee -->
 		<link name="${name}_link3">
-			<!-- Collision created from STL mesh without color -->
 	    	<collision>
 				<origin xyz="0 0 0" rpy="0 0 0"/>
@@ -103,16 +102,17 @@
 	    		</geometry>
 			</collision>
-			<!-- Visualisation created from Color dae -->
-	    	<visual>
-				<origin xyz="0 0 0" rpy="0 0 0"/>
-	    		<geometry>
-					<mesh filename="package://ginko_description/models/ginko_auto/meshes/dae/link05_r_knee.dae"/>
-	    		</geometry>
-			</visual>
-			<!-- nothing worth -->
-			<inertial>
-				<origin xyz="0 0 0" rpy="0 0 0"/>
-				<mass value="6.1"/>
-				<inertia ixx="0.0001" ixy="0.0" ixz="0.0" iyy="0.0001" iyz="0.0" izz="0.0001"/>
+	    	<visual>
+				<origin xyz="0 0 0" rpy="0 0 0"/>
+	    		<geometry>
+					<mesh filename="package://ginko_description/models/ginko_auto/meshes/stl/link05_r_knee.stl"/>
+	    		</geometry>
+			</visual>
+			<inertial>
+				<mass value="0.01781176"/>
+				<origin xyz="0.00393357 -0.02364163 -0.01930000" rpy="0 0 0"/>
+				<inertia
+					ixx="0.00001301"
+					ixy="-0.00000008" iyy="0.00000700"
+					ixz="0.00000000" iyz="0.00000000" izz="0.00001388"/>
 			</inertial>
 		</link>
@@ -127,5 +127,4 @@
 		<!-- parallel link (lower-1st) -->
 		<link name="${name}_link4">
-			<!-- Collision created from STL mesh without color -->
 			<collision>
 				<origin xyz="0 0 0" rpy="0 0 0"/>
@@ -134,16 +133,17 @@
 	    		</geometry>
 			</collision>
-			<!-- Visualisation created from Color dae -->
-	    	<visual>
-				<origin xyz="0 0 0" rpy="0 0 0"/>
-	    		<geometry>
-					<mesh filename="package://ginko_description/models/ginko_auto/meshes/dae/link03_r_leg01.dae"/>
-	    		</geometry>
-			</visual>
-			<!-- nothing worth -->
-			<inertial>
-				<origin xyz="0 0 0" rpy="0 0 0"/>
-				<mass value="6.1"/>
-				<inertia ixx="0.0001" ixy="0.0" ixz="0.0" iyy="0.0001" iyz="0.0" izz="0.0001"/>
+	    	<visual>
+				<origin xyz="0 0 0" rpy="0 0 0"/>
+	    		<geometry>
+					<mesh filename="package://ginko_description/models/ginko_auto/meshes/stl/link03_r_leg01.stl"/>
+	    		</geometry>
+			</visual>
+			<inertial>
+				<mass value="0.18525690"/>
+				<origin xyz="0.05000000 -0.01719078 0.00068146" rpy="0 0 0"/>
+				<inertia
+					ixx="0.00055489"
+					ixy="-0.00004242" iyy="0.00027917"
+					ixz="0.00000000" iyz="-0.00000175" izz="0.00081028"/>
 			</inertial>
 		</link>
@@ -157,5 +157,4 @@
 		<!-- parallel link (lower-2nd) -->
 		<link name="${name}_link5">
-			<!-- Collision created from STL mesh without color -->
 	    	<collision>
 				<origin xyz="0 0 0" rpy="0 0 0"/>
@@ -164,16 +163,17 @@
 	    		</geometry>
 			</collision>
-			<!-- Visualisation created from Color dae -->
-	    	<visual>
-				<origin xyz="0 0 0" rpy="0 0 0"/>
-	    		<geometry>
-					<mesh filename="package://ginko_description/models/ginko_auto/meshes/dae/link04_r_leg02.dae"/>
-	    		</geometry>
-			</visual>
-			<!-- nothing worth -->
-			<inertial>
-				<origin xyz="0 0 0" rpy="0 0 0"/>
-				<mass value="6.1"/>
-				<inertia ixx="0.0001" ixy="0.0" ixz="0.0" iyy="0.0001" iyz="0.0" izz="0.0001"/>
+	    	<visual>
+				<origin xyz="0 0 0" rpy="0 0 0"/>
+	    		<geometry>
+					<mesh filename="package://ginko_description/models/ginko_auto/meshes/stl/link04_r_leg02.stl"/>
+	    		</geometry>
+			</visual>
+			<inertial>
+				<mass value="0.01646643"/>
+				<origin xyz="0.05000000 -0.02495100 -0.00491150" rpy="0 0 0"/>
+				<inertia
+					ixx="0.00000640"
+					ixy="0.00000000" iyy="0.00001642"
+					ixz="0.00000000" iyz="0.00000000" izz="0.00002264"/>
 			</inertial>
 		</link>
@@ -188,5 +188,4 @@
 		<!-- toe -->
 		<link name="${name}_link6">
-			<!-- Collision created from STL mesh without color -->
 	    	<collision>
 				<origin xyz="0 0 0" rpy="0 0 0"/>
@@ -195,16 +194,17 @@
 	    		</geometry>
 			</collision>
-			<!-- Visualisation created from Color dae -->
-	    	<visual>
-				<origin xyz="0 0 0" rpy="0 0 0"/>
-	    		<geometry>
-					<mesh filename="package://ginko_description/models/ginko_auto/meshes/dae/link06_r_toe01.dae"/>
-	    		</geometry>
-			</visual>
-			<!-- nothing worth -->
-			<inertial>
-				<origin xyz="0 0 0" rpy="0 0 0"/>
-				<mass value="6.1"/>
-				<inertia ixx="0.0001" ixy="0.0" ixz="0.0" iyy="0.0001" iyz="0.0" izz="0.0001"/>
+	    	<visual>
+				<origin xyz="0 0 0" rpy="0 0 0"/>
+	    		<geometry>
+					<mesh filename="package://ginko_description/models/ginko_auto/meshes/stl/link06_r_toe01.stl"/>
+	    		</geometry>
+			</visual>
+			<inertial>
+				<mass value="0.08799204"/>
+				<origin xyz="-0.04166125 -0.02463880 -0.02586249" rpy="0 0 0"/>
+				<inertia
+					ixx="0.00002815"
+					ixy="0.00000041" iyy="0.00006846"
+					ixz="0.00000980" iyz="0.00000026" izz="0.00006529"/>
 			</inertial>
 		</link>
@@ -218,5 +218,4 @@
 	  	</joint>
 		<link name="${name}_link7">
-			<!-- Collision created from STL mesh without color -->
 	    	<collision>
 				<origin xyz="0 0 0" rpy="0 0 0"/>
@@ -225,16 +224,17 @@
 	    		</geometry>
 			</collision>
-			<!-- Visualisation created from Color dae -->
-	    	<visual>
-				<origin xyz="0 0 0" rpy="0 0 0"/>
-	    		<geometry>
-					<mesh filename="package://ginko_description/models/ginko_auto/meshes/dae/link07_r_toe02.dae"/>
-	    		</geometry>
-			</visual>
-			<!-- nothing worth -->
-			<inertial>
-				<origin xyz="0 0 0" rpy="0 0 0"/>
-				<mass value="6.1"/>
-				<inertia ixx="0.0001" ixy="0.0" ixz="0.0" iyy="0.0001" iyz="0.0" izz="0.0001"/>
+	    	<visual>
+				<origin xyz="0 0 0" rpy="0 0 0"/>
+	    		<geometry>
+					<mesh filename="package://ginko_description/models/ginko_auto/meshes/stl/link07_r_toe02.stl"/>
+	    		</geometry>
+			</visual>
+			<inertial>
+				<mass value="0.10920041"/>
+				<origin xyz="0.02658756 -0.00000053 -0.01782468" rpy="0 0 0"/>
+				<inertia
+					ixx="0.00003853"
+					ixy="0.00000000" iyy="0.00005192"
+					ixz="-0.00000479" iyz="0.00000000" izz="0.00003521"/>
 			</inertial>
 		</link>
@@ -247,5 +247,4 @@
 	  	</joint>
 		<link name="${name}_link8">
-			<!-- Collision created from STL mesh without color -->
 	    	<collision>
 				<origin xyz="0 0 0" rpy="0 0 0"/>
@@ -254,16 +253,17 @@
 	    		</geometry>
 			</collision>
-			<!-- Visualisation created from Color dae -->
-	    	<visual>
-				<origin xyz="0 0 0" rpy="0 0 0"/>
-	    		<geometry>
-					<mesh filename="package://ginko_description/models/ginko_auto/meshes/dae/link08_r_toe03.dae"/>
-	    		</geometry>
-			</visual>
-			<!-- nothing worth -->
-			<inertial>
-				<origin xyz="0 0 0" rpy="0 0 0"/>
-				<mass value="6.1"/>
-				<inertia ixx="0.0001" ixy="0.0" ixz="0.0" iyy="0.0001" iyz="0.0" izz="0.0001"/>
+	    	<visual>
+				<origin xyz="0 0 0" rpy="0 0 0"/>
+	    		<geometry>
+					<mesh filename="package://ginko_description/models/ginko_auto/meshes/stl/link08_r_toe03.stl"/>
+	    		</geometry>
+			</visual>
+			<inertial>
+				<mass value="0.05363111"/>
+				<origin xyz="0.00000000 0.00000000 -0.00269342" rpy="0 0 0"/>
+				<inertia
+					ixx="0.00002877"
+					ixy="0.00000000" iyy="0.00007083"
+					ixz="0.00000000" iyz="-0.00000000" izz="0.00009934"/>
 			</inertial>
 		</link>

File: ginko_description/models/ginko_auto/urdf/robot.urdf.xacro (robot description, xacro)
@@ -13,8 +13,8 @@
 	</joint>
 	<xacro:body name="body" parent="base"/>
-	<xacro:leg_r name="leg_r" parent="body_leg_r_link"/>
-	<xacro:leg_l name="leg_l" parent="body_leg_l_link"/>
-	<xacro:arm_r name="arm_r" parent="body_arm_r_link"/>
-	<xacro:arm_l name="arm_l" parent="body_arm_l_link"/>
+	<xacro:leg_r name="leg_r" parent="body_link1"/>
+	<xacro:leg_l name="leg_l" parent="body_link1"/>
+	<xacro:arm_r name="arm_r" parent="body_link0"/>
+	<xacro:arm_l name="arm_l" parent="body_link0"/>
 	<!-- <xacro:include filename="robot.transmission.xacro" /> -->
 	<!-- <xacro:include filename="robot.gazebo.xacro" /> -->

File: ginko_description/models/ginko_auto/urdf/robot_gazebo.urdf.xacro (robot description, xacro)
@@ -9,4 +9,6 @@
   <xacro:include filename="$(find ginko_description)/models/ginko_auto/urdf/modules/leg_l.urdf.xacro"/>
   <xacro:include filename="$(find ginko_description)/models/ginko_auto/urdf/gazebo_modules/leg_l.gazebo"/>
+  <xacro:include filename="$(find ginko_description)/models/ginko_auto/urdf/modules/leg_r.urdf.xacro"/>
+  <xacro:include filename="$(find ginko_description)/models/ginko_auto/urdf/gazebo_modules/leg_r.gazebo"/>
   <!-- Import all Gazebo-customization elements, including Gazebo colors -->
   <!-- <xacro:include filename="$(find rrbot_description)/urdf/rrbot.gazebo" /> -->
@@ -17,9 +19,11 @@
   <xacro:body name="body" parent="base"/>
   <xacro:body_gazebo name="body"/>
-<!--   <xacro:arm_l name="arm_l" parent="body_link0"/>
+  <xacro:arm_l name="arm_l" parent="body_link0"/>
   <xacro:arm_l_gazebo name="arm_l"/>
   <xacro:arm_r name="arm_r" parent="body_link0"/>
-  <xacro:arm_r_gazebo name="arm_r"/> -->
+  <xacro:arm_r_gazebo name="arm_r"/>
   <xacro:leg_l name="leg_l" parent="body_link1"/>
   <xacro:leg_l_gazebo name="leg_l"/>
+  <xacro:leg_r name="leg_r" parent="body_link1"/>
+  <xacro:leg_r_gazebo name="leg_r"/>
 </robot>
