Commit message: 平行リンクを含めたSDFを作成
rosrun xacro xacro --inorder -o robot_gazebo.urdf robot_gazebo.urdf.xacro
gz sdf -p robot_gazebo.urdf > ../sdf/robot_gazebo.sdf

File: ginko_description/urdf/leg_l.urdf (robot description, URDF)
Before this commit: robot ginko, 9 links, 8 joints
Links:
- link leg_l_link0: geometry collision mesh filename=package://ginko_description/meshes/stl/link02_l_femoral.stl; visual mesh filename=package://ginko_description/meshes/stl/link02_l_femoral.stl
- link leg_l_link1: geometry collision mesh filename=package://ginko_description/meshes/stl/link03_l_leg01.stl; visual mesh filename=package://ginko_description/meshes/stl/link03_l_leg01.stl
- link leg_l_link2: geometry collision mesh filename=package://ginko_description/meshes/stl/link04_l_leg02.stl; visual mesh filename=package://ginko_description/meshes/stl/link04_l_leg02.stl
- link leg_l_link3: geometry collision mesh filename=package://ginko_description/meshes/stl/link05_l_knee.stl; visual mesh filename=package://ginko_description/meshes/stl/link05_l_knee.stl
- link leg_l_link4: geometry collision mesh filename=package://ginko_description/meshes/stl/link03_l_leg01.stl; visual mesh filename=package://ginko_description/meshes/stl/link03_l_leg01.stl
- link leg_l_link5: geometry collision mesh filename=package://ginko_description/meshes/stl/link04_l_leg02.stl; visual mesh filename=package://ginko_description/meshes/stl/link04_l_leg02.stl
- link leg_l_link6: geometry collision mesh filename=package://ginko_description/meshes/stl/link06_l_toe01.stl; visual mesh filename=package://ginko_description/meshes/stl/link06_l_toe01.stl
- link leg_l_link7: geometry collision mesh filename=package://ginko_description/meshes/stl/link07_l_toe02.stl; visual mesh filename=package://ginko_description/meshes/stl/link07_l_toe02.stl
- link leg_l_link8: geometry collision mesh filename=package://ginko_description/meshes/stl/link08_l_toe03.stl; visual mesh filename=package://ginko_description/meshes/stl/link08_l_toe03.stl
