Commit message: urdfとsdfの共存を検証中

File: ginko_description/gazebo/pre_urdf/robot_gazebo.urdf.xacro (robot description, xacro)
@@ -13,4 +13,10 @@
   <!-- Used for fixing robot to Gazebo 'base_link' -->
   <!-- <link name="base"/> -->
+  <gazebo>
+    <plugin name="gazebo_ros_control" filename="libgazebo_ros_control.so">
+      <robotNamespace>/ginko</robotNamespace>
+      <robotSimType>gazebo_ros_control/DefaultRobotHWSim</robotSimType>
+    </plugin>
+  </gazebo>
   <xacro:body name="body" parent="base"/>
   <xacro:body_gazebo name="body"/>

File: ginko_description/urdf/robot_gazebo.urdf.xacro (robot description, xacro)
@@ -16,10 +16,6 @@
 	  </plugin>
 	</gazebo>
-	<!-- <link name="world"/> -->
+	<!-- <xacro:include filename="$(find ginko_description)/gazebo/sdf/robot_gazebo_sdf.urdf"/> -->
 	<link name="base"/>
-<!-- 	<joint name="fixed1" type="fixed">
-		<parent link="world"/>
-		<child link="base"/>
-	</joint> -->
 	<xacro:body name="body" parent="base"/>
 	<xacro:leg_r name="leg_r" parent="body_link1"/>
