Commit message: 表示用とgazebo用を分けて用意

File: ginko_description/gazebo/urdf_sim/modules/arm_l.urdf.xacro (robot description, xacro)
@@ -1,5 +1,5 @@
 <?xml version="1.0"?>
 <robot xmlns:xacro="http://www.ros.org/wiki/xacro">
-	<xacro:macro name="arm_l" params="name parent">
+	<xacro:macro name="arm_l_sim" params="name parent">
 		<!-- shoulder pitch. -->
 		<link name="${name}_link0">
@@ -30,5 +30,5 @@
 		    <origin xyz="0 0.10683 0.05115" rpy="0 0.3927 0"/>
 		    <axis xyz="0 -1 0"/>
-			<limit effort="1000.0" lower="-2.6" upper="2.6" velocity="0.5"/>
+			<limit effort="100.0" lower="-2.6" upper="2.6" velocity="10.0"/>
 		</joint>
 		<!-- shoulder roll -->
@@ -60,5 +60,5 @@
 			<origin xyz="0.035 0.0246 0" rpy="1.1781 0 0"/>
 			<axis xyz="1 0 0"/>
-			<limit effort="1000.0" lower="-0.85" upper="1.18" velocity="0.5"/>
+			<limit effort="100.0" lower="-0.85" upper="1.18" velocity="10.0"/>
 		</joint>
 		<!-- scissors -->
@@ -90,5 +90,5 @@
 	    	<origin xyz="0.0092 0.0547 -0.11295" rpy="0 0.7854 0"/>
 	    	<axis xyz="0 1 0"/>
-	    	<limit effort="1000.0" lower="-2.36" upper="2.36" velocity="0.5"/>
+	    	<limit effort="100.0" lower="-2.36" upper="2.36" velocity="10.0"/>
 	  	</joint>
 		<link name="${name}_link3">
@@ -119,5 +119,5 @@
 	    	<origin xyz="0.0092 -0.0018 -0.11295" rpy="0 0.7854 0"/>
 	    	<axis xyz="0 1 0"/>
-	    	<limit effort="1000.0" lower="-2.36" upper="2.36" velocity="0.5"/>
+	    	<limit effort="100.0" lower="-2.36" upper="2.36" velocity="10.0"/>
 	  	</joint>
 	  	<!-- LiDAR -->

File: ginko_description/gazebo/urdf_sim/modules/arm_r.urdf.xacro (robot description, xacro)
@@ -1,5 +1,5 @@
 <?xml version="1.0"?>
 <robot xmlns:xacro="http://www.ros.org/wiki/xacro">
-	<xacro:macro name="arm_r" params="name parent">
+	<xacro:macro name="arm_r_sim" params="name parent">
 		<!-- shoulder pitch. -->
 		<link name="${name}_link0">
@@ -30,5 +30,5 @@
 		    <origin xyz="0 -0.10683 0.05115" rpy="0 0.3927 0"/>
 		    <axis xyz="0 1 0"/>
-			<limit effort="1000.0" lower="-2.6" upper="2.6" velocity="0.5"/>
+			<limit effort="100.0" lower="-2.6" upper="2.6" velocity="10.0"/>
 		</joint>
 		<!-- shoulder roll -->
@@ -60,5 +60,5 @@
 			<origin xyz="0.035 -0.0246 0" rpy="-1.1781 0 0"/>
 			<axis xyz="1 0 0"/>
-			<limit effort="1000.0" lower="-0.85" upper="1.18" velocity="0.5"/>
+			<limit effort="100.0" lower="-0.85" upper="1.18" velocity="10.0"/>
 		</joint>
 		<!-- scissors -->
@@ -90,5 +90,5 @@
 	    	<origin xyz="0.0092 -0.0547 -0.11295" rpy="0 0.7854 0"/>
 	    	<axis xyz="0 -1 0"/>
-	    	<limit effort="1000.0" lower="-2.36" upper="2.36" velocity="0.5"/>
+	    	<limit effort="100.0" lower="-2.36" upper="2.36" velocity="10.0"/>
 	  	</joint>
 		<link name="${name}_link3">
@@ -119,5 +119,5 @@
 	    	<origin xyz="0.0092 0.0018 -0.11295" rpy="0 0.7854 0"/>
 	    	<axis xyz="0 -1 0"/>
-	    	<limit effort="1000.0" lower="-2.36" upper="2.36" velocity="0.5"/>
+	    	<limit effort="100.0" lower="-2.36" upper="2.36" velocity="10.0"/>
 	  	</joint>
 	  	<!-- LiDAR -->

File: ginko_description/gazebo/urdf_sim/modules/body.urdf.xacro (robot description, xacro)
@@ -1,5 +1,5 @@
 <?xml version="1.0"?>
 <robot xmlns:xacro="http://www.ros.org/wiki/xacro">
-	<xacro:macro name="body" params="name parent">
+	<xacro:macro name="body_sim" params="name">
 		<!-- chest -->
 		<link name="${name}_link0">
@@ -25,10 +25,4 @@
 			</inertial>
 		</link>
-<!-- 		<joint name="${name}_joint0" type="fixed">
-		    <parent link="${parent}"/>
-			<child link="${name}_link0"/>
-		    <origin xyz="0 0 0" rpy="0 0 0"/>
-		    <axis xyz="0 0 1"/>
-		</joint> -->
 		<!-- waist -->
 		<link name="${name}_link1">
@@ -59,5 +53,5 @@
 			<origin xyz="0 0 0" rpy="0 0 0"/>
 			<axis xyz="0 0 1"/>
-			<limit effort="1000.0" lower="-2.6" upper="2.6" velocity="0.5"/>
+			<limit effort="100.0" lower="-2.6" upper="2.6" velocity="10.0"/>
 		</joint>
 	</xacro:macro>

File: ginko_description/gazebo/urdf_sim/modules/leg_l.urdf.xacro (robot description, xacro)
@@ -1,9 +1,7 @@
 <?xml version="1.0"?>
-<robot name="leg_l" xmlns:xacro="http://www.ros.org/wiki/xacro">
-	<xacro:macro name="leg_l" params="name parent">
-	<!-- <xacro:property name="name" value="leg"/> -->
-		<!-- Link conencts from body. Femoral first. -->
+<robot xmlns:xacro="http://www.ros.org/wiki/xacro">
+	<xacro:macro name="leg_l_sim" params="name parent">
+		<!-- Femoral -->
 		<link name="${name}_link0">
-			<!-- Collision created from STL mesh without color -->
 			<collision>
 				<origin xyz="0 0 0" rpy="0 0 0"/>
@@ -12,10 +10,8 @@
 				</geometry>
 			</collision>
-			<!-- Visualisation created from Color dae -->
 			<visual>
 				<origin xyz="0 0 0" rpy="0 0 0"/>
 				<geometry>
 					<mesh filename="package://ginko_description/meshes/stl/link02_l_femoral.stl"/>
-					<!-- <mesh filename="package://ginko_description/models/ginko_auto/meshes/dae/link02_l_femoral.dae"/> -->
 				</geometry>
 			</visual>
@@ -34,9 +30,8 @@
 			<origin xyz="-0.0404 0.0 -0.0409" rpy="0 0 0"/>
 		    <axis xyz="-1 0 0"/>
-			<limit effort="1000.0" lower="-0.8" upper="1.1781" velocity="0.5"/>
+			<limit effort="100.0" lower="-0.8" upper="1.1781" velocity="10.0"/>
 		</joint>
 		<!-- parallel link (upper-1st) -->
 		<link name="${name}_link1">
-			<!-- Collision created from STL mesh without color -->
 			<collision>
 				<origin xyz="0 0 0" rpy="0 0 0"/>
@@ -45,10 +40,8 @@
 	    		</geometry>
 			</collision>
-			<!-- Visualisation created from Color dae -->
-	    	<visual>
-				<origin xyz="0 0 0" rpy="0 0 0"/>
-	    		<geometry>
-					<mesh filename="package://ginko_description/meshes/stl/link03_l_leg01.stl"/>
-					<!-- <mesh filename="package://ginko_description/models/ginko_auto/meshes/dae/link03_l_leg01.dae"/> -->
+	    	<visual>
+				<origin xyz="0 0 0" rpy="0 0 0"/>
+	    		<geometry>
+					<mesh filename="package://ginko_description/meshes/stl/link03_l_leg01.stl"/>
 	    		</geometry>
 			</visual>
@@ -67,21 +60,17 @@
 			<origin xyz="0.0433 0.0175 -0.0481" rpy="0 0.7854 0"/>
 			<axis xyz="0 -1 0"/>
-			<limit effort="1000.0" lower="-1.3" upper="0.7854" velocity="0.5"/>
+			<limit effort="100.0" lower="-1.3" upper="0.7854" velocity="10.0"/>
 		</joint>
-		<!-- parallel link (upper-2nd) -->
 		<link name="${name}_link2">
-			<!-- Collision created from STL mesh without color -->
-	    	<collision>
-				<origin xyz="0 0 0" rpy="0 0 0"/>
-	    		<geometry>
-					<mesh filename="package://ginko_description/meshes/stl/link04_l_leg02.stl"/>
-	    		</geometry>
-			</collision>
-			<!-- Visualisation created from Color dae -->
-	    	<visual>
-				<origin xyz="0 0 0" rpy="0 0 0"/>
-	    		<geometry>
-					<mesh filename="package://ginko_description/meshes/stl/link04_l_leg02.stl"/>
-					<!-- <mesh filename="package://ginko_description/models/ginko_auto/meshes/dae/link04_l_leg02.dae"/> -->
+	    	<collision>
+				<origin xyz="0 0 0" rpy="0 0 0"/>
+	    		<geometry>
+					<mesh filename="package://ginko_description/meshes/stl/link04_l_leg02.stl"/>
+	    		</geometry>
+			</collision>
+	    	<visual>
+				<origin xyz="0 0 0" rpy="0 0 0"/>
+	    		<geometry>
+					<mesh filename="package://ginko_description/meshes/stl/link04_l_leg02.stl"/>
 	    		</geometry>
 			</visual>
@@ -100,6 +89,5 @@
 	    	<origin xyz="0.022 0.0175 -0.06015" rpy="0 0.7854 0"/>
 	    	<axis xyz="0 -1 0"/>
-	    	<limit effort="1000.0" lower="-3.141593" upper="3.141593" velocity="0.5"/>
-	    	<!-- <mimic joint="${name}_joint1" multiplier="1" offset="0"/>  -->
+	    	<limit effort="100.0" lower="-3.141593" upper="3.141593" velocity="10.0"/>
 	  	</joint>
 		<!-- knee -->
@@ -115,5 +103,4 @@
 	    		<geometry>
 					<mesh filename="package://ginko_description/meshes/stl/link05_l_knee.stl"/>
-					<!-- <mesh filename="package://ginko_description/models/ginko_auto/meshes/dae/link05_l_knee.dae"/> -->
 	    		</geometry>
 			</visual>
@@ -132,5 +119,5 @@
 	    	<origin xyz="0.1 0.0 0.0" rpy="0 -0.7854 0"/>
 	    	<axis xyz="0 1 0"/>
-	    	<limit effort="1000.0" lower="-3.141593" upper="3.141593" velocity="0.5"/>
+	    	<limit effort="100.0" lower="-3.141593" upper="3.141593" velocity="10.0"/>
 	  	</joint>
 		<!-- parallel link (lower-1st) -->
@@ -162,5 +149,5 @@
 			<origin xyz="0 0 -0.0386" rpy="0 2.3562 0"/>
 			<axis xyz="0 -1 0"/>
-			<limit effort="1000.0" lower="-0.7854" upper="1.3" velocity="0.5"/>
+			<limit effort="100.0" lower="-0.7854" upper="1.3" velocity="10.0"/>
 		</joint>
 		<!-- parallel link (lower-2nd) -->
@@ -192,6 +179,5 @@
 	    	<origin xyz="-0.0213 0 -0.02655" rpy="0 2.3562 0"/>
 	    	<axis xyz="0 -1 0"/>
-	    	<limit effort="1000.0" lower="-3.141593" upper="3.141593" velocity="0.5"/>
-	    	<mimic joint="${name}_joint4" multiplier="1" offset="0"/>
+	    	<limit effort="100.0" lower="-3.141593" upper="3.141593" velocity="10.0"/>
 	  	</joint>
 		<!-- toe -->
@@ -223,5 +209,5 @@
 	    	<origin xyz="0.1 0.0 0.0" rpy="0 -2.3562 0"/>
 	    	<axis xyz="0 1 0"/>
-	    	<limit effort="1000.0" lower="-3.141593" upper="3.141593" velocity="0.5"/>
+	    	<limit effort="100.0" lower="-3.141593" upper="3.141593" velocity="10.0"/>
 	  	</joint>
 		<link name="${name}_link7">
@@ -252,5 +238,5 @@
 	    	<origin xyz="-0.028 0.02475 -0.0391" rpy="0 0 0"/>
 	    	<axis xyz="-1 0 0"/>
-	    	<limit effort="1000.0" lower="-1.6" upper="1.6" velocity="0.5"/>
+	    	<limit effort="100.0" lower="-1.6" upper="1.6" velocity="10.0"/>
 	  	</joint>
 		<link name="${name}_link8">
@@ -281,5 +267,5 @@
 	    	<origin xyz="0.0342 0 -0.04" rpy="0 0 0"/>
 	    	<axis xyz="0 0 1"/>
-	    	<limit effort="1000.0" lower="-2.6" upper="2.6" velocity="0.5"/>
+	    	<limit effort="100.0" lower="-2.6" upper="2.6" velocity="10.0"/>
 	  	</joint>
 	</xacro:macro>

File: ginko_description/gazebo/urdf_sim/modules/leg_r.urdf.xacro (robot description, xacro)
@@ -1,7 +1,6 @@
 <?xml version="1.0"?>
-<robot name="leg_r" xmlns:xacro="http://www.ros.org/wiki/xacro">
-	<xacro:macro name="leg_r" params="name parent">
-	<!-- <xacro:property name="name" value="leg"/> -->
-		<!-- Link conencts from body. Femoral first. -->
+<robot xmlns:xacro="http://www.ros.org/wiki/xacro">
+	<xacro:macro name="leg_r_sim" params="name parent">
+		<!-- Femoral -->
 		<link name="${name}_link0">
 			<collision>
@@ -31,5 +30,5 @@
 		    <origin xyz="0.0205 0.0 -0.0409" rpy="0 0 0"/>
 		    <axis xyz="1 0 0"/>
-			<limit effort="1000.0" lower="-1.1781" upper="0.8" velocity="0.5"/>
+			<limit effort="100.0" lower="-1.1781" upper="0.8" velocity="10.0"/>
 		</joint>
 		<!-- parallel link (upper-1st) -->
@@ -61,5 +60,5 @@
 			<origin xyz="-0.0176 -0.0175 -0.0481" rpy="0 0.7854 0"/>
 			<axis xyz="0 1 0"/>
-			<limit effort="1000.0" lower="-0.7854" upper="1.3" velocity="0.5"/>
+			<limit effort="100.0" lower="-0.7854" upper="1.3" velocity="10.0"/>
 		</joint>
 		<!-- parallel link (upper-2nd) -->
@@ -91,6 +90,5 @@
 	    	<origin xyz="-0.0389 -0.0175 -0.06015" rpy="0 0.7854 0"/>
 	    	<axis xyz="0 1 0"/>
-	    	<limit effort="1000.0" lower="-3.141593" upper="3.141593" velocity="0.5"/>
-	    	<mimic joint="${name}_joint1" multiplier="1" offset="0"/>
+	    	<limit effort="100.0" lower="-3.141593" upper="3.141593" velocity="10.0"/>
 	  	</joint>
 		<!-- knee -->
@@ -122,6 +120,5 @@
 	    	<origin xyz="0.1 0.0 0.0" rpy="0 -0.7854 0"/>
 	    	<axis xyz="0 -1 0"/>
-	    	<limit effort="1000.0" lower="-3.141593" upper="3.141593" velocity="0.5"/>
-	    	<!-- <mimic joint="${name}_joint1" multiplier="1" offset="0"/>  -->
+	    	<limit effort="100.0" lower="-3.141593" upper="3.141593" velocity="10.0"/>
 	  	</joint>
 		<!-- parallel link (lower-1st) -->
@@ -153,5 +150,5 @@
 			<origin xyz="0 0 -0.0386" rpy="0 2.3562 0"/>
 			<axis xyz="0 1 0"/>
-			<limit effort="1000.0" lower="-1.3" upper="0.7854" velocity="0.5"/>
+			<limit effort="100.0" lower="-1.3" upper="0.7854" velocity="10.0"/>
 		</joint>
 		<!-- parallel link (lower-2nd) -->
@@ -183,6 +180,5 @@
 	    	<origin xyz="-0.0213 0 -0.02655" rpy="0 2.3562 0"/>
 	    	<axis xyz="0 1 0"/>
-	    	<limit effort="1000.0" lower="-3.141593" upper="3.141593" velocity="0.5"/>
-	    	<mimic joint="${name}_joint4" multiplier="1" offset="0"/>
+	    	<limit effort="100.0" lower="-3.141593" upper="3.141593" velocity="10.0"/>
 	  	</joint>
 		<!-- toe -->
@@ -214,6 +210,5 @@
 	    	<origin xyz="0.1 0.0 0.0" rpy="0 -2.3562 0"/>
 	    	<axis xyz="0 -1 0"/>
-	    	<limit effort="1000.0" lower="-3.141593" upper="3.141593" velocity="0.5"/>
-	    	<!-- <mimic joint="${name}_joint4" multiplier="1" offset="0"/>  -->
+	    	<limit effort="100.0" lower="-3.141593" upper="3.141593" velocity="10.0"/>
 	  	</joint>
 		<link name="${name}_link7">
@@ -244,5 +239,5 @@
 	    	<origin xyz="-0.028 -0.02475 -0.0391" rpy="0 0 0"/>
 	    	<axis xyz="-1 0 0"/>
-	    	<limit effort="1000.0" lower="-1.6" upper="1.6" velocity="0.5"/>
+	    	<limit effort="100.0" lower="-1.6" upper="1.6" velocity="10.0"/>
 	  	</joint>
 		<link name="${name}_link8">
@@ -273,5 +268,5 @@
 	    	<origin xyz="0.0342 0 -0.04" rpy="0 0 0"/>
 	    	<axis xyz="0 0 1"/>
-	    	<limit effort="1000.0" lower="-2.6" upper="2.6" velocity="0.5"/>
+	    	<limit effort="100.0" lower="-2.6" upper="2.6" velocity="10.0"/>
 	  	</joint>
 	</xacro:macro>

File: ginko_description/gazebo/urdf_sim/robot_gazebo.urdf.xacro (robot description, xacro)
@@ -1,13 +1,13 @@
 <?xml version="1.0"?>
 <robot name="ginko" xmlns:xacro="http://www.ros.org/wiki/xacro">
-  <xacro:include filename="$(find ginko_description)/gazebo/pre_urdf/modules/body.urdf.xacro"/>
+  <xacro:include filename="$(find ginko_description)/gazebo/urdf_sim/modules/body.urdf.xacro"/>
   <xacro:include filename="$(find ginko_description)/gazebo/transmission/body.gazebo"/>
-  <xacro:include filename="$(find ginko_description)/gazebo/pre_urdf/modules/arm_l.urdf.xacro"/>
+  <xacro:include filename="$(find ginko_description)/gazebo/urdf_sim/modules/arm_l.urdf.xacro"/>
   <xacro:include filename="$(find ginko_description)/gazebo/transmission/arm_l.gazebo"/>
-  <xacro:include filename="$(find ginko_description)/gazebo/pre_urdf/modules/arm_r.urdf.xacro"/>
+  <xacro:include filename="$(find ginko_description)/gazebo/urdf_sim/modules/arm_r.urdf.xacro"/>
   <xacro:include filename="$(find ginko_description)/gazebo/transmission/arm_r.gazebo"/>
-  <xacro:include filename="$(find ginko_description)/gazebo/pre_urdf/modules/leg_l.urdf.xacro"/>
+  <xacro:include filename="$(find ginko_description)/gazebo/urdf_sim/modules/leg_l.urdf.xacro"/>
   <xacro:include filename="$(find ginko_description)/gazebo/transmission/leg_l.gazebo"/>
-  <xacro:include filename="$(find ginko_description)/gazebo/pre_urdf/modules/leg_r.urdf.xacro"/>
+  <xacro:include filename="$(find ginko_description)/gazebo/urdf_sim/modules/leg_r.urdf.xacro"/>
   <xacro:include filename="$(find ginko_description)/gazebo/transmission/leg_r.gazebo"/>
   <!-- Used for fixing robot to Gazebo 'base_link' -->
@@ -19,13 +19,13 @@
     </plugin>
   </gazebo>
-  <xacro:body name="body" parent="base"/>
+  <xacro:body_sim name="body"/>
   <xacro:body_gazebo name="body"/>
-  <xacro:arm_l name="arm_l" parent="body_link0"/>
+  <xacro:arm_l_sim name="arm_l" parent="body_link0"/>
   <xacro:arm_l_gazebo name="arm_l"/>
   <xacro:arm_r name="arm_r" parent="body_link0"/>
   <xacro:arm_r_gazebo name="arm_r"/>
-  <xacro:leg_l name="leg_l" parent="body_link1"/>
+  <xacro:leg_l_sim name="leg_l" parent="body_link1"/>
   <xacro:leg_l_gazebo name="leg_l"/>
-  <xacro:leg_r name="leg_r" parent="body_link1"/>
+  <xacro:leg_r_sim name="leg_r" parent="body_link1"/>
   <xacro:leg_r_gazebo name="leg_r"/>
 </robot>

File: ginko_description/gazebo/urdf_viz/robot_gazebo.urdf.xacro (robot description, xacro)
@@ -1,13 +1,13 @@
 <?xml version="1.0"?>
 <robot name="ginko" xmlns:xacro="http://www.ros.org/wiki/xacro">
-  <xacro:include filename="$(find ginko_description)/gazebo/pre_urdf/modules/body.urdf.xacro"/>
+  <xacro:include filename="$(find ginko_description)/gazebo/urdf_viz/modules/body.urdf.xacro"/>
   <xacro:include filename="$(find ginko_description)/gazebo/transmission/body.gazebo"/>
-  <xacro:include filename="$(find ginko_description)/gazebo/pre_urdf/modules/arm_l.urdf.xacro"/>
+  <xacro:include filename="$(find ginko_description)/gazebo/urdf_viz/modules/arm_l.urdf.xacro"/>
   <xacro:include filename="$(find ginko_description)/gazebo/transmission/arm_l.gazebo"/>
-  <xacro:include filename="$(find ginko_description)/gazebo/pre_urdf/modules/arm_r.urdf.xacro"/>
+  <xacro:include filename="$(find ginko_description)/gazebo/urdf_viz/modules/arm_r.urdf.xacro"/>
   <xacro:include filename="$(find ginko_description)/gazebo/transmission/arm_r.gazebo"/>
-  <xacro:include filename="$(find ginko_description)/gazebo/pre_urdf/modules/leg_l.urdf.xacro"/>
+  <xacro:include filename="$(find ginko_description)/gazebo/urdf_viz/modules/leg_l.urdf.xacro"/>
   <xacro:include filename="$(find ginko_description)/gazebo/transmission/leg_l.gazebo"/>
-  <xacro:include filename="$(find ginko_description)/gazebo/pre_urdf/modules/leg_r.urdf.xacro"/>
+  <xacro:include filename="$(find ginko_description)/gazebo/urdf_viz/modules/leg_r.urdf.xacro"/>
   <xacro:include filename="$(find ginko_description)/gazebo/transmission/leg_r.gazebo"/>
   <!-- Used for fixing robot to Gazebo 'base_link' -->
@@ -19,13 +19,13 @@
     </plugin>
   </gazebo>
-  <xacro:body name="body" parent="base"/>
+  <xacro:body_viz name="body" parent="base"/>
   <xacro:body_gazebo name="body"/>
-  <xacro:arm_l name="arm_l" parent="body_link0"/>
+  <xacro:arm_l_viz name="arm_l" parent="body_link0"/>
   <xacro:arm_l_gazebo name="arm_l"/>
-  <xacro:arm_r name="arm_r" parent="body_link0"/>
+  <xacro:arm_r_viz name="arm_r" parent="body_link0"/>
   <xacro:arm_r_gazebo name="arm_r"/>
-  <xacro:leg_l name="leg_l" parent="body_link1"/>
+  <xacro:leg_l_viz name="leg_l" parent="body_link1"/>
   <xacro:leg_l_gazebo name="leg_l"/>
-  <xacro:leg_r name="leg_r" parent="body_link1"/>
+  <xacro:leg_r_viz name="leg_r" parent="body_link1"/>
   <xacro:leg_r_gazebo name="leg_r"/>
 </robot>
