Commit message: urdfにバネを追加

File: ginko_description/gazebo/urdf_sim/modules/leg_l_spring.urdf.xacro (robot description, xacro)
@@ -91,4 +91,63 @@
 	    	<limit effort="100.0" lower="-3.141593" upper="3.141593" velocity="10.0"/>
 	  	</joint>
+	  	<!-- spring -->
+	  	<link name="${name}_spring_link0">
+	    	<collision>
+				<origin xyz="0 0 0" rpy="0 0 0"/>
+	    		<geometry>
+					<mesh filename="package://ginko_description/meshes/stl/spring1.stl"/>
+	    		</geometry>
+			</collision>
+	    	<visual>
+				<origin xyz="0 0 0" rpy="0 0 0"/>
+	    		<geometry>
+					<mesh filename="package://ginko_description/meshes/stl/spring1.stl"/>
+	    		</geometry>
+			</visual>
+			<inertial>
+				<mass value="0.00143865"/>
+				<origin xyz="0.03091683 0.0 0.0" rpy="0 0 0"/>
+				<inertia
+					ixx="0.00000001"
+					ixy="0.00000000" iyy="0.00000060"
+					ixz="0.00000000" iyz="0.00000000" izz="0.00000060"/>
+			</inertial>
+		</link>
+		<joint name="${name}_spring_joint0" type="revolute">
+	    	<parent link="${name}_link0"/>
+	    	<child  link="${name}_spring_link0"/>
+	    	<origin xyz="0.022 0.0755 -0.06015" rpy="0 0.56756754 0"/>
+	    	<axis xyz="0 -1 0"/>
+	    	<limit effort="0.0" lower="-3.141593" upper="3.141593" velocity="10.0"/>
+	  	</joint>
+	  	<link name="${name}_spring_link1">
+	    	<collision>
+				<origin xyz="0 0 0" rpy="0 0 0"/>
+	    		<geometry>
+					<mesh filename="package://ginko_description/meshes/stl/spring2.stl"/>
+	    		</geometry>
+			</collision>
+	    	<visual>
+				<origin xyz="0 0 0" rpy="0 0 0"/>
+	    		<geometry>
+					<mesh filename="package://ginko_description/meshes/stl/spring2.stl"/>
+	    		</geometry>
+			</visual>
+			<inertial>
+				<mass value="0.00143865"/>
+				<origin xyz="0.03091683 0.0 0.0" rpy="0 0 0"/>
+				<inertia
+					ixx="0.00000001"
+					ixy="0.00000000" iyy="0.00000060"
+					ixz="0.00000000" iyz="0.00000000" izz="0.00000060"/>
+			</inertial>
+		</link>
+		<joint name="${name}_spring_joint1" type="prismatic">
+	    	<parent link="${name}_spring_link0"/>
+	    	<child  link="${name}_spring_link1"/>
+	    	<origin xyz="0.10911938 0.0 0.0" rpy="0 3.141593 0"/>
+	    	<axis xyz="0 -1 0"/>
+	    	<limit effort="1000.0" lower="-3.141593" upper="3.141593" velocity="10.0"/>
+	  	</joint>
 		<!-- knee -->
 		<link name="${name}_link3">
@@ -181,4 +240,63 @@
 	    	<limit effort="100.0" lower="-3.141593" upper="3.141593" velocity="10.0"/>
 	  	</joint>
+	  	<!-- spring -->
+	  	<link name="${name}_spring_link2">
+	    	<collision>
+				<origin xyz="0 0 0" rpy="0 0 0"/>
+	    		<geometry>
+					<mesh filename="package://ginko_description/meshes/stl/spring1.stl"/>
+	    		</geometry>
+			</collision>
+	    	<visual>
+				<origin xyz="0 0 0" rpy="0 0 0"/>
+	    		<geometry>
+					<mesh filename="package://ginko_description/meshes/stl/spring1.stl"/>
+	    		</geometry>
+			</visual>
+			<inertial>
+				<mass value="0.00143865"/>
+				<origin xyz="0.03091683 0.0 0.0" rpy="0 2.138363867 0"/>
+				<inertia
+					ixx="0.00000001"
+					ixy="0.00000000" iyy="0.00000060"
+					ixz="0.00000000" iyz="0.00000000" izz="0.00000060"/>
+			</inertial>
+		</link>
+		<joint name="${name}_spring_joint2" type="revolute">
+	    	<parent link="${name}_link3"/>
+	    	<child  link="${name}_spring_link2"/>
+			<origin xyz="0 0.058 -0.0386" rpy="0 2.574025114 0"/>
+	    	<axis xyz="0 -1 0"/>
+	    	<limit effort="0.0" lower="-3.141593" upper="3.141593" velocity="10.0"/>
+	  	</joint>
+	  	<link name="${name}_spring_link3">
+	    	<collision>
+				<origin xyz="0 0 0" rpy="0 0 0"/>
+	    		<geometry>
+					<mesh filename="package://ginko_description/meshes/stl/spring2.stl"/>
+	    		</geometry>
+			</collision>
+	    	<visual>
+				<origin xyz="0 0 0" rpy="0 0 0"/>
+	    		<geometry>
+					<mesh filename="package://ginko_description/meshes/stl/spring2.stl"/>
+	    		</geometry>
+			</visual>
+			<inertial>
+				<mass value="0.00143865"/>
+				<origin xyz="0.03091683 0.0 0.0" rpy="0 0 0"/>
+				<inertia
+					ixx="0.00000001"
+					ixy="0.00000000" iyy="0.00000060"
+					ixz="0.00000000" iyz="0.00000000" izz="0.00000060"/>
+			</inertial>
+		</link>
+		<joint name="${name}_spring_joint3" type="prismatic">
+	    	<parent link="${name}_spring_link2"/>
+	    	<child  link="${name}_spring_link3"/>
+	    	<origin xyz="0.10911938 0.0 0.0" rpy="0 3.141593 0"/>
+	    	<axis xyz="0 -1 0"/>
+	    	<limit effort="1000.0" lower="-3.141593" upper="3.141593" velocity="10.0"/>
+	  	</joint>
 		<!-- toe -->
 		<link name="${name}_link6">

File: ginko_description/gazebo/urdf_sim/modules/leg_r_spring.urdf.xacro (robot description, xacro)
@@ -92,4 +92,63 @@
 	    	<limit effort="100.0" lower="-3.141593" upper="3.141593" velocity="10.0"/>
 	  	</joint>
+	  	<!-- spring -->
+	  	<link name="${name}_spring_link0">
+	    	<collision>
+				<origin xyz="0 0 0" rpy="0 0 0"/>
+	    		<geometry>
+					<mesh filename="package://ginko_description/meshes/stl/spring1.stl"/>
+	    		</geometry>
+			</collision>
+	    	<visual>
+				<origin xyz="0 0 0" rpy="0 0 0"/>
+	    		<geometry>
+					<mesh filename="package://ginko_description/meshes/stl/spring1.stl"/>
+	    		</geometry>
+			</visual>
+			<inertial>
+				<mass value="0.00143865"/>
+				<origin xyz="0.03091683 0.0 0.0" rpy="0 0 0"/>
+				<inertia
+					ixx="0.00000001"
+					ixy="0.00000000" iyy="0.00000060"
+					ixz="0.00000000" iyz="0.00000000" izz="0.00000060"/>
+			</inertial>
+		</link>
+		<joint name="${name}_spring_joint0" type="revolute">
+	    	<parent link="${name}_link0"/>
+	    	<child  link="${name}_spring_link0"/>
+			<origin xyz="-0.0389 -0.0755 -0.06015" rpy="0 0.56756754 0"/>
+	    	<axis xyz="0 -1 0"/>
+	    	<limit effort="0.0" lower="-3.141593" upper="3.141593" velocity="10.0"/>
+	  	</joint>
+	  	<link name="${name}_spring_link1">
+	    	<collision>
+				<origin xyz="0 0 0" rpy="0 0 0"/>
+	    		<geometry>
+					<mesh filename="package://ginko_description/meshes/stl/spring2.stl"/>
+	    		</geometry>
+			</collision>
+	    	<visual>
+				<origin xyz="0 0 0" rpy="0 0 0"/>
+	    		<geometry>
+					<mesh filename="package://ginko_description/meshes/stl/spring2.stl"/>
+	    		</geometry>
+			</visual>
+			<inertial>
+				<mass value="0.00143865"/>
+				<origin xyz="0.03091683 0.0 0.0" rpy="0 0 0"/>
+				<inertia
+					ixx="0.00000001"
+					ixy="0.00000000" iyy="0.00000060"
+					ixz="0.00000000" iyz="0.00000000" izz="0.00000060"/>
+			</inertial>
+		</link>
+		<joint name="${name}_spring_joint1" type="prismatic">
+	    	<parent link="${name}_spring_link0"/>
+	    	<child  link="${name}_spring_link1"/>
+	    	<origin xyz="0.10911938 0.0 0.0" rpy="0 3.141593 0"/>
+	    	<axis xyz="0 -1 0"/>
+	    	<limit effort="1000.0" lower="-3.141593" upper="3.141593" velocity="10.0"/>
+	  	</joint>
 		<!-- knee -->
 		<link name="${name}_link3">
@@ -182,4 +241,63 @@
 	    	<limit effort="100.0" lower="-3.141593" upper="3.141593" velocity="10.0"/>
 	  	</joint>
+	  	<!-- spring -->
+	  	<link name="${name}_spring_link2">
+	    	<collision>
+				<origin xyz="0 0 0" rpy="0 0 0"/>
+	    		<geometry>
+					<mesh filename="package://ginko_description/meshes/stl/spring1.stl"/>
+	    		</geometry>
+			</collision>
+	    	<visual>
+				<origin xyz="0 0 0" rpy="0 0 0"/>
+	    		<geometry>
+					<mesh filename="package://ginko_description/meshes/stl/spring1.stl"/>
+	    		</geometry>
+			</visual>
+			<inertial>
+				<mass value="0.00143865"/>
+				<origin xyz="0.03091683 0.0 0.0" rpy="0 2.138363867 0"/>
+				<inertia
+					ixx="0.00000001"
+					ixy="0.00000000" iyy="0.00000060"
+					ixz="0.00000000" iyz="0.00000000" izz="0.00000060"/>
+			</inertial>
+		</link>
+		<joint name="${name}_spring_joint2" type="revolute">
+	    	<parent link="${name}_link3"/>
+	    	<child  link="${name}_spring_link2"/>
+			<origin xyz="0 -0.058 -0.0386" rpy="0 2.574025114 0"/>
+	    	<axis xyz="0 -1 0"/>
+	    	<limit effort="0.0" lower="-3.141593" upper="3.141593" velocity="10.0"/>
+	  	</joint>
+	  	<link name="${name}_spring_link3">
+	    	<collision>
+				<origin xyz="0 0 0" rpy="0 0 0"/>
+	    		<geometry>
+					<mesh filename="package://ginko_description/meshes/stl/spring2.stl"/>
+	    		</geometry>
+			</collision>
+	    	<visual>
+				<origin xyz="0 0 0" rpy="0 0 0"/>
+	    		<geometry>
+					<mesh filename="package://ginko_description/meshes/stl/spring2.stl"/>
+	    		</geometry>
+			</visual>
+			<inertial>
+				<mass value="0.00143865"/>
+				<origin xyz="0.03091683 0.0 0.0" rpy="0 0 0"/>
+				<inertia
+					ixx="0.00000001"
+					ixy="0.00000000" iyy="0.00000060"
+					ixz="0.00000000" iyz="0.00000000" izz="0.00000060"/>
+			</inertial>
+		</link>
+		<joint name="${name}_spring_joint3" type="prismatic">
+	    	<parent link="${name}_spring_link2"/>
+	    	<child  link="${name}_spring_link3"/>
+	    	<origin xyz="0.10911938 0.0 0.0" rpy="0 3.141593 0"/>
+	    	<axis xyz="0 -1 0"/>
+	    	<limit effort="1000.0" lower="-3.141593" upper="3.141593" velocity="10.0"/>
+	  	</joint>
 		<!-- toe -->
 		<link name="${name}_link6">

File: ginko_description/gazebo/urdf_sim/robot_gazebo_spring.urdf.xacro (robot description, xacro)
@@ -8,5 +8,5 @@
   <xacro:include filename="$(find ginko_description)/gazebo/transmission/arm_r.gazebo"/>
   <xacro:include filename="$(find ginko_description)/gazebo/urdf_sim/modules/leg_l_spring.urdf.xacro"/>
-  <xacro:include filename="$(find ginko_description)/gazebo/transmission/leg_l_sprong.gazebo"/>
+  <xacro:include filename="$(find ginko_description)/gazebo/transmission/leg_l_spring.gazebo"/>
   <xacro:include filename="$(find ginko_description)/gazebo/urdf_sim/modules/leg_r_spring.urdf.xacro"/>
   <xacro:include filename="$(find ginko_description)/gazebo/transmission/leg_r_spring.gazebo"/>

Commit message: 部品の弾性係数を変更(ode)

File: ginko_description/gazebo/urdf_sim/modules/leg_l_spring.urdf.xacro (robot description, xacro)
@@ -93,10 +93,10 @@
 	  	<!-- spring -->
 	  	<link name="${name}_spring_link0">
-	    	<collision>
+<!-- 	    	<collision>
 				<origin xyz="0 0 0" rpy="0 0 0"/>
 	    		<geometry>
 					<mesh filename="package://ginko_description/meshes/stl/spring1.stl"/>
 	    		</geometry>
-			</collision>
+			</collision> -->
 	    	<visual>
 				<origin xyz="0 0 0" rpy="0 0 0"/>
@@ -122,10 +122,10 @@
 	  	</joint>
 	  	<link name="${name}_spring_link1">
-	    	<collision>
+<!-- 	    	<collision>
 				<origin xyz="0 0 0" rpy="0 0 0"/>
 	    		<geometry>
 					<mesh filename="package://ginko_description/meshes/stl/spring2.stl"/>
 	    		</geometry>
-			</collision>
+			</collision> -->
 	    	<visual>
 				<origin xyz="0 0 0" rpy="0 0 0"/>
@@ -242,10 +242,10 @@
 	  	<!-- spring -->
 	  	<link name="${name}_spring_link2">
-	    	<collision>
+<!-- 	    	<collision>
 				<origin xyz="0 0 0" rpy="0 0 0"/>
 	    		<geometry>
 					<mesh filename="package://ginko_description/meshes/stl/spring1.stl"/>
 	    		</geometry>
-			</collision>
+			</collision> -->
 	    	<visual>
 				<origin xyz="0 0 0" rpy="0 0 0"/>
@@ -271,10 +271,10 @@
 	  	</joint>
 	  	<link name="${name}_spring_link3">
-	    	<collision>
+<!-- 	    	<collision>
 				<origin xyz="0 0 0" rpy="0 0 0"/>
 	    		<geometry>
 					<mesh filename="package://ginko_description/meshes/stl/spring2.stl"/>
 	    		</geometry>
-			</collision>
+			</collision> -->
 	    	<visual>
 				<origin xyz="0 0 0" rpy="0 0 0"/>

File: ginko_description/gazebo/urdf_sim/modules/leg_r_spring.urdf.xacro (robot description, xacro)
@@ -94,10 +94,10 @@
 	  	<!-- spring -->
 	  	<link name="${name}_spring_link0">
-	    	<collision>
+<!-- 	    	<collision>
 				<origin xyz="0 0 0" rpy="0 0 0"/>
 	    		<geometry>
 					<mesh filename="package://ginko_description/meshes/stl/spring1.stl"/>
 	    		</geometry>
-			</collision>
+			</collision> -->
 	    	<visual>
 				<origin xyz="0 0 0" rpy="0 0 0"/>
@@ -123,10 +123,10 @@
 	  	</joint>
 	  	<link name="${name}_spring_link1">
-	    	<collision>
+<!-- 	    	<collision>
 				<origin xyz="0 0 0" rpy="0 0 0"/>
 	    		<geometry>
 					<mesh filename="package://ginko_description/meshes/stl/spring2.stl"/>
 	    		</geometry>
-			</collision>
+			</collision> -->
 	    	<visual>
 				<origin xyz="0 0 0" rpy="0 0 0"/>
@@ -243,10 +243,10 @@
 	  	<!-- spring -->
 	  	<link name="${name}_spring_link2">
-	    	<collision>
+<!-- 	    	<collision>
 				<origin xyz="0 0 0" rpy="0 0 0"/>
 	    		<geometry>
 					<mesh filename="package://ginko_description/meshes/stl/spring1.stl"/>
 	    		</geometry>
-			</collision>
+			</collision> -->
 	    	<visual>
 				<origin xyz="0 0 0" rpy="0 0 0"/>
@@ -272,10 +272,10 @@
 	  	</joint>
 	  	<link name="${name}_spring_link3">
-	    	<collision>
+<!-- 	    	<collision>
 				<origin xyz="0 0 0" rpy="0 0 0"/>
 	    		<geometry>
 					<mesh filename="package://ginko_description/meshes/stl/spring2.stl"/>
 	    		</geometry>
-			</collision>
+			</collision> -->
 	    	<visual>
 				<origin xyz="0 0 0" rpy="0 0 0"/>

Commit message: バネのcollisionを復活

File: ginko_description/gazebo/urdf_sim/modules/leg_l_spring.urdf.xacro (robot description, xacro)
@@ -93,10 +93,10 @@
 	  	<!-- spring -->
 	  	<link name="${name}_spring_link0">
-<!-- 	    	<collision>
+	    	<collision>
 				<origin xyz="0 0 0" rpy="0 0 0"/>
 	    		<geometry>
 					<mesh filename="package://ginko_description/meshes/stl/spring1.stl"/>
 	    		</geometry>
-			</collision> -->
+			</collision>
 	    	<visual>
 				<origin xyz="0 0 0" rpy="0 0 0"/>
@@ -122,10 +122,10 @@
 	  	</joint>
 	  	<link name="${name}_spring_link1">
-<!-- 	    	<collision>
+	    	<collision>
 				<origin xyz="0 0 0" rpy="0 0 0"/>
 	    		<geometry>
 					<mesh filename="package://ginko_description/meshes/stl/spring2.stl"/>
 	    		</geometry>
-			</collision> -->
+			</collision>
 	    	<visual>
 				<origin xyz="0 0 0" rpy="0 0 0"/>
@@ -242,10 +242,10 @@
 	  	<!-- spring -->
 	  	<link name="${name}_spring_link2">
-<!-- 	    	<collision>
+	    	<collision>
 				<origin xyz="0 0 0" rpy="0 0 0"/>
 	    		<geometry>
 					<mesh filename="package://ginko_description/meshes/stl/spring1.stl"/>
 	    		</geometry>
-			</collision> -->
+			</collision>
 	    	<visual>
 				<origin xyz="0 0 0" rpy="0 0 0"/>
@@ -271,10 +271,10 @@
 	  	</joint>
 	  	<link name="${name}_spring_link3">
-<!-- 	    	<collision>
+	    	<collision>
 				<origin xyz="0 0 0" rpy="0 0 0"/>
 	    		<geometry>
 					<mesh filename="package://ginko_description/meshes/stl/spring2.stl"/>
 	    		</geometry>
-			</collision> -->
+			</collision>
 	    	<visual>
 				<origin xyz="0 0 0" rpy="0 0 0"/>

File: ginko_description/gazebo/urdf_sim/modules/leg_r_spring.urdf.xacro (robot description, xacro)
@@ -94,10 +94,10 @@
 	  	<!-- spring -->
 	  	<link name="${name}_spring_link0">
-<!-- 	    	<collision>
+	    	<collision>
 				<origin xyz="0 0 0" rpy="0 0 0"/>
 	    		<geometry>
 					<mesh filename="package://ginko_description/meshes/stl/spring1.stl"/>
 	    		</geometry>
-			</collision> -->
+			</collision>
 	    	<visual>
 				<origin xyz="0 0 0" rpy="0 0 0"/>
@@ -123,10 +123,10 @@
 	  	</joint>
 	  	<link name="${name}_spring_link1">
-<!-- 	    	<collision>
+	    	<collision>
 				<origin xyz="0 0 0" rpy="0 0 0"/>
 	    		<geometry>
 					<mesh filename="package://ginko_description/meshes/stl/spring2.stl"/>
 	    		</geometry>
-			</collision> -->
+			</collision>
 	    	<visual>
 				<origin xyz="0 0 0" rpy="0 0 0"/>
@@ -243,10 +243,10 @@
 	  	<!-- spring -->
 	  	<link name="${name}_spring_link2">
-<!-- 	    	<collision>
+	    	<collision>
 				<origin xyz="0 0 0" rpy="0 0 0"/>
 	    		<geometry>
 					<mesh filename="package://ginko_description/meshes/stl/spring1.stl"/>
 	    		</geometry>
-			</collision> -->
+			</collision>
 	    	<visual>
 				<origin xyz="0 0 0" rpy="0 0 0"/>
@@ -272,10 +272,10 @@
 	  	</joint>
 	  	<link name="${name}_spring_link3">
-<!-- 	    	<collision>
+	    	<collision>
 				<origin xyz="0 0 0" rpy="0 0 0"/>
 	    		<geometry>
 					<mesh filename="package://ginko_description/meshes/stl/spring2.stl"/>
 	    		</geometry>
-			</collision> -->
+			</collision>
 	    	<visual>
 				<origin xyz="0 0 0" rpy="0 0 0"/>
