Commit message: 表示用urdf作成

File: ginko_description/gazebo/urdf_viz/modules/arm_l.urdf.xacro (robot description, xacro)
@@ -1,5 +1,5 @@
 <?xml version="1.0"?>
 <robot xmlns:xacro="http://www.ros.org/wiki/xacro">
-	<xacro:macro name="arm_l_sim" params="name parent">
+	<xacro:macro name="arm_l_viz" params="name parent">
 		<!-- shoulder pitch. -->
 		<link name="${name}_link0">

File: ginko_description/gazebo/urdf_viz/modules/arm_r.urdf.xacro (robot description, xacro)
@@ -1,5 +1,5 @@
 <?xml version="1.0"?>
 <robot xmlns:xacro="http://www.ros.org/wiki/xacro">
-	<xacro:macro name="arm_r_sim" params="name parent">
+	<xacro:macro name="arm_r_viz" params="name parent">
 		<!-- shoulder pitch. -->
 		<link name="${name}_link0">

File: ginko_description/gazebo/urdf_viz/modules/body.urdf.xacro (robot description, xacro)
@@ -1,5 +1,5 @@
 <?xml version="1.0"?>
 <robot xmlns:xacro="http://www.ros.org/wiki/xacro">
-	<xacro:macro name="body_sim" params="name">
+	<xacro:macro name="body_viz" params="name">
 		<!-- chest -->
 		<link name="${name}_link0">

File: ginko_description/gazebo/urdf_viz/modules/leg_l.urdf.xacro (robot description, xacro)
@@ -1,5 +1,5 @@
 <?xml version="1.0"?>
 <robot xmlns:xacro="http://www.ros.org/wiki/xacro">
-	<xacro:macro name="leg_l_sim" params="name parent">
+	<xacro:macro name="leg_l_viz" params="name parent">
 		<!-- Femoral -->
 		<link name="${name}_link0">
@@ -62,4 +62,5 @@
 			<limit effort="100.0" lower="-1.3" upper="0.7854" velocity="10.0"/>
 		</joint>
+		<!-- parallel link (upper-2nd) -->
 		<link name="${name}_link2">
 	    	<collision>
@@ -90,4 +91,5 @@
 	    	<axis xyz="0 -1 0"/>
 	    	<limit effort="100.0" lower="-3.141593" upper="3.141593" velocity="10.0"/>
+	    	<mimic joint="${name}_joint1" multiplier="1" offset="0"/>
 	  	</joint>
 		<!-- knee -->
@@ -120,4 +122,5 @@
 	    	<axis xyz="0 1 0"/>
 	    	<limit effort="100.0" lower="-3.141593" upper="3.141593" velocity="10.0"/>
+	    	<mimic joint="${name}_joint1" multiplier="1" offset="0"/>
 	  	</joint>
 		<!-- parallel link (lower-1st) -->
@@ -180,4 +183,5 @@
 	    	<axis xyz="0 -1 0"/>
 	    	<limit effort="100.0" lower="-3.141593" upper="3.141593" velocity="10.0"/>
+	    	<mimic joint="${name}_joint4" multiplier="1" offset="0"/>
 	  	</joint>
 		<!-- toe -->
@@ -210,4 +214,5 @@
 	    	<axis xyz="0 1 0"/>
 	    	<limit effort="100.0" lower="-3.141593" upper="3.141593" velocity="10.0"/>
+	    	<mimic joint="${name}_joint4" multiplier="1" offset="0"/>
 	  	</joint>
 		<link name="${name}_link7">

File: ginko_description/gazebo/urdf_viz/modules/leg_r.urdf.xacro (robot description, xacro)
@@ -1,5 +1,5 @@
 <?xml version="1.0"?>
 <robot xmlns:xacro="http://www.ros.org/wiki/xacro">
-	<xacro:macro name="leg_r_sim" params="name parent">
+	<xacro:macro name="leg_r_viz" params="name parent">
 		<!-- Femoral -->
 		<link name="${name}_link0">
@@ -91,4 +91,5 @@
 	    	<axis xyz="0 1 0"/>
 	    	<limit effort="100.0" lower="-3.141593" upper="3.141593" velocity="10.0"/>
+	    	<mimic joint="${name}_joint1" multiplier="1" offset="0"/>
 	  	</joint>
 		<!-- knee -->
@@ -121,4 +122,5 @@
 	    	<axis xyz="0 -1 0"/>
 	    	<limit effort="100.0" lower="-3.141593" upper="3.141593" velocity="10.0"/>
+	    	<mimic joint="${name}_joint1" multiplier="1" offset="0"/>
 	  	</joint>
 		<!-- parallel link (lower-1st) -->
@@ -181,4 +183,5 @@
 	    	<axis xyz="0 1 0"/>
 	    	<limit effort="100.0" lower="-3.141593" upper="3.141593" velocity="10.0"/>
+	    	<mimic joint="${name}_joint4" multiplier="1" offset="0"/>
 	  	</joint>
 		<!-- toe -->
@@ -211,4 +214,5 @@
 	    	<axis xyz="0 -1 0"/>
 	    	<limit effort="100.0" lower="-3.141593" upper="3.141593" velocity="10.0"/>
+	    	<mimic joint="${name}_joint4" multiplier="1" offset="0"/>
 	  	</joint>
 		<link name="${name}_link7">
