Commit message: サーボIDとの対応がずれている

File: ginko_description/gazebo/sdf/robot_sim_mimic.urdf (robot description, URDF)
Before this commit: robot ginko, 30 links, 29 joints
Links:
- added link base_link
Joints:
- added joint base_joint: type fixed, parent base_link, child body_link0, origin xyz=0 0 0 rpy=0 0 0, axis 0 0 1, limit lower=0.0 upper=0.0 effort=0.0 velocity=0.0

Commit message: gazeboでモーションが動いた
※注意
・urdfの関節角度制限：gazeboのサーボの角度指令値に制限がかかる
・sdfの関節角度制限：物理シミュレータの角度が制限される

File: ginko_description/gazebo/sdf/robot_sim_mimic.urdf (robot description, URDF)
Before this commit: robot ginko, 31 links, 30 joints
Joints:
- joint arm_l_joint1: limit lower=-0.85 upper=1.18 effort=100.0 velocity=10.0 -> lower=-2.6 upper=2.6 effort=100.0 velocity=10.0
- joint arm_r_joint1: limit lower=-0.85 upper=1.18 effort=100.0 velocity=10.0 -> lower=-2.6 upper=2.6 effort=100.0 velocity=10.0
