Commit message: rvizで表示できるように修正

File: ginko_description/gazebo/sdf/robot_sim.urdf (robot description, URDF)
Before this commit: robot ginko, 30 links, 29 joints
Joints:
- joint arm_l_urg_joint: type revolute -> fixed
- joint arm_r_urg_joint: type revolute -> fixed
- joint leg_l_joint2: mimic (none) -> joint=leg_l_joint1 multiplier=1 offset=0
- joint leg_l_joint3: mimic (none) -> joint=leg_l_joint1 multiplier=1 offset=0
- joint leg_l_joint5: mimic (none) -> joint=leg_l_joint4 multiplier=1 offset=0
- joint leg_l_joint6: mimic (none) -> joint=leg_l_joint4 multiplier=1 offset=0
- joint leg_r_joint2: mimic (none) -> joint=leg_r_joint1 multiplier=1 offset=0
- joint leg_r_joint3: mimic (none) -> joint=leg_r_joint1 multiplier=1 offset=0
- joint leg_r_joint5: mimic (none) -> joint=leg_r_joint4 multiplier=1 offset=0
- joint leg_r_joint6: mimic (none) -> joint=leg_r_joint4 multiplier=1 offset=0

Commit message: 弾性係数を変更してsdf出力

File: ginko_description/gazebo/sdf/robot_sim.urdf (robot description, URDF)
Before this commit: robot ginko, 30 links, 29 joints
Joints:
- joint leg_l_joint2: mimic joint=leg_l_joint1 multiplier=1 offset=0 -> (none)
- joint leg_l_joint3: mimic joint=leg_l_joint1 multiplier=1 offset=0 -> (none)
- joint leg_l_joint5: mimic joint=leg_l_joint4 multiplier=1 offset=0 -> (none)
- joint leg_l_joint6: mimic joint=leg_l_joint4 multiplier=1 offset=0 -> (none)
- joint leg_r_joint2: mimic joint=leg_r_joint1 multiplier=1 offset=0 -> (none)
- joint leg_r_joint3: mimic joint=leg_r_joint1 multiplier=1 offset=0 -> (none)
- joint leg_r_joint5: mimic joint=leg_r_joint4 multiplier=1 offset=0 -> (none)
- joint leg_r_joint6: mimic joint=leg_r_joint4 multiplier=1 offset=0 -> (none)
