Commit message: 左足の根元側のバネだけ再現できた

File: ginko_description/gazebo/sdf/robot_sim_spring.urdf (robot description, URDF)
Before this commit: robot ginko, 38 links, 37 joints
Links:
- link leg_l_spring_link0: geometry collision mesh filename=package://ginko_description/meshes/stl/spring1.stl; visual mesh filename=package://ginko_description/meshes/stl/spring1.stl
- link leg_l_spring_link1: geometry collision mesh filename=package://ginko_description/meshes/stl/spring2.stl; visual mesh filename=package://ginko_description/meshes/stl/spring2.stl
- link leg_l_spring_link2: geometry collision mesh filename=package://ginko_description/meshes/stl/spring1.stl; visual mesh filename=package://ginko_description/meshes/stl/spring1.stl
- link leg_l_spring_link3: geometry collision mesh filename=package://ginko_description/meshes/stl/spring2.stl; visual mesh filename=package://ginko_description/meshes/stl/spring2.stl
- link leg_r_spring_link0: geometry collision mesh filename=package://ginko_description/meshes/stl/spring1.stl; visual mesh filename=package://ginko_description/meshes/stl/spring1.stl
- link leg_r_spring_link1: geometry collision mesh filename=package://ginko_description/meshes/stl/spring2.stl; visual mesh filename=package://ginko_description/meshes/stl/spring2.stl
- link leg_r_spring_link2: geometry collision mesh filename=package://ginko_description/meshes/stl/spring1.stl; visual mesh filename=package://ginko_description/meshes/stl/spring1.stl
- link leg_r_spring_link3: geometry collision mesh filename=package://ginko_description/meshes/stl/spring2.stl; visual mesh filename=package://ginko_description/meshes/stl/spring2.stl
Joints:
- joint leg_l_spring_joint1: axis 0 -1 0 -> 1 0 0
- joint leg_l_spring_joint3: axis 0 -1 0 -> 1 0 0
- joint leg_r_spring_joint1: axis 0 -1 0 -> 1 0 0
- joint leg_r_spring_joint3: axis 0 -1 0 -> 1 0 0

File: ginko_description/gazebo/urdf_sim/modules/leg_l_spring.urdf.xacro (robot description, xacro)
@@ -147,5 +147,5 @@
 	    	<child  link="${name}_spring_link1"/>
 	    	<origin xyz="0.10911938 0.0 0.0" rpy="0 3.141593 0"/>
-	    	<axis xyz="0 -1 0"/>
+	    	<axis xyz="1 0 0"/>
 	    	<limit effort="1000.0" lower="-3.141593" upper="3.141593" velocity="10.0"/>
 	  	</joint>
@@ -296,5 +296,5 @@
 	    	<child  link="${name}_spring_link3"/>
 	    	<origin xyz="0.10911938 0.0 0.0" rpy="0 3.141593 0"/>
-	    	<axis xyz="0 -1 0"/>
+	    	<axis xyz="1 0 0"/>
 	    	<limit effort="1000.0" lower="-3.141593" upper="3.141593" velocity="10.0"/>
 	  	</joint>

File: ginko_description/gazebo/urdf_sim/modules/leg_r_spring.urdf.xacro (robot description, xacro)
@@ -148,5 +148,5 @@
 	    	<child  link="${name}_spring_link1"/>
 	    	<origin xyz="0.10911938 0.0 0.0" rpy="0 3.141593 0"/>
-	    	<axis xyz="0 -1 0"/>
+	    	<axis xyz="1 0 0"/>
 	    	<limit effort="1000.0" lower="-3.141593" upper="3.141593" velocity="10.0"/>
 	  	</joint>
@@ -297,5 +297,5 @@
 	    	<child  link="${name}_spring_link3"/>
 	    	<origin xyz="0.10911938 0.0 0.0" rpy="0 3.141593 0"/>
-	    	<axis xyz="0 -1 0"/>
+	    	<axis xyz="1 0 0"/>
 	    	<limit effort="1000.0" lower="-3.141593" upper="3.141593" velocity="10.0"/>
 	  	</joint>
