Commit message: rvizもobjで表示するように変更

File: ginko_description/gazebo/sdf/original_sim_mimic.urdf (robot description, URDF)
Before this commit: robot ginko, 31 links, 30 joints
Links:
- link arm_l_link0: geometry collision mesh filename=package://ginko_description/meshes/stl/link09_l_arm01.stl; visual mesh filename=package://ginko_description/meshes/obj/link09_l_arm01.obj
- link arm_l_link1: geometry collision mesh filename=package://ginko_description/meshes/stl/link10_l_arm02.stl; visual mesh filename=package://ginko_description/meshes/obj/link10_l_arm02.obj
- link arm_l_link2: geometry collision mesh filename=package://ginko_description/meshes/stl/link11_l_scissor01.s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; visual mesh filename=package://ginko_description/meshes/obj/link11_l_scissor01.o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
- link arm_l_link3: geometry collision mesh filename=package://ginko_description/meshes/stl/link12_l_scissor02.s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; visual mesh filename=package://ginko_description/meshes/obj/link12_l_scissor02.o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
- link arm_l_urg_link: geometry collision mesh filename=package://ginko_description/meshes/stl/urg.stl; visual mesh filename=package://ginko_description/meshes/obj/urg.obj
- link arm_r_link0: geometry collision mesh filename=package://ginko_description/meshes/stl/link09_r_arm01.stl; visual mesh filename=package://ginko_description/meshes/obj/link09_r_arm01.obj
- link arm_r_link1: geometry collision mesh filename=package://ginko_description/meshes/stl/link10_r_arm02.stl; visual mesh filename=package://ginko_description/meshes/obj/link10_r_arm02.obj
- link arm_r_link2: geometry collision mesh filename=package://ginko_description/meshes/stl/link11_r_scissor01.s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; visual mesh filename=package://ginko_description/meshes/obj/link11_r_scissor01.o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
- link arm_r_link3: geometry collision mesh filename=package://ginko_description/meshes/stl/link12_r_scissor02.s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; visual mesh filename=package://ginko_description/meshes/obj/link12_r_scissor02.o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
- link arm_r_urg_link: geometry collision mesh filename=package://ginko_description/meshes/stl/urg.stl; visual mesh filename=package://ginko_description/meshes/obj/urg.obj
- link body_link0: geometry collision mesh filename=package://ginko_description/meshes/stl/link00_chest.stl; visual mesh filename=package://ginko_description/meshes/obj/link00_chest.obj
- link body_link1: geometry collision mesh filename=package://ginko_description/meshes/stl/link01_waist.stl; visual mesh filename=package://ginko_description/meshes/obj/link01_waist.obj
- link leg_l_link0: geometry collision mesh filename=package://ginko_description/meshes/stl/link02_l_femoral.stl; visual mesh filename=package://ginko_description/meshes/obj/link02_l_femoral.obj
- link leg_l_link1: geometry collision mesh filename=package://ginko_description/meshes/stl/link03_l_leg01.stl; visual mesh filename=package://ginko_description/meshes/obj/link03_l_leg01.obj
- link leg_l_link2: geometry collision mesh filename=package://ginko_description/meshes/stl/link04_l_leg02.stl; visual mesh filename=package://ginko_description/meshes/obj/link04_l_leg02.obj
- link leg_l_link3: geometry collision mesh filename=package://ginko_description/meshes/stl/link05_l_knee.stl; visual mesh filename=package://ginko_description/meshes/obj/link05_l_knee.obj
- link leg_l_link4: geometry collision mesh filename=package://ginko_description/meshes/stl/link03_l_leg01.stl; visual mesh filename=package://ginko_description/meshes/obj/link03_l_leg01.obj
- link leg_l_link5: geometry collision mesh filename=package://ginko_description/meshes/stl/link04_l_leg02.stl; visual mesh filename=package://ginko_description/meshes/obj/link04_l_leg02.obj
- link leg_l_link6: geometry collision mesh filename=package://ginko_description/meshes/stl/link06_l_toe01.stl; visual mesh filename=package://ginko_description/meshes/obj/link06_l_toe01.obj
- link leg_l_link7: geometry collision mesh filename=package://ginko_description/meshes/stl/link07_l_toe02.stl; visual mesh filename=package://ginko_description/meshes/obj/link07_l_toe02.obj
- link leg_l_link8: geometry collision mesh filename=package://ginko_description/meshes/stl/link08_l_toe03.stl; visual mesh filename=package://ginko_description/meshes/obj/link08_l_toe03.obj
- link leg_r_link0: geometry collision mesh filename=package://ginko_description/meshes/stl/link02_r_femoral.stl; visual mesh filename=package://ginko_description/meshes/obj/link02_r_femoral.obj
- link leg_r_link1: geometry collision mesh filename=package://ginko_description/meshes/stl/link03_r_leg01.stl; visual mesh filename=package://ginko_description/meshes/obj/link03_r_leg01.obj
- link leg_r_link2: geometry collision mesh filename=package://ginko_description/meshes/stl/link04_r_leg02.stl; visual mesh filename=package://ginko_description/meshes/obj/link04_r_leg02.obj
- link leg_r_link3: geometry collision mesh filename=package://ginko_description/meshes/stl/link05_r_knee.stl; visual mesh filename=package://ginko_description/meshes/obj/link05_r_knee.obj
- link leg_r_link4: geometry collision mesh filename=package://ginko_description/meshes/stl/link03_r_leg01.stl; visual mesh filename=package://ginko_description/meshes/obj/link03_r_leg01.obj
- link leg_r_link5: geometry collision mesh filename=package://ginko_description/meshes/stl/link04_r_leg02.stl; visual mesh filename=package://ginko_description/meshes/obj/link04_r_leg02.obj
- link leg_r_link6: geometry collision mesh filename=package://ginko_description/meshes/stl/link06_r_toe01.stl; visual mesh filename=package://ginko_description/meshes/obj/link06_r_toe01.obj
- link leg_r_link7: geometry collision mesh filename=package://ginko_description/meshes/stl/link07_r_toe02.stl; visual mesh filename=package://ginko_description/meshes/obj/link07_r_toe02.obj
- link leg_r_link8: geometry collision mesh filename=package://ginko_description/meshes/stl/link08_r_toe03.stl; visual mesh filename=package://ginko_description/meshes/obj/link08_r_toe03.obj
