Commit message: 不要なファイルを削除

File: ginko_description/urdf/modules/arm_l.urdf.xacro (robot description, xacro)
@@ -9,6 +9,6 @@
 				<origin xyz="0 0 0" rpy="0 0 0"/>
 				<geometry>
-					<!-- <mesh filename="package://ginko_description/models/ginko_auto/meshes/stl/link01_waist.stl"/> -->
-					<mesh filename="package://ginko_description/models/ginko_auto/meshes/stl/link09_l_arm01.stl"/>
+					<!-- <mesh filename="package://ginko_description/meshes/stl/link01_waist.stl"/> -->
+					<mesh filename="package://ginko_description/meshes/stl/link09_l_arm01.stl"/>
 				</geometry>
 			</collision>
@@ -17,7 +17,7 @@
 				<origin xyz="0 0 0" rpy="0 0 0"/>
 				<geometry>
-					<!-- <mesh filename="package://ginko_description/models/ginko_auto/meshes/stl/link01_waist.stl"/> -->
-					<mesh filename="package://ginko_description/models/ginko_auto/meshes/stl/link09_l_arm01.stl"/>
-					<!-- <mesh filename="package://ginko_description/models/ginko_auto/meshes/dae/link09_l_arm01.dae"/> -->
+					<!-- <mesh filename="package://ginko_description/meshes/stl/link01_waist.stl"/> -->
+					<mesh filename="package://ginko_description/meshes/stl/link09_l_arm01.stl"/>
+					<!-- <mesh filename="package://ginko_description/meshes/dae/link09_l_arm01.dae"/> -->
 				</geometry>
 			</visual>
@@ -45,5 +45,5 @@
 				<origin xyz="0 0 0" rpy="0 0 0"/>
 	    		<geometry>
-					<mesh filename="package://ginko_description/models/ginko_auto/meshes/stl/link10_l_arm02.stl"/>
+					<mesh filename="package://ginko_description/meshes/stl/link10_l_arm02.stl"/>
 	    		</geometry>
 			</collision>
@@ -52,6 +52,6 @@
 				<origin xyz="0 0 0" rpy="0 0 0"/>
 	    		<geometry>
-					<mesh filename="package://ginko_description/models/ginko_auto/meshes/stl/link10_l_arm02.stl"/>
-					<!-- <mesh filename="package://ginko_description/models/ginko_auto/meshes/dae/link10_l_arm02.dae"/> -->
+					<mesh filename="package://ginko_description/meshes/stl/link10_l_arm02.stl"/>
+					<!-- <mesh filename="package://ginko_description/meshes/dae/link10_l_arm02.dae"/> -->
 	    		</geometry>
 			</visual>
@@ -88,5 +88,5 @@
 				<origin xyz="0 0 0" rpy="0 0 0"/>
 	    		<geometry>
-					<mesh filename="package://ginko_description/models/ginko_auto/meshes/stl/link11_l_scissor01.stl"/>
+					<mesh filename="package://ginko_description/meshes/stl/link11_l_scissor01.stl"/>
 	    		</geometry>
 			</collision>
@@ -95,6 +95,6 @@
 				<origin xyz="0 0 0" rpy="0 0 0"/>
 	    		<geometry>
-					<mesh filename="package://ginko_description/models/ginko_auto/meshes/stl/link11_l_scissor01.stl"/>
-					<!-- <mesh filename="package://ginko_description/models/ginko_auto/meshes/dae/link11_l_scissor01.dae"/> -->
+					<mesh filename="package://ginko_description/meshes/stl/link11_l_scissor01.stl"/>
+					<!-- <mesh filename="package://ginko_description/meshes/dae/link11_l_scissor01.dae"/> -->
 	    		</geometry>
 			</visual>
@@ -121,5 +121,5 @@
 				<origin xyz="0 0 0" rpy="0 0 0"/>
 	    		<geometry>
-					<mesh filename="package://ginko_description/models/ginko_auto/meshes/stl/link12_l_scissor02.stl"/>
+					<mesh filename="package://ginko_description/meshes/stl/link12_l_scissor02.stl"/>
 	    		</geometry>
 			</collision>
@@ -128,6 +128,6 @@
 				<origin xyz="0 0 0" rpy="0 0 0"/>
 	    		<geometry>
-					<mesh filename="package://ginko_description/models/ginko_auto/meshes/stl/link12_l_scissor02.stl"/>
-					<!-- <mesh filename="package://ginko_description/models/ginko_auto/meshes/dae/link12_l_scissor02.dae"/> -->
+					<mesh filename="package://ginko_description/meshes/stl/link12_l_scissor02.stl"/>
+					<!-- <mesh filename="package://ginko_description/meshes/dae/link12_l_scissor02.dae"/> -->
 	    		</geometry>
 			</visual>
@@ -154,5 +154,5 @@
 				<origin xyz="0 0 0" rpy="0 0 0"/>
 	    		<geometry>
-					<mesh filename="package://ginko_description/models/ginko_auto/meshes/stl/urg.stl"/>
+					<mesh filename="package://ginko_description/meshes/stl/urg.stl"/>
 	    		</geometry>
 			</collision>
@@ -161,6 +161,6 @@
 				<origin xyz="0 0 0" rpy="0 0 0"/>
 	    		<geometry>
-	    			<mesh filename="package://ginko_description/models/ginko_auto/meshes/stl/urg.stl"/>
-					<!-- <mesh filename="package://ginko_description/models/ginko_auto/meshes/dae/urg.dae"/> -->
+	    			<mesh filename="package://ginko_description/meshes/stl/urg.stl"/>
+					<!-- <mesh filename="package://ginko_description/meshes/dae/urg.dae"/> -->
 	    		</geometry>
 			</visual>

File: ginko_description/urdf/modules/arm_r.urdf.xacro (robot description, xacro)
@@ -9,5 +9,5 @@
 				<origin xyz="0 0 0" rpy="0 0 0"/>
 				<geometry>
-					<mesh filename="package://ginko_description/models/ginko_auto/meshes/stl/link09_r_arm01.stl"/>
+					<mesh filename="package://ginko_description/meshes/stl/link09_r_arm01.stl"/>
 				</geometry>
 			</collision>
@@ -16,6 +16,6 @@
 				<origin xyz="0 0 0" rpy="0 0 0"/>
 				<geometry>
-					<mesh filename="package://ginko_description/models/ginko_auto/meshes/stl/link09_r_arm01.stl"/>
-					<!-- <mesh filename="package://ginko_description/models/ginko_auto/meshes/dae/link09_r_arm01.dae"/> -->
+					<mesh filename="package://ginko_description/meshes/stl/link09_r_arm01.stl"/>
+					<!-- <mesh filename="package://ginko_description/meshes/dae/link09_r_arm01.dae"/> -->
 				</geometry>
 			</visual>
@@ -40,5 +40,5 @@
 				<origin xyz="0 0 0" rpy="0 0 0"/>
 	    		<geometry>
-					<mesh filename="package://ginko_description/models/ginko_auto/meshes/stl/link10_r_arm02.stl"/>
+					<mesh filename="package://ginko_description/meshes/stl/link10_r_arm02.stl"/>
 	    		</geometry>
 			</collision>
@@ -47,6 +47,6 @@
 				<origin xyz="0 0 0" rpy="0 0 0"/>
 	    		<geometry>
-					<mesh filename="package://ginko_description/models/ginko_auto/meshes/stl/link10_r_arm02.stl"/>
-					<!-- <mesh filename="package://ginko_description/models/ginko_auto/meshes/dae/link10_r_arm02.dae"/> -->
+					<mesh filename="package://ginko_description/meshes/stl/link10_r_arm02.stl"/>
+					<!-- <mesh filename="package://ginko_description/meshes/dae/link10_r_arm02.dae"/> -->
 	    		</geometry>
 			</visual>
@@ -80,5 +80,5 @@
 				<origin xyz="0 0 0" rpy="0 0 0"/>
 	    		<geometry>
-					<mesh filename="package://ginko_description/models/ginko_auto/meshes/stl/link11_r_scissor01.stl"/>
+					<mesh filename="package://ginko_description/meshes/stl/link11_r_scissor01.stl"/>
 	    		</geometry>
 			</collision>
@@ -87,6 +87,6 @@
 				<origin xyz="0 0 0" rpy="0 0 0"/>
 	    		<geometry>
-					<mesh filename="package://ginko_description/models/ginko_auto/meshes/stl/link11_r_scissor01.stl"/>
-					<!-- <mesh filename="package://ginko_description/models/ginko_auto/meshes/dae/link11_r_scissor01.dae"/> -->
+					<mesh filename="package://ginko_description/meshes/stl/link11_r_scissor01.stl"/>
+					<!-- <mesh filename="package://ginko_description/meshes/dae/link11_r_scissor01.dae"/> -->
 	    		</geometry>
 			</visual>
@@ -110,5 +110,5 @@
 				<origin xyz="0 0 0" rpy="0 0 0"/>
 	    		<geometry>
-					<mesh filename="package://ginko_description/models/ginko_auto/meshes/stl/link12_r_scissor02.stl"/>
+					<mesh filename="package://ginko_description/meshes/stl/link12_r_scissor02.stl"/>
 	    		</geometry>
 			</collision>
@@ -117,6 +117,6 @@
 				<origin xyz="0 0 0" rpy="0 0 0"/>
 	    		<geometry>
-					<mesh filename="package://ginko_description/models/ginko_auto/meshes/stl/link12_r_scissor02.stl"/>
-					<!-- <mesh filename="package://ginko_description/models/ginko_auto/meshes/dae/link12_r_scissor02.dae"/> -->
+					<mesh filename="package://ginko_description/meshes/stl/link12_r_scissor02.stl"/>
+					<!-- <mesh filename="package://ginko_description/meshes/dae/link12_r_scissor02.dae"/> -->
 	    		</geometry>
 			</visual>
@@ -140,5 +140,5 @@
 				<origin xyz="0 0 0" rpy="0 0 0"/>
 	    		<geometry>
-					<mesh filename="package://ginko_description/models/ginko_auto/meshes/stl/urg.stl"/>
+					<mesh filename="package://ginko_description/meshes/stl/urg.stl"/>
 	    		</geometry>
 			</collision>
@@ -147,6 +147,6 @@
 				<origin xyz="0 0 0" rpy="0 0 0"/>
 	    		<geometry>
-	    			<mesh filename="package://ginko_description/models/ginko_auto/meshes/stl/urg.stl"/>
-					<!-- <mesh filename="package://ginko_description/models/ginko_auto/meshes/dae/urg.dae"/> -->
+	    			<mesh filename="package://ginko_description/meshes/stl/urg.stl"/>
+					<!-- <mesh filename="package://ginko_description/meshes/dae/urg.dae"/> -->
 	    		</geometry>
 			</visual>

File: ginko_description/urdf/modules/body.urdf.xacro (robot description, xacro)
@@ -9,5 +9,5 @@
 				<origin xyz="0 0 0" rpy="0 0 0"/>
 				<geometry>
-					<mesh filename="package://ginko_description/models/ginko_auto/meshes/stl/link00_chest.stl"/>
+					<mesh filename="package://ginko_description/meshes/stl/link00_chest.stl"/>
 				</geometry>
 			</collision>
@@ -16,7 +16,7 @@
 				<origin xyz="0 0 0" rpy="0 0 0"/>
 				<geometry>
-					<!-- <mesh filename="package://ginko_description/models/ginko_auto/meshes/obj/link00_chest.obj"/> -->
-					<mesh filename="package://ginko_description/models/ginko_auto/meshes/stl/link00_chest.stl"/>
-					<!-- <mesh filename="package://ginko_description/models/ginko_auto/meshes/dae/link00_chest.dae"/> -->
+					<!-- <mesh filename="package://ginko_description/meshes/obj/link00_chest.obj"/> -->
+					<mesh filename="package://ginko_description/meshes/stl/link00_chest.stl"/>
+					<!-- <mesh filename="package://ginko_description/meshes/dae/link00_chest.dae"/> -->
 				</geometry>
 			</visual>
@@ -42,5 +42,5 @@
 				<origin xyz="0 0 0" rpy="0 0 0"/>
 	    		<geometry>
-					<mesh filename="package://ginko_description/models/ginko_auto/meshes/stl/link01_waist.stl"/>
+					<mesh filename="package://ginko_description/meshes/stl/link01_waist.stl"/>
 	    		</geometry>
 			</collision>
@@ -49,7 +49,7 @@
 				<origin xyz="0 0 0" rpy="0 0 0"/>
 	    		<geometry>
-	    			<!-- <mesh filename="package://ginko_description/models/ginko_auto/meshes/obj/link01_waist.obj"/> -->
-					<mesh filename="package://ginko_description/models/ginko_auto/meshes/stl/link01_waist.stl"/>
-					<!-- <mesh filename="package://ginko_description/models/ginko_auto/meshes/dae/link01_waist.dae"/> -->
+	    			<!-- <mesh filename="package://ginko_description/meshes/obj/link01_waist.obj"/> -->
+					<mesh filename="package://ginko_description/meshes/stl/link01_waist.stl"/>
+					<!-- <mesh filename="package://ginko_description/meshes/dae/link01_waist.dae"/> -->
 	    		</geometry>
 			</visual>

File: ginko_description/urdf/modules/leg_l.urdf.xacro (robot description, xacro)
@@ -9,5 +9,5 @@
 				<origin xyz="0 0 0" rpy="0 0 0"/>
 				<geometry>
-					<mesh filename="package://ginko_description/models/ginko_auto/meshes/stl/link02_l_femoral.stl"/>
+					<mesh filename="package://ginko_description/meshes/stl/link02_l_femoral.stl"/>
 				</geometry>
 			</collision>
@@ -16,6 +16,6 @@
 				<origin xyz="0 0 0" rpy="0 0 0"/>
 				<geometry>
-					<mesh filename="package://ginko_description/models/ginko_auto/meshes/stl/link02_l_femoral.stl"/>
-					<!-- <mesh filename="package://ginko_description/models/ginko_auto/meshes/dae/link02_l_femoral.dae"/> -->
+					<mesh filename="package://ginko_description/meshes/stl/link02_l_femoral.stl"/>
+					<!-- <mesh filename="package://ginko_description/meshes/dae/link02_l_femoral.dae"/> -->
 				</geometry>
 			</visual>
@@ -42,5 +42,5 @@
 				<origin xyz="0 0 0" rpy="0 0 0"/>
 	    		<geometry>
-					<mesh filename="package://ginko_description/models/ginko_auto/meshes/stl/link03_l_leg01.stl"/>
+					<mesh filename="package://ginko_description/meshes/stl/link03_l_leg01.stl"/>
 	    		</geometry>
 			</collision>
@@ -49,6 +49,6 @@
 				<origin xyz="0 0 0" rpy="0 0 0"/>
 	    		<geometry>
-					<mesh filename="package://ginko_description/models/ginko_auto/meshes/stl/link03_l_leg01.stl"/>
-					<!-- <mesh filename="package://ginko_description/models/ginko_auto/meshes/dae/link03_l_leg01.dae"/> -->
+					<mesh filename="package://ginko_description/meshes/stl/link03_l_leg01.stl"/>
+					<!-- <mesh filename="package://ginko_description/meshes/dae/link03_l_leg01.dae"/> -->
 	    		</geometry>
 			</visual>
@@ -75,5 +75,5 @@
 				<origin xyz="0 0 0" rpy="0 0 0"/>
 	    		<geometry>
-					<mesh filename="package://ginko_description/models/ginko_auto/meshes/stl/link04_l_leg02.stl"/>
+					<mesh filename="package://ginko_description/meshes/stl/link04_l_leg02.stl"/>
 	    		</geometry>
 			</collision>
@@ -82,6 +82,6 @@
 				<origin xyz="0 0 0" rpy="0 0 0"/>
 	    		<geometry>
-					<mesh filename="package://ginko_description/models/ginko_auto/meshes/stl/link04_l_leg02.stl"/>
-					<!-- <mesh filename="package://ginko_description/models/ginko_auto/meshes/dae/link04_l_leg02.dae"/> -->
+					<mesh filename="package://ginko_description/meshes/stl/link04_l_leg02.stl"/>
+					<!-- <mesh filename="package://ginko_description/meshes/dae/link04_l_leg02.dae"/> -->
 	    		</geometry>
 			</visual>
@@ -108,12 +108,12 @@
 				<origin xyz="0 0 0" rpy="0 0 0"/>
 	    		<geometry>
-					<mesh filename="package://ginko_description/models/ginko_auto/meshes/stl/link05_l_knee.stl"/>
-	    		</geometry>
-			</collision>
-	    	<visual>
-				<origin xyz="0 0 0" rpy="0 0 0"/>
-	    		<geometry>
-					<mesh filename="package://ginko_description/models/ginko_auto/meshes/stl/link05_l_knee.stl"/>
-					<!-- <mesh filename="package://ginko_description/models/ginko_auto/meshes/dae/link05_l_knee.dae"/> -->
+					<mesh filename="package://ginko_description/meshes/stl/link05_l_knee.stl"/>
+	    		</geometry>
+			</collision>
+	    	<visual>
+				<origin xyz="0 0 0" rpy="0 0 0"/>
+	    		<geometry>
+					<mesh filename="package://ginko_description/meshes/stl/link05_l_knee.stl"/>
+					<!-- <mesh filename="package://ginko_description/meshes/dae/link05_l_knee.dae"/> -->
 	    		</geometry>
 			</visual>
@@ -139,11 +139,11 @@
 				<origin xyz="0 0 0" rpy="0 0 0"/>
 	    		<geometry>
-					<mesh filename="package://ginko_description/models/ginko_auto/meshes/stl/link03_l_leg01.stl"/>
-	    		</geometry>
-			</collision>
-	    	<visual>
-				<origin xyz="0 0 0" rpy="0 0 0"/>
-	    		<geometry>
-					<mesh filename="package://ginko_description/models/ginko_auto/meshes/stl/link03_l_leg01.stl"/>
+					<mesh filename="package://ginko_description/meshes/stl/link03_l_leg01.stl"/>
+	    		</geometry>
+			</collision>
+	    	<visual>
+				<origin xyz="0 0 0" rpy="0 0 0"/>
+	    		<geometry>
+					<mesh filename="package://ginko_description/meshes/stl/link03_l_leg01.stl"/>
 	    		</geometry>
 			</visual>
@@ -169,11 +169,11 @@
 				<origin xyz="0 0 0" rpy="0 0 0"/>
 	    		<geometry>
-					<mesh filename="package://ginko_description/models/ginko_auto/meshes/stl/link04_l_leg02.stl"/>
-	    		</geometry>
-			</collision>
-	    	<visual>
-				<origin xyz="0 0 0" rpy="0 0 0"/>
-	    		<geometry>
-					<mesh filename="package://ginko_description/models/ginko_auto/meshes/stl/link04_l_leg02.stl"/>
+					<mesh filename="package://ginko_description/meshes/stl/link04_l_leg02.stl"/>
+	    		</geometry>
+			</collision>
+	    	<visual>
+				<origin xyz="0 0 0" rpy="0 0 0"/>
+	    		<geometry>
+					<mesh filename="package://ginko_description/meshes/stl/link04_l_leg02.stl"/>
 	    		</geometry>
 			</visual>
@@ -200,11 +200,11 @@
 				<origin xyz="0 0 0" rpy="0 0 0"/>
 	    		<geometry>
-					<mesh filename="package://ginko_description/models/ginko_auto/meshes/stl/link06_l_toe01.stl"/>
-	    		</geometry>
-			</collision>
-	    	<visual>
-				<origin xyz="0 0 0" rpy="0 0 0"/>
-	    		<geometry>
-					<mesh filename="package://ginko_description/models/ginko_auto/meshes/stl/link06_l_toe01.stl"/>
+					<mesh filename="package://ginko_description/meshes/stl/link06_l_toe01.stl"/>
+	    		</geometry>
+			</collision>
+	    	<visual>
+				<origin xyz="0 0 0" rpy="0 0 0"/>
+	    		<geometry>
+					<mesh filename="package://ginko_description/meshes/stl/link06_l_toe01.stl"/>
 	    		</geometry>
 			</visual>
@@ -229,11 +229,11 @@
 				<origin xyz="0 0 0" rpy="0 0 0"/>
 	    		<geometry>
-					<mesh filename="package://ginko_description/models/ginko_auto/meshes/stl/link07_l_toe02.stl"/>
-	    		</geometry>
-			</collision>
-	    	<visual>
-				<origin xyz="0 0 0" rpy="0 0 0"/>
-	    		<geometry>
-					<mesh filename="package://ginko_description/models/ginko_auto/meshes/stl/link07_l_toe02.stl"/>
+					<mesh filename="package://ginko_description/meshes/stl/link07_l_toe02.stl"/>
+	    		</geometry>
+			</collision>
+	    	<visual>
+				<origin xyz="0 0 0" rpy="0 0 0"/>
+	    		<geometry>
+					<mesh filename="package://ginko_description/meshes/stl/link07_l_toe02.stl"/>
 	    		</geometry>
 			</visual>
@@ -258,11 +258,11 @@
 				<origin xyz="0 0 0" rpy="0 0 0"/>
 	    		<geometry>
-					<mesh filename="package://ginko_description/models/ginko_auto/meshes/stl/link08_l_toe03.stl"/>
-	    		</geometry>
-			</collision>
-	    	<visual>
-				<origin xyz="0 0 0" rpy="0 0 0"/>
-	    		<geometry>
-					<mesh filename="package://ginko_description/models/ginko_auto/meshes/stl/link08_l_toe03.stl"/>
+					<mesh filename="package://ginko_description/meshes/stl/link08_l_toe03.stl"/>
+	    		</geometry>
+			</collision>
+	    	<visual>
+				<origin xyz="0 0 0" rpy="0 0 0"/>
+	    		<geometry>
+					<mesh filename="package://ginko_description/meshes/stl/link08_l_toe03.stl"/>
 	    		</geometry>
 			</visual>
