Commit message: 不要なファイルを削除

File: ginko_description/urdf/modules/leg_r.urdf.xacro (robot description, xacro)
@@ -8,5 +8,5 @@
 				<origin xyz="0 0 0" rpy="0 0 0"/>
 				<geometry>
-					<mesh filename="package://ginko_description/models/ginko_auto/meshes/stl/link02_r_femoral.stl"/>
+					<mesh filename="package://ginko_description/meshes/stl/link02_r_femoral.stl"/>
 				</geometry>
 			</collision>
@@ -14,5 +14,5 @@
 				<origin xyz="0 0 0" rpy="0 0 0"/>
 				<geometry>
-					<mesh filename="package://ginko_description/models/ginko_auto/meshes/stl/link02_r_femoral.stl"/>
+					<mesh filename="package://ginko_description/meshes/stl/link02_r_femoral.stl"/>
 				</geometry>
 			</visual>
@@ -38,11 +38,11 @@
 				<origin xyz="0 0 0" rpy="0 0 0"/>
 	    		<geometry>
-					<mesh filename="package://ginko_description/models/ginko_auto/meshes/stl/link03_r_leg01.stl"/>
-	    		</geometry>
-			</collision>
-	    	<visual>
-				<origin xyz="0 0 0" rpy="0 0 0"/>
-	    		<geometry>
-					<mesh filename="package://ginko_description/models/ginko_auto/meshes/stl/link03_r_leg01.stl"/>
+					<mesh filename="package://ginko_description/meshes/stl/link03_r_leg01.stl"/>
+	    		</geometry>
+			</collision>
+	    	<visual>
+				<origin xyz="0 0 0" rpy="0 0 0"/>
+	    		<geometry>
+					<mesh filename="package://ginko_description/meshes/stl/link03_r_leg01.stl"/>
 	    		</geometry>
 			</visual>
@@ -68,11 +68,11 @@
 				<origin xyz="0 0 0" rpy="0 0 0"/>
 	    		<geometry>
-					<mesh filename="package://ginko_description/models/ginko_auto/meshes/stl/link04_r_leg02.stl"/>
-	    		</geometry>
-			</collision>
-	    	<visual>
-				<origin xyz="0 0 0" rpy="0 0 0"/>
-	    		<geometry>
-					<mesh filename="package://ginko_description/models/ginko_auto/meshes/stl/link04_r_leg02.stl"/>
+					<mesh filename="package://ginko_description/meshes/stl/link04_r_leg02.stl"/>
+	    		</geometry>
+			</collision>
+	    	<visual>
+				<origin xyz="0 0 0" rpy="0 0 0"/>
+	    		<geometry>
+					<mesh filename="package://ginko_description/meshes/stl/link04_r_leg02.stl"/>
 	    		</geometry>
 			</visual>
@@ -99,11 +99,11 @@
 				<origin xyz="0 0 0" rpy="0 0 0"/>
 	    		<geometry>
-					<mesh filename="package://ginko_description/models/ginko_auto/meshes/stl/link05_r_knee.stl"/>
-	    		</geometry>
-			</collision>
-	    	<visual>
-				<origin xyz="0 0 0" rpy="0 0 0"/>
-	    		<geometry>
-					<mesh filename="package://ginko_description/models/ginko_auto/meshes/stl/link05_r_knee.stl"/>
+					<mesh filename="package://ginko_description/meshes/stl/link05_r_knee.stl"/>
+	    		</geometry>
+			</collision>
+	    	<visual>
+				<origin xyz="0 0 0" rpy="0 0 0"/>
+	    		<geometry>
+					<mesh filename="package://ginko_description/meshes/stl/link05_r_knee.stl"/>
 	    		</geometry>
 			</visual>
@@ -130,11 +130,11 @@
 				<origin xyz="0 0 0" rpy="0 0 0"/>
 	    		<geometry>
-					<mesh filename="package://ginko_description/models/ginko_auto/meshes/stl/link03_r_leg01.stl"/>
-	    		</geometry>
-			</collision>
-	    	<visual>
-				<origin xyz="0 0 0" rpy="0 0 0"/>
-	    		<geometry>
-					<mesh filename="package://ginko_description/models/ginko_auto/meshes/stl/link03_r_leg01.stl"/>
+					<mesh filename="package://ginko_description/meshes/stl/link03_r_leg01.stl"/>
+	    		</geometry>
+			</collision>
+	    	<visual>
+				<origin xyz="0 0 0" rpy="0 0 0"/>
+	    		<geometry>
+					<mesh filename="package://ginko_description/meshes/stl/link03_r_leg01.stl"/>
 	    		</geometry>
 			</visual>
@@ -160,11 +160,11 @@
 				<origin xyz="0 0 0" rpy="0 0 0"/>
 	    		<geometry>
-					<mesh filename="package://ginko_description/models/ginko_auto/meshes/stl/link04_r_leg02.stl"/>
-	    		</geometry>
-			</collision>
-	    	<visual>
-				<origin xyz="0 0 0" rpy="0 0 0"/>
-	    		<geometry>
-					<mesh filename="package://ginko_description/models/ginko_auto/meshes/stl/link04_r_leg02.stl"/>
+					<mesh filename="package://ginko_description/meshes/stl/link04_r_leg02.stl"/>
+	    		</geometry>
+			</collision>
+	    	<visual>
+				<origin xyz="0 0 0" rpy="0 0 0"/>
+	    		<geometry>
+					<mesh filename="package://ginko_description/meshes/stl/link04_r_leg02.stl"/>
 	    		</geometry>
 			</visual>
@@ -191,11 +191,11 @@
 				<origin xyz="0 0 0" rpy="0 0 0"/>
 	    		<geometry>
-					<mesh filename="package://ginko_description/models/ginko_auto/meshes/stl/link06_r_toe01.stl"/>
-	    		</geometry>
-			</collision>
-	    	<visual>
-				<origin xyz="0 0 0" rpy="0 0 0"/>
-	    		<geometry>
-					<mesh filename="package://ginko_description/models/ginko_auto/meshes/stl/link06_r_toe01.stl"/>
+					<mesh filename="package://ginko_description/meshes/stl/link06_r_toe01.stl"/>
+	    		</geometry>
+			</collision>
+	    	<visual>
+				<origin xyz="0 0 0" rpy="0 0 0"/>
+	    		<geometry>
+					<mesh filename="package://ginko_description/meshes/stl/link06_r_toe01.stl"/>
 	    		</geometry>
 			</visual>
@@ -221,11 +221,11 @@
 				<origin xyz="0 0 0" rpy="0 0 0"/>
 	    		<geometry>
-					<mesh filename="package://ginko_description/models/ginko_auto/meshes/stl/link07_r_toe02.stl"/>
-	    		</geometry>
-			</collision>
-	    	<visual>
-				<origin xyz="0 0 0" rpy="0 0 0"/>
-	    		<geometry>
-					<mesh filename="package://ginko_description/models/ginko_auto/meshes/stl/link07_r_toe02.stl"/>
+					<mesh filename="package://ginko_description/meshes/stl/link07_r_toe02.stl"/>
+	    		</geometry>
+			</collision>
+	    	<visual>
+				<origin xyz="0 0 0" rpy="0 0 0"/>
+	    		<geometry>
+					<mesh filename="package://ginko_description/meshes/stl/link07_r_toe02.stl"/>
 	    		</geometry>
 			</visual>
@@ -250,11 +250,11 @@
 				<origin xyz="0 0 0" rpy="0 0 0"/>
 	    		<geometry>
-					<mesh filename="package://ginko_description/models/ginko_auto/meshes/stl/link08_r_toe03.stl"/>
-	    		</geometry>
-			</collision>
-	    	<visual>
-				<origin xyz="0 0 0" rpy="0 0 0"/>
-	    		<geometry>
-					<mesh filename="package://ginko_description/models/ginko_auto/meshes/stl/link08_r_toe03.stl"/>
+					<mesh filename="package://ginko_description/meshes/stl/link08_r_toe03.stl"/>
+	    		</geometry>
+			</collision>
+	    	<visual>
+				<origin xyz="0 0 0" rpy="0 0 0"/>
+	    		<geometry>
+					<mesh filename="package://ginko_description/meshes/stl/link08_r_toe03.stl"/>
 	    		</geometry>
 			</visual>

Commit message: sdfを統合するパッチを検証中

File: ginko_description/urdf/modules/arm_l.urdf.xacro (robot description, xacro)
@@ -9,5 +9,4 @@
 				<origin xyz="0 0 0" rpy="0 0 0"/>
 				<geometry>
-					<!-- <mesh filename="package://ginko_description/meshes/stl/link01_waist.stl"/> -->
 					<mesh filename="package://ginko_description/meshes/stl/link09_l_arm01.stl"/>
 				</geometry>
@@ -17,7 +16,5 @@
 				<origin xyz="0 0 0" rpy="0 0 0"/>
 				<geometry>
-					<!-- <mesh filename="package://ginko_description/meshes/stl/link01_waist.stl"/> -->
-					<mesh filename="package://ginko_description/meshes/stl/link09_l_arm01.stl"/>
-					<!-- <mesh filename="package://ginko_description/meshes/dae/link09_l_arm01.dae"/> -->
+					<mesh filename="package://ginko_description/meshes/obj/link09_l_arm01.obj"/>
 				</geometry>
 			</visual>
@@ -49,10 +46,9 @@
 			</collision>
 			<!-- Visualisation created from Color dae -->
-	    	<visual>
+			<visual>
 				<origin xyz="0 0 0" rpy="0 0 0"/>
-	    		<geometry>
-					<mesh filename="package://ginko_description/meshes/stl/link10_l_arm02.stl"/>
-					<!-- <mesh filename="package://ginko_description/meshes/dae/link10_l_arm02.dae"/> -->
-	    		</geometry>
+				<geometry>
+					<mesh filename="package://ginko_description/meshes/obj/link10_l_arm02.obj"/>
+				</geometry>
 			</visual>
 			<!-- nothing worth -->
@@ -92,10 +88,9 @@
 			</collision>
 			<!-- Visualisation created from Color dae -->
-	    	<visual>
+			<visual>
 				<origin xyz="0 0 0" rpy="0 0 0"/>
-	    		<geometry>
-					<mesh filename="package://ginko_description/meshes/stl/link11_l_scissor01.stl"/>
-					<!-- <mesh filename="package://ginko_description/meshes/dae/link11_l_scissor01.dae"/> -->
-	    		</geometry>
+				<geometry>
+					<mesh filename="package://ginko_description/meshes/obj/link11_l_scissor01.obj"/>
+				</geometry>
 			</visual>
 			<!-- nothing worth -->
@@ -125,10 +120,9 @@
 			</collision>
 			<!-- Visualisation created from Color dae -->
-	    	<visual>
+			<visual>
 				<origin xyz="0 0 0" rpy="0 0 0"/>
-	    		<geometry>
-					<mesh filename="package://ginko_description/meshes/stl/link12_l_scissor02.stl"/>
-					<!-- <mesh filename="package://ginko_description/meshes/dae/link12_l_scissor02.dae"/> -->
-	    		</geometry>
+				<geometry>
+					<mesh filename="package://ginko_description/meshes/obj/link12_l_scissor02.obj"/>
+				</geometry>
 			</visual>
 			<!-- nothing worth -->
@@ -158,10 +152,9 @@
 			</collision>
 			<!-- Visualisation created from Color dae -->
-	    	<visual>
+			<visual>
 				<origin xyz="0 0 0" rpy="0 0 0"/>
-	    		<geometry>
-	    			<mesh filename="package://ginko_description/meshes/stl/urg.stl"/>
-					<!-- <mesh filename="package://ginko_description/meshes/dae/urg.dae"/> -->
-	    		</geometry>
+				<geometry>
+					<mesh filename="package://ginko_description/meshes/obj/urg.obj"/>
+				</geometry>
 			</visual>
 			<!-- nothing worth -->

File: ginko_description/urdf/modules/arm_r.urdf.xacro (robot description, xacro)
@@ -16,6 +16,5 @@
 				<origin xyz="0 0 0" rpy="0 0 0"/>
 				<geometry>
-					<mesh filename="package://ginko_description/meshes/stl/link09_r_arm01.stl"/>
-					<!-- <mesh filename="package://ginko_description/meshes/dae/link09_r_arm01.dae"/> -->
+					<mesh filename="package://ginko_description/meshes/obj/link09_r_arm01.obj"/>
 				</geometry>
 			</visual>
@@ -44,10 +43,9 @@
 			</collision>
 			<!-- Visualisation created from Color dae -->
-	    	<visual>
+			<visual>
 				<origin xyz="0 0 0" rpy="0 0 0"/>
-	    		<geometry>
-					<mesh filename="package://ginko_description/meshes/stl/link10_r_arm02.stl"/>
-					<!-- <mesh filename="package://ginko_description/meshes/dae/link10_r_arm02.dae"/> -->
-	    		</geometry>
+				<geometry>
+					<mesh filename="package://ginko_description/meshes/obj/link10_r_arm02.obj"/>
+				</geometry>
 			</visual>
 			<!-- nothing worth -->
@@ -84,10 +82,9 @@
 			</collision>
 			<!-- Visualisation created from Color dae -->
-	    	<visual>
+			<visual>
 				<origin xyz="0 0 0" rpy="0 0 0"/>
-	    		<geometry>
-					<mesh filename="package://ginko_description/meshes/stl/link11_r_scissor01.stl"/>
-					<!-- <mesh filename="package://ginko_description/meshes/dae/link11_r_scissor01.dae"/> -->
-	    		</geometry>
+				<geometry>
+					<mesh filename="package://ginko_description/meshes/obj/link11_r_scissor01.obj"/>
+				</geometry>
 			</visual>
 			<!-- nothing worth -->
@@ -114,10 +111,9 @@
 			</collision>
 			<!-- Visualisation created from Color dae -->
-	    	<visual>
+			<visual>
 				<origin xyz="0 0 0" rpy="0 0 0"/>
-	    		<geometry>
-					<mesh filename="package://ginko_description/meshes/stl/link12_r_scissor02.stl"/>
-					<!-- <mesh filename="package://ginko_description/meshes/dae/link12_r_scissor02.dae"/> -->
-	    		</geometry>
+				<geometry>
+					<mesh filename="package://ginko_description/meshes/obj/link12_r_scissor02.obj"/>
+				</geometry>
 			</visual>
 			<!-- nothing worth -->
@@ -144,10 +140,9 @@
 			</collision>
 			<!-- Visualisation created from Color dae -->
-	    	<visual>
+			<visual>
 				<origin xyz="0 0 0" rpy="0 0 0"/>
-	    		<geometry>
-	    			<mesh filename="package://ginko_description/meshes/stl/urg.stl"/>
-					<!-- <mesh filename="package://ginko_description/meshes/dae/urg.dae"/> -->
-	    		</geometry>
+				<geometry>
+					<mesh filename="package://ginko_description/meshes/obj/urg.obj"/>
+				</geometry>
 			</visual>
 			<!-- nothing worth -->

File: ginko_description/urdf/modules/body.urdf.xacro (robot description, xacro)
@@ -16,7 +16,5 @@
 				<origin xyz="0 0 0" rpy="0 0 0"/>
 				<geometry>
-					<!-- <mesh filename="package://ginko_description/meshes/obj/link00_chest.obj"/> -->
-					<mesh filename="package://ginko_description/meshes/stl/link00_chest.stl"/>
-					<!-- <mesh filename="package://ginko_description/meshes/dae/link00_chest.dae"/> -->
+					<mesh filename="package://ginko_description/meshes/obj/link00_chest.obj"/>
 				</geometry>
 			</visual>
@@ -46,11 +44,9 @@
 			</collision>
 			<!-- Visualisation created from Color dae -->
-	    	<visual>
+			<visual>
 				<origin xyz="0 0 0" rpy="0 0 0"/>
-	    		<geometry>
-	    			<!-- <mesh filename="package://ginko_description/meshes/obj/link01_waist.obj"/> -->
-					<mesh filename="package://ginko_description/meshes/stl/link01_waist.stl"/>
-					<!-- <mesh filename="package://ginko_description/meshes/dae/link01_waist.dae"/> -->
-	    		</geometry>
+				<geometry>
+					<mesh filename="package://ginko_description/meshes/obj/link01_waist.obj"/>
+				</geometry>
 			</visual>
 			<inertial>

File: ginko_description/urdf/modules/leg_l.urdf.xacro (robot description, xacro)
@@ -16,6 +16,5 @@
 				<origin xyz="0 0 0" rpy="0 0 0"/>
 				<geometry>
-					<mesh filename="package://ginko_description/meshes/stl/link02_l_femoral.stl"/>
-					<!-- <mesh filename="package://ginko_description/meshes/dae/link02_l_femoral.dae"/> -->
+					<mesh filename="package://ginko_description/meshes/obj/link02_l_femoral.obj"/>
 				</geometry>
 			</visual>
@@ -46,10 +45,9 @@
 			</collision>
 			<!-- Visualisation created from Color dae -->
-	    	<visual>
-				<origin xyz="0 0 0" rpy="0 0 0"/>
-	    		<geometry>
-					<mesh filename="package://ginko_description/meshes/stl/link03_l_leg01.stl"/>
-					<!-- <mesh filename="package://ginko_description/meshes/dae/link03_l_leg01.dae"/> -->
-	    		</geometry>
+			<visual>
+				<origin xyz="0 0 0" rpy="0 0 0"/>
+				<geometry>
+					<mesh filename="package://ginko_description/meshes/obj/link03_l_leg01.obj"/>
+				</geometry>
 			</visual>
 			<inertial>
@@ -79,10 +77,9 @@
 			</collision>
 			<!-- Visualisation created from Color dae -->
-	    	<visual>
-				<origin xyz="0 0 0" rpy="0 0 0"/>
-	    		<geometry>
-					<mesh filename="package://ginko_description/meshes/stl/link04_l_leg02.stl"/>
-					<!-- <mesh filename="package://ginko_description/meshes/dae/link04_l_leg02.dae"/> -->
-	    		</geometry>
+			<visual>
+				<origin xyz="0 0 0" rpy="0 0 0"/>
+				<geometry>
+					<mesh filename="package://ginko_description/meshes/obj/link04_l_leg02.obj"/>
+				</geometry>
 			</visual>
 			<inertial>
@@ -111,10 +108,9 @@
 	    		</geometry>
 			</collision>
-	    	<visual>
-				<origin xyz="0 0 0" rpy="0 0 0"/>
-	    		<geometry>
-					<mesh filename="package://ginko_description/meshes/stl/link05_l_knee.stl"/>
-					<!-- <mesh filename="package://ginko_description/meshes/dae/link05_l_knee.dae"/> -->
-	    		</geometry>
+			<visual>
+				<origin xyz="0 0 0" rpy="0 0 0"/>
+				<geometry>
+					<mesh filename="package://ginko_description/meshes/obj/link05_l_knee.obj"/>
+				</geometry>
 			</visual>
 			<inertial>
@@ -142,9 +138,9 @@
 	    		</geometry>
 			</collision>
-	    	<visual>
-				<origin xyz="0 0 0" rpy="0 0 0"/>
-	    		<geometry>
-					<mesh filename="package://ginko_description/meshes/stl/link03_l_leg01.stl"/>
-	    		</geometry>
+			<visual>
+				<origin xyz="0 0 0" rpy="0 0 0"/>
+				<geometry>
+					<mesh filename="package://ginko_description/meshes/obj/link03_l_leg01.obj"/>
+				</geometry>
 			</visual>
 			<inertial>
@@ -172,9 +168,9 @@
 	    		</geometry>
 			</collision>
-	    	<visual>
-				<origin xyz="0 0 0" rpy="0 0 0"/>
-	    		<geometry>
-					<mesh filename="package://ginko_description/meshes/stl/link04_l_leg02.stl"/>
-	    		</geometry>
+			<visual>
+				<origin xyz="0 0 0" rpy="0 0 0"/>
+				<geometry>
+					<mesh filename="package://ginko_description/meshes/obj/link04_l_leg02.obj"/>
+				</geometry>
 			</visual>
 			<inertial>
@@ -197,15 +193,15 @@
 		<!-- toe -->
 		<link name="${name}_link6">
-	    	<collision>
-				<origin xyz="0 0 0" rpy="0 0 0"/>
-	    		<geometry>
-					<mesh filename="package://ginko_description/meshes/stl/link06_l_toe01.stl"/>
-	    		</geometry>
-			</collision>
-	    	<visual>
-				<origin xyz="0 0 0" rpy="0 0 0"/>
-	    		<geometry>
-					<mesh filename="package://ginko_description/meshes/stl/link06_l_toe01.stl"/>
-	    		</geometry>
+			<collision>
+				<origin xyz="0 0 0" rpy="0 0 0"/>
+				<geometry>
+					<mesh filename="package://ginko_description/meshes/stl/link06_r_toe01.stl"/>
+				</geometry>
+			</collision>
+			<visual>
+				<origin xyz="0 0 0" rpy="0 0 0"/>
+				<geometry>
+					<mesh filename="package://ginko_description/meshes/obj/link06_l_toe01.obj"/>
+				</geometry>
 			</visual>
 			<inertial>
@@ -232,9 +228,9 @@
 	    		</geometry>
 			</collision>
-	    	<visual>
-				<origin xyz="0 0 0" rpy="0 0 0"/>
-	    		<geometry>
-					<mesh filename="package://ginko_description/meshes/stl/link07_l_toe02.stl"/>
-	    		</geometry>
+			<visual>
+				<origin xyz="0 0 0" rpy="0 0 0"/>
+				<geometry>
+					<mesh filename="package://ginko_description/meshes/obj/link07_l_toe02.obj"/>
+				</geometry>
 			</visual>
 			<inertial>
@@ -255,15 +251,17 @@
 	  	</joint>
 		<link name="${name}_link8">
-	    	<collision>
-				<origin xyz="0 0 0" rpy="0 0 0"/>
-	    		<geometry>
-					<mesh filename="package://ginko_description/meshes/stl/link08_l_toe03.stl"/>
-	    		</geometry>
-			</collision>
-	    	<visual>
-				<origin xyz="0 0 0" rpy="0 0 0"/>
-	    		<geometry>
-					<mesh filename="package://ginko_description/meshes/stl/link08_l_toe03.stl"/>
-	    		</geometry>
+			<collision>
+				<origin xyz="0 0 -0.003" rpy="0 0 0"/>
+				<geometry>
+					<box>
+						<size>0.128 0.08 0.006</size>
+					</box>
+				</geometry>
+			</collision>
+			<visual>
+				<origin xyz="0 0 0" rpy="0 0 0"/>
+				<geometry>
+					<mesh filename="package://ginko_description/meshes/obj/link08_l_toe03.obj"/>
+				</geometry>
 			</visual>
 			<inertial>

File: ginko_description/urdf/modules/leg_r.urdf.xacro (robot description, xacro)
@@ -14,5 +14,5 @@
 				<origin xyz="0 0 0" rpy="0 0 0"/>
 				<geometry>
-					<mesh filename="package://ginko_description/meshes/stl/link02_r_femoral.stl"/>
+					<mesh filename="package://ginko_description/meshes/obj/link02_r_femoral.obj"/>
 				</geometry>
 			</visual>
@@ -41,9 +41,9 @@
 	    		</geometry>
 			</collision>
-	    	<visual>
-				<origin xyz="0 0 0" rpy="0 0 0"/>
-	    		<geometry>
-					<mesh filename="package://ginko_description/meshes/stl/link03_r_leg01.stl"/>
-	    		</geometry>
+			<visual>
+				<origin xyz="0 0 0" rpy="0 0 0"/>
+				<geometry>
+					<mesh filename="package://ginko_description/meshes/obj/link03_r_leg01.obj"/>
+				</geometry>
 			</visual>
 			<inertial>
@@ -71,9 +71,9 @@
 	    		</geometry>
 			</collision>
-	    	<visual>
-				<origin xyz="0 0 0" rpy="0 0 0"/>
-	    		<geometry>
-					<mesh filename="package://ginko_description/meshes/stl/link04_r_leg02.stl"/>
-	    		</geometry>
+			<visual>
+				<origin xyz="0 0 0" rpy="0 0 0"/>
+				<geometry>
+					<mesh filename="package://ginko_description/meshes/obj/link04_r_leg02.obj"/>
+				</geometry>
 			</visual>
 			<inertial>
@@ -102,9 +102,9 @@
 	    		</geometry>
 			</collision>
-	    	<visual>
-				<origin xyz="0 0 0" rpy="0 0 0"/>
-	    		<geometry>
-					<mesh filename="package://ginko_description/meshes/stl/link05_r_knee.stl"/>
-	    		</geometry>
+			<visual>
+				<origin xyz="0 0 0" rpy="0 0 0"/>
+				<geometry>
+					<mesh filename="package://ginko_description/meshes/obj/link05_r_knee.obj"/>
+				</geometry>
 			</visual>
 			<inertial>
@@ -133,9 +133,9 @@
 	    		</geometry>
 			</collision>
-	    	<visual>
-				<origin xyz="0 0 0" rpy="0 0 0"/>
-	    		<geometry>
-					<mesh filename="package://ginko_description/meshes/stl/link03_r_leg01.stl"/>
-	    		</geometry>
+			<visual>
+				<origin xyz="0 0 0" rpy="0 0 0"/>
+				<geometry>
+					<mesh filename="package://ginko_description/meshes/obj/link03_r_leg01.obj"/>
+				</geometry>
 			</visual>
 			<inertial>
@@ -163,9 +163,9 @@
 	    		</geometry>
 			</collision>
-	    	<visual>
-				<origin xyz="0 0 0" rpy="0 0 0"/>
-	    		<geometry>
-					<mesh filename="package://ginko_description/meshes/stl/link04_r_leg02.stl"/>
-	    		</geometry>
+			<visual>
+				<origin xyz="0 0 0" rpy="0 0 0"/>
+				<geometry>
+					<mesh filename="package://ginko_description/meshes/obj/link04_r_leg02.obj"/>
+				</geometry>
 			</visual>
 			<inertial>
@@ -188,15 +188,15 @@
 		<!-- toe -->
 		<link name="${name}_link6">
-	    	<collision>
-				<origin xyz="0 0 0" rpy="0 0 0"/>
-	    		<geometry>
+			<collision>
+				<origin xyz="0 0 0" rpy="0 0 0"/>
+				<geometry>
 					<mesh filename="package://ginko_description/meshes/stl/link06_r_toe01.stl"/>
-	    		</geometry>
-			</collision>
-	    	<visual>
-				<origin xyz="0 0 0" rpy="0 0 0"/>
-	    		<geometry>
-					<mesh filename="package://ginko_description/meshes/stl/link06_r_toe01.stl"/>
-	    		</geometry>
+				</geometry>
+			</collision>
+			<visual>
+				<origin xyz="0 0 0" rpy="0 0 0"/>
+				<geometry>
+					<mesh filename="package://ginko_description/meshes/obj/link06_r_toe01.obj"/>
+				</geometry>
 			</visual>
 			<inertial>
@@ -224,9 +224,9 @@
 	    		</geometry>
 			</collision>
-	    	<visual>
-				<origin xyz="0 0 0" rpy="0 0 0"/>
-	    		<geometry>
-					<mesh filename="package://ginko_description/meshes/stl/link07_r_toe02.stl"/>
-	    		</geometry>
+			<visual>
+				<origin xyz="0 0 0" rpy="0 0 0"/>
+				<geometry>
+					<mesh filename="package://ginko_description/meshes/obj/link07_r_toe02.obj"/>
+				</geometry>
 			</visual>
 			<inertial>
@@ -247,15 +247,17 @@
 	  	</joint>
 		<link name="${name}_link8">
-	    	<collision>
-				<origin xyz="0 0 0" rpy="0 0 0"/>
-	    		<geometry>
-					<mesh filename="package://ginko_description/meshes/stl/link08_r_toe03.stl"/>
-	    		</geometry>
-			</collision>
-	    	<visual>
-				<origin xyz="0 0 0" rpy="0 0 0"/>
-	    		<geometry>
-					<mesh filename="package://ginko_description/meshes/stl/link08_r_toe03.stl"/>
-	    		</geometry>
+			<collision>
+				<origin xyz="0 0 -0.003" rpy="0 0 0"/>
+				<geometry>
+					<box>
+						<size>0.128 0.08 0.006</size>
+					</box>
+				</geometry>
+			</collision>
+			<visual>
+				<origin xyz="0 0 0" rpy="0 0 0"/>
+				<geometry>
+					<mesh filename="package://ginko_description/meshes/obj/link08_r_toe03.obj"/>
+				</geometry>
 			</visual>
 			<inertial>
