Commit message: sed,trコマンドでの置換は煩雑だったためpythonで対応→右足だけはうまく行った

File: ginko_description/gazebo/xacro/modules/leg_r.xacro (robot description, xacro)
@@ -172,5 +172,7 @@
 						<mesh filename="package://ginko_description/meshes/stl/spring1.stl"/>
 					</geometry>
-					<color rgba="1.0 1.0 1.0 0.5"/>
+					<material name="spring">
+						<color rgba="0.5 0.5 0.5 1.0"/>
+					</material>
 				</visual>
 				<inertial>
@@ -183,5 +185,5 @@
 				</inertial>
 			</link>
-			<joint name="leg_r_spring0_joint1" type="prismatic">
+			<joint name="spring0_leg_r_joint" type="prismatic">
 				<parent link="leg_r_spring0_link0"/>
 				<child  link="leg_r_spring0_link1"/>
@@ -204,5 +206,7 @@
 						<mesh filename="package://ginko_description/meshes/stl/spring2.stl"/>
 		    		</geometry>
-		    		<color rgba="1.0 1.0 1.0 0.5"/>
+					<material name="spring">
+						<color rgba="0.5 0.5 0.5 1.0"/>
+					</material>
 				</visual>
 				<inertial>
@@ -349,5 +353,7 @@
 						<mesh filename="package://ginko_description/meshes/stl/spring1.stl"/>
 					</geometry>
-					<color rgba="1.0 1.0 1.0 0.5"/>
+					<material name="spring">
+						<color rgba="0.5 0.5 0.5 1.0"/>
+					</material>
 				</visual>
 				<inertial>
@@ -360,5 +366,5 @@
 				</inertial>
 			</link>
-			<joint name="leg_r_spring1_joint1" type="prismatic">
+			<joint name="spring1_leg_r_joint" type="prismatic">
 				<parent link="leg_r_spring1_link0"/>
 				<child  link="leg_r_spring1_link1"/>
@@ -366,4 +372,5 @@
 				<axis xyz="1 0 0"/>
 				<limit effort="1000.0" lower="-0.035" upper="0.055" velocity="10.0"/>
+				<dynamics damping="0.0" friction="0.0"/>
 			</joint>
 			<link name="leg_r_spring1_link1">
@@ -379,5 +386,7 @@
 						<mesh filename="package://ginko_description/meshes/stl/spring2.stl"/>
 					</geometry>
-					<color rgba="1.0 1.0 1.0 0.5"/>
+					<material name="spring">
+						<color rgba="0.5 0.5 0.5 1.0"/>
+					</material>
 				</visual>
 				<inertial>
