Commit message: アームのダブルサーボを再現

File: ginko_description/gazebo/xacro/modules/arm_l.xacro (robot description, xacro)
@@ -39,5 +39,5 @@
 			<origin xyz="0.035 0.0246 0" rpy="1.1781 0 0"/>
 			<axis xyz="1 0 0"/>
-			<limit effort="1000.0" lower="-0.85" upper="1.18" velocity="10.0"/>
+			<limit effort="1000.0" lower="-1.18" upper="1.5" velocity="10.0"/>
 			<dynamics damping="0.1" friction="0.1"/>
 		</joint>
@@ -62,4 +62,22 @@
 					ixy="0.00015366" iyy="0.00113572"
 					ixz="-0.00031848" iyz="-0.00037104" izz="0.00064743"/>
+			</inertial>
+		</link>
+		<joint name="arm_l_joint1_rev" type="revolute">
+			<parent link="arm_l_link0"/>
+			<child  link="dummy0_arm_l_link1"/>
+			<origin xyz="-0.0562 0.0246 0" rpy="1.1781 0 0"/>
+			<axis xyz="-1 0 0"/>
+			<limit effort="1000.0" lower="-1.5" upper="1.18" velocity="10.0"/>
+			<dynamics damping="0.0" friction="0.0"/>
+		</joint>
+		<link name="dummy0_arm_l_link1">
+			<inertial>
+				<mass value="0.00001"/>
+				<origin xyz="-0.0912 0 0" rpy="0 0 0"/>
+				<inertia
+					ixx="0.00000001"
+					ixy="0.00000000" iyy="0.00000001"
+					ixz="0.00000000" iyz="0.00000000" izz="0.00000001"/>
 			</inertial>
 		</link>

File: ginko_description/gazebo/xacro/modules/arm_r.xacro (robot description, xacro)
@@ -39,5 +39,5 @@
 			<origin xyz="0.035 -0.0246 0" rpy="-1.1781 0 0"/>
 			<axis xyz="1 0 0"/>
-			<limit effort="1000.0" lower="-0.85" upper="1.18" velocity="10.0"/>
+			<limit effort="1000.0" lower="-1.5" upper="1.18" velocity="10.0"/>
 			<dynamics damping="0.1" friction="0.1"/>
 		</joint>
@@ -62,4 +62,22 @@
 					ixy="-0.00015366" iyy="0.00113572"
 					ixz="-0.00031848" iyz="0.00037104" izz="0.00064743"/>
+			</inertial>
+		</link>
+		<joint name="arm_r_joint1_rev" type="revolute">
+			<parent link="arm_r_link0"/>
+			<child  link="dummy0_arm_r_link1"/>
+			<origin xyz="-0.0562 -0.0246 0" rpy="-1.1781 0 0"/>
+			<axis xyz="-1 0 0"/>
+			<limit effort="1000.0" lower="-1.18" upper="1.5" velocity="10.0"/>
+			<dynamics damping="0.0" friction="0.0"/>
+		</joint>
+		<link name="dummy0_arm_r_link1">
+			<inertial>
+				<mass value="0.00001"/>
+				<origin xyz="-0.0912 0 0" rpy="0 0 0"/>
+				<inertia
+					ixx="0.00000001"
+					ixy="0.00000000" iyy="0.00000001"
+					ixz="0.00000000" iyz="0.00000000" izz="0.00000001"/>
 			</inertial>
 		</link>

Commit message: バグ修正

File: ginko_description/gazebo/xacro/modules/arm_l.xacro (robot description, xacro)
@@ -4,5 +4,5 @@
 		<!-- shoulder pitch. -->
 		<joint name="arm_l_joint0" type="revolute">
-		    <parent link="body_link1"/>
+		    <parent link="body_link0"/>
 			<child link="arm_l_link0"/>
 		    <origin xyz="0 0.10683 0.05115" rpy="0 0.3927 0"/>

File: ginko_description/gazebo/xacro/modules/arm_r.xacro (robot description, xacro)
@@ -4,5 +4,5 @@
 		<!-- shoulder pitch. -->
 		<joint name="arm_r_joint0" type="revolute">
-		    <parent link="body_link1"/>
+		    <parent link="body_link0"/>
 			<child link="arm_r_link0"/>
 		    <origin xyz="0 -0.10683 0.05115" rpy="0 0.3927 0"/>

File: ginko_description/gazebo/xacro/modules/leg_l.xacro (robot description, xacro)
@@ -155,5 +155,5 @@
 	  	<!-- spring -->
 		<xacro:if value="${model_mode!='rviz'}">
-			<joint name="leg_l_spring_joint0" type="revolute">
+			<joint name="leg_l_spring0_joint0" type="revolute">
 		    	<parent link="leg_l_link0"/>
 		    	<child  link="leg_l_spring0_link0"/>
@@ -167,5 +167,5 @@
 					<origin xyz="0 0 0" rpy="0 0 0"/>
 		    		<geometry>
-						<!-- <mesh filename="package://ginko_description/meshes/stl/spring1.stl"/> -->
+						<mesh filename="package://ginko_description/meshes/stl/spring1.stl"/>
 		    		</geometry>
 				</collision>
@@ -200,5 +200,5 @@
 					<origin xyz="0 0 0" rpy="0 0 0"/>
 		    		<geometry>
-						<!-- <mesh filename="package://ginko_description/meshes/stl/spring2.stl"/> -->
+						<mesh filename="package://ginko_description/meshes/stl/spring2.stl"/>
 		    		</geometry>
 				</collision>
@@ -221,5 +221,5 @@
 				</inertial>
 			</link>
-			<joint name="close_leg_l_spring0_joint2" type="revolute">
+			<joint name="close_leg_l_spring0_joint1" type="revolute">
 				<parent link="leg_l_spring0_link1"/>
 				<child  link="dummy1_leg_l_link3"/>
@@ -340,10 +340,10 @@
 		<xacro:if value="${model_mode!='rviz'}">
 			<joint name="leg_l_spring1_joint0" type="revolute">
-				<parent link="leg_l_link3"/>
+				<parent link="leg_l_link4"/>
 				<child  link="leg_l_spring1_link0"/>
-				<origin xyz="0 0.058 -0.0386" rpy="0 2.574025114 0"/>
+				<origin xyz="0 0.058 0" rpy="0 0.217830624 0"/>
 				<axis xyz="0 -1 0"/>
-				<limit effort="0.0" lower="-3.141593" upper="3.141593" velocity="10.0"/>
-				<dynamics damping="0.0" friction="0.0"/>
+				<limit effort="1000.0" lower="-3.141593" upper="3.141593" velocity="10.0"/>
+				<dynamics damping="0.01" friction="0.01"/>
 			</joint>
 			<link name="leg_l_spring1_link0">
@@ -351,5 +351,5 @@
 					<origin xyz="0 0 0" rpy="0 0 0"/>
 					<geometry>
-						<!-- <mesh filename="package://ginko_description/meshes/stl/spring1.stl"/> -->
+						<mesh filename="package://ginko_description/meshes/stl/spring1.stl"/>
 					</geometry>
 				</collision>
@@ -378,5 +378,5 @@
 				<axis xyz="1 0 0"/>
 				<limit effort="1000.0" lower="-0.03" upper="0.06" velocity="10.0"/>
-				<dynamics damping="0.0" friction="0.0"/>
+				<dynamics damping="0.01" friction="0.01"/>
 			</joint>
 			<link name="leg_l_spring1_link1">
@@ -384,5 +384,5 @@
 					<origin xyz="0 0 0" rpy="0 0 0"/>
 					<geometry>
-						<!-- <mesh filename="package://ginko_description/meshes/stl/spring2.stl"/> -->
+						<mesh filename="package://ginko_description/meshes/stl/spring2.stl"/>
 					</geometry>
 				</collision>
@@ -405,11 +405,11 @@
 				</inertial>
 			</link>
-			<joint name="close_leg_l_spring1_joint2" type="revolute">
+			<joint name="close_leg_l_spring1_joint1" type="revolute">
 				<parent link="leg_l_spring1_link1"/>
 				<child  link="dummy3_leg_l_link6"/>
 				<origin xyz="0 0 0" rpy="0 0 0"/>
 				<axis xyz="0 -1 0"/>
-				<limit effort="0.0" lower="-3.141593" upper="3.141593" velocity="10.0"/>
-				<dynamics damping="0.0" friction="0.0"/>
+				<limit effort="1000.0" lower="-3.141593" upper="3.141593" velocity="10.0"/>
+				<dynamics damping="0.01" friction="0.01"/>
 			</joint>
 			<link name="dummy3_leg_l_link6">

File: ginko_description/gazebo/xacro/modules/leg_r.xacro (robot description, xacro)
@@ -167,5 +167,5 @@
 					<origin xyz="0 0 0" rpy="0 0 0"/>
 					<geometry>
-						<!-- <mesh filename="package://ginko_description/meshes/stl/spring1.stl"/> -->
+						<mesh filename="package://ginko_description/meshes/stl/spring1.stl"/>
 					</geometry>
 				</collision>
@@ -200,5 +200,5 @@
 					<origin xyz="0 0 0" rpy="0 0 0"/>
 		    		<geometry>
-						<!-- <mesh filename="package://ginko_description/meshes/stl/spring2.stl"/> -->
+						<mesh filename="package://ginko_description/meshes/stl/spring2.stl"/>
 		    		</geometry>
 				</collision>
@@ -221,5 +221,5 @@
 				</inertial>
 			</link>
-			<joint name="close_leg_r_spring0_joint2" type="revolute">
+			<joint name="close_leg_r_spring0_joint1" type="revolute">
 				<parent link="leg_r_spring0_link1"/>
 				<child  link="dummy1_leg_r_link3"/>
@@ -340,10 +340,10 @@
 		<xacro:if value="${model_mode!='rviz'}">
 			<joint name="leg_r_spring1_joint0" type="revolute">
-				<parent link="leg_r_link3"/>
+				<parent link="leg_r_link4"/>
 				<child  link="leg_r_spring1_link0"/>
-				<origin xyz="0 -0.058 -0.0386" rpy="0 2.574025114 0"/>
+				<origin xyz="0 -0.058 0" rpy="0 0.217830624 0"/>
 				<axis xyz="0 -1 0"/>
-				<limit effort="0.0" lower="-3.141593" upper="3.141593" velocity="10.0"/>
-				<dynamics damping="0.0" friction="0.0"/>
+				<limit effort="1000.0" lower="-3.141593" upper="3.141593" velocity="10.0"/>
+				<dynamics damping="0.01" friction="0.01"/>
 			</joint>
 			<link name="leg_r_spring1_link0">
@@ -351,5 +351,5 @@
 					<origin xyz="0 0 0" rpy="0 0 0"/>
 					<geometry>
-						<!-- <mesh filename="package://ginko_description/meshes/stl/spring1.stl"/> -->
+						<mesh filename="package://ginko_description/meshes/stl/spring1.stl"/>
 					</geometry>
 				</collision>
@@ -378,5 +378,5 @@
 				<axis xyz="1 0 0"/>
 				<limit effort="1000.0" lower="-0.03" upper="0.06" velocity="10.0"/>
-				<dynamics damping="0.0" friction="0.0"/>
+				<dynamics damping="0.01" friction="0.01"/>
 			</joint>
 			<link name="leg_r_spring1_link1">
@@ -384,5 +384,5 @@
 					<origin xyz="0 0 0" rpy="0 0 0"/>
 					<geometry>
-						<!-- <mesh filename="package://ginko_description/meshes/stl/spring2.stl"/> -->
+						<mesh filename="package://ginko_description/meshes/stl/spring2.stl"/>
 					</geometry>
 				</collision>
@@ -405,11 +405,11 @@
 				</inertial>
 			</link>
-			<joint name="close_leg_r_spring1_joint2" type="revolute">
+			<joint name="close_leg_r_spring1_joint1" type="revolute">
 				<parent link="leg_r_spring1_link1"/>
 				<child  link="dummy3_leg_r_link6"/>
 				<origin xyz="0 0 0" rpy="0 0 0"/>
 				<axis xyz="0 -1 0"/>
-				<limit effort="0.0" lower="-3.141593" upper="3.141593" velocity="10.0"/>
-				<dynamics damping="0.0" friction="0.0"/>
+				<limit effort="1000.0" lower="-3.141593" upper="3.141593" velocity="10.0"/>
+				<dynamics damping="0.01" friction="0.01"/>
 			</joint>
 			<link name="dummy3_leg_r_link6">

Commit message: 摩擦を修正・rviz上でのURGの表示を反映

File: ginko_description/gazebo/xacro/modules/arm_l.xacro (robot description, xacro)
@@ -145,12 +145,21 @@
 	  	<!-- LiDAR -->
 		<!-- use zero-limited revolute joint for fixed joint (SDF) -->
-		<joint name="arm_l_urg_joint" type="revolute">
-	    	<parent link="arm_l_link1"/>
-	    	<child  link="arm_l_urg_link"/>
-	    	<origin xyz="-0.0456 -0.01715 -0.06795" rpy="0 1.57 -1.57"/>
-	    	<axis xyz="0 0 1"/>
-	    	<limit effort="0.0" lower="0.0" upper="0.0" velocity="0.0"/>
-			<dynamics damping="0.1" friction="0.1"/>
-		</joint>
+		<xacro:if value="${model_mode!='rviz'}">
+			<joint name="arm_l_urg_joint" type="revolute">
+				<parent link="arm_l_link1"/>
+				<child  link="arm_l_urg_link"/>
+				<origin xyz="-0.0456 -0.01715 -0.06795" rpy="0 1.57 -1.57"/>
+				<axis xyz="0 0 1"/>
+				<limit effort="0.0" lower="0.0" upper="0.0" velocity="0.0"/>
+				<dynamics damping="0.1" friction="0.1"/>
+			</joint>
+		</xacro:if>
+		<xacro:if value="${model_mode=='rviz'}">
+			<joint name="arm_l_urg_joint" type="fixed">
+				<parent link="arm_l_link1"/>
+				<child  link="arm_l_urg_link"/>
+				<origin xyz="-0.0456 -0.01715 -0.06795" rpy="0 1.57 -1.57"/>
+			</joint>
+		</xacro:if>
 		<link name="arm_l_urg_link">
 	    	<collision>

File: ginko_description/gazebo/xacro/modules/arm_r.xacro (robot description, xacro)
@@ -145,12 +145,21 @@
 	  	<!-- LiDAR -->
 		<!-- use zero-limited revolute joint for fixed joint (SDF) -->
-		<joint name="arm_r_urg_joint"  type="revolute">
-	    	<parent link="arm_r_link1"/>
-	    	<child  link="arm_r_urg_link"/>
-	    	<origin xyz="-0.0456 0.01715 -0.06795" rpy="0 1.57 1.57"/>
-	    	<axis xyz="0 0 1"/>
-	    	<limit effort="0.0" lower="0.0" upper="0.0" velocity="0.0"/>
-			<dynamics damping="0.1" friction="0.1"/>
-		</joint>
+		<xacro:if value="${model_mode!='rviz'}">
+			<joint name="arm_r_urg_joint"  type="revolute">
+				<parent link="arm_r_link1"/>
+				<child  link="arm_r_urg_link"/>
+				<origin xyz="-0.0456 0.01715 -0.06795" rpy="0 1.57 1.57"/>
+				<axis xyz="0 0 1"/>
+				<limit effort="0.0" lower="0.0" upper="0.0" velocity="0.0"/>
+				<dynamics damping="0.1" friction="0.1"/>
+			</joint>
+		</xacro:if>
+		<xacro:if value="${model_mode=='rviz'}">
+			<joint name="arm_r_urg_joint" type="fixed">
+				<parent link="arm_r_link1"/>
+				<child  link="arm_r_urg_link"/>
+				<origin xyz="-0.0456 0.01715 -0.06795" rpy="0 1.57 1.57"/>
+			</joint>
+		</xacro:if>
 		<link name="arm_r_urg_link">
 	    	<collision>

File: ginko_description/gazebo/xacro/modules/leg_l.xacro (robot description, xacro)
@@ -180,10 +180,10 @@
 				</visual>
 				<inertial>
-					<mass value="0.00143865"/>
+					<mass value="0.0143865"/>
 					<origin xyz="0.03091683 0.0 0.0" rpy="0 0 0"/>
 					<inertia
-						ixx="0.00000001"
-						ixy="0.00000000" iyy="0.00000060"
-						ixz="0.00000000" iyz="0.00000000" izz="0.00000060"/>
+						ixx="0.0000001"
+						ixy="0.00000000" iyy="0.0000060"
+						ixz="0.00000000" iyz="0.00000000" izz="0.0000060"/>
 				</inertial>
 			</link>
@@ -213,10 +213,10 @@
 				</visual>
 				<inertial>
-					<mass value="0.00143865"/>
+					<mass value="0.0143865"/>
 					<origin xyz="0.03091683 0.0 0.0" rpy="0 0 0"/>
 					<inertia
-						ixx="0.00000001"
-						ixy="0.00000000" iyy="0.00000060"
-						ixz="0.00000000" iyz="0.00000000" izz="0.00000060"/>
+						ixx="0.0000001"
+						ixy="0.00000000" iyy="0.0000060"
+						ixz="0.00000000" iyz="0.00000000" izz="0.0000060"/>
 				</inertial>
 			</link>
@@ -364,10 +364,10 @@
 				</visual>
 				<inertial>
-					<mass value="0.00143865"/>
+					<mass value="0.0143865"/>
 					<origin xyz="0.03091683 0.0 0.0" rpy="0 0 0"/>
 					<inertia
-						ixx="0.00000001"
-						ixy="0.00000000" iyy="0.00000060"
-						ixz="0.00000000" iyz="0.00000000" izz="0.00000060"/>
+						ixx="0.0000001"
+						ixy="0.00000000" iyy="0.0000060"
+						ixz="0.00000000" iyz="0.00000000" izz="0.0000060"/>
 				</inertial>
 			</link>
@@ -400,7 +400,7 @@
 					<origin xyz="0.03091683 0.0 0.0" rpy="0 0 0"/>
 					<inertia
-						ixx="0.00000001"
-						ixy="0.00000000" iyy="0.00000060"
-						ixz="0.00000000" iyz="0.00000000" izz="0.00000060"/>
+						ixx="0.0000001"
+						ixy="0.00000000" iyy="0.0000060"
+						ixz="0.00000000" iyz="0.00000000" izz="0.0000060"/>
 				</inertial>
 			</link>
@@ -507,4 +507,37 @@
 			</inertial>
 		</link>
+		<!-- toe edges -->
+		<xacro:if value="${model_mode=='rviz'}">
+			<joint name="leg_l_toe_joint0" type="fixed">
+				<parent link="leg_l_link8"/>
+				<child  link="leg_l_toe_link0"/>
+				<origin xyz="0.064 0.040 -0.005" rpy="0 0 0"/>
+			</joint>
+			<link name="leg_l_toe_link0"/>
+			<joint name="leg_l_toe_joint1" type="fixed">
+				<parent link="leg_l_link8"/>
+				<child  link="leg_l_toe_link1"/>
+				<origin xyz="-0.064 0.040 -0.005" rpy="0 0 0"/>
+			</joint>
+			<link name="leg_l_toe_link1"/>
+			<joint name="leg_l_toe_joint2" type="fixed">
+				<parent link="leg_l_link8"/>
+				<child  link="leg_l_toe_link2"/>
+				<origin xyz="-0.064 -0.040 -0.005" rpy="0 0 0"/>
+			</joint>
+			<link name="leg_l_toe_link2"/>
+			<joint name="leg_l_toe_joint3" type="fixed">
+				<parent link="leg_l_link8"/>
+				<child  link="leg_l_toe_link3"/>
+				<origin xyz="0.064 -0.040 -0.005" rpy="0 0 0"/>
+			</joint>
+			<link name="leg_l_toe_link3"/>
+			<joint name="leg_l_toe_center_joint" type="fixed">
+				<parent link="leg_l_link8"/>
+				<child  link="leg_l_toe_center"/>
+				<origin xyz="0.0 0.0 -0.005" rpy="0 0 0"/>
+			</joint>
+			<link name="leg_l_toe_center"/>
+		</xacro:if>
 	</xacro:macro>
 </robot>

File: ginko_description/gazebo/xacro/modules/leg_r.xacro (robot description, xacro)
@@ -73,5 +73,5 @@
 			<xacro:if value="${model_mode=='rviz'}">
 				<mimic joint="leg_r_joint1" multiplier="1" offset="0"/>
-    		</xacro:if>
+			</xacro:if>
 		</joint>
 		<!-- parallel link (upper-2nd) -->
@@ -180,10 +180,10 @@
 				</visual>
 				<inertial>
-					<mass value="0.00143865"/>
+					<mass value="0.0143865"/>
 					<origin xyz="0.03091683 0.0 0.0" rpy="0 0 0"/>
 					<inertia
-						ixx="0.00000001"
-						ixy="0.00000000" iyy="0.00000060"
-						ixz="0.00000000" iyz="0.00000000" izz="0.00000060"/>
+						ixx="0.0000001"
+						ixy="0.00000000" iyy="0.0000060"
+						ixz="0.00000000" iyz="0.00000000" izz="0.0000060"/>
 				</inertial>
 			</link>
@@ -213,10 +213,10 @@
 				</visual>
 				<inertial>
-					<mass value="0.00143865"/>
+					<mass value="0.0143865"/>
 					<origin xyz="0.03091683 0.0 0.0" rpy="0 0 0"/>
 					<inertia
-						ixx="0.00000001"
-						ixy="0.00000000" iyy="0.00000060"
-						ixz="0.00000000" iyz="0.00000000" izz="0.00000060"/>
+						ixx="0.0000001"
+						ixy="0.00000000" iyy="0.0000060"
+						ixz="0.00000000" iyz="0.00000000" izz="0.0000060"/>
 				</inertial>
 			</link>
@@ -364,10 +364,10 @@
 				</visual>
 				<inertial>
-					<mass value="0.00143865"/>
+					<mass value="0.0143865"/>
 					<origin xyz="0.03091683 0.0 0.0" rpy="0 0 0"/>
 					<inertia
-						ixx="0.00000001"
-						ixy="0.00000000" iyy="0.00000060"
-						ixz="0.00000000" iyz="0.00000000" izz="0.00000060"/>
+						ixx="0.0000001"
+						ixy="0.00000000" iyy="0.0000060"
+						ixz="0.00000000" iyz="0.00000000" izz="0.0000060"/>
 				</inertial>
 			</link>
@@ -397,10 +397,10 @@
 				</visual>
 				<inertial>
-					<mass value="0.00143865"/>
+					<mass value="0.0143865"/>
 					<origin xyz="0.03091683 0.0 0.0" rpy="0 0 0"/>
 					<inertia
-						ixx="0.00000001"
-						ixy="0.00000000" iyy="0.00000060"
-						ixz="0.00000000" iyz="0.00000000" izz="0.00000060"/>
+						ixx="0.0000001"
+						ixy="0.00000000" iyy="0.0000060"
+						ixz="0.00000000" iyz="0.00000000" izz="0.0000060"/>
 				</inertial>
 			</link>
@@ -507,4 +507,37 @@
 			</inertial>
 		</link>
+		<!-- toe edges -->
+		<xacro:if value="${model_mode=='rviz'}">
+			<joint name="leg_r_toe_joint0" type="fixed">
+				<parent link="leg_r_link8"/>
+				<child  link="leg_r_toe_link0"/>
+				<origin xyz="0.064 0.040 -0.005" rpy="0 0 0"/>
+			</joint>
+			<link name="leg_r_toe_link0"/>
+			<joint name="leg_r_toe_joint1" type="fixed">
+				<parent link="leg_r_link8"/>
+				<child  link="leg_r_toe_link1"/>
+				<origin xyz="-0.064 0.040 -0.005" rpy="0 0 0"/>
+			</joint>
+			<link name="leg_r_toe_link1"/>
+			<joint name="leg_r_toe_joint2" type="fixed">
+				<parent link="leg_r_link8"/>
+				<child  link="leg_r_toe_link2"/>
+				<origin xyz="-0.064 -0.040 -0.005" rpy="0 0 0"/>
+			</joint>
+			<link name="leg_r_toe_link2"/>
+			<joint name="leg_r_toe_joint3" type="fixed">
+				<parent link="leg_r_link8"/>
+				<child  link="leg_r_toe_link3"/>
+				<origin xyz="0.064 -0.040 -0.005" rpy="0 0 0"/>
+			</joint>
+			<link name="leg_r_toe_link3"/>
+			<joint name="leg_r_toe_center_joint" type="fixed">
+				<parent link="leg_r_link8"/>
+				<child  link="leg_r_toe_center"/>
+				<origin xyz="0.0 0.0 -0.005" rpy="0 0 0"/>
+			</joint>
+			<link name="leg_r_toe_center"/>
+		</xacro:if>
 	</xacro:macro>
 </robot>

Commit message: gazeboのモーション再生プログラムを修正

File: ginko_description/gazebo/xacro/modules/arm_l.xacro (robot description, xacro)
@@ -39,5 +39,5 @@
 			<origin xyz="0.035 0.0246 0" rpy="1.1781 0 0"/>
 			<axis xyz="1 0 0"/>
-			<limit effort="1000.0" lower="-1.18" upper="1.5" velocity="10.0"/>
+			<limit effort="1000.0" lower="-1.18" upper="1.6" velocity="10.0"/>
 			<dynamics damping="0.1" friction="0.1"/>
 		</joint>
@@ -69,5 +69,5 @@
 			<origin xyz="-0.0562 0.0246 0" rpy="1.1781 0 0"/>
 			<axis xyz="-1 0 0"/>
-			<limit effort="1000.0" lower="-1.5" upper="1.18" velocity="10.0"/>
+			<limit effort="1000.0" lower="-1.6" upper="1.18" velocity="10.0"/>
 			<dynamics damping="0.0" friction="0.0"/>
 		</joint>

File: ginko_description/gazebo/xacro/modules/arm_r.xacro (robot description, xacro)
@@ -39,5 +39,5 @@
 			<origin xyz="0.035 -0.0246 0" rpy="-1.1781 0 0"/>
 			<axis xyz="1 0 0"/>
-			<limit effort="1000.0" lower="-1.5" upper="1.18" velocity="10.0"/>
+			<limit effort="1000.0" lower="-1.6" upper="1.18" velocity="10.0"/>
 			<dynamics damping="0.1" friction="0.1"/>
 		</joint>
@@ -69,5 +69,5 @@
 			<origin xyz="-0.0562 -0.0246 0" rpy="-1.1781 0 0"/>
 			<axis xyz="-1 0 0"/>
-			<limit effort="1000.0" lower="-1.18" upper="1.5" velocity="10.0"/>
+			<limit effort="1000.0" lower="-1.18" upper="1.6" velocity="10.0"/>
 			<dynamics damping="0.0" friction="0.0"/>
 		</joint>
