Commit message: バネ部分inertialの誤入力を修正

File: ginko_description/gazebo/xacro/modules/leg_l.xacro (robot description, xacro)
@@ -339,11 +339,11 @@
 	  	<!-- spring -->
 		<xacro:if value="${model_mode!='rviz'}">
-			<joint name="leg_l_spring1_joint0" type="revolute">
+			<joint name="leg_l_spring1_joint0" type="continuous">
 				<parent link="leg_l_link4"/>
 				<child  link="leg_l_spring1_link0"/>
 				<origin xyz="0 0.058 0" rpy="0 0.217830624 0"/>
 				<axis xyz="0 -1 0"/>
-				<limit effort="1000.0" lower="-3.141593" upper="3.141593" velocity="10.0"/>
-				<dynamics damping="0.01" friction="0.01"/>
+				<limit effort="0.0" lower="-3.141593" upper="3.141593" velocity="10.0"/>
+				<dynamics damping="0.01" friction="0.0"/>
 			</joint>
 			<link name="leg_l_spring1_link0">
@@ -365,5 +365,5 @@
 				<inertial>
 					<mass value="0.00143865"/>
-					<origin xyz="0.03091683 0.0 0.0" rpy="0 2.138363867 0"/>
+					<origin xyz="0.03091683 0.0 0.0" rpy="0 0 0"/>
 					<inertia
 						ixx="0.00000001"
@@ -378,5 +378,5 @@
 				<axis xyz="1 0 0"/>
 				<limit effort="1000.0" lower="-0.03" upper="0.06" velocity="10.0"/>
-				<dynamics damping="0.01" friction="0.01"/>
+				<dynamics damping="0.01" friction="0.0"/>
 			</joint>
 			<link name="leg_l_spring1_link1">
@@ -405,11 +405,11 @@
 				</inertial>
 			</link>
-			<joint name="close_leg_l_spring1_joint1" type="revolute">
+			<joint name="close_leg_l_spring1_joint1" type="continuous">
 				<parent link="leg_l_spring1_link1"/>
 				<child  link="dummy3_leg_l_link6"/>
-				<origin xyz="0 0 0" rpy="0 0 0"/>
+				<origin xyz="0 0 0" rpy="0 -2.574025114 0"/>
 				<axis xyz="0 -1 0"/>
-				<limit effort="1000.0" lower="-3.141593" upper="3.141593" velocity="10.0"/>
-				<dynamics damping="0.01" friction="0.01"/>
+				<limit effort="0.0" lower="-3.141593" upper="3.141593" velocity="10.0"/>
+				<dynamics damping="0.01" friction="0.0"/>
 			</joint>
 			<link name="dummy3_leg_l_link6">

File: ginko_description/gazebo/xacro/modules/leg_r.xacro (robot description, xacro)
@@ -339,11 +339,11 @@
 		<!-- spring -->
 		<xacro:if value="${model_mode!='rviz'}">
-			<joint name="leg_r_spring1_joint0" type="revolute">
+			<joint name="leg_r_spring1_joint0" type="continuous">
 				<parent link="leg_r_link4"/>
 				<child  link="leg_r_spring1_link0"/>
 				<origin xyz="0 -0.058 0" rpy="0 0.217830624 0"/>
 				<axis xyz="0 -1 0"/>
-				<limit effort="1000.0" lower="-3.141593" upper="3.141593" velocity="10.0"/>
-				<dynamics damping="0.01" friction="0.01"/>
+				<limit effort="0.0" lower="-3.141593" upper="3.141593" velocity="10.0"/>
+				<dynamics damping="0.01" friction="0.0"/>
 			</joint>
 			<link name="leg_r_spring1_link0">
@@ -365,5 +365,5 @@
 				<inertial>
 					<mass value="0.00143865"/>
-					<origin xyz="0.03091683 0.0 0.0" rpy="0 2.138363867 0"/>
+					<origin xyz="0.03091683 0.0 0.0" rpy="0 0 0"/>
 					<inertia
 						ixx="0.00000001"
@@ -378,5 +378,5 @@
 				<axis xyz="1 0 0"/>
 				<limit effort="1000.0" lower="-0.03" upper="0.06" velocity="10.0"/>
-				<dynamics damping="0.01" friction="0.01"/>
+				<dynamics damping="0.01" friction="0.0"/>
 			</joint>
 			<link name="leg_r_spring1_link1">
@@ -405,11 +405,11 @@
 				</inertial>
 			</link>
-			<joint name="close_leg_r_spring1_joint1" type="revolute">
+			<joint name="close_leg_r_spring1_joint1" type="continuous">
 				<parent link="leg_r_spring1_link1"/>
 				<child  link="dummy3_leg_r_link6"/>
-				<origin xyz="0 0 0" rpy="0 0 0"/>
+				<origin xyz="0 0 0" rpy="0 -2.574025114 0"/>
 				<axis xyz="0 -1 0"/>
-				<limit effort="1000.0" lower="-3.141593" upper="3.141593" velocity="10.0"/>
-				<dynamics damping="0.01" friction="0.01"/>
+				<limit effort="0.0" lower="-3.141593" upper="3.141593" velocity="10.0"/>
+				<dynamics damping="0.01" friction="0.0"/>
 			</joint>
 			<link name="dummy3_leg_r_link6">

Commit message: 脚部品のinertial誤入力を修正

File: ginko_description/gazebo/xacro/modules/leg_l.xacro (robot description, xacro)
@@ -56,10 +56,10 @@
 			</visual>
 			<inertial>
-				<mass value="0.18525692"/>
-				<origin xyz="0.05000000 0.03285059 0.00068146" rpy="0 0 0"/>
-				<inertia
-					ixx="0.00041331"
-					ixy="-0.00003605" iyy="0.00027917"
-					ixz="-0.00000000" iyz="-0.00000184" izz="0.00066510"/>
+				<mass value="0.15115113"/>
+				<origin xyz="0.05000000 0.02587267 0.00000000" rpy="0 0 0"/>
+				<inertia
+					ixx="0.00003721"
+					ixy="0.00000000" iyy="0.00026035"
+					ixz="0.00000000" iyz="0.00000000" izz="0.00028077"/>
 			</inertial>
 		</link>
@@ -263,10 +263,10 @@
 			</visual>
 			<inertial>
-				<mass value="0.18525692"/>
-				<origin xyz="0.05000000 0.03285059 0.00068146" rpy="0 0 0"/>
-				<inertia
-					ixx="0.00041331"
-					ixy="-0.00003605" iyy="0.00027917"
-					ixz="-0.00000000" iyz="-0.00000184" izz="0.00066510"/>
+				<mass value="0.15115113"/>
+				<origin xyz="0.05000000 0.02587267 0.00000000" rpy="0 0 0"/>
+				<inertia
+					ixx="0.00003721"
+					ixy="0.00000000" iyy="0.00026035"
+					ixz="0.00000000" iyz="0.00000000" izz="0.00028077"/>
 			</inertial>
 		</link>

File: ginko_description/gazebo/xacro/modules/leg_r.xacro (robot description, xacro)
@@ -56,10 +56,10 @@
 			</visual>
 			<inertial>
-				<mass value="0.18525690"/>
-				<origin xyz="0.05000000 -0.01719078 0.00068146" rpy="0 0 0"/>
-				<inertia
-					ixx="0.00055489"
-					ixy="-0.00004242" iyy="0.00027917"
-					ixz="0.00000000" iyz="-0.00000175" izz="0.00081028"/>
+				<mass value="0.15115113"/>
+				<origin xyz="0.05000000 -0.02587267 0.00000000" rpy="0 0 0"/>
+				<inertia
+					ixx="0.00003721"
+					ixy="0.00000000" iyy="0.00026035"
+					ixz="0.00000000" iyz="0.00000000" izz="0.00028077"/>
 			</inertial>
 		</link>
@@ -263,10 +263,10 @@
 			</visual>
 			<inertial>
-				<mass value="0.18525690"/>
-				<origin xyz="0.05000000 -0.01719078 0.00068146" rpy="0 0 0"/>
-				<inertia
-					ixx="0.00055489"
-					ixy="-0.00004242" iyy="0.00027917"
-					ixz="0.00000000" iyz="-0.00000175" izz="0.00081028"/>
+				<mass value="0.15115113"/>
+				<origin xyz="0.05000000 -0.02587267 0.00000000" rpy="0 0 0"/>
+				<inertia
+					ixx="0.00003721"
+					ixy="0.00000000" iyy="0.00026035"
+					ixz="0.00000000" iyz="0.00000000" izz="0.00028077"/>
 			</inertial>
 		</link>

Commit message: 実機の挙動に寄せるため物理パラメータを修正

File: ginko_description/gazebo/xacro/modules/leg_l.xacro (robot description, xacro)
@@ -397,5 +397,5 @@
 				</visual>
 				<inertial>
-					<mass value="0.00143865"/>
+					<mass value="0.0143865"/>
 					<origin xyz="0.03091683 0.0 0.0" rpy="0 0 0"/>
 					<inertia

Commit message: 実機に寄せるためパラメータ調整中

File: ginko_description/gazebo/xacro/modules/leg_l.xacro (robot description, xacro)
@@ -9,5 +9,5 @@
 		    <axis xyz="-1 0 0"/>
 			<limit effort="1000.0" lower="-0.8" upper="1.0" velocity="10.0"/>
-			<dynamics damping="0.1" friction="0.1"/>
+			<dynamics damping="0.0" friction="0.3"/>
 		</joint>
 		<link name="leg_l_link0">
@@ -40,5 +40,5 @@
 			<axis xyz="0 -1 0"/>
 			<limit effort="1000.0" lower="-1.3" upper="0.7854" velocity="10.0"/>
-			<dynamics damping="0.1" friction="0.1"/>
+			<dynamics damping="0.0" friction="0.3"/>
 		</joint>
 		<link name="leg_l_link1">
@@ -70,5 +70,5 @@
 	    	<axis xyz="0 1 0"/>
 			<limit effort="1000.0" lower="-1.3" upper="0.7854" velocity="10.0"/>
-			<dynamics damping="0.1" friction="0.1"/>
+			<dynamics damping="0.0" friction="0.3"/>
 			<xacro:if value="${model_mode=='rviz'}">
 				<mimic joint="leg_l_joint1" multiplier="1" offset="0"/>
@@ -82,5 +82,5 @@
 			<axis xyz="0 -1 0"/>
 			<limit effort="1000.0" lower="-1.3" upper="0.7854" velocity="10.0"/>
-			<dynamics damping="0.1" friction="0.1"/>
+			<dynamics damping="0.0" friction="0.3"/>
 			<xacro:if value="${model_mode=='rviz'}">
 				<mimic joint="leg_l_joint1" multiplier="1" offset="0"/>
@@ -247,5 +247,5 @@
 			<axis xyz="0 -1 0"/>
 			<limit effort="1000.0" lower="-0.7854" upper="1.3" velocity="10.0"/>
-			<dynamics damping="0.1" friction="0.1"/>
+			<dynamics damping="0.0" friction="0.3"/>
 		</joint>
 		<link name="leg_l_link4">
@@ -277,5 +277,5 @@
 	    	<axis xyz="0 1 0"/>
 			<limit effort="1000.0" lower="-0.7854" upper="1.3" velocity="10.0"/>
-			<dynamics damping="0.1" friction="0.1"/>
+			<dynamics damping="0.0" friction="0.3"/>
 			<xacro:if value="${model_mode=='rviz'}">
 	    		<mimic joint="leg_l_joint4" multiplier="1" offset="0"/>
@@ -453,5 +453,5 @@
 	    	<axis xyz="-1 0 0"/>
 	    	<limit effort="1000.0" lower="-1.6" upper="1.6" velocity="10.0"/>
-			<dynamics damping="0.1" friction="0.1"/>
+			<dynamics damping="0.0" friction="0.3"/>
 		</joint>
 		<link name="leg_l_link7">
@@ -483,5 +483,5 @@
 			<axis xyz="0 0 1"/>
 			<limit effort="1000.0" lower="-2.6" upper="2.6" velocity="10.0"/>
-			<dynamics damping="0.1" friction="0.1"/>
+			<dynamics damping="0.0" friction="0.3"/>
 		</joint>
 		<link name="leg_l_link8">

File: ginko_description/gazebo/xacro/modules/leg_r.xacro (robot description, xacro)
@@ -9,5 +9,5 @@
 		    <axis xyz="1 0 0"/>
 			<limit effort="1000.0" lower="-1.0" upper="0.8" velocity="10.0"/>
-			<dynamics damping="0.1" friction="0.1"/>
+			<dynamics damping="0.0" friction="0.3"/>
 		</joint>
 		<link name="leg_r_link0">
@@ -40,5 +40,5 @@
 			<axis xyz="0 1 0"/>
 			<limit effort="1000.0" lower="-0.7854" upper="1.3" velocity="10.0"/>
-			<dynamics damping="0.1" friction="0.1"/>
+			<dynamics damping="0.0" friction="0.3"/>
 		</joint>
 		<link name="leg_r_link1">
@@ -70,5 +70,5 @@
 			<axis xyz="0 -1 0"/>
 			<limit effort="1000.0" lower="-0.7854" upper="1.3" velocity="10.0"/>
-			<dynamics damping="0.1" friction="0.1"/>
+			<dynamics damping="0.0" friction="0.3"/>
 			<xacro:if value="${model_mode=='rviz'}">
 				<mimic joint="leg_r_joint1" multiplier="1" offset="0"/>
@@ -247,5 +247,5 @@
 			<axis xyz="0 1 0"/>
 			<limit effort="1000.0" lower="-1.3" upper="0.7854" velocity="10.0"/>
-			<dynamics damping="0.1" friction="0.1"/>
+			<dynamics damping="0.0" friction="0.3"/>
 		</joint>
 		<link name="leg_r_link4">
@@ -277,5 +277,5 @@
 			<axis xyz="0 -1 0"/>
 			<limit effort="1000.0" lower="-1.3" upper="0.7854" velocity="10.0"/>
-			<dynamics damping="0.1" friction="0.1"/>
+			<dynamics damping="0.0" friction="0.3"/>
 			<xacro:if value="${model_mode=='rviz'}">
 				<mimic joint="leg_r_joint4" multiplier="1" offset="0"/>
@@ -453,5 +453,5 @@
 			<axis xyz="-1 0 0"/>
 			<limit effort="1000.0" lower="-1.6" upper="1.6" velocity="10.0"/>
-			<dynamics damping="0.1" friction="0.1"/>
+			<dynamics damping="0.0" friction="0.3"/>
 		</joint>
 		<link name="leg_r_link7">
@@ -483,5 +483,5 @@
 			<axis xyz="0 0 1"/>
 			<limit effort="1000.0" lower="-2.6" upper="2.6" velocity="10.0"/>
-			<dynamics damping="0.1" friction="0.1"/>
+			<dynamics damping="0.0" friction="0.3"/>
 		</joint>
 		<link name="leg_r_link8">
