Commit message: xacroファイル作り直し

File: ginko_description/gazebo/xacro/ginko.xacro (robot description, xacro)
@@ -1,51 +1,21 @@
 <?xml version="1.0"?>
-<robot name="ginko" xmlns:xacro="http://www.ros.org/wiki/xacro">
+<robot name="ginko_xacro" xmlns:xacro="http://www.ros.org/wiki/xacro">
   <xacro:arg name="model_mode" default="rviz"/>
-  <xacro:include filename="$(find ginko_description)/gazebo/xacro/modules/body.urdf.xacro"/>
+  <xacro:include filename="$(find ginko_description)/gazebo/xacro/modules/body.xacro"/>
   <xacro:include filename="$(find ginko_description)/gazebo/transmission/body.gazebo"/>
-  <xacro:include filename="$(find ginko_description)/gazebo/xacro/modules/arm_l.urdf.xacro"/>
+  <xacro:include filename="$(find ginko_description)/gazebo/xacro/modules/arm_l.xacro"/>
   <xacro:include filename="$(find ginko_description)/gazebo/transmission/arm_l.gazebo"/>
-  <xacro:include filename="$(find ginko_description)/gazebo/xacro/modules/arm_r.urdf.xacro"/>
+  <xacro:include filename="$(find ginko_description)/gazebo/xacro/modules/arm_r.xacro"/>
   <xacro:include filename="$(find ginko_description)/gazebo/transmission/arm_r.gazebo"/>
-  <xacro:include filename="$(find ginko_description)/gazebo/xacro/modules/leg_l_spring.urdf.xacro"/>
-  <xacro:include filename="$(find ginko_description)/gazebo/transmission/leg_l_spring.gazebo"/>
-  <xacro:include filename="$(find ginko_description)/gazebo/xacro/modules/leg_r_spring.urdf.xacro"/>
-  <xacro:include filename="$(find ginko_description)/gazebo/transmission/leg_r_spring.gazebo"/>
-  <xacro:macro name="if_macro" params="rviz_or_gazebo">
-    <xacro:if value="${rviz_or_gazebo=='rviz'}">
-      <xacro:body_sim name="body"/>
+  <xacro:include filename="$(find ginko_description)/gazebo/xacro/modules/leg_l.xacro"/>
+  <xacro:include filename="$(find ginko_description)/gazebo/transmission/leg_l.gazebo"/>
+  <xacro:include filename="$(find ginko_description)/gazebo/xacro/modules/leg_r.xacro"/>
+  <xacro:include filename="$(find ginko_description)/gazebo/transmission/leg_r.gazebo"/>
+  <xacro:macro name="ginko_xacro" params="model_mode">
+    <xacro:if value="${model_mode=='rviz'}">
+      <xacro:body_xacro name="body" model_mode="rviz" />
       <xacro:body_gazebo name="body"/>
-      <xacro:leg_l_sim name="leg_l" parent="body_link1"/>
-      <xacro:leg_l_gazebo name="leg_l"/>
-      <xacro:leg_r_sim name="leg_r" parent="body_link1"/>
-      <xacro:leg_r_gazebo name="leg_r"/>
-    </xacro:if>
-    <xacro:if value="${rviz_or_gazebo=='gazebo'}">
-      <xacro:body_sim name="body"/>
-      <xacro:body_gazebo name="body"/>
-      <xacro:arm_l_sim name="arm_l" parent="body_link0"/>
-      <xacro:arm_l_gazebo name="arm_l"/>
-    </xacro:if>
-    <xacro:if value="${rviz_or_gazebo=='left_arm'}">
-      <xacro:body_sim name="body"/>
-      <xacro:body_gazebo name="body"/>
-      <xacro:leg_l_sim name="leg_l" parent="body_link1"/>
-      <xacro:leg_l_gazebo name="leg_l"/>
-      <xacro:leg_r_sim name="leg_r" parent="body_link1"/>
-      <xacro:leg_r_gazebo name="leg_r"/>
-      <xacro:arm_l_sim name="arm_l" parent="body_link0"/>
-      <xacro:arm_l_gazebo name="arm_l"/>
-    </xacro:if>
-    <xacro:if value="${rviz_or_gazebo=='right_arm'}">
-      <xacro:body_sim name="body"/>
-      <xacro:body_gazebo name="body"/>
-      <xacro:leg_l_sim name="leg_l" parent="body_link1"/>
-      <xacro:leg_l_gazebo name="leg_l"/>
-      <xacro:leg_r_sim name="leg_r" parent="body_link1"/>
-      <xacro:leg_r_gazebo name="leg_r"/>
-      <xacro:arm_r_sim name="arm_r" parent="body_link0"/>
-      <xacro:arm_r_gazebo name="arm_r"/>
     </xacro:if>
   </xacro:macro>
-  <xacro:if_macro rviz_or_gazebo="$(arg mode)"/>
+  <xacro:ginko_xacro model_mode="$(arg model_mode)"/>
 </robot>

File: ginko_description/gazebo/xacro/modules/body.xacro (robot description, xacro)
@@ -1,5 +1,5 @@
 <?xml version="1.0"?>
 <robot xmlns:xacro="http://www.ros.org/wiki/xacro">
-	<xacro:macro name="body_sim" params="name">
+	<xacro:macro name="body_xacro" params="name model_mode">
 		<!-- chest -->
 		<link name="${name}_link0">

Commit message: sedコマンドで閉ループ部分を置換できないか検証

File: ginko_description/gazebo/xacro/ginko.xacro (robot description, xacro)
@@ -2,4 +2,5 @@
 <robot name="ginko_xacro" xmlns:xacro="http://www.ros.org/wiki/xacro">
   <xacro:arg name="model_mode" default="rviz"/>
+  <xacro:arg name="gazebo_control_mode" default="ginko"/>
   <xacro:include filename="$(find ginko_description)/gazebo/xacro/modules/body.xacro"/>
   <xacro:include filename="$(find ginko_description)/gazebo/transmission/body.gazebo"/>
@@ -12,10 +13,50 @@
   <xacro:include filename="$(find ginko_description)/gazebo/xacro/modules/leg_r.xacro"/>
   <xacro:include filename="$(find ginko_description)/gazebo/transmission/leg_r.gazebo"/>
-  <xacro:macro name="ginko_xacro" params="model_mode">
-    <xacro:if value="${model_mode=='rviz'}">
-      <xacro:body_xacro name="body" model_mode="rviz" />
-      <xacro:body_gazebo name="body"/>
+  <!-- MACRO:Loading Gazebo Controllers for joints -->
+  <xacro:macro name="gazebo_plugin_xacro" params="gazebo_control_mode">
+    <xacro:if value="${gazebo_control_mode=='ginko'}">
+      <gazebo>
+        <plugin name="gazebo_ros_control" filename="libgazebo_ros_control.so">
+          <robotNamespace>/ginko</robotNamespace>
+          <robotSimType>gazebo_ros_control/GinkoRobotHWSim</robotSimType>
+          <legacyModeNS>true</legacyModeNS>
+        </plugin>
+      </gazebo>
+    </xacro:if>
+    <xacro:if value="${gazebo_control_mode!='ginko'}">
+      <gazebo>
+        <plugin name="gazebo_ros_control" filename="libgazebo_ros_control.so">
+          <robotNamespace>/ginko</robotNamespace>
+          <robotSimType>gazebo_ros_control/DefaultRobotHWSim</robotSimType>
+          <legacyModeNS>true</legacyModeNS>
+        </plugin>
+      </gazebo>
     </xacro:if>
   </xacro:macro>
-  <xacro:ginko_xacro model_mode="$(arg model_mode)"/>
+  <!-- MACRO:Setting up a Robot Model -->
+  <xacro:macro name="ginko_xacro" params="model_mode gazebo_control_mode">
+    <xacro:body_xacro model_mode="${model_mode}"/>
+    <xacro:body_gazebo gazebo_control_mode="${gazebo_control_mode}"/>
+    <xacro:leg_r model_mode="${model_mode}"/>
+    <xacro:leg_r_gazebo name="leg_r" gazebo_control_mode="${gazebo_control_mode}"/>
+<!--     <xacro:if value="${model_mode=='rviz'}">
+      <xacro:leg_r model_mode="common"/>
+      <xacro:leg_r_gazebo name="leg_r"/>
+    </xacro:if>
+    <xacro:if value="${model_mode=='common'}">
+      <xacro:leg_r model_mode="common"/>
+      <xacro:leg_r_gazebo name="leg_r"/>
+    </xacro:if>
+    <xacro:if value="${model_mode=='gazebo_part1'}">
+      <xacro:leg_r model_mode="gazebo_part1"/>
+      <xacro:leg_r_gazebo name="leg_r"/>
+    </xacro:if>
+    <xacro:if value="${model_mode=='gazebo_part2'}">
+      <xacro:leg_r model_mode="common"/>
+      <xacro:leg_r_gazebo name="leg_r"/>
+    </xacro:if> -->
+  </xacro:macro>
+  <!-- Load Macros -->
+  <xacro:ginko_xacro model_mode="$(arg model_mode)" gazebo_control_mode="$(arg gazebo_control_mode)"/>
+  <xacro:gazebo_plugin_xacro gazebo_control_mode="$(arg gazebo_control_mode)"/>
 </robot>

File: ginko_description/gazebo/xacro/modules/body.xacro (robot description, xacro)
@@ -1,8 +1,7 @@
 <?xml version="1.0"?>
 <robot xmlns:xacro="http://www.ros.org/wiki/xacro">
-	<xacro:macro name="body_xacro" params="name model_mode">
+	<xacro:macro name="body_xacro" params="model_mode">
 		<!-- chest -->
-		<link name="${name}_link0">
-			<!-- Collision created from STL mesh without color -->
+		<link name="body_link0">
 			<collision>
 				<origin xyz="0 0 0" rpy="0 0 0"/>
@@ -11,5 +10,4 @@
 				</geometry>
 			</collision>
-			<!-- Visualisation created from Color dae -->
 			<visual>
 				<origin xyz="0 0 0" rpy="0 0 0"/>
@@ -27,7 +25,15 @@
 			</inertial>
 		</link>
+		<!-- Joint1 -->
+		<joint name="body_joint1" type="revolute">
+			<parent link="body_link0"/>
+			<child  link="body_link1"/>
+			<origin xyz="0.0 0 0" rpy="0 0 0"/>
+			<axis xyz="0 0 1"/>
+			<limit effort="1000.0" lower="-2.6" upper="2.6" velocity="10.0"/>
+			<dynamics damping="0.1" friction="0.1"/>
+		</joint>
 		<!-- waist -->
-		<link name="${name}_link1">
-			<!-- Collision created from STL mesh without color -->
+		<link name="body_link1">
 			<collision>
 				<origin xyz="0 0 0" rpy="0 0 0"/>
@@ -36,5 +42,4 @@
 	    		</geometry>
 			</collision>
-			<!-- Visualisation created from Color dae -->
 			<visual>
 				<origin xyz="0 0 0" rpy="0 0 0"/>
@@ -52,11 +57,4 @@
 			</inertial>
 		</link>
-		<joint name="${name}_joint1" type="revolute">
-			<parent link="${name}_link0"/>
-			<child  link="${name}_link1"/>
-			<origin xyz="0 0 0" rpy="0 0 0"/>
-			<axis xyz="0 0 1"/>
-			<limit effort="1000.0" lower="-2.6" upper="2.6" velocity="10.0"/>
-		</joint>
 	</xacro:macro>
 </robot>

File: ginko_description/gazebo/xacro/modules/leg_r.xacro (robot description, xacro)
@@ -1,8 +1,15 @@
 <?xml version="1.0"?>
 <robot xmlns:xacro="http://www.ros.org/wiki/xacro">
-	<xacro:macro name="leg_r_sim" params="name parent">
-		<!-- Femoral -->
+	<xacro:macro name="leg_r" params="model_mode">
 		<!-- Link conencts from body. Femoral first. -->
-		<link name="${name}_link0">
+		<joint name="leg_r_joint0" type="revolute">
+		    <parent link="body_link1"/>
+			<child link="leg_r_link0"/>
+		    <origin xyz="0.0205 0.0 -0.0409" rpy="0 0 0"/>
+		    <axis xyz="1 0 0"/>
+			<limit effort="1000.0" lower="-1.0" upper="0.8" velocity="10.0"/>
+			<dynamics damping="0.1" friction="0.1"/>
+		</joint>
+		<link name="leg_r_link0">
 			<collision>
 				<origin xyz="0 0 0" rpy="0 0 0"/>
@@ -26,13 +33,14 @@
 			</inertial>
 		</link>
-		<joint name="${name}_joint0" type="revolute">
-		    <parent link="${parent}"/>
-			<child link="${name}_link0"/>
-		    <origin xyz="0.0205 0.0 -0.0409" rpy="0 0 0"/>
-		    <axis xyz="1 0 0"/>
-			<limit effort="1000.0" lower="-1.1781" upper="0.8" velocity="10.0"/>
-		</joint>
 		<!-- parallel link (upper-1st) -->
-		<link name="${name}_link1">
+		<joint name="leg_r_joint1" type="revolute">
+			<parent link="leg_r_link0"/>
+			<child  link="leg_r_link1"/>
+			<origin xyz="-0.0176 -0.0175 -0.0481" rpy="0 0.7854 0"/>
+			<axis xyz="0 1 0"/>
+			<limit effort="1000.0" lower="-0.7854" upper="1.3" velocity="10.0"/>
+			<dynamics damping="0.1" friction="0.1"/>
+		</joint>
+		<link name="leg_r_link1">
 			<collision>
 				<origin xyz="0 0 0" rpy="0 0 0"/>
@@ -56,13 +64,27 @@
 			</inertial>
 		</link>
-		<joint name="${name}_joint1" type="revolute">
-			<parent link="${name}_link0"/>
-			<child  link="${name}_link1"/>
-			<origin xyz="-0.0176 -0.0175 -0.0481" rpy="0 0.7854 0"/>
+		<joint name="leg_r_joint3" type="revolute">
+			<parent link="leg_r_link1"/>
+			<child  link="leg_r_link3"/>
+			<origin xyz="0.1 0.0 0.0" rpy="0 -0.7854 0"/>
+			<axis xyz="0 -1 0"/>
+			<limit effort="1000.0" lower="-0.7854" upper="1.3" velocity="10.0"/>
+			<dynamics damping="0.1" friction="0.1"/>
+			<xacro:if value="${model_mode=='rviz'}">
+				<mimic joint="leg_r_joint1" multiplier="1" offset="0"/>
+    		</xacro:if>
+		</joint>
+		<!-- parallel link (upper-2nd) -->
+		<joint name="leg_r_joint2" type="revolute">
+			<parent link="leg_r_link0"/>
+			<child  link="leg_r_link2"/>
+			<origin xyz="-0.0389 -0.0175 -0.06015" rpy="0 0.7854 0"/>
 			<axis xyz="0 1 0"/>
 			<limit effort="1000.0" lower="-0.7854" upper="1.3" velocity="10.0"/>
-		</joint>
-		<!-- parallel link (upper-2nd) -->
-		<link name="${name}_link2">
+			<xacro:if value="${model_mode=='rviz'}">
+				<mimic joint="leg_r_joint1" multiplier="1" offset="0"/>
+    		</xacro:if>
+		</joint>
+		<link name="leg_r_link2">
 	    	<collision>
 				<origin xyz="0 0 0" rpy="0 0 0"/>
@@ -86,14 +108,26 @@
 			</inertial>
 		</link>
-		<joint name="${name}_joint2" type="revolute">
-	    	<parent link="${name}_link0"/>
-	    	<child  link="${name}_link2"/>
-	    	<origin xyz="-0.0389 -0.0175 -0.06015" rpy="0 0.7854 0"/>
-	    	<axis xyz="0 1 0"/>
-	    	<limit effort="1000.0" lower="-3.141593" upper="3.141593" velocity="10.0"/>
-			<mimic joint="${name}_joint1" multiplier="1" offset="0"/>
-	  	</joint>
+		<joint name="close_leg_r_joint0" type="revolute">
+			<parent link="leg_r_link2"/>
+			<child  link="dummy0_leg_r_link3"/>
+			<origin xyz="0.1 0.0 0.0" rpy="0 -0.7854 0"/>
+			<axis xyz="0 -1 0"/>
+			<limit effort="1000.0" lower="-0.7854" upper="1.3" velocity="10.0"/>
+			<xacro:if value="${model_mode=='rviz'}">
+				<mimic joint="leg_r_joint1" multiplier="1" offset="0"/>
+			</xacro:if>
+		</joint>
+		<link name="dummy0_leg_r_link3">
+			<inertial>
+				<mass value="0.00001"/>
+				<origin xyz="-0.021 0 -0.012" rpy="0 0 0"/>
+				<inertia
+					ixx="0.00000001"
+					ixy="0.00000000" iyy="0.00000001"
+					ixz="0.00000000" iyz="0.00000000" izz="0.00000001"/>
+			</inertial>
+		</link>
 		<!-- knee -->
-		<link name="${name}_link3">
+		<link name="leg_r_link3">
 	    	<collision>
 				<origin xyz="0 0 0" rpy="0 0 0"/>
@@ -117,14 +151,96 @@
 			</inertial>
 		</link>
-		<joint name="${name}_joint3" type="revolute">
-	    	<parent link="${name}_link1"/>
-	    	<child  link="${name}_link3"/>
-	    	<origin xyz="0.1 0.0 0.0" rpy="0 -0.7854 0"/>
-	    	<axis xyz="0 -1 0"/>
-	    	<limit effort="1000.0" lower="-3.141593" upper="3.141593" velocity="10.0"/>
-			<mimic joint="${name}_joint1" multiplier="1" offset="0"/>
-	  	</joint>
+		<!-- spring -->
+		<xacro:if value="${model_mode!='rviz'}">
+			<joint name="leg_r_spring0_joint0" type="revolute">
+				<parent link="leg_r_link0"/>
+				<child  link="leg_r_spring0_link0"/>
+				<origin xyz="-0.0389 -0.0755 -0.06015" rpy="0 0.56756754 0"/>
+				<axis xyz="0 -1 0"/>
+				<limit effort="0.0" lower="-3.141593" upper="3.141593" velocity="10.0"/>
+			</joint>
+			<link name="leg_r_spring0_link0">
+				<collision>
+					<origin xyz="0 0 0" rpy="0 0 0"/>
+					<geometry>
+						<mesh filename="package://ginko_description/meshes/stl/spring1.stl"/>
+					</geometry>
+				</collision>
+				<visual>
+					<origin xyz="0 0 0" rpy="0 0 0"/>
+					<geometry>
+						<mesh filename="package://ginko_description/meshes/stl/spring1.stl"/>
+					</geometry>
+					<color rgba="1.0 1.0 1.0 0.5"/>
+				</visual>
+				<inertial>
+					<mass value="0.00143865"/>
+					<origin xyz="0.03091683 0.0 0.0" rpy="0 0 0"/>
+					<inertia
+						ixx="0.00000001"
+						ixy="0.00000000" iyy="0.00000060"
+						ixz="0.00000000" iyz="0.00000000" izz="0.00000060"/>
+				</inertial>
+			</link>
+			<joint name="leg_r_spring0_joint1" type="prismatic">
+				<parent link="leg_r_spring0_link0"/>
+				<child  link="leg_r_spring0_link1"/>
+				<origin xyz="0.10911938 0.0 0.0" rpy="0 3.141593 0"/>
+				<axis xyz="1 0 0"/>
+				<limit effort="1000.0" lower="-0.035" upper="0.055" velocity="10.0"/>
+				<dynamics damping="0.0" friction="0.0"/>
+			</joint>
+		  	<link name="leg_r_spring0_link1">
+		    	<collision>
+					<origin xyz="0 0 0" rpy="0 0 0"/>
+		    		<geometry>
+						<mesh filename="package://ginko_description/meshes/stl/spring2.stl"/>
+		    		</geometry>
+					<color rgba="1.0 1.0 1.0 0.5"/>
+				</collision>
+		    	<visual>
+					<origin xyz="0 0 0" rpy="0 0 0"/>
+		    		<geometry>
+						<mesh filename="package://ginko_description/meshes/stl/spring2.stl"/>
+		    		</geometry>
+		    		<color rgba="1.0 1.0 1.0 0.5"/>
+				</visual>
+				<inertial>
+					<mass value="0.00143865"/>
+					<origin xyz="0.03091683 0.0 0.0" rpy="0 0 0"/>
+					<inertia
+						ixx="0.00000001"
+						ixy="0.00000000" iyy="0.00000060"
+						ixz="0.00000000" iyz="0.00000000" izz="0.00000060"/>
+				</inertial>
+			</link>
+			<joint name="close_leg_r_spring0_joint2" type="revolute">
+				<parent link="leg_r_spring0_link1"/>
+				<child  link="dummy1_leg_r_link3"/>
+				<origin xyz="0 0 0" rpy="0 0 0"/>
+				<axis xyz="0 -1 0"/>
+				<limit effort="0.0" lower="-3.141593" upper="3.141593" velocity="10.0"/>
+			</joint>
+			<link name="dummy1_leg_r_link3">
+				<inertial>
+					<mass value="0.00001"/>
+					<origin xyz="0 -0.058 0" rpy="0 0 0"/>
+					<inertia
+						ixx="0.00000001"
+						ixy="0.00000000" iyy="0.00000001"
+						ixz="0.00000000" iyz="0.00000000" izz="0.00000001"/>
+				</inertial>
+			</link>
+		</xacro:if>
 		<!-- parallel link (lower-1st) -->
-		<link name="${name}_link4">
+		<joint name="leg_r_joint4" type="revolute">
+			<parent link="leg_r_link3"/>
+			<child  link="leg_r_link4"/>
+			<origin xyz="0 0 -0.0386" rpy="0 2.3562 0"/>
+			<axis xyz="0 1 0"/>
+			<limit effort="1000.0" lower="-1.3" upper="0.7854" velocity="10.0"/>
+			<dynamics damping="0.1" friction="0.1"/>
+		</joint>
+		<link name="leg_r_link4">
 			<collision>
 				<origin xyz="0 0 0" rpy="0 0 0"/>
@@ -148,18 +264,32 @@
 			</inertial>
 		</link>
-		<joint name="${name}_joint4" type="revolute">
-			<parent link="${name}_link3"/>
-			<child  link="${name}_link4"/>
-			<origin xyz="0 0 -0.0386" rpy="0 2.3562 0"/>
+		<joint name="leg_r_joint6" type="revolute">
+			<parent link="leg_r_link4"/>
+			<child  link="leg_r_link6"/>
+			<origin xyz="0.1 0.0 0.0" rpy="0 -2.3562 0"/>
+			<axis xyz="0 -1 0"/>
+			<limit effort="1000.0" lower="-1.3" upper="0.7854" velocity="10.0"/>
+			<dynamics damping="0.1" friction="0.1"/>
+			<xacro:if value="${model_mode=='rviz'}">
+				<mimic joint="leg_r_joint4" multiplier="1" offset="0"/>
+			</xacro:if>
+		</joint>
+		<!-- parallel link (lower-2nd) -->
+		<joint name="leg_r_joint5" type="revolute">
+			<parent link="leg_r_link3"/>
+			<child  link="leg_r_link5"/>
+			<origin xyz="-0.0213 0 -0.02655" rpy="0 2.3562 0"/>
 			<axis xyz="0 1 0"/>
-			<limit effort="1000.0" lower="-1.3" upper="0.7854" velocity="10.0"/>
-		</joint>
-		<!-- parallel link (lower-2nd) -->
-		<link name="${name}_link5">
-	    	<collision>
-				<origin xyz="0 0 0" rpy="0 0 0"/>
-	    		<geometry>
+			<limit effort="0.0" lower="-1.3" upper="0.7854" velocity="10.0"/>
+			<xacro:if value="${model_mode=='rviz'}">
+				<mimic joint="leg_r_joint4" multiplier="1" offset="0"/>
+			</xacro:if>
+		</joint>
+		<link name="leg_r_link5">
+			<collision>
+				<origin xyz="0 0 0" rpy="0 0 0"/>
+				<geometry>
 					<mesh filename="package://ginko_description/meshes/stl/link04_r_leg02.stl"/>
-	    		</geometry>
+				</geometry>
 			</collision>
 			<visual>
@@ -178,14 +308,106 @@
 			</inertial>
 		</link>
-		<joint name="${name}_joint5" type="revolute">
-	    	<parent link="${name}_link3"/>
-	    	<child  link="${name}_link5"/>
-	    	<origin xyz="-0.0213 0 -0.02655" rpy="0 2.3562 0"/>
-	    	<axis xyz="0 1 0"/>
-	    	<limit effort="1000.0" lower="-3.141593" upper="3.141593" velocity="10.0"/>
-	    	<mimic joint="${name}_joint4" multiplier="1" offset="0"/>
-	  	</joint>
+		<joint name="close_leg_r_joint1" type="revolute">
+			<parent link="leg_r_link5"/>
+			<child  link="dummy2_leg_r_link6"/>
+			<origin xyz="0.1 0.0 0.0" rpy="0 -2.3562 0"/>
+			<axis xyz="0 -1 0"/>
+			<limit effort="0.0" lower="-1.3" upper="0.7854" velocity="10.0"/>
+			<xacro:if value="${model_mode=='rviz'}">
+				<mimic joint="leg_r_joint4" multiplier="1" offset="0"/>
+			</xacro:if>
+		</joint>
+		<link name="dummy2_leg_r_link6">
+			<inertial>
+				<mass value="0.00001"/>
+				<origin xyz="-0.021 0 0.012" rpy="0 0 0"/>
+				<inertia
+					ixx="0.00000001"
+					ixy="0.00000000" iyy="0.00000001"
+					ixz="0.00000000" iyz="0.00000000" izz="0.00000001"/>
+			</inertial>
+		</link>
+		<!-- spring -->
+		<xacro:if value="${model_mode!='rviz'}">
+			<joint name="leg_r_spring1_joint0" type="revolute">
+				<parent link="leg_r_link3"/>
+				<child  link="leg_r_spring1_link0"/>
+				<origin xyz="0 -0.058 -0.0386" rpy="0 2.574025114 0"/>
+				<axis xyz="0 -1 0"/>
+				<limit effort="0.0" lower="-3.141593" upper="3.141593" velocity="10.0"/>
+			</joint>
+			<link name="leg_r_spring1_link0">
+				<collision>
+					<origin xyz="0 0 0" rpy="0 0 0"/>
+					<geometry>
+						<mesh filename="package://ginko_description/meshes/stl/spring1.stl"/>
+					</geometry>
+				</collision>
+				<visual>
+					<origin xyz="0 0 0" rpy="0 0 0"/>
+					<geometry>
+						<mesh filename="package://ginko_description/meshes/stl/spring1.stl"/>
+					</geometry>
+					<color rgba="1.0 1.0 1.0 0.5"/>
+				</visual>
+				<inertial>
+					<mass value="0.00143865"/>
+					<origin xyz="0.03091683 0.0 0.0" rpy="0 2.138363867 0"/>
+					<inertia
+						ixx="0.00000001"
+						ixy="0.00000000" iyy="0.00000060"
+						ixz="0.00000000" iyz="0.00000000" izz="0.00000060"/>
+				</inertial>
+			</link>
+			<joint name="leg_r_spring1_joint1" type="prismatic">
+				<parent link="leg_r_spring1_link0"/>
+				<child  link="leg_r_spring1_link1"/>
+				<origin xyz="0.10911938 0.0 0.0" rpy="0 3.141593 0"/>
+				<axis xyz="1 0 0"/>
+				<limit effort="1000.0" lower="-0.035" upper="0.055" velocity="10.0"/>
+			</joint>
+			<link name="leg_r_spring1_link1">
+				<collision>
+					<origin xyz="0 0 0" rpy="0 0 0"/>
+					<geometry>
+						<mesh filename="package://ginko_description/meshes/stl/spring2.stl"/>
+					</geometry>
+				</collision>
+				<visual>
+					<origin xyz="0 0 0" rpy="0 0 0"/>
+					<geometry>
+						<mesh filename="package://ginko_description/meshes/stl/spring2.stl"/>
+					</geometry>
+					<color rgba="1.0 1.0 1.0 0.5"/>
+				</visual>
+				<inertial>
+					<mass value="0.00143865"/>
+					<origin xyz="0.03091683 0.0 0.0" rpy="0 0 0"/>
+					<inertia
+						ixx="0.00000001"
+						ixy="0.00000000" iyy="0.00000060"
+						ixz="0.00000000" iyz="0.00000000" izz="0.00000060"/>
+				</inertial>
+			</link>
+			<joint name="close_leg_r_spring1_joint2" type="revolute">
+				<parent link="leg_r_spring1_link1"/>
+				<child  link="dummy3_leg_r_link6"/>
+				<origin xyz="0 0 0" rpy="0 0 0"/>
+				<axis xyz="0 -1 0"/>
+				<limit effort="0.0" lower="-3.141593" upper="3.141593" velocity="10.0"/>
+			</joint>
+			<link name="dummy3_leg_r_link6">
+				<inertial>
+					<mass value="0.00001"/>
+					<origin xyz="-0.021 -0.058 0.012" rpy="0 0 0"/>
+					<inertia
+						ixx="0.00000001"
+						ixy="0.00000000" iyy="0.00000001"
+						ixz="0.00000000" iyz="0.00000000" izz="0.00000001"/>
+				</inertial>
+			</link>
+		</xacro:if>
 		<!-- toe -->
-		<link name="${name}_link6">
+		<link name="leg_r_link6">
 			<collision>
 				<origin xyz="0 0 0" rpy="0 0 0"/>
@@ -209,13 +431,5 @@
 			</inertial>
 		</link>
-		<joint name="${name}_joint6" type="revolute">
-	    	<parent link="${name}_link4"/>
-	    	<child  link="${name}_link6"/>
-	    	<origin xyz="0.1 0.0 0.0" rpy="0 -2.3562 0"/>
-	    	<axis xyz="0 -1 0"/>
-	    	<limit effort="1000.0" lower="-3.141593" upper="3.141593" velocity="10.0"/>
-	    	<mimic joint="${name}_joint4" multiplier="1" offset="0"/>
-	  	</joint>
-		<link name="${name}_link7">
+		<link name="leg_r_link7">
 	    	<collision>
 				<origin xyz="0 0 0" rpy="0 0 0"/>
@@ -239,12 +453,12 @@
 			</inertial>
 		</link>
-		<joint name="${name}_joint7" type="revolute">
-	    	<parent link="${name}_link6"/>
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