Commit message: 腕を追加

File: ginko_description/gazebo/xacro/ginko.xacro (robot description, xacro)
@@ -42,4 +42,8 @@
     <xacro:leg_l model_mode="${model_mode}"/>
     <xacro:leg_l_gazebo gazebo_control_mode="${gazebo_control_mode}"/>
+    <xacro:arm_r model_mode="${model_mode}"/>
+    <xacro:arm_r_gazebo gazebo_control_mode="${gazebo_control_mode}"/>
+    <xacro:arm_l model_mode="${model_mode}"/>
+    <xacro:arm_l_gazebo gazebo_control_mode="${gazebo_control_mode}"/>
     <!-- <xacro:leg_l model_mode="${model_mode}"/> -->
     <!-- <xacro:leg_l_gazebo name="leg_l" gazebo_control_mode="${gazebo_control_mode}"/> -->

File: ginko_description/gazebo/xacro/modules/arm_l.xacro (robot description, xacro)
@@ -1,8 +1,15 @@
 <?xml version="1.0"?>
 <robot xmlns:xacro="http://www.ros.org/wiki/xacro">
-	<xacro:macro name="arm_l_sim" params="name parent">
+	<xacro:macro name="arm_l" params="model_mode">
 		<!-- shoulder pitch. -->
-		<link name="${name}_link0">
-			<!-- Collision created from STL mesh without color -->
+		<joint name="arm_l_joint0" type="revolute">
+		    <parent link="body_link1"/>
+			<child link="arm_l_link0"/>
+		    <origin xyz="0 0.10683 0.05115" rpy="0 0.3927 0"/>
+		    <axis xyz="0 -1 0"/>
+			<limit effort="1000.0" lower="-2.6" upper="2.6" velocity="10.0"/>
+			<dynamics damping="0.1" friction="0.1"/>
+		</joint>
+		<link name="arm_l_link0">
 			<collision>
 				<origin xyz="0 0 0" rpy="0 0 0"/>
@@ -11,5 +18,4 @@
 				</geometry>
 			</collision>
-			<!-- Visualisation created from Color dae -->
 			<visual>
 				<origin xyz="0 0 0" rpy="0 0 0"/>
@@ -27,14 +33,14 @@
 			</inertial>
 		</link>
-		<joint name="${name}_joint0" type="revolute">
-		    <parent link="${parent}"/>
-			<child link="${name}_link0"/>
-		    <origin xyz="0 0.10683 0.05115" rpy="0 0.3927 0"/>
-		    <axis xyz="0 -1 0"/>
-			<limit effort="1000.0" lower="-2.6" upper="2.6" velocity="10.0"/>
+		<!-- shoulder roll -->
+		<joint name="arm_l_joint1" type="revolute">
+			<parent link="arm_l_link0"/>
+			<child  link="arm_l_link1"/>
+			<origin xyz="0.035 0.0246 0" rpy="1.1781 0 0"/>
+			<axis xyz="1 0 0"/>
+			<limit effort="1000.0" lower="-0.85" upper="1.18" velocity="10.0"/>
+			<dynamics damping="0.1" friction="0.1"/>
 		</joint>
-		<!-- shoulder roll -->
-		<link name="${name}_link1">
-			<!-- Collision created from STL mesh without color -->
+		<link name="arm_l_link1">
 			<collision>
 				<origin xyz="0 0 0" rpy="0 0 0"/>
@@ -43,5 +49,4 @@
 	    		</geometry>
 			</collision>
-			<!-- Visualisation created from Color dae -->
 			<visual>
 				<origin xyz="0 0 0" rpy="0 0 0"/>
@@ -59,14 +64,14 @@
 			</inertial>
 		</link>
-		<joint name="${name}_joint1" type="revolute">
-			<parent link="${name}_link0"/>
-			<child  link="${name}_link1"/>
-			<origin xyz="0.035 0.0246 0" rpy="1.1781 0 0"/>
-			<axis xyz="1 0 0"/>
-			<limit effort="1000.0" lower="-0.85" upper="1.18" velocity="10.0"/>
+		<!-- scissors -->
+		<joint name="arm_l_joint2" type="revolute">
+	    	<parent link="arm_l_link1"/>
+	    	<child  link="arm_l_link2"/>
+	    	<origin xyz="0.0092 0.0547 -0.11295" rpy="0 0.7854 0"/>
+	    	<axis xyz="0 1 0"/>
+	    	<limit effort="1000.0" lower="-2.36" upper="2.36" velocity="10.0"/>
+			<dynamics damping="0.1" friction="0.1"/>
 		</joint>
-		<!-- scissors -->
-		<link name="${name}_link2">
-			<!-- Collision created from STL mesh without color -->
+		<link name="arm_l_link2">
 	    	<collision>
 				<origin xyz="0 0 0" rpy="0 0 0"/>
@@ -75,5 +80,4 @@
 	    		</geometry>
 			</collision>
-			<!-- Visualisation created from Color dae -->
 			<visual>
 				<origin xyz="0 0 0" rpy="0 0 0"/>
@@ -91,13 +95,13 @@
 			</inertial>
 		</link>
-		<joint name="${name}_joint2" type="revolute">
-	    	<parent link="${name}_link1"/>
-	    	<child  link="${name}_link2"/>
-	    	<origin xyz="0.0092 0.0547 -0.11295" rpy="0 0.7854 0"/>
+		<joint name="arm_l_joint3" type="revolute">
+	    	<parent link="arm_l_link1"/>
+	    	<child  link="arm_l_link3"/>
+	    	<origin xyz="0.0092 -0.0018 -0.11295" rpy="0 0.7854 0"/>
 	    	<axis xyz="0 1 0"/>
 	    	<limit effort="1000.0" lower="-2.36" upper="2.36" velocity="10.0"/>
-	  	</joint>
-		<link name="${name}_link3">
-			<!-- Collision created from STL mesh without color -->
+			<dynamics damping="0.1" friction="0.1"/>
+		</joint>
+		<link name="arm_l_link3">
 	    	<collision>
 				<origin xyz="0 0 0" rpy="0 0 0"/>
@@ -106,5 +110,4 @@
 	    		</geometry>
 			</collision>
-			<!-- Visualisation created from Color dae -->
 			<visual>
 				<origin xyz="0 0 0" rpy="0 0 0"/>
@@ -113,5 +116,4 @@
 				</geometry>
 			</visual>
-			<!-- nothing worth -->
 			<inertial>
 				<mass value="0.02936110"/>
@@ -123,13 +125,15 @@
 			</inertial>
 		</link>
-		<joint name="${name}_joint3" type="revolute">
-	    	<parent link="${name}_link1"/>
-	    	<child  link="${name}_link3"/>
-	    	<origin xyz="0.0092 -0.0018 -0.11295" rpy="0 0.7854 0"/>
-	    	<axis xyz="0 1 0"/>
-	    	<limit effort="1000.0" lower="-2.36" upper="2.36" velocity="10.0"/>
-	  	</joint>
 	  	<!-- LiDAR -->
-		<link name="${name}_urg_link">
+		<!-- use zero-limited revolute joint for fixed joint (SDF) -->
+		<joint name="arm_l_urg_joint" type="revolute">
+	    	<parent link="arm_l_link1"/>
+	    	<child  link="arm_l_urg_link"/>
+	    	<origin xyz="-0.0456 -0.01715 -0.06795" rpy="0 1.57 -1.57"/>
+	    	<axis xyz="0 0 1"/>
+	    	<limit effort="0.0" lower="0.0" upper="0.0" velocity="0.0"/>
+			<dynamics damping="0.1" friction="0.1"/>
+		</joint>
+		<link name="arm_l_urg_link">
 	    	<collision>
 				<origin xyz="0 0 0" rpy="0 0 0"/>
@@ -138,5 +142,4 @@
 	    		</geometry>
 			</collision>
-			<!-- Visualisation created from Color dae -->
 			<visual>
 				<origin xyz="0 0 0" rpy="0 0 0"/>
@@ -145,5 +148,4 @@
 				</geometry>
 			</visual>
-			<!-- nothing worth -->
 			<inertial>
 				<mass value="0.16705492"/>
@@ -155,12 +157,4 @@
 			</inertial>
 		</link>
-		<!-- use zero-limited revolute joint for fixed joint (SDF) -->
-		<joint name="${name}_urg_joint" type="revolute">
-	    	<parent link="${name}_link1"/>
-	    	<child  link="${name}_urg_link"/>
-	    	<origin xyz="-0.0456 -0.01715 -0.06795" rpy="0 1.57 -1.57"/>
-	    	<axis xyz="0 0 1"/>
-	    	<limit effort="0.0" lower="0.0" upper="0.0" velocity="0.0"/>
-		</joint>
 	</xacro:macro>
 </robot>

File: ginko_description/gazebo/xacro/modules/arm_r.xacro (robot description, xacro)
@@ -1,8 +1,15 @@
 <?xml version="1.0"?>
 <robot xmlns:xacro="http://www.ros.org/wiki/xacro">
-	<xacro:macro name="arm_r_sim" params="name parent">
+	<xacro:macro name="arm_r" params="model_mode">
 		<!-- shoulder pitch. -->
-		<link name="${name}_link0">
-			<!-- Collision created from STL mesh without color -->
+		<joint name="arm_r_joint0" type="revolute">
+		    <parent link="body_link1"/>
+			<child link="arm_r_link0"/>
+		    <origin xyz="0 -0.10683 0.05115" rpy="0 0.3927 0"/>
+		    <axis xyz="0 1 0"/>
+			<limit effort="1000.0" lower="-2.6" upper="2.6" velocity="10.0"/>
+			<dynamics damping="0.1" friction="0.1"/>
+		</joint>
+		<link name="arm_r_link0">
 			<collision>
 				<origin xyz="0 0 0" rpy="0 0 0"/>
@@ -11,5 +18,4 @@
 				</geometry>
 			</collision>
-			<!-- Visualisation created from Color dae -->
 			<visual>
 				<origin xyz="0 0 0" rpy="0 0 0"/>
@@ -27,14 +33,14 @@
 			</inertial>
 		</link>
-		<joint name="${name}_joint0" type="revolute">
-		    <parent link="${parent}"/>
-			<child link="${name}_link0"/>
-		    <origin xyz="0 -0.10683 0.05115" rpy="0 0.3927 0"/>
-		    <axis xyz="0 1 0"/>
-			<limit effort="1000.0" lower="-2.6" upper="2.6" velocity="10.0"/>
+		<!-- shoulder roll -->
+		<joint name="arm_r_joint1" type="revolute">
+			<parent link="arm_r_link0"/>
+			<child  link="arm_r_link1"/>
+			<origin xyz="0.035 -0.0246 0" rpy="-1.1781 0 0"/>
+			<axis xyz="1 0 0"/>
+			<limit effort="1000.0" lower="-0.85" upper="1.18" velocity="10.0"/>
+			<dynamics damping="0.1" friction="0.1"/>
 		</joint>
-		<!-- shoulder roll -->
-		<link name="${name}_link1">
-			<!-- Collision created from STL mesh without color -->
+		<link name="arm_r_link1">
 			<collision>
 				<origin xyz="0 0 0" rpy="0 0 0"/>
@@ -43,5 +49,4 @@
 	    		</geometry>
 			</collision>
-			<!-- Visualisation created from Color dae -->
 			<visual>
 				<origin xyz="0 0 0" rpy="0 0 0"/>
@@ -59,14 +64,14 @@
 			</inertial>
 		</link>
-		<joint name="${name}_joint1" type="revolute">
-			<parent link="${name}_link0"/>
-			<child  link="${name}_link1"/>
-			<origin xyz="0.035 -0.0246 0" rpy="-1.1781 0 0"/>
-			<axis xyz="1 0 0"/>
-			<limit effort="1000.0" lower="-0.85" upper="1.18" velocity="10.0"/>
+		<!-- scissors -->
+		<joint name="arm_r_joint2" type="revolute">
+			<parent link="arm_r_link1"/>
+			<child  link="arm_r_link2"/>
+			<origin xyz="0.0092 -0.0547 -0.11295" rpy="0 0.7854 0"/>
+			<axis xyz="0 -1 0"/>
+			<limit effort="1000.0" lower="-2.36" upper="2.36" velocity="10.0"/>
+			<dynamics damping="0.1" friction="0.1"/>
 		</joint>
-		<!-- scissors -->
-		<link name="${name}_link2">
-			<!-- Collision created from STL mesh without color -->
+		<link name="arm_r_link2">
 	    	<collision>
 				<origin xyz="0 0 0" rpy="0 0 0"/>
@@ -75,5 +80,4 @@
 	    		</geometry>
 			</collision>
-			<!-- Visualisation created from Color dae -->
 			<visual>
 				<origin xyz="0 0 0" rpy="0 0 0"/>
@@ -82,5 +86,4 @@
 				</geometry>
 			</visual>
-			<!-- nothing worth -->
 			<inertial>
 				<mass value="0.03287850"/>
@@ -92,13 +95,13 @@
 			</inertial>
 		</link>
-		<joint name="${name}_joint2" type="revolute">
-	    	<parent link="${name}_link1"/>
-	    	<child  link="${name}_link2"/>
-	    	<origin xyz="0.0092 -0.0547 -0.11295" rpy="0 0.7854 0"/>
-	    	<axis xyz="0 -1 0"/>
-	    	<limit effort="1000.0" lower="-2.36" upper="2.36" velocity="10.0"/>
-	  	</joint>
-		<link name="${name}_link3">
-			<!-- Collision created from STL mesh without color -->
+		<joint name="arm_r_joint3" type="revolute">
+			<parent link="arm_r_link1"/>
+			<child  link="arm_r_link3"/>
+			<origin xyz="0.0092 0.0018 -0.11295" rpy="0 0.7854 0"/>
+			<axis xyz="0 -1 0"/>
+			<limit effort="1000.0" lower="-2.36" upper="2.36" velocity="10.0"/>
+			<dynamics damping="0.1" friction="0.1"/>
+		</joint>
+		<link name="arm_r_link3">
 	    	<collision>
 				<origin xyz="0 0 0" rpy="0 0 0"/>
@@ -107,5 +110,4 @@
 	    		</geometry>
 			</collision>
-			<!-- Visualisation created from Color dae -->
 			<visual>
 				<origin xyz="0 0 0" rpy="0 0 0"/>
@@ -123,13 +125,15 @@
 			</inertial>
 		</link>
-		<joint name="${name}_joint3" type="revolute">
-	    	<parent link="${name}_link1"/>
-	    	<child  link="${name}_link3"/>
-	    	<origin xyz="0.0092 0.0018 -0.11295" rpy="0 0.7854 0"/>
-	    	<axis xyz="0 -1 0"/>
-	    	<limit effort="1000.0" lower="-2.36" upper="2.36" velocity="10.0"/>
-	  	</joint>
 	  	<!-- LiDAR -->
-		<link name="${name}_urg_link">
+		<!-- use zero-limited revolute joint for fixed joint (SDF) -->
+		<joint name="arm_r_urg_joint"  type="revolute">
+	    	<parent link="arm_r_link1"/>
+	    	<child  link="arm_r_urg_link"/>
+	    	<origin xyz="-0.0456 0.01715 -0.06795" rpy="0 1.57 1.57"/>
+	    	<axis xyz="0 0 1"/>
+	    	<limit effort="0.0" lower="0.0" upper="0.0" velocity="0.0"/>
+			<dynamics damping="0.1" friction="0.1"/>
+		</joint>
+		<link name="arm_r_urg_link">
 	    	<collision>
 				<origin xyz="0 0 0" rpy="0 0 0"/>
@@ -138,5 +142,4 @@
 	    		</geometry>
 			</collision>
-			<!-- Visualisation created from Color dae -->
 			<visual>
 				<origin xyz="0 0 0" rpy="0 0 0"/>
@@ -145,5 +148,4 @@
 				</geometry>
 			</visual>
-			<!-- nothing worth -->
 			<inertial>
 				<mass value="0.16705492"/>
@@ -155,12 +157,4 @@
 			</inertial>
 		</link>
-		<!-- use zero-limited revolute joint for fixed joint (SDF) -->
-		<joint name="${name}_urg_joint"  type="revolute">
-	    	<parent link="${name}_link1"/>
-	    	<child  link="${name}_urg_link"/>
-	    	<origin xyz="-0.0456 0.01715 -0.06795" rpy="0 1.57 1.57"/>
-	    	<axis xyz="0 0 1"/>
-	    	<limit effort="0.0" lower="0.0" upper="0.0" velocity="0.0"/>
-		</joint>
 	</xacro:macro>
 </robot>

Commit message: gazeboモデルにurgを追加

File: ginko_description/gazebo/xacro/ginko.xacro (robot description, xacro)
@@ -3,5 +3,6 @@
   <xacro:arg name="model_mode" default="rviz"/>
   <xacro:arg name="gazebo_control_mode" default="ginko"/>
-  <xacro:include filename="$(find ginko_description)/gazebo/xacro/modules/imu_macro.xacro"/>
+  <xacro:include filename="$(find ginko_description)/gazebo/xacro/sensors/imu.xacro"/>
+  <xacro:include filename="$(find ginko_description)/gazebo/xacro/sensors/urg.xacro"/>
   <xacro:include filename="$(find ginko_description)/gazebo/xacro/modules/body.xacro"/>
   <xacro:include filename="$(find ginko_description)/gazebo/transmission/body.gazebo"/>
@@ -53,26 +54,10 @@
     <xacro:arm_l model_mode="${model_mode}"/>
     <xacro:arm_l_gazebo gazebo_control_mode="${gazebo_control_mode}"/>
-    <!-- <xacro:leg_l model_mode="${model_mode}"/> -->
-    <!-- <xacro:leg_l_gazebo name="leg_l" gazebo_control_mode="${gazebo_control_mode}"/> -->
-<!--     <xacro:if value="${model_mode=='rviz'}">
-      <xacro:leg_r model_mode="common"/>
-      <xacro:leg_r_gazebo name="leg_r"/>
-    </xacro:if>
-    <xacro:if value="${model_mode=='common'}">
-      <xacro:leg_r model_mode="common"/>
-      <xacro:leg_r_gazebo name="leg_r"/>
-    </xacro:if>
-    <xacro:if value="${model_mode=='gazebo_part1'}">
-      <xacro:leg_r model_mode="gazebo_part1"/>
-      <xacro:leg_r_gazebo name="leg_r"/>
-    </xacro:if>
-    <xacro:if value="${model_mode=='gazebo_part2'}">
-      <xacro:leg_r model_mode="common"/>
-      <xacro:leg_r_gazebo name="leg_r"/>
-    </xacro:if> -->
   </xacro:macro>
   <!-- Load Macros -->
   <xacro:ginko_xacro model_mode="$(arg model_mode)" gazebo_control_mode="$(arg gazebo_control_mode)"/>
   <xacro:gazebo_plugin_xacro gazebo_control_mode="$(arg gazebo_control_mode)"/>
-  <xacro:imu_macro model_mode="$(arg model_mode)"/>
+  <xacro:imu_xacro model_mode="$(arg model_mode)"/>
+  <xacro:urg_xacro firame_id="arm_r_urg_link" topic_name="/sensor/urg/right/scan_raw" sensor_name="urg_right"/>
+  <xacro:urg_xacro firame_id="arm_l_urg_link" topic_name="/sensor/urg/left/scan_raw" sensor_name="urg_left"/>
 </robot>

File: ginko_description/gazebo/xacro/sensors/imu.xacro (robot description, xacro)
@@ -1,5 +1,5 @@
 <?xml version="1.0"?>
 <robot xmlns:xacro="http://www.ros.org/wiki/xacro">
-	<xacro:macro name="imu_macro" params="model_mode">
+	<xacro:macro name="imu_xacro" params="model_mode">
 		<xacro:if value="${model_mode!='rviz'}">
 			<link name="body_imu_attached_link">
@@ -58,5 +58,5 @@
 				<alwaysOn>true</alwaysOn>
 				<bodyName>body_imu_base_link</bodyName>
-				<topicName>/sensor/imu/madgwick</topicName>
+				<topicName>/sensor/imu/raw</topicName>
 				<serviceName>gazebo_imu_service</serviceName>
 				<gaussianNoise>0.0</gaussianNoise>
