Commit message: imuのトピック名修正

File: ginko_description/gazebo/xacro/sensors/imu.xacro (robot description, xacro)
@@ -5,5 +5,5 @@
 			<link name="body_imu_attached_link">
 				<inertial>
-					<mass value="0.00052271"/>
+					<mass value="0.0005"/>
 					<origin xyz="0 0 0" rpy="0 0 0"/>
 					<inertia
@@ -23,5 +23,5 @@
 			<link name="body_imu_base_link">
 				<inertial>
-					<mass value="0.00052271"/>
+					<mass value="0.0005"/>
 					<origin xyz="0 0 0" rpy="0 0 0"/>
 					<inertia
@@ -58,8 +58,8 @@
 				<alwaysOn>true</alwaysOn>
 				<bodyName>body_imu_base_link</bodyName>
-				<topicName>/sensor/imu/raw</topicName>
+				<topicName>/sensor/imu/raw/data</topicName>
 				<serviceName>gazebo_imu_service</serviceName>
 				<gaussianNoise>0.0</gaussianNoise>
-				<updateRate>50.0</updateRate>
+				<updateRate>400.0</updateRate>
 			</plugin>
 		</gazebo>

File: ginko_description/gazebo/xacro/tmp/urdf/ginko_common.urdf (robot description, URDF)
Before this commit: robot ginko_xacro, 51 links, 50 joints
Links:
- link body_imu_attached_link: mass 0.00052271 -> 0.0005
- link body_imu_base_link: mass 0.00052271 -> 0.0005
