Commit message: gazeboにimuを追加

File: ginko_description/gazebo/urdf/ginko_rviz.urdf (robot description, URDF)
Before this commit: robot ginko_xacro, 46 links, 45 joints
Links:
- added link body_imu_attached_link
- added link body_imu_base_link
- added link root_link
Joints:
- added joint body_imu_attached_joint: type fixed, parent body_link1, child body_imu_attached_link, origin xyz=-0.09 0 -0.0379 rpy=0 1.5708 0
- added joint imu_joint: type fixed, parent body_link1, child body_imu_base_link, origin xyz=-0.09 0 -0.0379 rpy=0 1.5708 0
- added joint root_joint: type fixed, parent root_link, child body_link0, origin xyz=0 0 0 rpy=0 0 0

File: ginko_description/gazebo/xacro/ginko.xacro (robot description, xacro)
@@ -3,4 +3,5 @@
   <xacro:arg name="model_mode" default="rviz"/>
   <xacro:arg name="gazebo_control_mode" default="ginko"/>
+  <xacro:include filename="$(find ginko_description)/gazebo/xacro/modules/imu_macro.xacro"/>
   <xacro:include filename="$(find ginko_description)/gazebo/xacro/modules/body.xacro"/>
   <xacro:include filename="$(find ginko_description)/gazebo/transmission/body.gazebo"/>
@@ -36,4 +37,10 @@
   <!-- MACRO:Setting up a Robot Model -->
   <xacro:macro name="ginko_xacro" params="model_mode gazebo_control_mode">
+    <link name="root_link"/>
+    <joint name="root_joint" type="fixed">
+        <parent link="root_link"/>
+        <child  link="body_link0"/>
+        <origin xyz="0 0 0" rpy="0 0 0"/>
+    </joint>
     <xacro:body_xacro model_mode="${model_mode}"/>
     <xacro:body_gazebo gazebo_control_mode="${gazebo_control_mode}"/>
@@ -68,3 +75,4 @@
   <xacro:ginko_xacro model_mode="$(arg model_mode)" gazebo_control_mode="$(arg gazebo_control_mode)"/>
   <xacro:gazebo_plugin_xacro gazebo_control_mode="$(arg gazebo_control_mode)"/>
+  <xacro:imu_macro model_mode="$(arg model_mode)"/>
 </robot>

File: ginko_description/gazebo/xacro/tmp/urdf/ginko_common.urdf (robot description, URDF)
Before this commit: robot ginko_xacro, 48 links, 47 joints
Links:
- added link body_imu_attached_link, mass 0.00052271
- added link body_imu_base_link, mass 0.00052271
- added link root_link
Joints:
- added joint body_imu_attached_joint: type revolute, parent body_link1, child body_imu_attached_link, origin xyz=-0.09 0 -0.0379 rpy=0 1.5708 0, axis 0 0 1, limit lower=0.0 upper=0.0 effort=0.0 velocity=0.0
- added joint imu_joint: type revolute, parent body_link1, child body_imu_base_link, origin xyz=-0.09 0 -0.0379 rpy=0 0 0, axis 0 0 1, limit lower=0.0 upper=0.0 effort=0.0 velocity=0.0
- added joint root_joint: type fixed, parent root_link, child body_link0, origin xyz=0 0 0 rpy=0 0 0

Commit message: gazeboにおけるIMUの加速度センサの値を重力加速度のみにして上書き

File: ginko_description/gazebo/urdf/ginko_rviz.urdf (robot description, URDF)
Before this commit: robot ginko_xacro, 49 links, 48 joints
Joints:
- joint imu_joint: origin xyz=-0.09 0 -0.0379 rpy=0 1.5708 0 -> xyz=-0.09 0 -0.0379 rpy=0 0 0

File: ginko_description/gazebo/xacro/sensors/imu.xacro (robot description, xacro)
@@ -19,5 +19,5 @@
 				<axis xyz="0 0 1"/>
 				<limit effort="0.0" lower="0.0" upper="0.0" velocity="0.0"/>
-				<dynamics damping="0.1" friction="0.1"/>
+				<dynamics damping="0.0" friction="0.0"/>
 			</joint>
 			<link name="body_imu_base_link">
@@ -34,8 +34,8 @@
 				<parent link="body_link1"/>
 				<child  link="body_imu_base_link"/>
-			<origin xyz="-0.09 0 -0.0379" rpy="0 0 0"/>
+				<origin xyz="-0.09 0 -0.0379" rpy="0 0 0"/>
 				<axis xyz="0 0 1"/>
 				<limit effort="0.0" lower="0.0" upper="0.0" velocity="0.0"/>
-				<dynamics damping="0.1" friction="0.1"/>
+				<dynamics damping="0.0" friction="0.0"/>
 			</joint>
 		</xacro:if>
@@ -51,5 +51,5 @@
 				<parent link="body_link1"/>
 				<child  link="body_imu_base_link"/>
-				<origin xyz="-0.09 0 -0.0379" rpy="0 1.5708 0"/>
+				<origin xyz="-0.09 0 -0.0379" rpy="0 0 0"/>
 			</joint>
 		</xacro:if>
@@ -57,6 +57,6 @@
 			<plugin name="imu_plugin" filename="libgazebo_ros_imu.so">
 				<alwaysOn>true</alwaysOn>
-				<bodyName>body_imu_base_link</bodyName>
-				<topicName>/sensor/imu/raw/data</topicName>
+				<bodyName>body_imu_attached_link</bodyName>
+				<topicName>/sensor/imu/raw/gazebo</topicName>
 				<serviceName>gazebo_imu_service</serviceName>
 				<gaussianNoise>0.0</gaussianNoise>
