Commit message: 左足モデルを作成

File: ginko_description/gazebo/transmission/default_gazebo_params.xacro (robot description, xacro)
@@ -34,9 +34,9 @@
 			<kd>100.0</kd>
 			<mu1>${friction}</mu1>
-			<maxVel>3.0</maxVel>
+			<maxVel>10.0</maxVel>
 			<minDepth>0.0001</minDepth>
-			<maxContacts>5</maxContacts>
+			<maxContacts>6</maxContacts>
 			<selfCollide>false</selfCollide>
-			<dampingFactor>0.001</dampingFactor>
+			<dampingFactor>0.00</dampingFactor>
 		</gazebo>
 	</xacro:macro>

File: ginko_description/gazebo/xacro/ginko.xacro (robot description, xacro)
@@ -39,5 +39,9 @@
     <xacro:body_gazebo gazebo_control_mode="${gazebo_control_mode}"/>
     <xacro:leg_r model_mode="${model_mode}"/>
-    <xacro:leg_r_gazebo name="leg_r" gazebo_control_mode="${gazebo_control_mode}"/>
+    <xacro:leg_r_gazebo gazebo_control_mode="${gazebo_control_mode}"/>
+    <xacro:leg_l model_mode="${model_mode}"/>
+    <xacro:leg_l_gazebo gazebo_control_mode="${gazebo_control_mode}"/>
+    <!-- <xacro:leg_l model_mode="${model_mode}"/> -->
+    <!-- <xacro:leg_l_gazebo name="leg_l" gazebo_control_mode="${gazebo_control_mode}"/> -->
 <!--     <xacro:if value="${model_mode=='rviz'}">
       <xacro:leg_r model_mode="common"/>

File: ginko_description/gazebo/xacro/modules/leg_l.xacro (robot description, xacro)
@@ -1,9 +1,15 @@
 <?xml version="1.0"?>
 <robot xmlns:xacro="http://www.ros.org/wiki/xacro">
-	<xacro:macro name="leg_l_sim" params="name parent">
-		<!-- Femoral -->
+	<xacro:macro name="leg_l" params="model_mode">
 		<!-- Link conencts from body. Femoral first. -->
-		<link name="${name}_link0">
-			<!-- Collision created from STL mesh without color -->
+		<joint name="leg_l_joint0" type="revolute">
+		    <parent link="body_link1"/>
+			<child link="leg_l_link0"/>
+			<origin xyz="-0.0404 0.0 -0.0409" rpy="0 0 0"/>
+		    <axis xyz="-1 0 0"/>
+			<limit effort="1000.0" lower="-0.8" upper="1.0" velocity="10.0"/>
+			<dynamics damping="0.1" friction="0.1"/>
+		</joint>
+		<link name="leg_l_link0">
 			<collision>
 				<origin xyz="0 0 0" rpy="0 0 0"/>
@@ -12,5 +18,4 @@
 				</geometry>
 			</collision>
-			<!-- Visualisation created from Color dae -->
 			<visual>
 				<origin xyz="0 0 0" rpy="0 0 0"/>
@@ -28,14 +33,14 @@
 			</inertial>
 		</link>
-		<joint name="${name}_joint0" type="revolute">
-		    <parent link="${parent}"/>
-			<child link="${name}_link0"/>
-			<origin xyz="-0.0404 0.0 -0.0409" rpy="0 0 0"/>
-		    <axis xyz="-1 0 0"/>
-			<limit effort="1000.0" lower="-0.8" upper="1.1781" velocity="10.0"/>
-		</joint>
 		<!-- parallel link (upper-1st) -->
-		<link name="${name}_link1">
-			<!-- Collision created from STL mesh without color -->
+		<joint name="leg_l_joint1" type="revolute">
+			<parent link="leg_l_link0"/>
+			<child  link="leg_l_link1"/>
+			<origin xyz="0.0433 0.0175 -0.0481" rpy="0 0.7854 0"/>
+			<axis xyz="0 -1 0"/>
+			<limit effort="1000.0" lower="-1.3" upper="0.7854" velocity="10.0"/>
+			<dynamics damping="0.1" friction="0.1"/>
+		</joint>
+		<link name="leg_l_link1">
 			<collision>
 				<origin xyz="0 0 0" rpy="0 0 0"/>
@@ -44,5 +49,4 @@
 	    		</geometry>
 			</collision>
-			<!-- Visualisation created from Color dae -->
 			<visual>
 				<origin xyz="0 0 0" rpy="0 0 0"/>
@@ -60,14 +64,28 @@
 			</inertial>
 		</link>
-		<joint name="${name}_joint1" type="revolute">
-			<parent link="${name}_link0"/>
-			<child  link="${name}_link1"/>
-			<origin xyz="0.0433 0.0175 -0.0481" rpy="0 0.7854 0"/>
+		<joint name="leg_l_joint3" type="revolute">
+	    	<parent link="leg_l_link1"/>
+	    	<child  link="leg_l_link3"/>
+	    	<origin xyz="0.1 0.0 0.0" rpy="0 -0.7854 0"/>
+	    	<axis xyz="0 1 0"/>
+			<limit effort="1000.0" lower="-1.3" upper="0.7854" velocity="10.0"/>
+			<dynamics damping="0.1" friction="0.1"/>
+			<xacro:if value="${model_mode=='rviz'}">
+				<mimic joint="leg_l_joint1" multiplier="1" offset="0"/>
+			</xacro:if>
+	  	</joint>
+		<!-- parallel link (upper-2nd) -->
+		<joint name="leg_l_joint2" type="revolute">
+			<parent link="leg_l_link0"/>
+			<child  link="leg_l_link2"/>
+			<origin xyz="0.022 0.0175 -0.06015" rpy="0 0.7854 0"/>
 			<axis xyz="0 -1 0"/>
 			<limit effort="1000.0" lower="-1.3" upper="0.7854" velocity="10.0"/>
-		</joint>
-		<!-- parallel link (upper-2nd) -->
-		<link name="${name}_link2">
-			<!-- Collision created from STL mesh without color -->
+			<dynamics damping="0.1" friction="0.1"/>
+			<xacro:if value="${model_mode=='rviz'}">
+				<mimic joint="leg_l_joint1" multiplier="1" offset="0"/>
+    		</xacro:if>
+		</joint>
+		<link name="leg_l_link2">
 	    	<collision>
 				<origin xyz="0 0 0" rpy="0 0 0"/>
@@ -76,5 +94,4 @@
 	    		</geometry>
 			</collision>
-			<!-- Visualisation created from Color dae -->
 			<visual>
 				<origin xyz="0 0 0" rpy="0 0 0"/>
@@ -92,14 +109,27 @@
 			</inertial>
 		</link>
-		<joint name="${name}_joint2" type="revolute">
-	    	<parent link="${name}_link0"/>
-	    	<child  link="${name}_link2"/>
-	    	<origin xyz="0.022 0.0175 -0.06015" rpy="0 0.7854 0"/>
-	    	<axis xyz="0 -1 0"/>
-	    	<limit effort="1000.0" lower="-3.141593" upper="3.141593" velocity="10.0"/>
-			<mimic joint="${name}_joint1" multiplier="1" offset="0"/>
-	  	</joint>
+		<joint name="close_leg_l_joint0" type="revolute">
+			<parent link="leg_l_link2"/>
+			<child  link="dummy0_leg_l_link3"/>
+			<origin xyz="0.1 0.0 0.0" rpy="0 -0.7854 0"/>
+			<axis xyz="0 1 0"/>
+			<limit effort="1000.0" lower="-1.3" upper="0.7854" velocity="10.0"/>
+			<dynamics damping="0.0" friction="0.0"/>
+			<xacro:if value="${model_mode=='rviz'}">
+				<mimic joint="leg_l_joint1" multiplier="1" offset="0"/>
+			</xacro:if>
+		</joint>
+		<link name="dummy0_leg_l_link3">
+			<inertial>
+				<mass value="0.00001"/>
+				<origin xyz="-0.021 0 -0.012" rpy="0 0 0"/>
+				<inertia
+					ixx="0.00000001"
+					ixy="0.00000000" iyy="0.00000001"
+					ixz="0.00000000" iyz="0.00000000" izz="0.00000001"/>
+			</inertial>
+		</link>
 		<!-- knee -->
-		<link name="${name}_link3">
+		<link name="leg_l_link3">
 	    	<collision>
 				<origin xyz="0 0 0" rpy="0 0 0"/>
@@ -123,14 +153,101 @@
 			</inertial>
 		</link>
-		<joint name="${name}_joint3" type="revolute">
-	    	<parent link="${name}_link1"/>
-	    	<child  link="${name}_link3"/>
-	    	<origin xyz="0.1 0.0 0.0" rpy="0 -0.7854 0"/>
-	    	<axis xyz="0 1 0"/>
-	    	<limit effort="1000.0" lower="-3.141593" upper="3.141593" velocity="10.0"/>
-			<mimic joint="${name}_joint1" multiplier="1" offset="0"/>
-	  	</joint>
+	  	<!-- spring -->
+		<xacro:if value="${model_mode!='rviz'}">
+			<joint name="leg_l_spring_joint0" type="revolute">
+		    	<parent link="leg_l_link0"/>
+		    	<child  link="leg_l_spring0_link0"/>
+		    	<origin xyz="0.022 0.0755 -0.06015" rpy="0 0.56756754 0"/>
+		    	<axis xyz="0 -1 0"/>
+				<dynamics damping="0.0" friction="0.0"/>
+		    	<limit effort="0.0" lower="-3.141593" upper="3.141593" velocity="10.0"/>
+		  	</joint>
+		  	<link name="leg_l_spring0_link0">
+		    	<collision>
+					<origin xyz="0 0 0" rpy="0 0 0"/>
+		    		<geometry>
+						<!-- <mesh filename="package://ginko_description/meshes/stl/spring1.stl"/> -->
+		    		</geometry>
+				</collision>
+		    	<visual>
+					<origin xyz="0 0 0" rpy="0 0 0"/>
+		    		<geometry>
+						<mesh filename="package://ginko_description/meshes/stl/spring1.stl"/>
+		    		</geometry>
+					<material name="spring">
+						<color rgba="0.5 0.5 0.5 1.0"/>
+					</material>
+				</visual>
+				<inertial>
+					<mass value="0.00143865"/>
+					<origin xyz="0.03091683 0.0 0.0" rpy="0 0 0"/>
+					<inertia
+						ixx="0.00000001"
+						ixy="0.00000000" iyy="0.00000060"
+						ixz="0.00000000" iyz="0.00000000" izz="0.00000060"/>
+				</inertial>
+			</link>
+			<joint name="spring0_leg_l_joint" type="prismatic">
+				<parent link="leg_l_spring0_link0"/>
+				<child  link="leg_l_spring0_link1"/>
+				<origin xyz="0.10911938 0.0 0.0" rpy="0 3.141593 0"/>
+				<axis xyz="1 0 0"/>
+				<limit effort="1000.0" lower="-0.03" upper="0.06" velocity="10.0"/>
+				<dynamics damping="0.0" friction="0.0"/>
+			</joint>
+		  	<link name="leg_l_spring0_link1">
+		    	<collision>
+					<origin xyz="0 0 0" rpy="0 0 0"/>
+		    		<geometry>
+						<!-- <mesh filename="package://ginko_description/meshes/stl/spring2.stl"/> -->
+		    		</geometry>
+				</collision>
+		    	<visual>
+					<origin xyz="0 0 0" rpy="0 0 0"/>
+		    		<geometry>
+						<mesh filename="package://ginko_description/meshes/stl/spring2.stl"/>
+		    		</geometry>
+					<material name="spring">
+						<color rgba="0.5 0.5 0.5 1.0"/>
+					</material>
+				</visual>
+				<inertial>
+					<mass value="0.00143865"/>
+					<origin xyz="0.03091683 0.0 0.0" rpy="0 0 0"/>
+					<inertia
+						ixx="0.00000001"
+						ixy="0.00000000" iyy="0.00000060"
+						ixz="0.00000000" iyz="0.00000000" izz="0.00000060"/>
+				</inertial>
+			</link>
+			<joint name="close_leg_l_spring0_joint2" type="revolute">
+				<parent link="leg_l_spring0_link1"/>
+				<child  link="dummy1_leg_l_link3"/>
+				<origin xyz="0 0 0" rpy="0 0 0"/>
+				<axis xyz="0 -1 0"/>
+				<limit effort="0.0" lower="-3.141593" upper="3.141593" velocity="10.0"/>
+				<dynamics damping="0.0" friction="0.0"/>
+			</joint>
+			<link name="dummy1_leg_l_link3">
+				<inertial>
+					<mass value="0.00001"/>
+					<origin xyz="0 0.058 0" rpy="0 0 0"/>
+					<inertia
+						ixx="0.00000001"
+						ixy="0.00000000" iyy="0.00000001"
+						ixz="0.00000000" iyz="0.00000000" izz="0.00000001"/>
+				</inertial>
+			</link>
+		</xacro:if>
 		<!-- parallel link (lower-1st) -->
-		<link name="${name}_link4">
+		<joint name="leg_l_joint4" type="revolute">
+			<parent link="leg_l_link3"/>
+			<child  link="leg_l_link4"/>
+			<origin xyz="0 0 -0.0386" rpy="0 2.3562 0"/>
+			<axis xyz="0 -1 0"/>
+			<limit effort="1000.0" lower="-0.7854" upper="1.3" velocity="10.0"/>
+			<dynamics damping="0.1" friction="0.1"/>
+		</joint>
+		<link name="leg_l_link4">
 			<collision>
 				<origin xyz="0 0 0" rpy="0 0 0"/>
@@ -154,13 +271,28 @@
 			</inertial>
 		</link>
-		<joint name="${name}_joint4" type="revolute">
-			<parent link="${name}_link3"/>
-			<child  link="${name}_link4"/>
-			<origin xyz="0 0 -0.0386" rpy="0 2.3562 0"/>
+		<joint name="leg_l_joint6" type="revolute">
+	    	<parent link="leg_l_link4"/>
+	    	<child  link="leg_l_link6"/>
+	    	<origin xyz="0.1 0.0 0.0" rpy="0 -2.3562 0"/>
+	    	<axis xyz="0 1 0"/>
+			<limit effort="1000.0" lower="-0.7854" upper="1.3" velocity="10.0"/>
+			<dynamics damping="0.1" friction="0.1"/>
+			<xacro:if value="${model_mode=='rviz'}">
+	    		<mimic joint="leg_l_joint4" multiplier="1" offset="0"/>
+			</xacro:if>
+		</joint>
+		<!-- parallel link (lower-2nd) -->
+		<joint name="leg_l_joint5" type="revolute">
+			<parent link="leg_l_link3"/>
+			<child  link="leg_l_link5"/>
+			<origin xyz="-0.0213 0 -0.02655" rpy="0 2.3562 0"/>
 			<axis xyz="0 -1 0"/>
-			<limit effort="1000.0" lower="-0.7854" upper="1.3" velocity="10.0"/>
-		</joint>
-		<!-- parallel link (lower-2nd) -->
-		<link name="${name}_link5">
+			<limit effort="0.0" lower="-0.7854" upper="1.3" velocity="10.0"/>
+			<dynamics damping="0.0" friction="0.0"/>
+			<xacro:if value="${model_mode=='rviz'}">
+				<mimic joint="leg_l_joint4" multiplier="1" offset="0"/>
+			</xacro:if>
+		</joint>
+		<link name="leg_l_link5">
 	    	<collision>
 				<origin xyz="0 0 0" rpy="0 0 0"/>
@@ -184,14 +316,114 @@
 			</inertial>
 		</link>
-		<joint name="${name}_joint5" type="revolute">
-	    	<parent link="${name}_link3"/>
-	    	<child  link="${name}_link5"/>
-	    	<origin xyz="-0.0213 0 -0.02655" rpy="0 2.3562 0"/>
-	    	<axis xyz="0 -1 0"/>
-	    	<limit effort="1000.0" lower="-3.141593" upper="3.141593" velocity="10.0"/>
-	    	<mimic joint="${name}_joint4" multiplier="1" offset="0"/>
-	  	</joint>
+		<joint name="close_leg_l_joint1" type="revolute">
+			<parent link="leg_l_link5"/>
+			<child  link="dummy2_leg_l_link6"/>
+			<origin xyz="0.1 0.0 0.0" rpy="0 -2.3562 0"/>
+			<axis xyz="0 1 0"/>
+			<limit effort="0.0" lower="-1.3" upper="0.7854" velocity="10.0"/>
+			<dynamics damping="0.0" friction="0.0"/>
+			<xacro:if value="${model_mode=='rviz'}">
+				<mimic joint="leg_l_joint4" multiplier="1" offset="0"/>
+			</xacro:if>
+		</joint>
+		<link name="dummy2_leg_l_link6">
+			<inertial>
+				<mass value="0.00001"/>
+				<origin xyz="-0.021 0 0.012" rpy="0 0 0"/>
+				<inertia
+					ixx="0.00000001"
+					ixy="0.00000000" iyy="0.00000001"
+					ixz="0.00000000" iyz="0.00000000" izz="0.00000001"/>
+			</inertial>
+		</link>
+	  	<!-- spring -->
+		<xacro:if value="${model_mode!='rviz'}">
+			<joint name="leg_l_spring1_joint0" type="revolute">
+				<parent link="leg_l_link3"/>
+				<child  link="leg_l_spring1_link0"/>
+				<origin xyz="0 0.058 -0.0386" rpy="0 2.574025114 0"/>
+				<axis xyz="0 -1 0"/>
+				<limit effort="0.0" lower="-3.141593" upper="3.141593" velocity="10.0"/>
+				<dynamics damping="0.0" friction="0.0"/>
+			</joint>
+			<link name="leg_l_spring1_link0">
+				<collision>
+					<origin xyz="0 0 0" rpy="0 0 0"/>
+					<geometry>
+						<!-- <mesh filename="package://ginko_description/meshes/stl/spring1.stl"/> -->
+					</geometry>
+				</collision>
+				<visual>
+					<origin xyz="0 0 0" rpy="0 0 0"/>
+					<geometry>
+						<mesh filename="package://ginko_description/meshes/stl/spring1.stl"/>
+					</geometry>
+					<material name="spring">
+						<color rgba="0.5 0.5 0.5 1.0"/>
+					</material>
+				</visual>
+				<inertial>
+					<mass value="0.00143865"/>
+					<origin xyz="0.03091683 0.0 0.0" rpy="0 2.138363867 0"/>
+					<inertia
+						ixx="0.00000001"
+						ixy="0.00000000" iyy="0.00000060"
+						ixz="0.00000000" iyz="0.00000000" izz="0.00000060"/>
+				</inertial>
+			</link>
+			<joint name="spring1_leg_l_joint" type="prismatic">
+				<parent link="leg_l_spring1_link0"/>
+				<child  link="leg_l_spring1_link1"/>
+				<origin xyz="0.10911938 0.0 0.0" rpy="0 3.141593 0"/>
+				<axis xyz="1 0 0"/>
+				<limit effort="1000.0" lower="-0.03" upper="0.06" velocity="10.0"/>
+				<dynamics damping="0.0" friction="0.0"/>
+			</joint>
+			<link name="leg_l_spring1_link1">
+				<collision>
+					<origin xyz="0 0 0" rpy="0 0 0"/>
+					<geometry>
+						<!-- <mesh filename="package://ginko_description/meshes/stl/spring2.stl"/> -->
+					</geometry>
+				</collision>
+				<visual>
+					<origin xyz="0 0 0" rpy="0 0 0"/>
+					<geometry>
+						<mesh filename="package://ginko_description/meshes/stl/spring2.stl"/>
+					</geometry>
+					<material name="spring">
+						<color rgba="0.5 0.5 0.5 1.0"/>
+					</material>
+				</visual>
+				<inertial>
+					<mass value="0.00143865"/>
+					<origin xyz="0.03091683 0.0 0.0" rpy="0 0 0"/>
+					<inertia
+						ixx="0.00000001"
+						ixy="0.00000000" iyy="0.00000060"
+						ixz="0.00000000" iyz="0.00000000" izz="0.00000060"/>
+				</inertial>
+			</link>
+			<joint name="close_leg_l_spring1_joint2" type="revolute">
+				<parent link="leg_l_spring1_link1"/>
+				<child  link="dummy3_leg_l_link6"/>
+				<origin xyz="0 0 0" rpy="0 0 0"/>
+				<axis xyz="0 -1 0"/>
+				<limit effort="0.0" lower="-3.141593" upper="3.141593" velocity="10.0"/>
+				<dynamics damping="0.0" friction="0.0"/>
+			</joint>
+			<link name="dummy3_leg_l_link6">
+				<inertial>
+					<mass value="0.00001"/>
+					<origin xyz="-0.021 0.058 0.012" rpy="0 0 0"/>
+					<inertia
+						ixx="0.00000001"
+						ixy="0.00000000" iyy="0.00000001"
+						ixz="0.00000000" iyz="0.00000000" izz="0.00000001"/>
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
File: ginko_description/gazebo/xacro/modules/leg_r.xacro (robot description, xacro)
@@ -82,4 +82,5 @@
 			<axis xyz="0 1 0"/>
 			<limit effort="1000.0" lower="-0.7854" upper="1.3" velocity="10.0"/>
+			<dynamics damping="0.0" friction="0.0"/>
 			<xacro:if value="${model_mode=='rviz'}">
 				<mimic joint="leg_r_joint1" multiplier="1" offset="0"/>
@@ -114,4 +115,5 @@
 			<axis xyz="0 -1 0"/>
 			<limit effort="1000.0" lower="-0.7854" upper="1.3" velocity="10.0"/>
+			<dynamics damping="0.0" friction="0.0"/>
 			<xacro:if value="${model_mode=='rviz'}">
 				<mimic joint="leg_r_joint1" multiplier="1" offset="0"/>
@@ -158,4 +160,5 @@
 				<origin xyz="-0.0389 -0.0755 -0.06015" rpy="0 0.56756754 0"/>
 				<axis xyz="0 -1 0"/>
+				<dynamics damping="0.0" friction="0.0"/>
 				<limit effort="0.0" lower="-3.141593" upper="3.141593" velocity="10.0"/>
 			</joint>
@@ -164,5 +167,5 @@
 					<origin xyz="0 0 0" rpy="0 0 0"/>
 					<geometry>
-						<mesh filename="package://ginko_description/meshes/stl/spring1.stl"/>
+						<!-- <mesh filename="package://ginko_description/meshes/stl/spring1.stl"/> -->
 					</geometry>
 				</collision>
@@ -190,5 +193,5 @@
 				<origin xyz="0.10911938 0.0 0.0" rpy="0 3.141593 0"/>
 				<axis xyz="1 0 0"/>
-				<limit effort="1000.0" lower="-0.035" upper="0.055" velocity="10.0"/>
+				<limit effort="1000.0" lower="-0.03" upper="0.06" velocity="10.0"/>
 				<dynamics damping="0.0" friction="0.0"/>
 			</joint>
@@ -197,7 +200,6 @@
 					<origin xyz="0 0 0" rpy="0 0 0"/>
 		    		<geometry>
-						<mesh filename="package://ginko_description/meshes/stl/spring2.stl"/>
+						<!-- <mesh filename="package://ginko_description/meshes/stl/spring2.stl"/> -->
 		    		</geometry>
-					<color rgba="1.0 1.0 1.0 0.5"/>
 				</collision>
 		    	<visual>
@@ -225,4 +227,5 @@
 				<axis xyz="0 -1 0"/>
 				<limit effort="0.0" lower="-3.141593" upper="3.141593" velocity="10.0"/>
+				<dynamics damping="0.0" friction="0.0"/>
 			</joint>
 			<link name="dummy1_leg_r_link3">
@@ -286,4 +289,5 @@
 			<axis xyz="0 1 0"/>
 			<limit effort="0.0" lower="-1.3" upper="0.7854" velocity="10.0"/>
+			<dynamics damping="0.0" friction="0.0"/>
 			<xacro:if value="${model_mode=='rviz'}">
 				<mimic joint="leg_r_joint4" multiplier="1" offset="0"/>
@@ -318,4 +322,5 @@
 			<axis xyz="0 -1 0"/>
 			<limit effort="0.0" lower="-1.3" upper="0.7854" velocity="10.0"/>
+			<dynamics damping="0.0" friction="0.0"/>
 			<xacro:if value="${model_mode=='rviz'}">
 				<mimic joint="leg_r_joint4" multiplier="1" offset="0"/>
@@ -340,4 +345,5 @@
 				<axis xyz="0 -1 0"/>
 				<limit effort="0.0" lower="-3.141593" upper="3.141593" velocity="10.0"/>
+				<dynamics damping="0.0" friction="0.0"/>
 			</joint>
 			<link name="leg_r_spring1_link0">
@@ -345,5 +351,5 @@
 					<origin xyz="0 0 0" rpy="0 0 0"/>
 					<geometry>
-						<mesh filename="package://ginko_description/meshes/stl/spring1.stl"/>
+						<!-- <mesh filename="package://ginko_description/meshes/stl/spring1.stl"/> -->
 					</geometry>
 				</collision>
@@ -371,5 +377,5 @@
 				<origin xyz="0.10911938 0.0 0.0" rpy="0 3.141593 0"/>
 				<axis xyz="1 0 0"/>
-				<limit effort="1000.0" lower="-0.035" upper="0.055" velocity="10.0"/>
+				<limit effort="1000.0" lower="-0.03" upper="0.06" velocity="10.0"/>
 				<dynamics damping="0.0" friction="0.0"/>
 			</joint>
@@ -378,5 +384,5 @@
 					<origin xyz="0 0 0" rpy="0 0 0"/>
 					<geometry>
-						<mesh filename="package://ginko_description/meshes/stl/spring2.stl"/>
+						<!-- <mesh filename="package://ginko_description/meshes/stl/spring2.stl"/> -->
 					</geometry>
 				</collision>
@@ -405,4 +411,5 @@
 				<axis xyz="0 -1 0"/>
 				<limit effort="0.0" lower="-3.141593" upper="3.141593" velocity="10.0"/>
+				<dynamics damping="0.0" friction="0.0"/>
 			</joint>
 			<link name="dummy3_leg_r_link6">
@@ -440,4 +447,12 @@
 			</inertial>
 		</link>
+		<joint name="leg_r_joint7" type="revolute">
+			<parent link="leg_r_link6"/>
+			<child  link="leg_r_link7"/>
+			<origin xyz="-0.028 -0.02475 -0.0391" rpy="0 0 0"/>
+			<axis xyz="-1 0 0"/>
+			<limit effort="1000.0" lower="-1.6" upper="1.6" velocity="10.0"/>
+			<dynamics damping="0.1" friction="0.1"/>
+		</joint>
 		<link name="leg_r_link7">
 	    	<collision>
@@ -462,11 +477,12 @@
 			</inertial>
 		</link>
-		<joint name="leg_r_joint7" type="revolute">
-	    	<parent link="leg_r_link6"/>
-	    	<child  link="leg_r_link7"/>
-	    	<origin xyz="-0.028 -0.02475 -0.0391" rpy="0 0 0"/>
-	    	<axis xyz="-1 0 0"/>
-	    	<limit effort="1000.0" lower="-1.6" upper="1.6" velocity="10.0"/>
-	  	</joint>
+		<joint name="leg_r_joint8" type="revolute">
+			<parent link="leg_r_link7"/>
+			<child  link="leg_r_link8"/>
+			<origin xyz="0.0342 0 -0.04" rpy="0 0 0"/>
+			<axis xyz="0 0 1"/>
+			<limit effort="1000.0" lower="-2.6" upper="2.6" velocity="10.0"/>
+			<dynamics damping="0.1" friction="0.1"/>
+		</joint>
 		<link name="leg_r_link8">
 			<collision>
@@ -491,11 +507,4 @@
 			</inertial>
 		</link>
-		<joint name="leg_r_joint8" type="revolute">
-	    	<parent link="leg_r_link7"/>
-	    	<child  link="leg_r_link8"/>
-	    	<origin xyz="0.0342 0 -0.04" rpy="0 0 0"/>
-	    	<axis xyz="0 0 1"/>
-	    	<limit effort="1000.0" lower="-2.6" upper="2.6" velocity="10.0"/>
-	  	</joint>
 	</xacro:macro>
 </robot>
