Commit message: Testing gazebo_dc_motor

File: ginko_description/gazebo/transmission/default_gazebo_params.xacro (robot description, xacro)
@@ -1,27 +1,30 @@
 <?xml version="1.0"?>
 <robot xmlns:xacro="http://www.ros.org/wiki/xacro">
-	<xacro:macro name="default_motor_transmission" params="joint_name gazebo_control_mode">
+	<xacro:macro name="default_motor_transmission" params="joint_name gazebo_hw_interface">
+		<gazebo reference="${joint_name}">
+  		<implicitSpringDamper>1</implicitSpringDamper>
+		</gazebo>
 		<transmission name="${joint_name}_trans">
 			<type>transmission_interface/SimpleTransmission</type>
 			<joint name="${joint_name}">
-				<xacro:if value="${gazebo_control_mode=='ginko'}">
-					<hardwareInterface>PositionDutyPidMotorInterface</hardwareInterface>
+				<xacro:if value="${gazebo_hw_interface=='ginko'}">
+					<hardwareInterface>hardware_interface/PositionDutyPidMotorInterface</hardwareInterface>
 				</xacro:if>
-				<xacro:if value="${gazebo_control_mode=='effort'}">
-					<hardwareInterface>EffortJointInterface</hardwareInterface>
+				<xacro:if value="${gazebo_hw_interface=='effort'}">
+					<hardwareInterface>hardware_interface/EffortJointInterface</hardwareInterface>
 				</xacro:if>
-				<xacro:if value="${gazebo_control_mode=='position'}">
-					<hardwareInterface>PositionJointInterface</hardwareInterface>
+				<xacro:if value="${gazebo_hw_interface=='position'}">
+					<hardwareInterface>hardware_interface/PositionJointInterface</hardwareInterface>
 				</xacro:if>
 			</joint>
 			<actuator name="${joint_name}_motor">
-				<xacro:if value="${gazebo_control_mode=='ginko'}">
-					<hardwareInterface>PositionDutyPidMotorInterface</hardwareInterface>
+				<xacro:if value="${gazebo_hw_interface=='ginko'}">
+					<hardwareInterface>hardware_interface/PositionDutyPidMotorInterface</hardwareInterface>
 				</xacro:if>
-				<xacro:if value="${gazebo_control_mode=='effort'}">
-					<hardwareInterface>EffortJointInterface</hardwareInterface>
+				<xacro:if value="${gazebo_hw_interface=='effort'}">
+					<hardwareInterface>hardware_interface/EffortJointInterface</hardwareInterface>
 				</xacro:if>
-				<xacro:if value="${gazebo_control_mode=='position'}">
-					<hardwareInterface>PositionJointInterface</hardwareInterface>
+				<xacro:if value="${gazebo_hw_interface=='position'}">
+          <hardwareInterface>hardware_interface/PositionJointInterface</hardwareInterface>
 				</xacro:if>
 				<mechanicalReduction>1</mechanicalReduction>

File: ginko_description/gazebo/xacro/ginko.xacro (robot description, xacro)
@@ -1,6 +1,8 @@
 <?xml version="1.0"?>
-<robot name="ginko_xacro" xmlns:xacro="http://www.ros.org/wiki/xacro">
+<robot name="ginko" xmlns:xacro="http://www.ros.org/wiki/xacro">
   <xacro:arg name="model_mode" default="rviz"/>
-  <xacro:arg name="gazebo_control_mode" default="ginko"/>
+  <xacro:arg name="gazebo_motor_model" default="dc"/>
+  <!-- <xacro:arg name="gazebo_motor_model" default="ginko"/> -->
+  <xacro:arg name="gazebo_hw_interface" default="position"/>
   <xacro:include filename="$(find ginko_description)/gazebo/xacro/sensors/imu.xacro"/>
   <xacro:include filename="$(find ginko_description)/gazebo/xacro/sensors/urg.xacro"/>
@@ -16,6 +18,6 @@
   <xacro:include filename="$(find ginko_description)/gazebo/transmission/leg_r.gazebo"/>
   <!-- MACRO:Loading Gazebo Controllers for joints -->
-  <xacro:macro name="gazebo_plugin_xacro" params="gazebo_control_mode">
-    <xacro:if value="${gazebo_control_mode=='ginko'}">
+  <xacro:macro name="gazebo_plugin_xacro" params="gazebo_motor_model">
+    <xacro:if value="${gazebo_motor_model=='ginko'}">
       <gazebo>
         <plugin name="gazebo_ros_control" filename="libgazebo_ros_control.so">
@@ -26,5 +28,5 @@
       </gazebo>
     </xacro:if>
-    <xacro:if value="${gazebo_control_mode!='ginko'}">
+    <xacro:if value="${gazebo_motor_model=='default'}">
       <gazebo>
         <plugin name="gazebo_ros_control" filename="libgazebo_ros_control.so">
@@ -35,7 +37,16 @@
       </gazebo>
     </xacro:if>
+    <xacro:if value="${gazebo_motor_model=='dc'}">
+      <gazebo>
+        <plugin name="gazebo_ros_control" filename="libgazebo_dc_motor.so">
+          <robotNamespace>ginko</robotNamespace>
+          <robotSimType>gazebo_dc_motor/DefaultRobotHWSim</robotSimType>
+          <legacyModeNS>false</legacyModeNS>
+        </plugin>
+      </gazebo>
+    </xacro:if>
   </xacro:macro>
   <!-- MACRO:Setting up a Robot Model -->
-  <xacro:macro name="ginko_xacro" params="model_mode gazebo_control_mode">
+  <xacro:macro name="ginko_xacro" params="model_mode gazebo_hw_interface">
     <link name="root_link"/>
     <joint name="root_joint" type="fixed">
@@ -45,17 +56,17 @@
     </joint>
     <xacro:body_xacro model_mode="${model_mode}"/>
-    <xacro:body_gazebo gazebo_control_mode="${gazebo_control_mode}"/>
+    <xacro:body_gazebo gazebo_hw_interface="${gazebo_hw_interface}"/>
     <xacro:leg_r model_mode="${model_mode}"/>
-    <xacro:leg_r_gazebo gazebo_control_mode="${gazebo_control_mode}"/>
+    <xacro:leg_r_gazebo gazebo_hw_interface="${gazebo_hw_interface}"/>
     <xacro:leg_l model_mode="${model_mode}"/>
-    <xacro:leg_l_gazebo gazebo_control_mode="${gazebo_control_mode}"/>
+    <xacro:leg_l_gazebo gazebo_hw_interface="${gazebo_hw_interface}"/>
     <xacro:arm_r model_mode="${model_mode}"/>
-    <xacro:arm_r_gazebo gazebo_control_mode="${gazebo_control_mode}"/>
+    <xacro:arm_r_gazebo gazebo_hw_interface="${gazebo_hw_interface}"/>
     <xacro:arm_l model_mode="${model_mode}"/>
-    <xacro:arm_l_gazebo gazebo_control_mode="${gazebo_control_mode}"/>
+    <xacro:arm_l_gazebo gazebo_hw_interface="${gazebo_hw_interface}"/>
   </xacro:macro>
   <!-- Load Macros -->
-  <xacro:ginko_xacro model_mode="$(arg model_mode)" gazebo_control_mode="$(arg gazebo_control_mode)"/>
-  <xacro:gazebo_plugin_xacro gazebo_control_mode="$(arg gazebo_control_mode)"/>
+  <xacro:ginko_xacro model_mode="$(arg model_mode)" gazebo_hw_interface="$(arg gazebo_hw_interface)"/>
+  <xacro:gazebo_plugin_xacro gazebo_motor_model="$(arg gazebo_motor_model)"/>
   <xacro:imu_xacro model_mode="$(arg model_mode)"/>
   <xacro:urg_xacro firame_id="arm_r_urg_link" topic_name="/sensor/urg/right/scan_raw" sensor_name="urg_right"/>
