Commit message: refactoring file path

File: ginko_description/xacro/ginko_rs406/parts/arm_l.xacro (robot description, xacro)
@@ -15,5 +15,5 @@
 				<origin xyz="0 0 0" rpy="0 0 0"/>
 				<geometry>
-					<mesh filename="package://ginko_description/meshes/stl/link09_l_arm01.stl"/>
+					<mesh filename="package://ginko_description/meshes/ginko_rs406/stl/link09_l_arm01.stl"/>
 				</geometry>
 			</collision>
@@ -21,5 +21,5 @@
 				<origin xyz="0 0 0" rpy="0 0 0"/>
 				<geometry>
-					<mesh filename="package://ginko_description/meshes/obj/link09_l_arm01.obj"/>
+					<mesh filename="package://ginko_description/meshes/ginko_rs406/obj/link09_l_arm01.obj"/>
 				</geometry>
 			</visual>
@@ -46,5 +46,5 @@
 				<origin xyz="0 0 0" rpy="0 0 0"/>
 	    		<geometry>
-					<mesh filename="package://ginko_description/meshes/stl/link10_l_arm02.stl"/>
+					<mesh filename="package://ginko_description/meshes/ginko_rs406/stl/link10_l_arm02.stl"/>
 	    		</geometry>
 			</collision>
@@ -52,5 +52,5 @@
 				<origin xyz="0 0 0" rpy="0 0 0"/>
 				<geometry>
-					<mesh filename="package://ginko_description/meshes/obj/link10_l_arm02.obj"/>
+					<mesh filename="package://ginko_description/meshes/ginko_rs406/obj/link10_l_arm02.obj"/>
 				</geometry>
 			</visual>
@@ -95,5 +95,5 @@
 				<origin xyz="0 0 0" rpy="0 0 0"/>
 	    		<geometry>
-					<mesh filename="package://ginko_description/meshes/stl/link11_l_scissor01.stl"/>
+					<mesh filename="package://ginko_description/meshes/ginko_rs406/stl/link11_l_scissor01.stl"/>
 	    		</geometry>
 			</collision>
@@ -101,5 +101,5 @@
 				<origin xyz="0 0 0" rpy="0 0 0"/>
 				<geometry>
-					<mesh filename="package://ginko_description/meshes/obj/link11_l_scissor01.obj"/>
+					<mesh filename="package://ginko_description/meshes/ginko_rs406/obj/link11_l_scissor01.obj"/>
 				</geometry>
 			</visual>
@@ -125,5 +125,5 @@
 				<origin xyz="0 0 0" rpy="0 0 0"/>
 	    		<geometry>
-					<mesh filename="package://ginko_description/meshes/stl/link12_l_scissor02.stl"/>
+					<mesh filename="package://ginko_description/meshes/ginko_rs406/stl/link12_l_scissor02.stl"/>
 	    		</geometry>
 			</collision>
@@ -131,5 +131,5 @@
 				<origin xyz="0 0 0" rpy="0 0 0"/>
 				<geometry>
-					<mesh filename="package://ginko_description/meshes/obj/link12_l_scissor02.obj"/>
+					<mesh filename="package://ginko_description/meshes/ginko_rs406/obj/link12_l_scissor02.obj"/>
 				</geometry>
 			</visual>
@@ -166,5 +166,5 @@
 				<origin xyz="0 0 0" rpy="0 0 0"/>
 	    		<geometry>
-					<mesh filename="package://ginko_description/meshes/stl/urg.stl"/>
+					<mesh filename="package://ginko_description/meshes/ginko_rs406/stl/urg.stl"/>
 	    		</geometry>
 			</collision>
@@ -172,5 +172,5 @@
 				<origin xyz="0 0 0" rpy="0 0 0"/>
 				<geometry>
-					<mesh filename="package://ginko_description/meshes/obj/urg.obj"/>
+					<mesh filename="package://ginko_description/meshes/ginko_rs406/obj/urg.obj"/>
 				</geometry>
 			</visual>

File: ginko_description/xacro/ginko_rs406/parts/arm_r.xacro (robot description, xacro)
@@ -15,5 +15,5 @@
 				<origin xyz="0 0 0" rpy="0 0 0"/>
 				<geometry>
-					<mesh filename="package://ginko_description/meshes/stl/link09_r_arm01.stl"/>
+					<mesh filename="package://ginko_description/meshes/ginko_rs406/stl/link09_r_arm01.stl"/>
 				</geometry>
 			</collision>
@@ -21,5 +21,5 @@
 				<origin xyz="0 0 0" rpy="0 0 0"/>
 				<geometry>
-					<mesh filename="package://ginko_description/meshes/obj/link09_r_arm01.obj"/>
+					<mesh filename="package://ginko_description/meshes/ginko_rs406/obj/link09_r_arm01.obj"/>
 				</geometry>
 			</visual>
@@ -46,5 +46,5 @@
 				<origin xyz="0 0 0" rpy="0 0 0"/>
 	    		<geometry>
-					<mesh filename="package://ginko_description/meshes/stl/link10_r_arm02.stl"/>
+					<mesh filename="package://ginko_description/meshes/ginko_rs406/stl/link10_r_arm02.stl"/>
 	    		</geometry>
 			</collision>
@@ -52,5 +52,5 @@
 				<origin xyz="0 0 0" rpy="0 0 0"/>
 				<geometry>
-					<mesh filename="package://ginko_description/meshes/obj/link10_r_arm02.obj"/>
+					<mesh filename="package://ginko_description/meshes/ginko_rs406/obj/link10_r_arm02.obj"/>
 				</geometry>
 			</visual>
@@ -95,5 +95,5 @@
 				<origin xyz="0 0 0" rpy="0 0 0"/>
 	    		<geometry>
-					<mesh filename="package://ginko_description/meshes/stl/link11_r_scissor01.stl"/>
+					<mesh filename="package://ginko_description/meshes/ginko_rs406/stl/link11_r_scissor01.stl"/>
 	    		</geometry>
 			</collision>
@@ -101,5 +101,5 @@
 				<origin xyz="0 0 0" rpy="0 0 0"/>
 				<geometry>
-					<mesh filename="package://ginko_description/meshes/obj/link11_r_scissor01.obj"/>
+					<mesh filename="package://ginko_description/meshes/ginko_rs406/obj/link11_r_scissor01.obj"/>
 				</geometry>
 			</visual>
@@ -125,5 +125,5 @@
 				<origin xyz="0 0 0" rpy="0 0 0"/>
 	    		<geometry>
-					<mesh filename="package://ginko_description/meshes/stl/link12_r_scissor02.stl"/>
+					<mesh filename="package://ginko_description/meshes/ginko_rs406/stl/link12_r_scissor02.stl"/>
 	    		</geometry>
 			</collision>
@@ -131,5 +131,5 @@
 				<origin xyz="0 0 0" rpy="0 0 0"/>
 				<geometry>
-					<mesh filename="package://ginko_description/meshes/obj/link12_r_scissor02.obj"/>
+					<mesh filename="package://ginko_description/meshes/ginko_rs406/obj/link12_r_scissor02.obj"/>
 				</geometry>
 			</visual>
@@ -166,5 +166,5 @@
 				<origin xyz="0 0 0" rpy="0 0 0"/>
 	    		<geometry>
-					<mesh filename="package://ginko_description/meshes/stl/urg.stl"/>
+					<mesh filename="package://ginko_description/meshes/ginko_rs406/stl/urg.stl"/>
 	    		</geometry>
 			</collision>
@@ -172,5 +172,5 @@
 				<origin xyz="0 0 0" rpy="0 0 0"/>
 				<geometry>
-					<mesh filename="package://ginko_description/meshes/obj/urg.obj"/>
+					<mesh filename="package://ginko_description/meshes/ginko_rs406/obj/urg.obj"/>
 				</geometry>
 			</visual>

File: ginko_description/xacro/ginko_rs406/parts/body.xacro (robot description, xacro)
@@ -7,5 +7,5 @@
 				<origin xyz="0 0 0" rpy="0 0 0"/>
 				<geometry>
-					<mesh filename="package://ginko_description/meshes/stl/link00_chest.stl"/>
+					<mesh filename="package://ginko_description/meshes/ginko_rs406/stl/link00_chest.stl"/>
 				</geometry>
 			</collision>
@@ -13,5 +13,5 @@
 				<origin xyz="0 0 0" rpy="0 0 0"/>
 				<geometry>
-					<mesh filename="package://ginko_description/meshes/obj/link00_chest.obj"/>
+					<mesh filename="package://ginko_description/meshes/ginko_rs406/obj/link00_chest.obj"/>
 				</geometry>
 			</visual>
@@ -39,5 +39,5 @@
 				<origin xyz="0 0 0" rpy="0 0 0"/>
 	    		<geometry>
-					<mesh filename="package://ginko_description/meshes/stl/link01_waist.stl"/>
+					<mesh filename="package://ginko_description/meshes/ginko_rs406/stl/link01_waist.stl"/>
 	    		</geometry>
 			</collision>
@@ -45,5 +45,5 @@
 				<origin xyz="0 0 0" rpy="0 0 0"/>
 				<geometry>
-					<mesh filename="package://ginko_description/meshes/obj/link01_waist.obj"/>
+					<mesh filename="package://ginko_description/meshes/ginko_rs406/obj/link01_waist.obj"/>
 				</geometry>
 			</visual>

File: ginko_description/xacro/ginko_rs406/parts/leg_l.xacro (robot description, xacro)
@@ -15,11 +15,11 @@
 				<origin xyz="0 0 0" rpy="0 0 0"/>
 				<geometry>
-					<mesh filename="package://ginko_description/meshes/stl/link02_l_femoral.stl"/>
-				</geometry>
-			</collision>
-			<visual>
-				<origin xyz="0 0 0" rpy="0 0 0"/>
-				<geometry>
-					<mesh filename="package://ginko_description/meshes/obj/link02_l_femoral.obj"/>
+					<mesh filename="package://ginko_description/meshes/ginko_rs406/stl/link02_l_femoral.stl"/>
+				</geometry>
+			</collision>
+			<visual>
+				<origin xyz="0 0 0" rpy="0 0 0"/>
+				<geometry>
+					<mesh filename="package://ginko_description/meshes/ginko_rs406/obj/link02_l_femoral.obj"/>
 				</geometry>
 			</visual>
@@ -46,5 +46,5 @@
 				<origin xyz="0 0 0" rpy="0 0 0"/>
 	    		<geometry>
-					<mesh filename="package://ginko_description/meshes/stl/link03_l_leg01.stl"/>
+					<mesh filename="package://ginko_description/meshes/ginko_rs406/stl/link03_l_leg01.stl"/>
 	    		</geometry>
 			</collision>
@@ -52,5 +52,5 @@
 				<origin xyz="0 0 0" rpy="0 0 0"/>
 				<geometry>
-					<mesh filename="package://ginko_description/meshes/obj/link03_l_leg01.obj"/>
+					<mesh filename="package://ginko_description/meshes/ginko_rs406/obj/link03_l_leg01.obj"/>
 				</geometry>
 			</visual>
@@ -91,5 +91,5 @@
 				<origin xyz="0 0 0" rpy="0 0 0"/>
 	    		<geometry>
-					<mesh filename="package://ginko_description/meshes/stl/link04_l_leg02.stl"/>
+					<mesh filename="package://ginko_description/meshes/ginko_rs406/stl/link04_l_leg02.stl"/>
 	    		</geometry>
 			</collision>
@@ -97,5 +97,5 @@
 				<origin xyz="0 0 0" rpy="0 0 0"/>
 				<geometry>
-					<mesh filename="package://ginko_description/meshes/obj/link04_l_leg02.obj"/>
+					<mesh filename="package://ginko_description/meshes/ginko_rs406/obj/link04_l_leg02.obj"/>
 				</geometry>
 			</visual>
@@ -135,5 +135,5 @@
 				<origin xyz="0 0 0" rpy="0 0 0"/>
 	    		<geometry>
-					<mesh filename="package://ginko_description/meshes/stl/link05_l_knee.stl"/>
+					<mesh filename="package://ginko_description/meshes/ginko_rs406/stl/link05_l_knee.stl"/>
 	    		</geometry>
 			</collision>
@@ -141,5 +141,5 @@
 				<origin xyz="0 0 0" rpy="0 0 0"/>
 				<geometry>
-					<mesh filename="package://ginko_description/meshes/obj/link05_l_knee.obj"/>
+					<mesh filename="package://ginko_description/meshes/ginko_rs406/obj/link05_l_knee.obj"/>
 				</geometry>
 			</visual>
@@ -167,5 +167,5 @@
 					<origin xyz="0 0 0" rpy="0 0 0"/>
 		    		<geometry>
-						<mesh filename="package://ginko_description/meshes/stl/spring1.stl"/>
+						<mesh filename="package://ginko_description/meshes/ginko_rs406/stl/spring1.stl"/>
 		    		</geometry>
 				</collision>
@@ -173,5 +173,5 @@
 					<origin xyz="0 0 0" rpy="0 0 0"/>
 		    		<geometry>
-						<mesh filename="package://ginko_description/meshes/stl/spring1.stl"/>
+						<mesh filename="package://ginko_description/meshes/ginko_rs406/stl/spring1.stl"/>
 		    		</geometry>
 					<material name="spring">
@@ -200,5 +200,5 @@
 					<origin xyz="0 0 0" rpy="0 0 0"/>
 		    		<geometry>
-						<mesh filename="package://ginko_description/meshes/stl/spring2.stl"/>
+						<mesh filename="package://ginko_description/meshes/ginko_rs406/stl/spring2.stl"/>
 		    		</geometry>
 				</collision>
@@ -206,5 +206,5 @@
 					<origin xyz="0 0 0" rpy="0 0 0"/>
 		    		<geometry>
-						<mesh filename="package://ginko_description/meshes/stl/spring2.stl"/>
+						<mesh filename="package://ginko_description/meshes/ginko_rs406/stl/spring2.stl"/>
 		    		</geometry>
 					<material name="spring">
@@ -253,5 +253,5 @@
 				<origin xyz="0 0 0" rpy="0 0 0"/>
 	    		<geometry>
-					<mesh filename="package://ginko_description/meshes/stl/link03_l_leg01.stl"/>
+					<mesh filename="package://ginko_description/meshes/ginko_rs406/stl/link03_l_leg01.stl"/>
 	    		</geometry>
 			</collision>
@@ -259,5 +259,5 @@
 				<origin xyz="0 0 0" rpy="0 0 0"/>
 				<geometry>
-					<mesh filename="package://ginko_description/meshes/obj/link03_l_leg01.obj"/>
+					<mesh filename="package://ginko_description/meshes/ginko_rs406/obj/link03_l_leg01.obj"/>
 				</geometry>
 			</visual>
@@ -298,5 +298,5 @@
 				<origin xyz="0 0 0" rpy="0 0 0"/>
 	    		<geometry>
-					<mesh filename="package://ginko_description/meshes/stl/link04_l_leg02.stl"/>
+					<mesh filename="package://ginko_description/meshes/ginko_rs406/stl/link04_l_leg02.stl"/>
 	    		</geometry>
 			</collision>
@@ -304,5 +304,5 @@
 				<origin xyz="0 0 0" rpy="0 0 0"/>
 				<geometry>
-					<mesh filename="package://ginko_description/meshes/obj/link04_l_leg02.obj"/>
+					<mesh filename="package://ginko_description/meshes/ginko_rs406/obj/link04_l_leg02.obj"/>
 				</geometry>
 			</visual>
@@ -351,5 +351,5 @@
 					<origin xyz="0 0 0" rpy="0 0 0"/>
 					<geometry>
-						<mesh filename="package://ginko_description/meshes/stl/spring1.stl"/>
+						<mesh filename="package://ginko_description/meshes/ginko_rs406/stl/spring1.stl"/>
 					</geometry>
 				</collision>
@@ -357,5 +357,5 @@
 					<origin xyz="0 0 0" rpy="0 0 0"/>
 					<geometry>
-						<mesh filename="package://ginko_description/meshes/stl/spring1.stl"/>
+						<mesh filename="package://ginko_description/meshes/ginko_rs406/stl/spring1.stl"/>
 					</geometry>
 					<material name="spring">
@@ -384,5 +384,5 @@
 					<origin xyz="0 0 0" rpy="0 0 0"/>
 					<geometry>
-						<mesh filename="package://ginko_description/meshes/stl/spring2.stl"/>
+						<mesh filename="package://ginko_description/meshes/ginko_rs406/stl/spring2.stl"/>
 					</geometry>
 				</collision>
@@ -390,5 +390,5 @@
 					<origin xyz="0 0 0" rpy="0 0 0"/>
 					<geometry>
-						<mesh filename="package://ginko_description/meshes/stl/spring2.stl"/>
+						<mesh filename="package://ginko_description/meshes/ginko_rs406/stl/spring2.stl"/>
 					</geometry>
 					<material name="spring">
@@ -429,11 +429,11 @@
 				<origin xyz="0 0 0" rpy="0 0 0"/>
 				<geometry>
-					<mesh filename="package://ginko_description/meshes/stl/link06_l_toe01.stl"/>
-				</geometry>
-			</collision>
-			<visual>
-				<origin xyz="0 0 0" rpy="0 0 0"/>
-				<geometry>
-					<mesh filename="package://ginko_description/meshes/obj/link06_l_toe01.obj"/>
+					<mesh filename="package://ginko_description/meshes/ginko_rs406/stl/link06_l_toe01.stl"/>
+				</geometry>
+			</collision>
+			<visual>
+				<origin xyz="0 0 0" rpy="0 0 0"/>
+				<geometry>
+					<mesh filename="package://ginko_description/meshes/ginko_rs406/obj/link06_l_toe01.obj"/>
 				</geometry>
 			</visual>
@@ -459,5 +459,5 @@
 				<origin xyz="0 0 0" rpy="0 0 0"/>
 	    		<geometry>
-					<mesh filename="package://ginko_description/meshes/stl/link07_l_toe02.stl"/>
+					<mesh filename="package://ginko_description/meshes/ginko_rs406/stl/link07_l_toe02.stl"/>
 	    		</geometry>
 			</collision>
@@ -465,5 +465,5 @@
 				<origin xyz="0 0 0" rpy="0 0 0"/>
 				<geometry>
-					<mesh filename="package://ginko_description/meshes/obj/link07_l_toe02.obj"/>
+					<mesh filename="package://ginko_description/meshes/ginko_rs406/obj/link07_l_toe02.obj"/>
 				</geometry>
 			</visual>
@@ -495,5 +495,5 @@
 				<origin xyz="0 0 0" rpy="0 0 0"/>
 				<geometry>
-					<mesh filename="package://ginko_description/meshes/obj/link08_l_toe03.obj"/>
+					<mesh filename="package://ginko_description/meshes/ginko_rs406/obj/link08_l_toe03.obj"/>
 				</geometry>
 			</visual>

File: ginko_description/xacro/ginko_rs406/parts/leg_r.xacro (robot description, xacro)
@@ -15,11 +15,11 @@
 				<origin xyz="0 0 0" rpy="0 0 0"/>
 				<geometry>
-					<mesh filename="package://ginko_description/meshes/stl/link02_r_femoral.stl"/>
-				</geometry>
-			</collision>
-			<visual>
-				<origin xyz="0 0 0" rpy="0 0 0"/>
-				<geometry>
-					<mesh filename="package://ginko_description/meshes/obj/link02_r_femoral.obj"/>
+					<mesh filename="package://ginko_description/meshes/ginko_rs406/stl/link02_r_femoral.stl"/>
+				</geometry>
+			</collision>
+			<visual>
+				<origin xyz="0 0 0" rpy="0 0 0"/>
+				<geometry>
+					<mesh filename="package://ginko_description/meshes/ginko_rs406/obj/link02_r_femoral.obj"/>
 				</geometry>
 			</visual>
@@ -46,5 +46,5 @@
 				<origin xyz="0 0 0" rpy="0 0 0"/>
 	    		<geometry>
-					<mesh filename="package://ginko_description/meshes/stl/link03_r_leg01.stl"/>
+					<mesh filename="package://ginko_description/meshes/ginko_rs406/stl/link03_r_leg01.stl"/>
 	    		</geometry>
 			</collision>
@@ -52,5 +52,5 @@
 				<origin xyz="0 0 0" rpy="0 0 0"/>
 				<geometry>
-					<mesh filename="package://ginko_description/meshes/obj/link03_r_leg01.obj"/>
+					<mesh filename="package://ginko_description/meshes/ginko_rs406/obj/link03_r_leg01.obj"/>
 				</geometry>
 			</visual>
@@ -91,5 +91,5 @@
 				<origin xyz="0 0 0" rpy="0 0 0"/>
 	    		<geometry>
-					<mesh filename="package://ginko_description/meshes/stl/link04_r_leg02.stl"/>
+					<mesh filename="package://ginko_description/meshes/ginko_rs406/stl/link04_r_leg02.stl"/>
 	    		</geometry>
 			</collision>
@@ -97,5 +97,5 @@
 				<origin xyz="0 0 0" rpy="0 0 0"/>
 				<geometry>
-					<mesh filename="package://ginko_description/meshes/obj/link04_r_leg02.obj"/>
+					<mesh filename="package://ginko_description/meshes/ginko_rs406/obj/link04_r_leg02.obj"/>
 				</geometry>
 			</visual>
@@ -135,5 +135,5 @@
 				<origin xyz="0 0 0" rpy="0 0 0"/>
 	    		<geometry>
-					<mesh filename="package://ginko_description/meshes/stl/link05_r_knee.stl"/>
+					<mesh filename="package://ginko_description/meshes/ginko_rs406/stl/link05_r_knee.stl"/>
 	    		</geometry>
 			</collision>
@@ -141,5 +141,5 @@
 				<origin xyz="0 0 0" rpy="0 0 0"/>
 				<geometry>
-					<mesh filename="package://ginko_description/meshes/obj/link05_r_knee.obj"/>
+					<mesh filename="package://ginko_description/meshes/ginko_rs406/obj/link05_r_knee.obj"/>
 				</geometry>
 			</visual>
@@ -167,5 +167,5 @@
 					<origin xyz="0 0 0" rpy="0 0 0"/>
 					<geometry>
-						<mesh filename="package://ginko_description/meshes/stl/spring1.stl"/>
+						<mesh filename="package://ginko_description/meshes/ginko_rs406/stl/spring1.stl"/>
 					</geometry>
 				</collision>
@@ -173,5 +173,5 @@
 					<origin xyz="0 0 0" rpy="0 0 0"/>
 					<geometry>
-						<mesh filename="package://ginko_description/meshes/stl/spring1.stl"/>
+						<mesh filename="package://ginko_description/meshes/ginko_rs406/stl/spring1.stl"/>
 					</geometry>
 					<material name="spring">
@@ -200,5 +200,5 @@
 					<origin xyz="0 0 0" rpy="0 0 0"/>
 		    		<geometry>
-						<mesh filename="package://ginko_description/meshes/stl/spring2.stl"/>
+						<mesh filename="package://ginko_description/meshes/ginko_rs406/stl/spring2.stl"/>
 		    		</geometry>
 				</collision>
@@ -206,5 +206,5 @@
 					<origin xyz="0 0 0" rpy="0 0 0"/>
 		    		<geometry>
-						<mesh filename="package://ginko_description/meshes/stl/spring2.stl"/>
+						<mesh filename="package://ginko_description/meshes/ginko_rs406/stl/spring2.stl"/>
 		    		</geometry>
 					<material name="spring">
@@ -253,5 +253,5 @@
 				<origin xyz="0 0 0" rpy="0 0 0"/>
 	    		<geometry>
-					<mesh filename="package://ginko_description/meshes/stl/link03_r_leg01.stl"/>
+					<mesh filename="package://ginko_description/meshes/ginko_rs406/stl/link03_r_leg01.stl"/>
 	    		</geometry>
 			</collision>
@@ -259,5 +259,5 @@
 				<origin xyz="0 0 0" rpy="0 0 0"/>
 				<geometry>
-					<mesh filename="package://ginko_description/meshes/obj/link03_r_leg01.obj"/>
+					<mesh filename="package://ginko_description/meshes/ginko_rs406/obj/link03_r_leg01.obj"/>
 				</geometry>
 			</visual>
@@ -298,11 +298,11 @@
 				<origin xyz="0 0 0" rpy="0 0 0"/>
 				<geometry>
-					<mesh filename="package://ginko_description/meshes/stl/link04_r_leg02.stl"/>
-				</geometry>
-			</collision>
-			<visual>
-				<origin xyz="0 0 0" rpy="0 0 0"/>
-				<geometry>
-					<mesh filename="package://ginko_description/meshes/obj/link04_r_leg02.obj"/>
+					<mesh filename="package://ginko_description/meshes/ginko_rs406/stl/link04_r_leg02.stl"/>
+				</geometry>
+			</collision>
+			<visual>
+				<origin xyz="0 0 0" rpy="0 0 0"/>
+				<geometry>
+					<mesh filename="package://ginko_description/meshes/ginko_rs406/obj/link04_r_leg02.obj"/>
 				</geometry>
 			</visual>
@@ -351,5 +351,5 @@
 					<origin xyz="0 0 0" rpy="0 0 0"/>
 					<geometry>
-						<mesh filename="package://ginko_description/meshes/stl/spring1.stl"/>
+						<mesh filename="package://ginko_description/meshes/ginko_rs406/stl/spring1.stl"/>
 					</geometry>
 				</collision>
@@ -357,5 +357,5 @@
 					<origin xyz="0 0 0" rpy="0 0 0"/>
 					<geometry>
-						<mesh filename="package://ginko_description/meshes/stl/spring1.stl"/>
+						<mesh filename="package://ginko_description/meshes/ginko_rs406/stl/spring1.stl"/>
 					</geometry>
 					<material name="spring">
@@ -384,5 +384,5 @@
 					<origin xyz="0 0 0" rpy="0 0 0"/>
 					<geometry>
-						<mesh filename="package://ginko_description/meshes/stl/spring2.stl"/>
+						<mesh filename="package://ginko_description/meshes/ginko_rs406/stl/spring2.stl"/>
 					</geometry>
 				</collision>
@@ -390,5 +390,5 @@
 					<origin xyz="0 0 0" rpy="0 0 0"/>
 					<geometry>
-						<mesh filename="package://ginko_description/meshes/stl/spring2.stl"/>
+						<mesh filename="package://ginko_description/meshes/ginko_rs406/stl/spring2.stl"/>
 					</geometry>
 					<material name="spring">
@@ -429,11 +429,11 @@
 				<origin xyz="0 0 0" rpy="0 0 0"/>
 				<geometry>
-					<mesh filename="package://ginko_description/meshes/stl/link06_r_toe01.stl"/>
-				</geometry>
-			</collision>
-			<visual>
-				<origin xyz="0 0 0" rpy="0 0 0"/>
-				<geometry>
-					<mesh filename="package://ginko_description/meshes/obj/link06_r_toe01.obj"/>
+					<mesh filename="package://ginko_description/meshes/ginko_rs406/stl/link06_r_toe01.stl"/>
+				</geometry>
+			</collision>
+			<visual>
+				<origin xyz="0 0 0" rpy="0 0 0"/>
+				<geometry>
+					<mesh filename="package://ginko_description/meshes/ginko_rs406/obj/link06_r_toe01.obj"/>
 				</geometry>
 			</visual>
@@ -459,5 +459,5 @@
 				<origin xyz="0 0 0" rpy="0 0 0"/>
 	    		<geometry>
-					<mesh filename="package://ginko_description/meshes/stl/link07_r_toe02.stl"/>
+					<mesh filename="package://ginko_description/meshes/ginko_rs406/stl/link07_r_toe02.stl"/>
 	    		</geometry>
 			</collision>
@@ -465,5 +465,5 @@
 				<origin xyz="0 0 0" rpy="0 0 0"/>
 				<geometry>
-					<mesh filename="package://ginko_description/meshes/obj/link07_r_toe02.obj"/>
+					<mesh filename="package://ginko_description/meshes/ginko_rs406/obj/link07_r_toe02.obj"/>
 				</geometry>
 			</visual>
@@ -495,5 +495,5 @@
 				<origin xyz="0 0 0" rpy="0 0 0"/>
 				<geometry>
-					<mesh filename="package://ginko_description/meshes/obj/link08_r_toe03.obj"/>
+					<mesh filename="package://ginko_description/meshes/ginko_rs406/obj/link08_r_toe03.obj"/>
 				</geometry>
 			</visual>
