Commit message: refactoring file path

File: ginko_description/xacro/ginko_rs406/sdf_generation/export/urdf/ginko_rviz.urdf (robot description, URDF)
Before this commit: robot ginko, 49 links, 48 joints
Links:
- link arm_l_link0: geometry collision mesh filename=package://ginko_description/meshes/ginko_rs406/stl/link09_l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; visual mesh filename=package://ginko_description/meshes/ginko_rs406/obj/link09_l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
- link arm_l_link1: geometry collision mesh filename=package://ginko_description/meshes/ginko_rs406/stl/link10_l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; visual mesh filename=package://ginko_description/meshes/ginko_rs406/obj/link10_l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
- link arm_l_link2: geometry collision mesh filename=package://ginko_description/meshes/ginko_rs406/stl/link11_l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; visual mesh filename=package://ginko_description/meshes/ginko_rs406/obj/link11_l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
- link arm_l_link3: geometry collision mesh filename=package://ginko_description/meshes/ginko_rs406/stl/link12_l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; visual mesh filename=package://ginko_description/meshes/ginko_rs406/obj/link12_l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
- link arm_l_urg_link: geometry collision mesh filename=package://ginko_description/meshes/ginko_rs406/stl/urg.stl; visual mesh filename=package://ginko_description/meshes/ginko_rs406/obj/urg.obj
- link arm_r_link0: geometry collision mesh filename=package://ginko_description/meshes/ginko_rs406/stl/link09_r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; visual mesh filename=package://ginko_description/meshes/ginko_rs406/obj/link09_r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
- link arm_r_link1: geometry collision mesh filename=package://ginko_description/meshes/ginko_rs406/stl/link10_r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; visual mesh filename=package://ginko_description/meshes/ginko_rs406/obj/link10_r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
- link arm_r_link2: geometry collision mesh filename=package://ginko_description/meshes/ginko_rs406/stl/link11_r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; visual mesh filename=package://ginko_description/meshes/ginko_rs406/obj/link11_r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
- link arm_r_link3: geometry collision mesh filename=package://ginko_description/meshes/ginko_rs406/stl/link12_r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; visual mesh filename=package://ginko_description/meshes/ginko_rs406/obj/link12_r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
- link arm_r_urg_link: geometry collision mesh filename=package://ginko_description/meshes/ginko_rs406/stl/urg.stl; visual mesh filename=package://ginko_description/meshes/ginko_rs406/obj/urg.obj
- link body_link0: geometry collision mesh filename=package://ginko_description/meshes/ginko_rs406/stl/link00_c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; visual mesh filename=package://ginko_description/meshes/ginko_rs406/obj/link00_c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
- link body_link1: geometry collision mesh filename=package://ginko_description/meshes/ginko_rs406/stl/link01_w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; visual mesh filename=package://ginko_description/meshes/ginko_rs406/obj/link01_w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
- link leg_l_link0: geometry collision mesh filename=package://ginko_description/meshes/ginko_rs406/stl/link02_l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; visual mesh filename=package://ginko_description/meshes/ginko_rs406/obj/link02_l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
- link leg_l_link1: geometry collision mesh filename=package://ginko_description/meshes/ginko_rs406/stl/link03_l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; visual mesh filename=package://ginko_description/meshes/ginko_rs406/obj/link03_l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
- link leg_l_link2: geometry collision mesh filename=package://ginko_description/meshes/ginko_rs406/stl/link04_l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; visual mesh filename=package://ginko_description/meshes/ginko_rs406/obj/link04_l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
- link leg_l_link3: geometry collision mesh filename=package://ginko_description/meshes/ginko_rs406/stl/link05_l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; visual mesh filename=package://ginko_description/meshes/ginko_rs406/obj/link05_l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
- link leg_l_link4: geometry collision mesh filename=package://ginko_description/meshes/ginko_rs406/stl/link03_l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; visual mesh filename=package://ginko_description/meshes/ginko_rs406/obj/link03_l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
- link leg_l_link5: geometry collision mesh filename=package://ginko_description/meshes/ginko_rs406/stl/link04_l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; visual mesh filename=package://ginko_description/meshes/ginko_rs406/obj/link04_l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
- link leg_l_link6: geometry collision mesh filename=package://ginko_description/meshes/ginko_rs406/stl/link06_l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; visual mesh filename=package://ginko_description/meshes/ginko_rs406/obj/link06_l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
- link leg_l_link7: geometry collision mesh filename=package://ginko_description/meshes/ginko_rs406/stl/link07_l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; visual mesh filename=package://ginko_description/meshes/ginko_rs406/obj/link07_l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
- link leg_l_link8: geometry collision box size=0.128 0.08 0.006; visual mesh filename=package://ginko_description/meshes/ginko_rs406/obj/link08_l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
- link leg_r_link0: geometry collision mesh filename=package://ginko_description/meshes/ginko_rs406/stl/link02_r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; visual mesh filename=package://ginko_description/meshes/ginko_rs406/obj/link02_r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
- link leg_r_link1: geometry collision mesh filename=package://ginko_description/meshes/ginko_rs406/stl/link03_r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; visual mesh filename=package://ginko_description/meshes/ginko_rs406/obj/link03_r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
- link leg_r_link2: geometry collision mesh filename=package://ginko_description/meshes/ginko_rs406/stl/link04_r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; visual mesh filename=package://ginko_description/meshes/ginko_rs406/obj/link04_r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
- link leg_r_link3: geometry collision mesh filename=package://ginko_description/meshes/ginko_rs406/stl/link05_r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; visual mesh filename=package://ginko_description/meshes/ginko_rs406/obj/link05_r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
- link leg_r_link4: geometry collision mesh filename=package://ginko_description/meshes/ginko_rs406/stl/link03_r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; visual mesh filename=package://ginko_description/meshes/ginko_rs406/obj/link03_r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
- link leg_r_link5: geometry collision mesh filename=package://ginko_description/meshes/ginko_rs406/stl/link04_r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; visual mesh filename=package://ginko_description/meshes/ginko_rs406/obj/link04_r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
- link leg_r_link6: geometry collision mesh filename=package://ginko_description/meshes/ginko_rs406/stl/link06_r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; visual mesh filename=package://ginko_description/meshes/ginko_rs406/obj/link06_r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
- link leg_r_link7: geometry collision mesh filename=package://ginko_description/meshes/ginko_rs406/stl/link07_r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; visual mesh filename=package://ginko_description/meshes/ginko_rs406/obj/link07_r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
- link leg_r_link8: geometry collision box size=0.128 0.08 0.006; visual mesh filename=package://ginko_description/meshes/ginko_rs406/obj/link08_r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

File: ginko_description/xacro/roboone_ring/large_ring.xacro (robot description, xacro)
@@ -7,5 +7,5 @@
 				<origin xyz="0 0 0" rpy="0 0 0"/>
 				<geometry>
-        			<mesh filename="package://ginko_description/meshes/stl/large_ring.stl"/>
+        			<mesh filename="package://ginko_description/meshes/roboone_ring/stl/large_ring.stl"/>
 				</geometry>
 			</collision>
@@ -13,5 +13,5 @@
 				<origin xyz="0 0 0" rpy="0 0 0"/>
 				<geometry>
-					<mesh filename="package://ginko_description/meshes/obj/large_ring.obj"/>
+					<mesh filename="package://ginko_description/meshes/roboone_ring/obj/large_ring.obj"/>
 				</geometry>
 			</visual>

File: ginko_description/xacro/roboone_ring/small_ring.xacro (robot description, xacro)
@@ -7,5 +7,5 @@
 				<origin xyz="0 0 0" rpy="0 0 0"/>
 				<geometry>
-        			<mesh filename="package://ginko_description/meshes/stl/small_ring.stl"/>
+        			<mesh filename="package://ginko_description/meshes/roboone_ring/stl/small_ring.stl"/>
 				</geometry>
 			</collision>
@@ -13,5 +13,5 @@
 				<origin xyz="0 0 0" rpy="0 0 0"/>
 				<geometry>
-					<mesh filename="package://ginko_description/meshes/obj/small_ring.obj"/>
+					<mesh filename="package://ginko_description/meshes/roboone_ring/obj/small_ring.obj"/>
 				</geometry>
 			</visual>
