Commit message: adding right leg

File: ginko_description/xacro/ginko_xm540/ginko.xacro (robot description, xacro)
@@ -9,4 +9,6 @@
   <xacro:include filename="$(find ginko_description)/xacro/ginko_xm540/parts/body.xacro"/>
   <xacro:include filename="$(find ginko_description)/xacro/ginko_xm540/transmission/body.gazebo"/>
+  <xacro:include filename="$(find ginko_description)/xacro/ginko_xm540/parts/leg_r.xacro"/>
+  <xacro:include filename="$(find ginko_description)/xacro/ginko_xm540/transmission/leg_r.gazebo"/>
   <!-- MACRO:Loading Gazebo Controllers for joints -->
   <xacro:macro name="gazebo_plugin_xacro" params="gazebo_motor_model">
@@ -49,4 +51,6 @@
     <xacro:body_xacro/>
     <xacro:body_gazebo gazebo_hw_interface="${gazebo_hw_interface}"/>
+    <xacro:leg_r_xacro/>
+    <xacro:leg_r_gazebo gazebo_hw_interface="${gazebo_hw_interface}"/>
   </xacro:macro>
   <!-- Load Macros -->

File: ginko_description/xacro/ginko_xm540/parts/body.xacro (robot description, xacro)
@@ -13,6 +13,6 @@
             <!-- waits collision -->
             <xacro:box_collision xyz="0 0 0.0305" rpy="0 0 0" size="0.084 0.04 0.0895"/>
-			<xacro:box_inertial xyz="0 0 0.03" rpy="0 0 0" size="0.068 0.0305 0.0738" mass="0.382"/>
-<!-- 			<inertial>
+			<xacro:box_inertial xyz="0 0 0.0305" rpy="0 0 0" size="0.084 0.04 0.0895" mass="0.382"/>
+			<!-- <inertial>
 				<mass value="0.382"/>
 				<origin xyz="0.000083485 0.0 0.03686607" rpy="0 0 0"/>
@@ -30,5 +30,5 @@
 			<axis xyz="0 0 1"/>
 			<limit effort="1000.0" lower="-3.1" upper="3.1" velocity="10.0"/>
-			<dynamics damping="0.1" friction="0.1"/>
+			<dynamics damping="0.0" friction="0.0"/>
 		</joint>
 		<!-- chest -->
@@ -44,6 +44,6 @@
             <!-- Head collision -->
             <xacro:box_collision xyz="0.052 0 0.067" rpy="0 0 0" size="0.09 0.06 0.06"/>
-			<xacro:box_inertial xyz="0 0 0.02" rpy="0 0 0" size="0.11 0.201 0.08" mass="0.665"/>
-<!-- 			<inertial>
+			<xacro:box_inertial xyz="0 0 0.012" rpy="0 0 0" size="0.11 0.201 0.053" mass="0.665"/>
+			<!-- <inertial>
 				<mass value="0.665"/>
 				<origin xyz="0.00121250 0.0 0.01189965" rpy="0 0 0"/>

File: ginko_description/xacro/physics/default_gazebo_params.xacro (robot description, xacro)
@@ -3,5 +3,5 @@
 	<xacro:macro name="default_motor_transmission" params="joint_name gazebo_hw_interface">
 		<gazebo reference="${joint_name}">
-  		<implicitSpringDamper>1</implicitSpringDamper>
+  		    <implicitSpringDamper>1</implicitSpringDamper>
 		</gazebo>
 		<transmission name="${joint_name}_trans">
@@ -26,5 +26,5 @@
 				</xacro:if>
 				<xacro:if value="${gazebo_hw_interface=='position'}">
-          <hardwareInterface>hardware_interface/PositionJointInterface</hardwareInterface>
+                    <hardwareInterface>hardware_interface/PositionJointInterface</hardwareInterface>
 				</xacro:if>
 				<mechanicalReduction>1</mechanicalReduction>
@@ -44,3 +44,8 @@
 		</gazebo>
 	</xacro:macro>
+	<xacro:macro name="default_passive_joint" params="joint_name">
+		<gazebo reference="${joint_name}">
+  		    <implicitSpringDamper>1</implicitSpringDamper>
+		</gazebo>
+	</xacro:macro>
 </robot>

Commit message: add arms

File: ginko_description/xacro/ginko_xm540/ginko.xacro (robot description, xacro)
@@ -13,4 +13,8 @@
   <xacro:include filename="$(find ginko_description)/xacro/ginko_xm540/parts/leg_l.xacro"/>
   <xacro:include filename="$(find ginko_description)/xacro/ginko_xm540/transmission/leg_l.gazebo"/>
+  <xacro:include filename="$(find ginko_description)/xacro/ginko_xm540/parts/arm_r.xacro"/>
+  <xacro:include filename="$(find ginko_description)/xacro/ginko_xm540/transmission/arm_r.gazebo"/>
+  <xacro:include filename="$(find ginko_description)/xacro/ginko_xm540/parts/arm_l.xacro"/>
+  <xacro:include filename="$(find ginko_description)/xacro/ginko_xm540/transmission/arm_l.gazebo"/>
   <!-- MACRO:Loading Gazebo Controllers for joints -->
   <xacro:macro name="gazebo_plugin_xacro" params="gazebo_motor_model">
@@ -57,4 +61,8 @@
     <xacro:leg_l_xacro/>
     <xacro:leg_l_gazebo gazebo_hw_interface="${gazebo_hw_interface}"/>
+    <xacro:arm_r_xacro/>
+    <xacro:arm_r_gazebo gazebo_hw_interface="${gazebo_hw_interface}"/>
+    <xacro:arm_l_xacro/>
+    <xacro:arm_l_gazebo gazebo_hw_interface="${gazebo_hw_interface}"/>
   </xacro:macro>
   <!-- Load Macros -->

File: ginko_description/xacro/ginko_xm540/parts/leg_r.xacro (robot description, xacro)
@@ -62,5 +62,5 @@
 		    <origin xyz="-0.016713 0 -0.027522" rpy="0 -0.5102 0"/>
 		    <axis xyz="0 1 0"/>
-			<limit effort="1000.0" lower="-1.4" upper="0.5" velocity="1000.0"/>
+			<limit effort="1000.0" lower="-3.1" upper="3.1" velocity="10.0"/>
 			<dynamics damping="0.0" friction="0.0"/>
 		</joint>
@@ -185,5 +185,5 @@
 		    <origin xyz="-0.0335 0 0" rpy="0 -0.7854 0"/>
 		    <axis xyz="0 1 0"/>
-			<limit effort="1000.0" lower="-1.4" upper="0.5" velocity="1000.0"/>
+			<limit effort="1000.0" lower="-3.1" upper="3.1" velocity="1000.0"/>
 			<dynamics damping="0.0" friction="0.0"/>
 			<mimic joint="leg_r_joint04" multiplier="1" offset="0"/>
@@ -233,5 +233,5 @@
 		    <origin xyz="0.07118 0 0.00834" rpy="0 1.5708 0"/>
 		    <axis xyz="0 1 0"/>
-			<limit effort="1000.0" lower="-1.0" upper="1.5" velocity="10.0"/>
+			<limit effort="1000.0" lower="-3.1" upper="3.1" velocity="10.0"/>
 			<dynamics damping="0.0" friction="0.0"/>
 			<!-- Only for Rviz. Not correct. -->
