Commit message: Change joint order

File: ginko_description/xacro/ginko_xm540/parts/leg_r.xacro (robot description, xacro)
@@ -18,11 +18,11 @@
 				</geometry>
 			</visual>
-            <xacro:box_collision xyz="0 -0.011 0" rpy="0 0 0" size="0.095 0.0415 0.02"/>
-			<xacro:box_inertial xyz="0 -0.011 0" rpy="0 0 0" size="0.095 0.0415 0.02" mass="0.024"/>
+            <xacro:box_collision xyz="0 -0.015 0" rpy="0 0 0" size="0.095 0.05 0.03"/>
+			<xacro:box_inertial xyz="0 -0.015 0" rpy="0 0 0" size="0.095 0.05 0.03" mass="0.025"/>
 		</link>
 		<joint name="leg_r_joint02" type="revolute">
 		    <parent link="leg_r_link01"/>
 			<child link="leg_r_link02"/>
-		    <origin xyz="0 -0.032 0" rpy="0 0 0"/>
+		    <origin xyz="0 -0.06085 0" rpy="0 0 0"/>
 		    <axis xyz="0 1 0"/>
 			<limit effort="1000.0" lower="-1.5708" upper="1.5708" velocity="10.0"/>
@@ -36,11 +36,11 @@
 				</geometry>
 			</visual>
-            <xacro:box_collision xyz="0 -0.058 -0.0037" rpy="0 0 0" size="0.067 0.095 0.077"/>
-			<xacro:box_inertial xyz="0 -0.058 -0.0037" rpy="0 0 0" size="0.067 0.095 0.077" mass="0.48"/>
+            <xacro:box_collision xyz="0 -0.02 -0.0037" rpy="0 0 0" size="0.067 0.095 0.077"/>
+			<xacro:box_inertial xyz="0 -0.02 -0.0037" rpy="0 0 0" size="0.067 0.095 0.077" mass="0.48"/>
 		</link>
 		<joint name="leg_r_joint03" type="revolute">
 		    <parent link="leg_r_link02"/>
 			<child link="leg_r_link03"/>
-		    <origin xyz="0.016713 -0.02935 -0.027522" rpy="0 0.7854 0"/>
+		    <origin xyz="0.016713 0 -0.027522" rpy="0 0.7854 0"/>
 		    <axis xyz="0 1 0"/>
 			<limit effort="1000.0" lower="-0.5" upper="1.4" velocity="10.0"/>
@@ -60,8 +60,7 @@
 		    <parent link="leg_r_link02"/>
 			<child link="leg_r_link04"/>
-		    <origin xyz="-0.016713 -0.02935 -0.027522" rpy="0 -0.5102 0"/>
-		    <axis xyz="0 1 0"/>
-			<!-- <limit effort="1000.0" lower="-1.42" upper="0.5" velocity="1000.0"/> -->
-			<limit effort="1000.0" lower="-3.1" upper="3.1" velocity="1000.0"/>
+		    <origin xyz="-0.016713 0 -0.027522" rpy="0 -0.5102 0"/>
+		    <axis xyz="0 1 0"/>
+			<limit effort="1000.0" lower="-1.4" upper="0.5" velocity="1000.0"/>
 			<dynamics damping="0.0" friction="0.0"/>
 		</joint>
@@ -75,41 +74,4 @@
             <xacro:box_collision xyz="-0.015 0 0" rpy="0 0 0" size="0.04565 0.0373 0.023"/>
 			<xacro:box_inertial xyz="-0.015 0 0" rpy="0 0 0" size="0.04565 0.0373 0.023" mass="0.011"/>
-		</link>
-		<joint name="leg_r_joint05" type="revolute">
-		    <parent link="leg_r_link02"/>
-			<child link="leg_r_link05"/>
-		    <origin xyz="-0.016713 -0.02935 -0.027522" rpy="0 0.7854 0"/>
-		    <axis xyz="0 1 0"/>
-			<limit effort="1000.0" lower="-3.1" upper="3.1" velocity="10.0"/>
-			<dynamics damping="0.0" friction="0.0"/>
-			<mimic joint="leg_l_joint03" multiplier="1" offset="0"/>
-		</joint>
-		<link name="leg_r_link05">
-			<visual>
-				<origin xyz="0 0 0" rpy="0 0 0"/>
-				<geometry>
-					<mesh filename="package://ginko_description/meshes/ginko_xm540/obj/leg_r_link05.obj"/>
-				</geometry>
-			</visual>
-            <xacro:box_collision xyz="0.05 0 0" rpy="0 0 0" size="0.1 0.0309 0.017"/>
-			<xacro:box_inertial xyz="0.05 0 0" rpy="0 0 0" size="0.1 0.0309 0.017" mass="0.020"/>
-		</link>
-		<joint name="leg_r_joint06" type="revolute">
-		    <parent link="leg_r_link04"/>
-			<child link="leg_r_link06"/>
-		    <origin xyz="-0.03 0 0" rpy="0 1.2956 0"/>
-		    <axis xyz="0 1 0"/>
-			<limit effort="1000.0" lower="-1.0" upper="1.6" velocity="10.0"/>
-			<dynamics damping="0.0" friction="0.0"/>
-		</joint>
-		<link name="leg_r_link06">
-			<visual>
-				<origin xyz="0 0 0" rpy="0 0 0"/>
-				<geometry>
-					<mesh filename="package://ginko_description/meshes/ginko_xm540/obj/leg_r_link06.obj"/>
-				</geometry>
-			</visual>
-            <xacro:box_collision xyz="0.05 0 0" rpy="0 0 0" size="0.1 0.0181 0.017"/>
-			<xacro:box_inertial xyz="0.05 0 0" rpy="0 0 0" size="0.1 0.0181 0.017" mass="0.015"/>
 		</link>
 		<joint name="leg_r_joint07" type="revolute">
@@ -120,4 +82,5 @@
 			<limit effort="1000.0" lower="-3.1" upper="3.1" velocity="1000.0"/>
 			<dynamics damping="0.0" friction="0.0"/>
+			<mimic joint="leg_r_joint03" multiplier="-1" offset="0"/>
 		</joint>
 		<link name="leg_r_link07">
@@ -131,9 +94,28 @@
 			<xacro:box_inertial xyz="-0.01 0 0" rpy="0 0 0" size="0.0605 0.0487 0.014" mass="0.009"/>
 		</link>
+		<joint name="leg_r_joint05" type="revolute">
+		    <parent link="leg_r_link07"/>
+			<child link="leg_r_link05"/>
+		    <origin xyz="-0.0335 0 0" rpy="0 0.7854 0"/>
+		    <axis xyz="0 1 0"/>
+			<limit effort="1000.0" lower="-0.5" upper="1.4" velocity="1000.0"/>
+			<dynamics damping="0.0" friction="0.0"/>
+			<mimic joint="leg_r_joint03" multiplier="1" offset="0"/>
+		</joint>
+		<link name="leg_r_link05">
+			<visual>
+				<origin xyz="-0.1 0 0" rpy="0 0 0"/>
+				<geometry>
+					<mesh filename="package://ginko_description/meshes/ginko_xm540/obj/leg_r_link05.obj"/>
+				</geometry>
+			</visual>
+            <xacro:box_collision xyz="-0.05 0 0" rpy="0 0 0" size="0.1 0.0309 0.017"/>
+			<xacro:box_inertial xyz="-0.05 0 0" rpy="0 0 0" size="0.1 0.0309 0.017" mass="0.020"/>
+		</link>
 	    <gazebo>
 	        <joint name="leg_r_loop_joint01" type="revolute">
-	            <parent>leg_r_link05</parent>
-	            <child>leg_r_link07</child>
-	            <pose>-0.0335 0 0 0 0 0</pose>
+	            <parent>leg_r_link02</parent>
+	            <child>leg_r_link05</child>
+	            <pose>-0.1 0 0 0 0 0</pose>
 	            <axis>
 	                <xyz>0 1 0</xyz>
@@ -165,6 +147,7 @@
 		    <origin xyz="0 0 0" rpy="0 -0.7854 0"/>
 		    <axis xyz="0 1 0"/>
-			<limit effort="1000.0" lower="-1.4" upper="0.5" velocity="1000.0"/>
-			<dynamics damping="0.0" friction="0.0"/>
+			<limit effort="1000.0" lower="-3.1" upper="3.1" velocity="10.0"/>
+			<dynamics damping="0.0" friction="0.0"/>
+			<mimic joint="leg_r_joint04" multiplier="1" offset="0"/>
 		</joint>
 		<link name="leg_r_link08">
@@ -178,27 +161,47 @@
 			<xacro:box_inertial xyz="-0.05 0 0" rpy="0 0 0" size="0.1 0.0301 0.0175" mass="0.021"/>
 		</link>
+		<joint name="leg_r_joint10" type="revolute">
+		    <parent link="leg_r_link08"/>
+			<child link="leg_r_link10"/>
+		    <origin xyz="-0.1 0 0" rpy="0 0.7854 0"/>
+		    <axis xyz="0 1 0"/>
+			<limit effort="1000.0" lower="-0.5" upper="1.4" velocity="1000.0"/>
+			<dynamics damping="0.0" friction="0.0"/>
+			<mimic joint="leg_r_joint04" multiplier="-1" offset="0"/>
+		</joint>
+		<link name="leg_r_link10">
+			<visual>
+				<origin xyz="0 0 0" rpy="0 0 0"/>
+				<geometry>
+					<mesh filename="package://ginko_description/meshes/ginko_xm540/obj/leg_r_link10.obj"/>
+				</geometry>
+			</visual>
+            <xacro:box_collision xyz="-0.03335 -0.0087 -0.0160" rpy="0 0 0" size="0.0873 0.0531 0.046"/>
+			<xacro:box_inertial xyz="-0.03335 -0.0087 -0.0160" rpy="0 0 0" size="0.0873 0.0531 0.046" mass="0.108"/>
+		</link>
 		<joint name="leg_r_joint09" type="revolute">
-		    <parent link="leg_r_link05"/>
+		    <parent link="leg_r_link10"/>
 			<child link="leg_r_link09"/>
-		    <origin xyz="0.1 0 0" rpy="0 -1.5708 0"/>
-		    <axis xyz="0 1 0"/>
-			<limit effort="1000.0" lower="-1.6" upper="1.0" velocity="1000.0"/>
-			<dynamics damping="0.0" friction="0.0"/>
+		    <origin xyz="-0.0335 0 0" rpy="0 -0.7854 0"/>
+		    <axis xyz="0 1 0"/>
+			<limit effort="1000.0" lower="-1.4" upper="0.5" velocity="1000.0"/>
+			<dynamics damping="0.0" friction="0.0"/>
+			<mimic joint="leg_r_joint04" multiplier="1" offset="0"/>
 		</joint>
 		<link name="leg_r_link09">
 			<visual>
-				<origin xyz="0 0 0" rpy="0 0 0"/>
+				<origin xyz="0.1 0 0" rpy="0 0 0"/>
 				<geometry>
 					<mesh filename="package://ginko_description/meshes/ginko_xm540/obj/leg_r_link09.obj"/>
 				</geometry>
 			</visual>
-            <xacro:box_collision xyz="-0.05 0 0" rpy="0 0 0" size="0.1 0.0237 0.0175"/>
-			<xacro:box_inertial xyz="-0.05 0 0" rpy="0 0 0" size="0.1 0.0237 0.0175" mass="0.022"/>
+            <xacro:box_collision xyz="0.05 0 0" rpy="0 0 0" size="0.1 0.0237 0.0175"/>
+			<xacro:box_inertial xyz="0.05 0 0" rpy="0 0 0" size="0.1 0.0237 0.0175" mass="0.022"/>
 		</link>
 	    <gazebo>
 	        <joint name="leg_r_loop_joint02" type="revolute">
-	            <parent>leg_r_link06</parent>
+	            <parent>leg_r_link07</parent>
 	            <child>leg_r_link09</child>
-	            <pose>-0.02882 0 0.00834 0 0 0</pose>
+	            <pose>0.1 0 0 0 0 0</pose>
 	            <axis>
 	                <xyz>0 1 0</xyz>
@@ -225,27 +228,29 @@
 	        </joint>
 	    </gazebo>
-		<joint name="leg_r_joint10" type="revolute">
-		    <parent link="leg_r_link08"/>
-			<child link="leg_r_link10"/>
-		    <origin xyz="-0.1 0 0" rpy="0 0.7854 0"/>
-		    <axis xyz="0 1 0"/>
-			<limit effort="1000.0" lower="-0.5" upper="1.42" velocity="1000.0"/>
-			<dynamics damping="0.0" friction="0.0"/>
-		</joint>
-		<link name="leg_r_link10">
-			<visual>
-				<origin xyz="0 0 0" rpy="0 0 0"/>
-				<geometry>
-					<mesh filename="package://ginko_description/meshes/ginko_xm540/obj/leg_r_link10.obj"/>
-				</geometry>
-			</visual>
-            <xacro:box_collision xyz="-0.03335 -0.0087 -0.0160" rpy="0 0 0" size="0.0873 0.0531 0.046"/>
-			<xacro:box_inertial xyz="-0.03335 -0.0087 -0.0160" rpy="0 0 0" size="0.0873 0.0531 0.046" mass="0.108"/>
+		<joint name="leg_r_joint06" type="revolute">
+		    <parent link="leg_r_link09"/>
+			<child link="leg_r_link06"/>
+		    <origin xyz="0.07118 0 0.00834" rpy="0 1.5708 0"/>
+		    <axis xyz="0 1 0"/>
+			<limit effort="1000.0" lower="-1.0" upper="1.5" velocity="10.0"/>
+			<dynamics damping="0.0" friction="0.0"/>
+			<!-- Only for Rviz. Not correct. -->
+			<mimic joint="leg_r_joint03" multiplier="1" offset="0"/>
+		</joint>
+		<link name="leg_r_link06">
+			<visual>
+				<origin xyz="-0.1 0 0" rpy="0 0 0"/>
+				<geometry>
+					<mesh filename="package://ginko_description/meshes/ginko_xm540/obj/leg_r_link06.obj"/>
+				</geometry>
+			</visual>
+            <xacro:box_collision xyz="-0.05 0 0" rpy="0 0 0" size="0.1 0.0181 0.017"/>
+			<xacro:box_inertial xyz="-0.05 0 0" rpy="0 0 0" size="0.1 0.0181 0.017" mass="0.015"/>
 		</link>
 	    <gazebo>
 	        <joint name="leg_r_loop_joint03" type="revolute">
-	            <parent>leg_r_link09</parent>
-	            <child>leg_r_link10</child>
-	            <pose>-0.0335 0 0 0 0 0</pose>
+	            <parent>leg_r_link04</parent>
+	            <child>leg_r_link06</child>
+	            <pose>-0.1 0 0 0 0 0</pose>
 	            <axis>
 	                <xyz>0 1 0</xyz>

Commit message: Revert unlimit

File: ginko_description/xacro/ginko_xm540/parts/leg_r.xacro (robot description, xacro)
@@ -62,5 +62,5 @@
 		    <origin xyz="-0.016713 0 -0.027522" rpy="0 -0.5102 0"/>
 		    <axis xyz="0 1 0"/>
-			<limit effort="1000.0" lower="-3.1" upper="3.1" velocity="10.0"/>
+			<limit effort="1000.0" lower="-1.4" upper="0.5" velocity="1000.0"/>
 			<dynamics damping="0.0" friction="0.0"/>
 		</joint>
@@ -185,5 +185,5 @@
 		    <origin xyz="-0.0335 0 0" rpy="0 -0.7854 0"/>
 		    <axis xyz="0 1 0"/>
-			<limit effort="1000.0" lower="-3.1" upper="3.1" velocity="1000.0"/>
+			<limit effort="1000.0" lower="-1.4" upper="0.5" velocity="1000.0"/>
 			<dynamics damping="0.0" friction="0.0"/>
 			<mimic joint="leg_r_joint04" multiplier="1" offset="0"/>
@@ -233,5 +233,5 @@
 		    <origin xyz="0.07118 0 0.00834" rpy="0 1.5708 0"/>
 		    <axis xyz="0 1 0"/>
-			<limit effort="1000.0" lower="-3.1" upper="3.1" velocity="10.0"/>
+			<limit effort="1000.0" lower="-1.0" upper="1.5" velocity="10.0"/>
 			<dynamics damping="0.0" friction="0.0"/>
 			<!-- Only for Rviz. Not correct. -->
