Commit message: Fix xacro

File: ginko_description/xacro/ginko_xm540/parts/leg_l.xacro (robot description, xacro)
@@ -133,5 +133,5 @@
 	                <ode>
 	                    <implicit_spring_damper>1</implicit_spring_damper>
-	                    <cfm_damping>1</cfm_damping>
+	                    <cfm_damping>0</cfm_damping>
 	                    <limit>
 	                        <cfm>0</cfm>
@@ -219,5 +219,5 @@
 	                <ode>
 	                    <implicit_spring_damper>1</implicit_spring_damper>
-	                    <cfm_damping>1</cfm_damping>
+	                    <cfm_damping>0</cfm_damping>
 	                    <limit>
 	                        <cfm>0</cfm>
@@ -268,5 +268,5 @@
 	                <ode>
 	                    <implicit_spring_damper>1</implicit_spring_damper>
-	                    <cfm_damping>1</cfm_damping>
+	                    <cfm_damping>0</cfm_damping>
 	                    <limit>
 	                        <cfm>0</cfm>
@@ -281,5 +281,5 @@
 			<child link="leg_l_link11"/>
 		    <origin xyz="-0.01675 0 -0.02475" rpy="0 0 0"/>
-		    <axis xyz="-1 0 0"/>
+		    <axis xyz="1 0 0"/>
 			<limit effort="1000.0" lower="-3.1" upper="3.1" velocity="1000.0"/>
 			<dynamics damping="0.0" friction="0.0"/>

File: ginko_description/xacro/ginko_xm540/parts/leg_r.xacro (robot description, xacro)
@@ -133,5 +133,5 @@
 	                <ode>
 	                    <implicit_spring_damper>1</implicit_spring_damper>
-	                    <cfm_damping>1</cfm_damping>
+	                    <cfm_damping>0</cfm_damping>
 	                    <limit>
 	                        <cfm>0</cfm>
@@ -219,5 +219,5 @@
 	                <ode>
 	                    <implicit_spring_damper>1</implicit_spring_damper>
-	                    <cfm_damping>1</cfm_damping>
+	                    <cfm_damping>0</cfm_damping>
 	                    <limit>
 	                        <cfm>0</cfm>
@@ -268,5 +268,5 @@
 	                <ode>
 	                    <implicit_spring_damper>1</implicit_spring_damper>
-	                    <cfm_damping>1</cfm_damping>
+	                    <cfm_damping>0</cfm_damping>
 	                    <limit>
 	                        <cfm>0</cfm>

File: ginko_description/xacro/physics/default_gazebo_params.xacro (robot description, xacro)
@@ -39,5 +39,5 @@
 			<maxVel>10.0</maxVel>
 			<minDepth>0.0001</minDepth>
-			<maxContacts>12</maxContacts>
+			<maxContacts>6</maxContacts>
 			<selfCollide>false</selfCollide>
 			<dampingFactor>0.00</dampingFactor>

Commit message: Edit cfm and erp

File: ginko_description/xacro/ginko_xm540/parts/leg_l.xacro (robot description, xacro)
@@ -8,5 +8,5 @@
 		    <origin xyz="0 0 0" rpy="0 0 0"/>
 		    <axis xyz="-1 0 0"/>
-			<limit effort="1000.0" lower="-0.7854" upper="0.7854" velocity="10.0"/>
+			<limit effort="1000.0" lower="-0.78539816" upper="0.78539816" velocity="10.0"/>
 			<dynamics damping="0.0" friction="0.0"/>
 		</joint>
@@ -26,5 +26,5 @@
 		    <origin xyz="0 0.06085 0" rpy="0 0 0"/>
 		    <axis xyz="0 -1 0"/>
-			<limit effort="1000.0" lower="-1.5708" upper="1.5708" velocity="10.0"/>
+			<limit effort="1000.0" lower="-1.57079633" upper="1.57079633" velocity="10.0"/>
 			<dynamics damping="0.0" friction="0.0"/>
 		</joint>
@@ -42,5 +42,5 @@
 		    <parent link="leg_l_link02"/>
 			<child link="leg_l_link03"/>
-		    <origin xyz="0.016713 0 -0.027522" rpy="0 0.7854 0"/>
+		    <origin xyz="0.016713 0 -0.027522" rpy="0 0.78539816 0"/>
 		    <axis xyz="0 -1 0"/>
 			<limit effort="1000.0" lower="-1.4" upper="0.5" velocity="10.0"/>
@@ -60,5 +60,5 @@
 		    <parent link="leg_l_link02"/>
 			<child link="leg_l_link04"/>
-		    <origin xyz="-0.016713 0 -0.027522" rpy="0 -0.5102 0"/>
+		    <origin xyz="-0.016713 0 -0.027522" rpy="0 -0.51016603 0"/>
 		    <axis xyz="0 -1 0"/>
 			<limit effort="1000.0" lower="-0.5" upper="1.4" velocity="1000.0"/>
@@ -78,5 +78,5 @@
 		    <parent link="leg_l_link03"/>
 			<child link="leg_l_link07"/>
-		    <origin xyz="0.1 0 0" rpy="0 -0.7854 0"/>
+		    <origin xyz="0.1 0 0" rpy="0 -0.78539816 0"/>
 		    <axis xyz="0 -1 0"/>
 			<limit effort="1000.0" lower="-3.1" upper="3.1" velocity="1000.0"/>
@@ -97,5 +97,5 @@
 		    <parent link="leg_l_link07"/>
 			<child link="leg_l_link05"/>
-		    <origin xyz="-0.0335 0 0" rpy="0 0.7854 0"/>
+		    <origin xyz="-0.0335 0 0" rpy="0 0.78539816 0"/>
 		    <axis xyz="0 -1 0"/>
 			<limit effort="1000.0" lower="-1.4" upper="0.5" velocity="1000.0"/>
@@ -135,6 +135,6 @@
 	                    <cfm_damping>0</cfm_damping>
 	                    <limit>
-	                        <cfm>0</cfm>
-	                        <erp>0</erp>
+	                        <cfm>1e-7</cfm>
+	                        <erp>0.8</erp>
 	                    </limit>
 	                </ode>
@@ -145,5 +145,5 @@
 		    <parent link="leg_l_link07"/>
 			<child link="leg_l_link08"/>
-		    <origin xyz="0 0 0" rpy="0 -0.7854 0"/>
+		    <origin xyz="0 0 0" rpy="0 -0.78539816 0"/>
 		    <axis xyz="0 -1 0"/>
 			<limit effort="1000.0" lower="-3.1" upper="3.1" velocity="10.0"/>
@@ -164,5 +164,5 @@
 		    <parent link="leg_l_link08"/>
 			<child link="leg_l_link10"/>
-		    <origin xyz="-0.1 0 0" rpy="0 0.7854 0"/>
+		    <origin xyz="-0.1 0 0" rpy="0 0.78539816 0"/>
 		    <axis xyz="0 -1 0"/>
 			<limit effort="1000.0" lower="-1.4" upper="0.5" velocity="1000.0"/>
@@ -183,5 +183,5 @@
 		    <parent link="leg_l_link10"/>
 			<child link="leg_l_link09"/>
-		    <origin xyz="-0.0335 0 0" rpy="0 -0.7854 0"/>
+		    <origin xyz="-0.0335 0 0" rpy="0 -0.78539816 0"/>
 		    <axis xyz="0 -1 0"/>
 			<limit effort="1000.0" lower="-0.5" upper="1.4" velocity="1000.0"/>
@@ -221,6 +221,6 @@
 	                    <cfm_damping>0</cfm_damping>
 	                    <limit>
-	                        <cfm>0</cfm>
-	                        <erp>0</erp>
+	                        <cfm>1e-7</cfm>
+	                        <erp>0.8</erp>
 	                    </limit>
 	                </ode>
@@ -231,5 +231,5 @@
 		    <parent link="leg_l_link09"/>
 			<child link="leg_l_link06"/>
-		    <origin xyz="0.07118 0 0.00834" rpy="0 1.5708 0"/>
+		    <origin xyz="0.07118 0 0.00834" rpy="0 1.57079633 0"/>
 		    <axis xyz="0 -1 0"/>
 			<limit effort="1000.0" lower="-1.5" upper="1.0" velocity="10.0"/>
@@ -270,6 +270,6 @@
 	                    <cfm_damping>0</cfm_damping>
 	                    <limit>
-	                        <cfm>0</cfm>
-	                        <erp>0</erp>
+	                        <cfm>1e-7</cfm>
+	                        <erp>0.8</erp>
 	                    </limit>
 	                </ode>

File: ginko_description/xacro/ginko_xm540/parts/leg_r.xacro (robot description, xacro)
@@ -8,5 +8,5 @@
 		    <origin xyz="0 0 0" rpy="0 0 0"/>
 		    <axis xyz="1 0 0"/>
-			<limit effort="1000.0" lower="-0.7854" upper="0.7854" velocity="10.0"/>
+			<limit effort="1000.0" lower="-0.78539816" upper="0.78539816" velocity="10.0"/>
 			<dynamics damping="0.0" friction="0.0"/>
 		</joint>
@@ -26,5 +26,5 @@
 		    <origin xyz="0 -0.06085 0" rpy="0 0 0"/>
 		    <axis xyz="0 1 0"/>
-			<limit effort="1000.0" lower="-1.5708" upper="1.5708" velocity="10.0"/>
+			<limit effort="1000.0" lower="-1.57079633" upper="1.57079633" velocity="10.0"/>
 			<dynamics damping="0.0" friction="0.0"/>
 		</joint>
@@ -42,5 +42,5 @@
 		    <parent link="leg_r_link02"/>
 			<child link="leg_r_link03"/>
-		    <origin xyz="0.016713 0 -0.027522" rpy="0 0.7854 0"/>
+		    <origin xyz="0.016713 0 -0.027522" rpy="0 0.78539816 0"/>
 		    <axis xyz="0 1 0"/>
 			<limit effort="1000.0" lower="-0.5" upper="1.4" velocity="10.0"/>
@@ -60,5 +60,5 @@
 		    <parent link="leg_r_link02"/>
 			<child link="leg_r_link04"/>
-		    <origin xyz="-0.016713 0 -0.027522" rpy="0 -0.5102 0"/>
+		    <origin xyz="-0.016713 0 -0.027522" rpy="0 -0.51016603 0"/>
 		    <axis xyz="0 1 0"/>
 			<limit effort="1000.0" lower="-1.4" upper="0.5" velocity="1000.0"/>
@@ -78,5 +78,5 @@
 		    <parent link="leg_r_link03"/>
 			<child link="leg_r_link07"/>
-		    <origin xyz="0.1 0 0" rpy="0 -0.7854 0"/>
+		    <origin xyz="0.1 0 0" rpy="0 -0.78539816 0"/>
 		    <axis xyz="0 1 0"/>
 			<limit effort="1000.0" lower="-3.1" upper="3.1" velocity="1000.0"/>
@@ -97,5 +97,5 @@
 		    <parent link="leg_r_link07"/>
 			<child link="leg_r_link05"/>
-		    <origin xyz="-0.0335 0 0" rpy="0 0.7854 0"/>
+		    <origin xyz="-0.0335 0 0" rpy="0 0.78539816 0"/>
 		    <axis xyz="0 1 0"/>
 			<limit effort="1000.0" lower="-0.5" upper="1.4" velocity="1000.0"/>
@@ -135,6 +135,6 @@
 	                    <cfm_damping>0</cfm_damping>
 	                    <limit>
-	                        <cfm>0</cfm>
-	                        <erp>0</erp>
+	                        <cfm>1e-7</cfm>
+	                        <erp>0.8</erp>
 	                    </limit>
 	                </ode>
@@ -145,5 +145,5 @@
 		    <parent link="leg_r_link07"/>
 			<child link="leg_r_link08"/>
-		    <origin xyz="0 0 0" rpy="0 -0.7854 0"/>
+		    <origin xyz="0 0 0" rpy="0 -0.78539816 0"/>
 		    <axis xyz="0 1 0"/>
 			<limit effort="1000.0" lower="-3.1" upper="3.1" velocity="10.0"/>
@@ -164,5 +164,5 @@
 		    <parent link="leg_r_link08"/>
 			<child link="leg_r_link10"/>
-		    <origin xyz="-0.1 0 0" rpy="0 0.7854 0"/>
+		    <origin xyz="-0.1 0 0" rpy="0 0.78539816 0"/>
 		    <axis xyz="0 1 0"/>
 			<limit effort="1000.0" lower="-0.5" upper="1.4" velocity="1000.0"/>
@@ -183,5 +183,5 @@
 		    <parent link="leg_r_link10"/>
 			<child link="leg_r_link09"/>
-		    <origin xyz="-0.0335 0 0" rpy="0 -0.7854 0"/>
+		    <origin xyz="-0.0335 0 0" rpy="0 -0.78539816 0"/>
 		    <axis xyz="0 1 0"/>
 			<limit effort="1000.0" lower="-1.4" upper="0.5" velocity="1000.0"/>
@@ -221,6 +221,6 @@
 	                    <cfm_damping>0</cfm_damping>
 	                    <limit>
-	                        <cfm>0</cfm>
-	                        <erp>0</erp>
+	                        <cfm>1e-7</cfm>
+	                        <erp>0.8</erp>
 	                    </limit>
 	                </ode>
@@ -231,5 +231,5 @@
 		    <parent link="leg_r_link09"/>
 			<child link="leg_r_link06"/>
-		    <origin xyz="0.07118 0 0.00834" rpy="0 1.5708 0"/>
+		    <origin xyz="0.07118 0 0.00834" rpy="0 1.57079633 0"/>
 		    <axis xyz="0 1 0"/>
 			<limit effort="1000.0" lower="-1.0" upper="1.5" velocity="10.0"/>
@@ -270,6 +270,6 @@
 	                    <cfm_damping>0</cfm_damping>
 	                    <limit>
-	                        <cfm>0</cfm>
-	                        <erp>0</erp>
+	                        <cfm>1e-7</cfm>
+	                        <erp>0.8</erp>
 	                    </limit>
 	                </ode>
