Commit message: Edit shoulder joint position

File: ginko_description/xacro/ginko_xm540/parts/arm_l.xacro (robot description, xacro)
@@ -6,5 +6,5 @@
 		    <parent link="chest_link01"/>
 			<child link="arm_l_link01"/>
-		    <origin xyz="0 0.117 0" rpy="0 0 0"/>
+		    <origin xyz="0 0.087 0" rpy="0 0 0"/>
 		    <axis xyz="0 1 0"/>
 			<limit effort="1000.0" lower="-3.1" upper="3.1" velocity="10.0"/>
@@ -13,16 +13,16 @@
 		<link name="arm_l_link01">
 			<visual>
-				<origin xyz="0 0.01 0" rpy="0 0 0"/>
+				<origin xyz="0 0.04 0" rpy="0 0 0"/>
 				<geometry>
 					<mesh filename="package://ginko_description/meshes/ginko_xm540/obj/arm_l_link01.obj"/>
 				</geometry>
 			</visual>
-            <xacro:box_collision xyz="0 0.00475 0" rpy="0 0 0" size="0.052 0.0365 0.0335"/>
-			<xacro:box_inertial xyz="0 0.00575 0" rpy="0 0 0" size="0.052 0.0365 0.0335" mass="0.03"/>
+            <xacro:box_collision xyz="0 0.03475 0" rpy="0 0 0" size="0.052 0.0365 0.0335"/>
+			<xacro:box_inertial xyz="0 0.03475 0" rpy="0 0 0" size="0.052 0.0365 0.0335" mass="0.03"/>
 		</link>
 		<joint name="arm_l_joint02" type="revolute">
 		    <parent link="arm_l_link01"/>
 			<child link="arm_l_link02"/>
-		    <origin xyz="0 0.01 0" rpy="0 0 0"/>
+		    <origin xyz="0 0.04 0" rpy="0 0 0"/>
 		    <axis xyz="1 0 0"/>
 			<limit effort="1000.0" lower="-3.1" upper="3.1" velocity="10.0"/>

File: ginko_description/xacro/ginko_xm540/parts/arm_r.xacro (robot description, xacro)
@@ -6,5 +6,5 @@
 		    <parent link="chest_link01"/>
 			<child link="arm_r_link01"/>
-		    <origin xyz="0 -0.117 0" rpy="0 0 0"/>
+		    <origin xyz="0 -0.087 0" rpy="0 0 0"/>
 		    <axis xyz="0 -1 0"/>
 			<limit effort="1000.0" lower="-3.1" upper="3.1" velocity="10.0"/>
@@ -13,16 +13,16 @@
 		<link name="arm_r_link01">
 			<visual>
-				<origin xyz="0 -0.01 0" rpy="0 0 0"/>
+				<origin xyz="0 -0.04 0" rpy="0 0 0"/>
 				<geometry>
 					<mesh filename="package://ginko_description/meshes/ginko_xm540/obj/arm_r_link01.obj"/>
 				</geometry>
 			</visual>
-            <xacro:box_collision xyz="0 -0.00475 0" rpy="0 0 0" size="0.052 0.0365 0.0335"/>
-			<xacro:box_inertial xyz="0 -0.00475 0" rpy="0 0 0" size="0.052 0.0365 0.0335" mass="0.03"/>
+            <xacro:box_collision xyz="0 -0.03475 0" rpy="0 0 0" size="0.052 0.0365 0.0335"/>
+			<xacro:box_inertial xyz="0 -0.03475 0" rpy="0 0 0" size="0.052 0.0365 0.0335" mass="0.03"/>
 		</link>
 		<joint name="arm_r_joint02" type="revolute">
 		    <parent link="arm_r_link01"/>
 			<child link="arm_r_link02"/>
-		    <origin xyz="0 -0.01 0" rpy="0 0 0"/>
+		    <origin xyz="0 -0.04 0" rpy="0 0 0"/>
 		    <axis xyz="1 0 0"/>
 			<limit effort="1000.0" lower="-3.1" upper="3.1" velocity="10.0"/>

Commit message: Set minimum inertia

File: ginko_description/xacro/ginko_xm540/parts/arm_l.xacro (robot description, xacro)
@@ -19,5 +19,5 @@
 			</visual>
             <xacro:box_collision xyz="0 0.03475 0" rpy="0 0 0" size="0.052 0.05 0.04"/>
-			<xacro:box_inertial xyz="0 0.03475 0" rpy="0 0 0" size="0.052 0.05 0.04" mass="0.05"/>
+			<xacro:box_inertial xyz="0 0.03475 0" rpy="0 0 0" size="0.052 0.05 0.04" mass="0.01"/>
 		</link>
 		<joint name="arm_l_joint02" type="revolute">

File: ginko_description/xacro/ginko_xm540/parts/arm_r.xacro (robot description, xacro)
@@ -19,5 +19,5 @@
 			</visual>
             <xacro:box_collision xyz="0 -0.03475 0" rpy="0 0 0" size="0.052 0.05 0.04"/>
-			<xacro:box_inertial xyz="0 -0.03475 0" rpy="0 0 0" size="0.052 0.05 0.04" mass="0.05"/>
+			<xacro:box_inertial xyz="0 -0.03475 0" rpy="0 0 0" size="0.052 0.05 0.04" mass="0.01"/>
 		</link>
 		<joint name="arm_r_joint02" type="revolute">

File: ginko_description/xacro/ginko_xm540/parts/leg_l.xacro (robot description, xacro)
@@ -73,5 +73,5 @@
 			</visual>
             <xacro:box_collision xyz="-0.015 0 0" rpy="0 0 0" size="0.04565 0.0373 0.023"/>
-			<xacro:box_inertial xyz="-0.015 0 0" rpy="0 0 0" size="0.04565 0.0373 0.023" mass="0.03"/>
+			<xacro:box_inertial xyz="-0.015 0 0" rpy="0 0 0" size="0.04565 0.0373 0.023" mass="0.011"/>
 		</link>
 		<joint name="leg_l_joint07" type="revolute">

File: ginko_description/xacro/ginko_xm540/parts/leg_r.xacro (robot description, xacro)
@@ -73,5 +73,5 @@
 			</visual>
             <xacro:box_collision xyz="-0.015 0 0" rpy="0 0 0" size="0.04565 0.0373 0.023"/>
-			<xacro:box_inertial xyz="-0.015 0 0" rpy="0 0 0" size="0.04565 0.0373 0.023" mass="0.03"/>
+			<xacro:box_inertial xyz="-0.015 0 0" rpy="0 0 0" size="0.04565 0.0373 0.023" mass="0.011"/>
 		</link>
 		<joint name="leg_r_joint07" type="revolute">

File: ginko_description/xacro/physics/box_physics.xacro (robot description, xacro)
@@ -5,10 +5,23 @@
     <xacro:property name="w" value="${float(size.split()[1])}" />
     <xacro:property name="h" value="${float(size.split()[2])}" />
+    <xacro:property name="ixx" value="${mass * (w ** 2 + h ** 2) / 12}" />
+    <xacro:property name="iyy" value="${mass * (d ** 2 + h ** 2) / 12}" />
+    <xacro:property name="izz" value="${mass * (w ** 2 + d ** 2) / 12}" />
+    <xacro:property name="inertia_min" value="0.00001" />
+    <xacro:if value="${int(inertia_min/ixx)}">
+      <xacro:property name="ixx" value="${inertia_min}" />
+    </xacro:if>
+    <xacro:if value="${int(inertia_min/iyy)}">
+      <xacro:property name="iyy" value="${inertia_min}" />
+    </xacro:if>
+    <xacro:if value="${int(inertia_min/izz)}">
+      <xacro:property name="izz" value="${inertia_min}" />
+    </xacro:if>
     <inertial>
       <origin xyz="${xyz}" rpy="${rpy}"/>
       <mass value="${mass}"/>
-      <inertia ixx="${mass * (w ** 2 + h ** 2) / 12}"
-               ixy="0.0" iyy="${mass * (d ** 2 + h ** 2) / 12}"
-               ixz="0.0" iyz="0.0" izz="${mass * (w ** 2 + d ** 2) / 12}"/>
+      <inertia ixx="${ixx}"
+               ixy="0.0" iyy="${iyy}"
+               ixz="0.0" iyz="0.0" izz="${izz}"/>
     </inertial>
   </xacro:macro>
