Commit message: Change inertia_min to param

File: ginko_description/xacro/physics/box_physics.xacro (robot description, xacro)
@@ -1,5 +1,5 @@
 <?xml version="1.0"?>
 <robot xmlns:xacro="http://www.ros.org/wiki/xacro">
-  <xacro:macro name="box_inertial" params="xyz:='0 0 0' rpy:='0 0 0' size mass">
+  <xacro:macro name="box_inertial" params="xyz:='0 0 0' rpy:='0 0 0' size mass inertia_min:=0.00001">
     <xacro:property name="d" value="${float(size.split()[0])}" />
     <xacro:property name="w" value="${float(size.split()[1])}" />
@@ -8,5 +8,4 @@
     <xacro:property name="iyy" value="${mass * (d ** 2 + h ** 2) / 12}" />
     <xacro:property name="izz" value="${mass * (w ** 2 + d ** 2) / 12}" />
-    <xacro:property name="inertia_min" value="0.00001" />
     <xacro:if value="${int(inertia_min/ixx)}">
       <xacro:property name="ixx" value="${inertia_min}" />
