Commit message: Edit ring

File: ginko_description/xacro/roboone_ring/large_ring.xacro (robot description, xacro)
@@ -5,5 +5,5 @@
 		<link name="large_ring_link0">
 			<collision>
-				<origin xyz="0 0 0" rpy="0 0 0"/>
+				<origin xyz="0 0 -0.97" rpy="0 0 0"/>
 				<geometry>
         			<mesh filename="package://ginko_description/meshes/roboone_ring/stl/large_ring.stl"/>

File: ginko_description/xacro/roboone_ring/small_ring.xacro (robot description, xacro)
@@ -5,5 +5,5 @@
 		<link name="small_ring_link0">
 			<collision>
-				<origin xyz="0 0 0" rpy="0 0 0"/>
+				<origin xyz="0 0 -0.97" rpy="0 0 0"/>
 				<geometry>
         			<mesh filename="package://ginko_description/meshes/roboone_ring/stl/small_ring.stl"/>
